File: furnace/furnace_controller/External.sch (KiCad schematic (older format))
At the start: 0 parts

Commit message: Add files via upload
Parts:
- added J?: Conn_01x10_Male, symbol Connector:Conn_01x10_Male
- added J?: Conn_01x24, symbol Connector_Generic:Conn_01x24
- added J?: Conn_01x04_Male, symbol Connector:Conn_01x04_Male
Changed lines of the file:
@@
 $Descr A4 11693 8268
 encoding utf-8
-Sheet 1 13
+Sheet 3 13
 Title ""
 Date ""
@@
 Comment4 ""
 $EndDescr
+$Comp
+L Connector:Conn_01x10_Male J?
+U 1 1 609EA720
+P 6750 3750
+F 0 "J?" H 6858 4331 50  0000 C CNN
+F 1 "Conn_01x10_Male" H 6858 4240 50  0000 C CNN
+F 2 "" H 6750 3750 50  0001 C CNN
+F 3 "~" H 6750 3750 50  0001 C CNN
+	1    6750 3750
+	1    0    0    -1
+$EndComp
+$Comp
+L Connector_Generic:Conn_01x24 J?
+U 1 1 609EA726
+P 8000 3800
+F 0 "J?" H 8080 3792 50  0000 L CNN
+F 1 "Conn_01x24" H 8080 3701 50  0000 L CNN
+F 2 "" H 8000 3800 50  0001 C CNN
+F 3 "~" H 8000 3800 50  0001 C CNN
+	1    8000 3800
+	1    0    0    -1
+$EndComp
+$Comp
+L Connector:Conn_01x04_Male J?
+U 1 1 609EAA53
+P 4600 3450
+F 0 "J?" H 4708 3731 50  0000 C CNN
+F 1 "Conn_01x04_Male" H 4708 3640 50  0000 C CNN
+F 2 "" H 4600 3450 50  0001 C CNN
+F 3 "~" H 4600 3450 50  0001 C CNN
+	1    4600 3450
+	1    0    0    -1
+$EndComp
 $EndSCHEMATC

Commit message: Add files via upload
Other:
- moved on the sheet: J?
Changed lines of the file:
@@
 $Descr A4 11693 8268
 encoding utf-8
-Sheet 3 13
+Sheet 3 14
 Title ""
 Date ""
@@
 L Connector:Conn_01x10_Male J?
 U 1 1 609EA720
-P 6750 3750
-F 0 "J?" H 6858 4331 50  0000 C CNN
-F 1 "Conn_01x10_Male" H 6858 4240 50  0000 C CNN
-F 2 "" H 6750 3750 50  0001 C CNN
-F 3 "~" H 6750 3750 50  0001 C CNN
-	1    6750 3750
+P 2600 4100
+F 0 "J?" H 2708 4681 50  0000 C CNN
+F 1 "Conn_01x10_Male" H 2708 4590 50  0000 C CNN
+F 2 "" H 2600 4100 50  0001 C CNN
+F 3 "~" H 2600 4100 50  0001 C CNN
+	1    2600 4100
 	1    0    0    -1
 $EndComp
@@
 L Connector:Conn_01x04_Male J?
 U 1 1 609EAA53
-P 4600 3450
-F 0 "J?" H 4708 3731 50  0000 C CNN
-F 1 "Conn_01x04_Male" H 4708 3640 50  0000 C CNN
-F 2 "" H 4600 3450 50  0001 C CNN
-F 3 "~" H 4600 3450 50  0001 C CNN
-	1    4600 3450
+P 2600 2850
+F 0 "J?" H 2708 3131 50  0000 C CNN
+F 1 "Conn_01x04_Male" H 2708 3040 50  0000 C CNN
+F 2 "" H 2600 2850 50  0001 C CNN
+F 3 "~" H 2600 2850 50  0001 C CNN
+	1    2600 2850
 	1    0    0    -1
 $EndComp

Commit message: Add files via upload
Parts:
- removed J?: Conn_01x10_Male, symbol Connector:Conn_01x10_Male
- removed J?: Conn_01x24, symbol Connector_Generic:Conn_01x24
- removed J?: Conn_01x04_Male, symbol Connector:Conn_01x04_Male
Changed lines of the file:
@@
 $Descr A4 11693 8268
 encoding utf-8
-Sheet 3 14
+Sheet 3 16
 Title ""
 Date ""
@@
 Comment4 ""
 $EndDescr
-$Comp
-L Connector:Conn_01x10_Male J?
-U 1 1 609EA720
-P 2600 4100
-F 0 "J?" H 2708 4681 50  0000 C CNN
-F 1 "Conn_01x10_Male" H 2708 4590 50  0000 C CNN
-F 2 "" H 2600 4100 50  0001 C CNN
-F 3 "~" H 2600 4100 50  0001 C CNN
-	1    2600 4100
-	1    0    0    -1
-$EndComp
-$Comp
-L Connector_Generic:Conn_01x24 J?
-U 1 1 609EA726
-P 8000 3800
-F 0 "J?" H 8080 3792 50  0000 L CNN
-F 1 "Conn_01x24" H 8080 3701 50  0000 L CNN
-F 2 "" H 8000 3800 50  0001 C CNN
-F 3 "~" H 8000 3800 50  0001 C CNN
-	1    8000 3800
-	1    0    0    -1
-$EndComp
-$Comp
-L Connector:Conn_01x04_Male J?
-U 1 1 609EAA53
-P 2600 2850
-F 0 "J?" H 2708 3131 50  0000 C CNN
-F 1 "Conn_01x04_Male" H 2708 3040 50  0000 C CNN
-F 2 "" H 2600 2850 50  0001 C CNN
-F 3 "~" H 2600 2850 50  0001 C CNN
-	1    2600 2850
-	1    0    0    -1
-$EndComp
 $EndSCHEMATC
