File: furnace/furnace_controller/Main.sch (KiCad schematic (older format))
At the start: 6 parts

Commit message: Add files via upload
Parts:
- added BZ?: Buzzer, symbol Device:Buzzer
- added Q?: BC847, Package_TO_SOT_SMD:SOT-23, symbol Transistor_BJT:BC847
Changed lines of the file:
@@
+	1    0    0    -1
+$EndComp
+$Comp
+L Device:Buzzer BZ?
+U 1 1 609E23B7
+P 3600 1900
+F 0 "BZ?" H 3752 1929 50  0000 L CNN
+F 1 "Buzzer" H 3752 1838 50  0000 L CNN
+F 2 "" V 3575 2000 50  0001 C CNN
+F 3 "~" V 3575 2000 50  0001 C CNN
+	1    3600 1900
+	1    0    0    -1
+$EndComp
+$Comp
+L Transistor_BJT:BC847 Q?
+U 1 1 609E3112
+P 3150 2400
+F 0 "Q?" H 3341 2446 50  0000 L CNN
+F 1 "BC847" H 3341 2355 50  0000 L CNN
+F 2 "Package_TO_SOT_SMD:SOT-23" H 3350 2325 50  0001 L CIN
+F 3 "http://www.infineon.com/dgdl/Infineon-BC847SERIES_BC848SERIES_BC849SERIES_BC850SERIES-DS-v01_01-en.pdf?fileId=db3a304314dca389011541d4630a1657" H 3150 2400 50  0001 L CNN
+	1    3150 2400
 	1    0    0    -1
 $EndComp

Commit message: Add files via upload
Parts:
- removed U?: AMS1117-3.3, Package_TO_SOT_SMD:SOT-223-3_TabPin2, symbol Regulator_Linear:AMS1117-3.3
Changed lines of the file:
@@
 $Descr A4 11693 8268
 encoding utf-8
-Sheet 2 13
+Sheet 2 14
 Title ""
 Date ""
@@
 	1    0    0    -1
 $EndComp
-$Comp
-L Regulator_Linear:AMS1117-3.3 U?
-U 1 1 609CF000
-P 3800 3500
-AR Path="/609CF000" Ref="U?"  Part="1"
-AR Path="/609C9D41/609CF000" Ref="U?"  Part="1"
-F 0 "U?" H 3800 3742 50  0000 C CNN
-F 1 "AMS1117-3.3" H 3800 3651 50  0000 C CNN
-F 2 "Package_TO_SOT_SMD:SOT-223-3_TabPin2" H 3800 3700 50  0001 C CNN
-F 3 "http://www.advanced-monolithic.com/pdf/ds1117.pdf" H 3900 3250 50  0001 C CNN
-	1    3800 3500
-	1    0    0    -1
-$EndComp
