File: furnace/furnace_controller/Temp_sensor.sch (KiCad schematic (older format))
At the start: 0 parts

Commit message: Add files via upload
Changed lines of the file:
@@
 $Descr A4 11693 8268
 encoding utf-8
-Sheet 4 13
+Sheet 4 14
 Title ""
 Date ""
@@
 $EndComp
 $Comp
-L power:GND1 #PWR?
+L furnace_controller-rescue:GND1-power #PWR?
 U 1 1 60A0EB0A
 P 3450 2350
@@
 	3450 2350 3550 2350
 $Comp
-L power:GND1 #PWR?
+L furnace_controller-rescue:GND1-power #PWR?
 U 1 1 60B09F47
 P 6450 2150
@@
 	6450 2150 6550 2150
 $Comp
-L power:GND1 #PWR?
+L furnace_controller-rescue:GND1-power #PWR?
 U 1 1 60B0A5B6
 P 6450 3450
@@
 ~CS5
 $Comp
-L power:GND1 #PWR?
+L furnace_controller-rescue:GND1-power #PWR?
 U 1 1 60B0F1ED
 P 3450 3350
@@
 	3450 3350 3550 3350
 $Comp
-L power:GND1 #PWR?
+L furnace_controller-rescue:GND1-power #PWR?
 U 1 1 60B0FB21
 P 3450 4350
@@
 	3450 4350 3550 4350
 $Comp
-L power:GND1 #PWR?
+L furnace_controller-rescue:GND1-power #PWR?
 U 1 1 60B108C7
 P 3450 5350
@@
 	3450 5350 3550 5350
 $Comp
-L power:GND1 #PWR?
+L furnace_controller-rescue:GND1-power #PWR?
 U 1 1 60B118E3
 P 3450 6350
@@
 	7550 4700 7650 4700
 $Comp
-L power:GND1 #PWR?
+L furnace_controller-rescue:GND1-power #PWR?
 U 1 1 60B14823
 P 6450 4700
@@
 	7550 5950 7650 5950
 $Comp
-L power:GND1 #PWR?
+L furnace_controller-rescue:GND1-power #PWR?
 U 1 1 60B180EF
 P 6450 5950
@@
 	4850 6050 4550 6050
 $Comp
-L power:GND1 #PWR?
+L furnace_controller-rescue:GND1-power #PWR?
 U 1 1 60B43E6A
 P 6450 4500
@@
 	6450 4500 6550 4500
 $Comp
-L power:GND1 #PWR?
+L furnace_controller-rescue:GND1-power #PWR?
 U 1 1 60B472DC
 P 6450 5750

Commit message: Add files via upload
Parts:
- added C?: 0,1, Capacitor_SMD:C_0603_1608Metric_Pad1.08x0.95mm_HandSolder, symbol Device:C
- added J?: Conn_01x03_Male, symbol Connector:Conn_01x03_Male
- added R? (x2): 4,7k, Resistor_SMD:R_0603_1608Metric_Pad0.98x0.95mm_HandSolder, symbol Device:R
- added U?: LM75A, symbol Sensor_Temperature:LM75B
Connections:
- net +3V3: now also C?.1, R?.1, R?.1, U?.8 (+Vs)
- net GND: now also C?.2, J?.3 (Pin_3), U?.4 (GND), U?.5 (A2), U?.6 (A1), U?.7 (A0)
- new net SCL: J?.1 (Pin_1), R?.2, U?.2 (SCL)
- new net SDA: J?.2 (Pin_2), R?.2, U?.1 (SDA)
- no-connect marks 2 -> 1
Other:
- note added: "Temperature sensor"
- note removed: "Isolated 5x temperature sensor"

Commit message: Add files via upload
Connections:
- net SCL renamed SCK
Changed lines of the file:
@@
 SDA
 Text HLabel 5000 4500 0    50   Input ~ 0
-SCL
+SCK
 $Comp
 L Connector:Conn_01x03_Male J?
