File: furnace/furnace_controller/furnace_controller.sch (KiCad schematic (older format))
At the start: 10 parts

Commit message: Add files via upload
Parts:
- removed J?: Conn_01x10_Male, symbol Connector:Conn_01x10_Male
- removed J?: Conn_01x24, symbol Connector_Generic:Conn_01x24
Other:
- moved on the sheet: TP?
Changed lines of the file:
@@
-$EndComp
-$Comp
-L Connector:Conn_01x10_Male J?
-U 1 1 609BABA5
-P 1550 6050
-F 0 "J?" H 1658 6631 50  0000 C CNN
-F 1 "Conn_01x10_Male" H 1658 6540 50  0000 C CNN
-F 2 "" H 1550 6050 50  0001 C CNN
-F 3 "~" H 1550 6050 50  0001 C CNN
-	1    1550 6050
-	1    0    0    -1
 $EndComp
 $Comp
 L Connector:TestPoint TP?
 U 1 1 609BBCCA
-P 3000 5950
-F 0 "TP?" H 3058 6068 50  0000 L CNN
-F 1 "TestPoint" H 3058 5977 50  0001 L CNN
-F 2 "" H 3200 5950 50  0001 C CNN
-F 3 "~" H 3200 5950 50  0001 C CNN
-	1    3000 5950
+P 5550 5650
+F 0 "TP?" H 5608 5768 50  0000 L CNN
+F 1 "TestPoint" H 5608 5677 50  0001 L CNN
+F 2 "" H 5750 5650 50  0001 C CNN
+F 3 "~" H 5750 5650 50  0001 C CNN
+	1    5550 5650
 	1    0    0    -1
 $EndComp
-$Comp
-L Connector_Generic:Conn_01x24 J?
-U 1 1 609BC9D9
-P 4350 6150
-F 0 "J?" H 4430 6142 50  0000 L CNN
-F 1 "Conn_01x24" H 4430 6051 50  0000 L CNN
-F 2 "" H 4350 6150 50  0001 C CNN
-F 3 "~" H 4350 6150 50  0001 C CNN
-	1    4350 6150
-	1    0    0    -1
-$EndComp

Commit message: Add files via upload
Changed lines of the file:
@@
 $Descr A4 11693 8268
 encoding utf-8
-Sheet 1 13
+Sheet 1 14
 Title ""
 Date ""
@@
 F6 "MISO" O R 2000 4400 50
 $EndSheet
+$Sheet
+S 1000 5000 1000 500
+U 609FED99
+F0 "POWER_3V3_10V" 50
+F1 "Power_3V3_10V.sch" 50
+F2 "CHARGE_PUMP_CLK" I L 1000 5400 50
+F3 "+5V_IN" I L 1000 5100 50
+F4 "-5V_IN" I L 1000 5200 50
+$EndSheet
 $EndSCHEMATC

Commit message: Add files via upload
Parts:
- added J?: Conn_01x04_Male, symbol Connector:Conn_01x04_Male
Other:
- note added: "I2C_DISPLAY"
- moved on the sheet: C?
Changed lines of the file:
@@
 $Descr A4 11693 8268
 encoding utf-8
-Sheet 1 14
+Sheet 1 15
 Title ""
 Date ""
@@
 L Device:C C?
 U 1 1 609B27F2
-P 4100 3400
-F 0 "C?" H 4215 3446 50  0000 L CNN
-F 1 "0603" H 4215 3355 50  0000 L CNN
-F 2 "Capacitor_SMD:C_0603_1608Metric_Pad1.08x0.95mm_HandSolder" H 4138 3250 50  0001 C CNN
-F 3 "~" H 4100 3400 50  0001 C CNN
-	1    4100 3400
+P 4050 3100
+F 0 "C?" H 4165 3146 50  0000 L CNN
+F 1 "0603" H 4165 3055 50  0000 L CNN
+F 2 "Capacitor_SMD:C_0603_1608Metric_Pad1.08x0.95mm_HandSolder" H 4088 2950 50  0001 C CNN
+F 3 "~" H 4050 3100 50  0001 C CNN
+	1    4050 3100
 	1    0    0    -1
 $EndComp
@@
 $EndComp
 $Sheet
-S 2550 3800 1400 850
+S 2500 3500 1400 850
 U 609C9D41
 F0 "MAIN" 50
 F1 "Main.sch" 50
-$EndSheet
-$Sheet
-S 4500 3850 1250 750
-U 609CA1D9
-F0 "EXTERNAL" 50
-F1 "External.sch" 50
 $EndSheet
 $Sheet
@@
 F4 "-5V_IN" I L 1000 5200 50
 $EndSheet
+$Sheet
+S 2500 5000 1000 500
+U 60A364EE
+F0 "OLED_DISPLAY_CONNECTOR" 50
+F1 "OLED_display_connector.sch" 50
+$EndSheet
+$Sheet
+S 4000 5000 1000 500
+U 60A36559
+F0 "KEYBOARD_CONNECTOR" 50
+F1 "Keyboard_connector.sch" 50
+$EndSheet
+$Comp
+L Connector:Conn_01x04_Male J?
+U 1 1 60A373FD
+P 7000 3950
+AR Path="/609CA1D9/60A373FD" Ref="J?"  Part="1"
+AR Path="/60A373FD" Ref="J?"  Part="1"
+F 0 "J?" H 7108 4231 50  0000 C CNN
+F 1 "Conn_01x04_Male" H 7108 4140 50  0000 C CNN
+F 2 "" H 7000 3950 50  0001 C CNN
+F 3 "~" H 7000 3950 50  0001 C CNN
+	1    7000 3950
+	1    0    0    -1
+$EndComp
+Text Notes 7450 4000 0    50   ~ 0
+I2C_DISPLAY
 $EndSCHEMATC

Commit message: Add files via upload
Parts:
- removed C?: 0603, Capacitor_SMD:C_0603_1608Metric_Pad1.08x0.95mm_HandSolder, symbol Device:C
- removed D?: PESD5Z3.3, symbol Device:D_Zener
- removed D?: SMAJ5.0CA, symbol Device:D_TVS
- removed D?: BAT54S, Package_TO_SOT_SMD:SOT-23, symbol Diode:BAT54S
- removed R?: 0603, Resistor_SMD:R_0603_1608Metric_Pad0.98x0.95mm_HandSolder, symbol Device:R
- removed TP?: TestPoint, symbol Connector:TestPoint
Connections:
- net labels removed: GND
- wire segments 1 -> 0
Other:
- moved on the sheet: J?
Changed lines of the file:
@@
 $Descr A4 11693 8268
 encoding utf-8
-Sheet 1 15
+Sheet 1 18
 Title ""
 Date ""
@@
 $EndDescr
 $Comp
-L Device:R R?
-U 1 1 609A6451
-P 6150 2600
-F 0 "R?" H 6220 2646 50  0000 L CNN
-F 1 "0603" H 6220 2555 50  0000 L CNN
-F 2 "Resistor_SMD:R_0603_1608Metric_Pad0.98x0.95mm_HandSolder" V 6080 2600 50  0001 C CNN
-F 3 "~" H 6150 2600 50  0001 C CNN
-	1    6150 2600
-	1    0    0    -1
-$EndComp
-$Comp
-L power:GND #PWR?
-U 1 1 609A7264
-P 4700 1850
-F 0 "#PWR?" H 4700 1600 50  0001 C CNN
-F 1 "GND" H 4705 1677 50  0000 C CNN
-F 2 "" H 4700 1850 50  0001 C CNN
-F 3 "" H 4700 1850 50  0001 C CNN
-	1    4700 1850
-	1    0    0    -1
-$EndComp
-Wire Wire Line
-	4700 1850 4900 1850
-$Comp
 L Connector:Screw_Terminal_01x02 J?
 U 1 1 609BACE5
@@
 F 3 "~" H 1800 1550 50  0001 C CNN
 	1    1800 1550
-	1    0    0    -1
-$EndComp
-$Comp
-L Device:D_Zener D?
-U 1 1 609A877C
-P 3900 2500
-F 0 "D?" V 3854 2580 50  0000 L CNN
-F 1 "PESD5Z3.3" V 3945 2580 50  0000 L CNN
-F 2 "" H 3900 2500 50  0001 C CNN
-F 3 "~" H 3900 2500 50  0001 C CNN
-	1    3900 2500
-	0    1    1    0
-$EndComp
-$Comp
-L Device:D_TVS D?
-U 1 1 609AD491
-P 2500 2350
-F 0 "D?" V 2546 2270 50  0000 R CNN
-F 1 "SMAJ5.0CA" V 2455 2270 50  0000 R CNN
-F 2 "" H 2500 2350 50  0001 C CNN
-F 3 "~" H 2500 2350 50  0001 C CNN
-	1    2500 2350
-	0    -1   -1   0
-$EndComp
-$Comp
-L Diode:BAT54S D?
-U 1 1 609B08DC
-P 2000 3300
-F 0 "D?" V 2200 3150 50  0000 C CNN
-F 1 "BAT54S" V 2100 3050 50  0000 C CNN
-F 2 "Package_TO_SOT_SMD:SOT-23" H 2075 3425 50  0001 L CNN
-F 3 "https://www.diodes.com/assets/Datasheets/ds11005.pdf" H 1880 3300 50  0001 C CNN
-	1    2000 3300
-	0    -1   -1   0
-$EndComp
-$Comp
-L Device:C C?
-U 1 1 609B27F2
-P 4050 3100
-F 0 "C?" H 4165 3146 50  0000 L CNN
-F 1 "0603" H 4165 3055 50  0000 L CNN
-F 2 "Capacitor_SMD:C_0603_1608Metric_Pad1.08x0.95mm_HandSolder" H 4088 2950 50  0001 C CNN
-F 3 "~" H 4050 3100 50  0001 C CNN
-	1    4050 3100
-	1    0    0    -1
-$EndComp
-$Comp
-L Connector:TestPoint TP?
-U 1 1 609BBCCA
-P 5550 5650
-F 0 "TP?" H 5608 5768 50  0000 L CNN
-F 1 "TestPoint" H 5608 5677 50  0001 L CNN
-F 2 "" H 5750 5650 50  0001 C CNN
-F 3 "~" H 5750 5650 50  0001 C CNN
-	1    5550 5650
 	1    0    0    -1
 $EndComp
@@
 $EndComp
 $Sheet
-S 2500 3500 1400 850
+S 6000 1500 1000 500
 U 609C9D41
-F0 "MAIN" 50
-F1 "Main.sch" 50
-$EndSheet
-$Sheet
-S 1000 4000 1000 500
-U 609CA6A8
-F0 "TEMP_SENSOR" 50
-F1 "Temp_sensor.sch" 50
-F2 "TC-" I L 1000 4350 50
-F3 "~CS" I R 2000 4100 50
-F4 "TC+" I L 1000 4150 50
-F5 "SCK" I R 2000 4200 50
-F6 "MISO" O R 2000 4400 50
+F0 "MCU" 50
+F1 "MCU.sch" 50
 $EndSheet
 $Sheet
@@
 $EndSheet
 $Sheet
-S 2500 5000 1000 500
+S 2500 5000 1000 700
 U 60A364EE
 F0 "OLED_DISPLAY_CONNECTOR" 50
 F1 "OLED_display_connector.sch" 50
+F2 "DPY_PWR_EN" I L 2500 5100 50
+F3 "~DPY_RST" I L 2500 5300 50
+F4 "SDA" I L 2500 5600 50
+F5 "SCK" I L 2500 5500 50
 $EndSheet
 $Sheet
@@
 F0 "KEYBOARD_CONNECTOR" 50
 F1 "Keyboard_connector.sch" 50
+F2 "KYBD" B L 4000 5250 50
 $EndSheet
 $Comp
@@
 F 3 "~" H 7000 3950 50  0001 C CNN
 	1    7000 3950
-	1    0    0    -1
+	-1   0    0    -1
 $EndComp
 Text Notes 7450 4000 0    50   ~ 0
 I2C_DISPLAY
+$Sheet
+S 1000 4000 1000 500
+U 609CA6A8
+F0 "ISOLATED_TEMP_SENSOR" 50
+F1 "Isolated_temp_sensor.sch" 50
+F2 "TC-" I L 1000 4350 50
+F3 "~CS" I R 2000 4100 50
+F4 "TC+" I L 1000 4150 50
+F5 "SCK" I R 2000 4200 50
+F6 "MISO" O R 2000 4400 50
+$EndSheet
+$Sheet
+S 4000 4000 1000 500
+U 60B0ABCB
+F0 "TEMP_SENSOR" 50
+F1 "Temp_sensor.sch" 50
+F2 "SDA" B L 4000 4200 50
+F3 "SCL" I L 4000 4100 50
+$EndSheet
+$Sheet
+S 5500 4000 1000 500
+U 60B1951B
+F0 "MICRO_SD_CARD" 50
+F1 "Micro_SD_card.sch" 50
+F2 "~CS~" I L 5500 4100 50
+F3 "MOSI" I L 5500 4300 50
+F4 "SCL" I L 5500 4200 50
+F5 "MISO" O L 5500 4400 50
+$EndSheet
+$Sheet
+S 5500 5000 1000 500
+U 60B39FE1
+F0 "BUZZER" 50
+F1 "Buzzer.sch" 50
+F2 "EN" I L 5500 5250 50
+$EndSheet
 $EndSCHEMATC

Commit message: Add files via upload
Changed lines of the file:
@@
-$EndSheet
-$Sheet
-S 4000 4000 1000 500
-U 60B0ABCB
-F0 "TEMP_SENSOR" 50
-F1 "Temp_sensor.sch" 50
-F2 "SDA" B L 4000 4200 50
-F3 "SCL" I L 4000 4100 50
 $EndSheet
 $Sheet
@@
 F2 "~CS~" I L 5500 4100 50
 F3 "MOSI" I L 5500 4300 50
-F4 "SCL" I L 5500 4200 50
+F4 "SCK" I L 5500 4200 50
 F5 "MISO" O L 5500 4400 50
 $EndSheet

Commit message: Add files via upload
Parts:
- added J? (x4): TC0, symbol Connector:Screw_Terminal_01x02
- J?: value Screw_Terminal_01x02 -> TC0
- J?: value Conn_01x04 -> CWF-4R
- J?: value Conn_01x04_Male -> PLS-4R
Connections:
- net POWER_3V3_10V/+5V_IN: now also J?.1 (Pin_1)
- net POWER_3V3_10V/-5V_IN: now also J?.4 (Pin_4)
- net TC+0: now reaches J?.1 (Pin_1)
- net TC-0: now reaches J?.2 (Pin_2)
- net MCU/EXT_UART_RX: now reaches J?.2 (Pin_2)
- net MCU/HEATER_CTRL: now reaches J?.3 (Pin_3)
- net MCU/DPY_I2C_SCK: now reaches J?.1 (Pin_1)
- net MCU/DPY_I2C_SDA: now reaches J?.2 (Pin_2)
- net +5V: now reaches J?.3 (Pin_3)
- net GND: now reaches J?.4 (Pin_4)
- new net TC+1: J?.1 (Pin_1)
- new net TC+2: J?.1 (Pin_1)
- new net TC+3: J?.1 (Pin_1)
- new net TC+4: J?.1 (Pin_1)
- new net TC-1: J?.2 (Pin_2)
- new net TC-2: J?.2 (Pin_2)
- new net TC-3: J?.2 (Pin_2)
- new net TC-4: J?.2 (Pin_2)
Other:
- note added: "I2C display (1602a)\ndo not use at the same time \nas OLED display\nbecause of 5V on data lines"
- note removed: "I2C_DISPLAY"
- moved on the sheet: J?

Commit message: Add files via upload
Parts:
- removed J?: PLS-4R, symbol Connector:Conn_01x04_Male
Connections:
- net POWER_3V3_10V/-5V_IN renamed POWER_3V3_10V/GND_IN
Changed lines of the file:
@@
 $Descr A4 11693 8268
 encoding utf-8
-Sheet 1 17
+Sheet 1 18
 Title ""
 Date ""
@@
 F2 "CHARGE_PUMP_CLK" I L 7500 1400 50
 F3 "+5V_IN" I L 7500 1100 50
-F4 "-5V_IN" I L 7500 1200 50
+F4 "GND_IN" I L 7500 1200 50
 $EndSheet
 $Sheet
@@
 F2 "KYBD" B L 8000 3750 50
 $EndSheet
-$Comp
-L Connector:Conn_01x04_Male J?
-U 1 1 60A373FD
-P 9800 3100
-AR Path="/609CA1D9/60A373FD" Ref="J?"  Part="1"
-AR Path="/60A373FD" Ref="J?"  Part="1"
-F 0 "J?" H 9908 3381 50  0000 C CNN
-F 1 "PLS-4R" H 9908 3290 50  0000 C CNN
-F 2 "" H 9800 3100 50  0001 C CNN
-F 3 "~" H 9800 3100 50  0001 C CNN
-	1    9800 3100
-	-1   0    0    -1
-$EndComp
-Text Notes 9600 2600 0    50   ~ 0
+Text Notes 9550 2750 0    50   ~ 0
 I2C display (1602a)\ndo not use at the same time \nas OLED display\nbecause of 5V on data lines
 $Sheet
@@
 	6500 3200 7650 3200
 Wire Wire Line
-	7650 3200 7650 3000
-Wire Wire Line
 	7650 2500 8000 2500
 Wire Wire Line
 	6500 3300 7850 3300
 Wire Wire Line
-	7850 3300 7850 3100
-Wire Wire Line
 	7850 2600 8000 2600
-Connection ~ 7650 3000
-Wire Wire Line
-	7650 3000 7650 2500
-Connection ~ 7850 3100
-Wire Wire Line
-	7850 3100 7850 2600
-$Comp
-L power:GND #PWR?
-U 1 1 60B5EB57
-P 9400 3300
-AR Path="/609FED99/60B5EB57" Ref="#PWR?"  Part="1"
-AR Path="/60B5EB57" Ref="#PWR?"  Part="1"
-F 0 "#PWR?" H 9400 3050 50  0001 C CNN
-F 1 "GND" H 9405 3127 50  0000 C CNN
-F 2 "" H 9400 3300 50  0001 C CNN
-F 3 "" H 9400 3300 50  0001 C CNN
-	1    9400 3300
-	1    0    0    -1
-$EndComp
-$Comp
-L power:+5V #PWR?
-U 1 1 60B5EB5D
-P 9400 2900
-AR Path="/609FED99/60B5EB5D" Ref="#PWR?"  Part="1"
-AR Path="/60B5EB5D" Ref="#PWR?"  Part="1"
-F 0 "#PWR?" H 9400 2750 50  0001 C CNN
-F 1 "+5V" H 9415 3073 50  0000 C CNN
-F 2 "" H 9400 2900 50  0001 C CNN
-F 3 "" H 9400 2900 50  0001 C CNN
-	1    9400 2900
-	1    0    0    -1
-$EndComp
-Wire Wire Line
-	7650 3000 9600 3000
-Wire Wire Line
-	7850 3100 9600 3100
-Wire Wire Line
-	9600 3200 9400 3200
-Wire Wire Line
-	9400 3200 9400 2900
-Wire Wire Line
-	9600 3300 9400 3300
 Wire Bus Line
 	8000 3750 7750 3750
@@
 Wire Wire Line
 	4750 3000 5000 3000
+$Sheet
+S 9500 3000 1000 500
+U 60B3D5E3
+F0 "I2C_DISPLAY_CONNECTOR" 50
+F1 "I2C_display_connector.sch" 50
+F2 "SCK" I L 9500 3100 50
+F3 "SDA" B L 9500 3200 50
+$EndSheet
+Wire Wire Line
+	7650 2500 7650 3100
+Wire Wire Line
+	7850 2600 7850 3200
+Wire Wire Line
+	9500 3100 7650 3100
+Connection ~ 7650 3100
+Wire Wire Line
+	7650 3100 7650 3200
+Wire Wire Line
+	9500 3200 7850 3200
 Wire Bus Line
 	2000 3150 2000 5500
 Wire Bus Line
 	2500 3350 2500 5600
+Connection ~ 7850 3200
+Wire Wire Line
+	7850 3200 7850 3300
 $EndSCHEMATC
