File: furnace/furnace_controller/furnace_controller.sch (KiCad schematic (older format))
At the start: 10 parts, among them J1 DG141R-2.54-02P, J2 DG141R-2.54-02P, J3 DG141R-2.54-02P, J4 DG141R-2.54-02P, J5 DG141R-2.54-02P, J6 IDC-6

Commit message: Add files via upload
Parts:
- added H4, H5: MountingHole, furnace_controller:hole_D3.5mm, symbol Mechanical:MountingHole
Connections:
- net TC+0: now also J1.1 (Pin_1); no longer J1.2 (Pin_2)
- net TC+1: now also J2.1 (Pin_1); no longer J2.2 (Pin_2)
- net TC+2: now also J3.1 (Pin_1); no longer J3.2 (Pin_2)
- net TC+3: now also J4.1 (Pin_1); no longer J4.2 (Pin_2)
- net TC+4: now also J5.1 (Pin_1); no longer J5.2 (Pin_2)
- net TC-0: now also J1.2 (Pin_2); no longer J1.1 (Pin_1)
- net TC-1: now also J2.2 (Pin_2); no longer J2.1 (Pin_1)
- net TC-2: now also J3.2 (Pin_2); no longer J3.1 (Pin_1)
- net TC-3: now also J4.2 (Pin_2); no longer J4.1 (Pin_1)
- net TC-4: now also J5.2 (Pin_2); no longer J5.1 (Pin_1)
Changed lines of the file:
@@
 Sheet 1 18
 Title "Furnace controller"
-Date "2021-09-24"
+Date "2021-09-30"
 Rev "1.0"
 Comp "Yuriy Volkov"
@@
 $EndSheet
 $Comp
-L Connector:Screw_Terminal_01x02 J2
-U 1 1 60B4A84C
-P 1300 4500
-F 0 "J2" H 1380 4492 50  0000 L CNN
-F 1 "DG141R-2.54-02P" H 1380 4401 50  0001 L CNN
-F 2 "furnace_controller:DG141R-2.54-02P" H 1300 4500 50  0001 C CNN
-F 3 "~" H 1300 4500 50  0001 C CNN
-	1    1300 4500
-	-1   0    0    -1
-$EndComp
-$Comp
 L Connector:Screw_Terminal_01x02 J3
 U 1 1 60B4A967
@@
 Wire Bus Line
 	3000 3850 2500 3850
-Entry Wire Line
-	1900 4100 2000 4200
-Entry Wire Line
-	2400 4000 2500 4100
 Text Label 1600 4100 0    50   ~ 0
+TC-0
+Text Label 1600 4600 0    50   ~ 0
+TC-1
+Text Label 1600 5100 0    50   ~ 0
+TC-2
+Text Label 1600 5600 0    50   ~ 0
+TC-3
+Text Label 1600 6100 0    50   ~ 0
+TC-4
+Text Label 1600 4000 0    50   ~ 0
 TC+0
-Text Label 1600 4600 0    50   ~ 0
+Text Label 1600 4500 0    50   ~ 0
 TC+1
-Text Label 1600 5100 0    50   ~ 0
+Text Label 1600 5000 0    50   ~ 0
 TC+2
-Text Label 1600 5600 0    50   ~ 0
+Text Label 1600 5500 0    50   ~ 0
 TC+3
-Text Label 1600 6100 0    50   ~ 0
+Text Label 1600 6000 0    50   ~ 0
 TC+4
-Text Label 1600 4000 0    50   ~ 0
-TC-0
-Text Label 1600 4500 0    50   ~ 0
-TC-1
-Text Label 1600 5000 0    50   ~ 0
-TC-2
-Text Label 1600 5500 0    50   ~ 0
-TC-3
-Text Label 1600 6000 0    50   ~ 0
-TC-4
 Wire Wire Line
 	4000 1600 4100 1600
@@
 Wire Wire Line
 	6700 4800 6500 4800
-Wire Wire Line
-	1900 4100 1500 4100
-Wire Wire Line
-	2400 4000 1500 4000
-Entry Wire Line
-	1900 4600 2000 4700
-Entry Wire Line
-	2400 4500 2500 4600
-Entry Wire Line
-	1900 5100 2000 5200
-Entry Wire Line
-	2400 5000 2500 5100
-Entry Wire Line
-	1900 5600 2000 5700
-Entry Wire Line
-	2400 5500 2500 5600
-Entry Wire Line
-	1900 6100 2000 6200
-Entry Wire Line
-	2400 6000 2500 6100
-Wire Wire Line
-	2400 4500 1500 4500
-Wire Wire Line
-	1900 4600 1500 4600
-Wire Wire Line
-	2400 5000 1500 5000
-Wire Wire Line
-	1900 5100 1500 5100
-Wire Wire Line
-	2400 5500 1500 5500
-Wire Wire Line
-	1900 5600 1500 5600
-Wire Wire Line
-	2400 6000 1500 6000
-Wire Wire Line
-	1900 6100 1500 6100
-Wire Bus Line
-	2000 3650 2000 6300
+$Comp
+L Connector:Screw_Terminal_01x02 J2
+U 1 1 60B4A84C
+P 1300 4500
+F 0 "J2" H 1380 4492 50  0000 L CNN
+F 1 "DG141R-2.54-02P" H 1380 4401 50  0001 L CNN
+F 2 "furnace_controller:DG141R-2.54-02P" H 1300 4500 50  0001 C CNN
+F 3 "~" H 1300 4500 50  0001 C CNN
+	1    1300 4500
+	-1   0    0    -1
+$EndComp
+Entry Wire Line
+	1900 4000 2000 3900
+Entry Wire Line
+	2400 4100 2500 4000
+Wire Wire Line
+	2400 4100 1500 4100
+Entry Wire Line
+	1900 4500 2000 4400
+Entry Wire Line
+	2400 4600 2500 4500
+Entry Wire Line
+	1900 5000 2000 4900
+Entry Wire Line
+	2400 5100 2500 5000
+Entry Wire Line
+	1900 5500 2000 5400
+Entry Wire Line
+	2400 5600 2500 5500
+Entry Wire Line
+	1900 6000 2000 5900
+Entry Wire Line
+	2400 6100 2500 6000
+Wire Wire Line
+	2400 6100 1500 6100
+Wire Wire Line
+	2400 5600 1500 5600
+Wire Wire Line
+	2400 4600 1500 4600
+Wire Wire Line
+	1500 4000 1900 4000
+Wire Wire Line
+	1500 4500 1900 4500
+Wire Wire Line
+	1500 5000 1900 5000
+Wire Wire Line
+	1500 5100 2400 5100
+Wire Wire Line
+	1500 5500 1900 5500
+Wire Wire Line
+	1500 6000 1900 6000
+$Comp
+L Mechanical:MountingHole H4
+U 1 1 6153166D
+P 5000 6500
+F 0 "H4" H 5100 6550 50  0000 L CNN
+F 1 "MountingHole" H 5100 6455 50  0001 L CNN
+F 2 "furnace_controller:hole_D3.5mm" H 5000 6500 50  0001 C CNN
+F 3 "~" H 5000 6500 50  0001 C CNN
+	1    5000 6500
+	1    0    0    -1
+$EndComp
+$Comp
+L Mechanical:MountingHole H5
+U 1 1 61533E8A
+P 5500 6500
+F 0 "H5" H 5600 6550 50  0000 L CNN
+F 1 "MountingHole" H 5600 6455 50  0001 L CNN
+F 2 "furnace_controller:hole_D3.5mm" H 5500 6500 50  0001 C CNN
+F 3 "~" H 5500 6500 50  0001 C CNN
+	1    5500 6500
+	1    0    0    -1
+$EndComp
+Wire Bus Line
+	2000 3650 2000 6200
 Wire Bus Line
 	2500 3850 2500 6200
