File: furnace/furnace_controller/Power_3V3_10V.sch (KiCad schematic (older format))
At the start: 25 parts

Commit message: Add files via upload
Connections:
- net +10V: now also TP?.1
- net +3V3: now also TP?.1
- net CHARGE_PUMP_CLK: now also D?.1; no longer D?.3
- net at R?.2: now also D?.3; no longer D?.2
Other:
- moved on the sheet: D?, Q?, R?
Changed lines of the file:
@@
 $Descr A4 11693 8268
 encoding utf-8
-Sheet 14 14
+Sheet 13 15
 Title ""
 Date ""
@@
 Connection ~ 7300 2550
 Wire Wire Line
-	7300 2550 7700 2550
+	7300 2550 7450 2550
 Wire Wire Line
 	7700 2450 7700 2550
@@
 L Transistor_FET:IRLML6402 Q?
 U 1 1 60A19F59
-P 6400 4550
-F 0 "Q?" H 6604 4504 50  0000 L CNN
-F 1 "IRLML6402" H 6604 4595 50  0000 L CNN
-F 2 "Package_TO_SOT_SMD:SOT-23" H 6600 4475 50  0001 L CIN
-F 3 "https://www.infineon.com/dgdl/irlml6402pbf.pdf?fileId=5546d462533600a401535668d5c2263c" H 6400 4550 50  0001 L CNN
-	1    6400 4550
+P 6400 4650
+F 0 "Q?" H 6604 4604 50  0000 L CNN
+F 1 "IRLML6402" H 6604 4695 50  0000 L CNN
+F 2 "Package_TO_SOT_SMD:SOT-23" H 6600 4575 50  0001 L CIN
+F 3 "https://www.infineon.com/dgdl/irlml6402pbf.pdf?fileId=5546d462533600a401535668d5c2263c" H 6400 4650 50  0001 L CNN
+	1    6400 4650
 	1    0    0    1
 $EndComp
@@
 L Diode:BAT54S D?
 U 1 1 60A281E0
-P 5400 4250
-F 0 "D?" H 5400 4475 50  0000 C CNN
-F 1 "BAT54S" H 5400 4384 50  0000 C CNN
-F 2 "Package_TO_SOT_SMD:SOT-23" H 5475 4375 50  0001 L CNN
-F 3 "https://www.diodes.com/assets/Datasheets/ds11005.pdf" H 5280 4250 50  0001 C CNN
-	1    5400 4250
-	1    0    0    -1
+P 5400 4350
+F 0 "D?" V 5500 4550 50  0000 C CNN
+F 1 "BAT54S" V 5400 4484 50  0000 C CNN
+F 2 "Package_TO_SOT_SMD:SOT-23" H 5475 4475 50  0001 L CNN
+F 3 "https://www.diodes.com/assets/Datasheets/ds11005.pdf" H 5280 4350 50  0001 C CNN
+	1    5400 4350
+	0    -1   -1   0
 $EndComp
 $Comp
@@
 L Device:R R?
 U 1 1 60A272DA
-P 5950 4250
+P 5950 4350
 AR Path="/60A272DA" Ref="R?"  Part="1"
 AR Path="/609FED99/60A272DA" Ref="R?"  Part="1"
-F 0 "R?" V 5850 4200 50  0000 L CNN
-F 1 "100" V 6050 4150 50  0000 L CNN
-F 2 "Resistor_SMD:R_0603_1608Metric_Pad0.98x0.95mm_HandSolder" V 5880 4250 50  0001 C CNN
-F 3 "~" H 5950 4250 50  0001 C CNN
-	1    5950 4250
+F 0 "R?" V 5850 4300 50  0000 L CNN
+F 1 "100" V 6050 4250 50  0000 L CNN
+F 2 "Resistor_SMD:R_0603_1608Metric_Pad0.98x0.95mm_HandSolder" V 5880 4350 50  0001 C CNN
+F 3 "~" H 5950 4350 50  0001 C CNN
+	1    5950 4350
 	0    1    1    0
 $EndComp
@@
 L Device:R R?
 U 1 1 60A440E9
-P 5950 4550
+P 5950 4650
 AR Path="/60A440E9" Ref="R?"  Part="1"
 AR Path="/609FED99/60A440E9" Ref="R?"  Part="1"
-F 0 "R?" V 5850 4500 50  0000 L CNN
-F 1 "680" V 6050 4450 50  0000 L CNN
-F 2 "Resistor_SMD:R_0603_1608Metric_Pad0.98x0.95mm_HandSolder" V 5880 4550 50  0001 C CNN
-F 3 "~" H 5950 4550 50  0001 C CNN
-	1    5950 4550
+F 0 "R?" V 5850 4600 50  0000 L CNN
+F 1 "680" V 6050 4550 50  0000 L CNN
+F 2 "Resistor_SMD:R_0603_1608Metric_Pad0.98x0.95mm_HandSolder" V 5880 4650 50  0001 C CNN
+F 3 "~" H 5950 4650 50  0001 C CNN
+	1    5950 4650
 	0    1    1    0
 $EndComp
@@
 	4500 3850 4500 3900
 Wire Wire Line
-	5800 4550 5400 4550
-Wire Wire Line
-	4500 4550 4500 4250
-Wire Wire Line
 	5800 5550 5400 5550
 Wire Wire Line
 	4500 5550 4500 4900
-Connection ~ 4500 4550
 Wire Wire Line
 	5400 5450 5400 5550
@@
 	5400 5550 4500 5550
 Wire Wire Line
-	5400 4450 5400 4550
-Connection ~ 5400 4550
-Wire Wire Line
-	5400 4550 4500 4550
-Wire Wire Line
-	5700 4250 5800 4250
-Wire Wire Line
-	6100 4250 6200 4250
-Wire Wire Line
-	6200 4250 6200 4550
-Wire Wire Line
-	6200 4550 6100 4550
-Connection ~ 6200 4550
+	6100 4350 6200 4350
+Wire Wire Line
+	6200 4350 6200 4650
+Wire Wire Line
+	6200 4650 6100 4650
+Connection ~ 6200 4650
 Wire Wire Line
 	5700 5250 5800 5250
@@
 Connection ~ 6200 5550
 Wire Wire Line
-	6500 4750 6500 5050
-Wire Wire Line
-	4500 3900 6500 3900
-Wire Wire Line
-	6500 3900 6500 4350
+	6500 4850 6500 5050
 Connection ~ 4500 3900
 Wire Wire Line
 	4500 3900 4500 3950
 NoConn ~ 5100 5250
-NoConn ~ 5100 4250
 Connection ~ 4500 4900
 Wire Wire Line
-	4500 4900 4500 4550
+	4500 4900 4500 4650
 Text HLabel 2900 4900 0    50   Input ~ 0
 CHARGE_PUMP_CLK
@@
 MCU pin should be \n5V tolerant and \nopen drain
 Wire Wire Line
-	7100 3900 6500 3900
-Connection ~ 6500 3900
-Wire Wire Line
-	7400 4100 7400 4400
-Wire Wire Line
 	7900 4400 7400 4400
-Connection ~ 7400 4400
 Wire Wire Line
 	7900 4700 7400 4700
@@
 Connection ~ 6500 5050
 Wire Wire Line
-	6500 5050 6500 5350
-Wire Wire Line
 	8900 4700 9400 4700
 Wire Wire Line
 	8900 4400 9400 4400
 Wire Wire Line
-	7700 3900 8900 3900
+	7700 3900 8450 3900
 Wire Wire Line
 	8900 3900 8900 3800
@@
 Wire Wire Line
 	5300 2850 5850 2850
+Wire Wire Line
+	4500 4650 5400 4650
+Connection ~ 4500 4650
+Wire Wire Line
+	4500 4250 4500 4650
+Wire Wire Line
+	4500 3900 6500 3900
+Wire Wire Line
+	5400 4650 5800 4650
+Wire Wire Line
+	6500 5050 6500 5350
+Connection ~ 5400 4650
+Wire Wire Line
+	5600 4350 5800 4350
+NoConn ~ 5400 4050
+Wire Wire Line
+	6500 4450 6500 3900
+Connection ~ 6500 3900
+Wire Wire Line
+	6500 3900 7100 3900
+Wire Wire Line
+	7400 4100 7400 4400
+Connection ~ 7400 4400
+Wire Wire Line
+	8450 3800 8450 3900
+Connection ~ 8450 3900
+Wire Wire Line
+	8450 3900 8900 3900
+Wire Wire Line
+	7450 2450 7450 2550
+Connection ~ 7450 2550
+Wire Wire Line
+	7450 2550 7700 2550
 $EndSCHEMATC

Commit message: Add files via upload
Other:
- moved on the sheet: TP?
Changed lines of the file:
@@
 $Descr A4 11693 8268
 encoding utf-8
-Sheet 13 15
+Sheet 3 18
 Title ""
 Date ""
@@
 Wire Wire Line
 	7000 2550 7300 2550
-Connection ~ 7300 2550
-Wire Wire Line
-	7300 2550 7450 2550
 Wire Wire Line
 	7700 2450 7700 2550
-Connection ~ 7700 2550
 Wire Wire Line
 	7700 2850 7300 2850
@@
 	8900 4400 9400 4400
 Wire Wire Line
-	7700 3900 8450 3900
-Wire Wire Line
 	8900 3900 8900 3800
 Wire Wire Line
@@
 L Connector:TestPoint TP?
 U 1 1 60AC6F73
-P 7450 2450
+P 7450 2550
 AR Path="/60AC6F73" Ref="TP?"  Part="1"
 AR Path="/609FED99/60AC6F73" Ref="TP?"  Part="1"
-F 0 "TP?" H 7508 2568 50  0000 L CNN
-F 1 "TestPoint" H 7508 2477 50  0001 L CNN
-F 2 "" H 7650 2450 50  0001 C CNN
-F 3 "~" H 7650 2450 50  0001 C CNN
-	1    7450 2450
+F 0 "TP?" H 7508 2668 50  0000 L CNN
+F 1 "TestPoint" H 7508 2577 50  0001 L CNN
+F 2 "" H 7650 2550 50  0001 C CNN
+F 3 "~" H 7650 2550 50  0001 C CNN
+	1    7450 2550
 	1    0    0    -1
 $EndComp
@@
 L Connector:TestPoint TP?
 U 1 1 60AC7FF7
-P 8450 3800
+P 8450 3900
 AR Path="/60AC7FF7" Ref="TP?"  Part="1"
 AR Path="/609FED99/60AC7FF7" Ref="TP?"  Part="1"
-F 0 "TP?" H 8508 3918 50  0000 L CNN
-F 1 "TestPoint" H 8508 3827 50  0001 L CNN
-F 2 "" H 8650 3800 50  0001 C CNN
-F 3 "~" H 8650 3800 50  0001 C CNN
-	1    8450 3800
+F 0 "TP?" H 8508 4018 50  0000 L CNN
+F 1 "TestPoint" H 8508 3927 50  0001 L CNN
+F 2 "" H 8650 3900 50  0001 C CNN
+F 3 "~" H 8650 3900 50  0001 C CNN
+	1    8450 3900
 	1    0    0    -1
 $EndComp
@@
 Wire Wire Line
 	4250 2850 4750 2850
-Connection ~ 4750 2850
-Wire Wire Line
-	4750 2850 5300 2850
 Wire Wire Line
 	6700 2850 7300 2850
 Wire Wire Line
 	5850 2950 5850 2850
-Connection ~ 5850 2850
 Wire Wire Line
 	5850 2850 6100 2850
@@
 L Connector:TestPoint TP?
 U 1 1 60AFF250
-P 5300 2750
+P 5300 2850
 AR Path="/60AFF250" Ref="TP?"  Part="1"
 AR Path="/609FED99/60AFF250" Ref="TP?"  Part="1"
-F 0 "TP?" H 5358 2868 50  0000 L CNN
-F 1 "TestPoint" H 5358 2777 50  0001 L CNN
-F 2 "" H 5500 2750 50  0001 C CNN
-F 3 "~" H 5500 2750 50  0001 C CNN
-	1    5300 2750
-	1    0    0    -1
-$EndComp
-Wire Wire Line
-	5300 2750 5300 2850
-Connection ~ 5300 2850
-Wire Wire Line
-	5300 2850 5850 2850
+F 0 "TP?" H 5358 2968 50  0000 L CNN
+F 1 "TestPoint" H 5358 2877 50  0001 L CNN
+F 2 "" H 5500 2850 50  0001 C CNN
+F 3 "~" H 5500 2850 50  0001 C CNN
+	1    5300 2850
+	1    0    0    -1
+$EndComp
 Wire Wire Line
 	4500 4650 5400 4650
@@
 Connection ~ 7400 4400
 Wire Wire Line
-	8450 3800 8450 3900
+	8450 3900 8900 3900
+Wire Wire Line
+	4750 2850 5300 2850
+Connection ~ 4750 2850
+Wire Wire Line
+	5300 2850 5850 2850
+Connection ~ 5300 2850
+Connection ~ 5850 2850
+Wire Wire Line
+	7300 2550 7450 2550
+Connection ~ 7300 2550
+Wire Wire Line
+	7450 2550 7700 2550
+Connection ~ 7450 2550
+Connection ~ 7700 2550
+Wire Wire Line
+	8450 3900 7700 3900
 Connection ~ 8450 3900
-Wire Wire Line
-	8450 3900 8900 3900
-Wire Wire Line
-	7450 2450 7450 2550
-Connection ~ 7450 2550
-Wire Wire Line
-	7450 2550 7700 2550
 $EndSCHEMATC

Commit message: Add files via upload
Changed lines of the file:
@@
 $Descr A4 11693 8268
 encoding utf-8
-Sheet 3 17
+Sheet 3 18
 Title ""
 Date ""
@@
 Wire Wire Line
 	5850 2850 6100 2850
-Text HLabel 2900 2850 0    50   Input ~ 0
--5V_IN
 Wire Wire Line
 	2900 2850 3700 2850
@@
 	8450 3900 7700 3900
 Connection ~ 8450 3900
+Text HLabel 2900 2850 0    50   Input ~ 0
+GND_IN
 $EndSCHEMATC

Commit message: Add files via upload
Parts:
- added Q?: BC847, Package_TO_SOT_SMD:SOT-23, symbol Transistor_BJT:BC847
- added R?: 56k, Resistor_SMD:R_0603_1608Metric_Pad0.98x0.95mm_HandSolder, symbol Device:R
- added R?: 3,3k, Resistor_SMD:R_0603_1608Metric_Pad0.98x0.95mm_HandSolder, symbol Device:R
Connections:
- net CHARGE_PUMP_CLK: now also R?.1; no longer D?.1, D?.3, R?.2, R?.2, R?.2
- net GND: now also Q?.2 (E), R?.2
- new net: D?.1, D?.3, Q?.3 (C), R?.2, R?.2, R?.2
- new net: Q?.1 (B), R?.1, R?.2
Other:
- note removed: "MCU pin should be \n5V tolerant and \nopen drain"
Changed lines of the file:
@@
 	5800 5550 5400 5550
-Wire Wire Line
-	4500 5550 4500 4900
 Wire Wire Line
 	5400 5450 5400 5550
@@
 	4500 3900 4500 3950
 NoConn ~ 5100 5250
-Connection ~ 4500 4900
-Wire Wire Line
-	4500 4900 4500 4650
-Text HLabel 2900 4900 0    50   Input ~ 0
+Text HLabel 3000 5750 0    50   Input ~ 0
 CHARGE_PUMP_CLK
-Text Notes 3050 4750 0    50   ~ 0
-MCU pin should be \n5V tolerant and \nopen drain
 Wire Wire Line
 	7900 4400 7400 4400
@@
 +5V_IN
 Wire Wire Line
-	2900 4900 4500 4900
-Wire Wire Line
 	2900 2550 3700 2550
 Connection ~ 6100 2550
@@
 Text HLabel 2900 2850 0    50   Input ~ 0
 GND_IN
+Wire Wire Line
+	4500 4650 4500 5550
+$Comp
+L Transistor_BJT:BC847 Q?
+U 1 1 60B184A0
+P 4400 5750
+AR Path="/609C9D41/60B184A0" Ref="Q?"  Part="1"
+AR Path="/60B39FE1/60B184A0" Ref="Q?"  Part="1"
+F 0 "Q?" H 4591 5796 50  0000 L CNN
+F 1 "BC847" H 4591 5705 50  0000 L CNN
+F 2 "Package_TO_SOT_SMD:SOT-23" H 4600 5675 50  0001 L CIN
+F 3 "http://www.infineon.com/dgdl/Infineon-BC847SERIES_BC848SERIES_BC849SERIES_BC850SERIES-DS-v01_01-en.pdf?fileId=db3a304314dca389011541d4630a1657" H 4400 5750 50  0001 L CNN
+	1    4400 5750
+	1    0    0    -1
+$EndComp
+$Comp
+L Device:R R?
+U 1 1 60B184A6
+P 4000 6000
+AR Path="/60B184A6" Ref="R?"  Part="1"
+AR Path="/60B39FE1/60B184A6" Ref="R?"  Part="1"
+F 0 "R?" H 4070 6046 50  0000 L CNN
+F 1 "56k" H 4070 5955 50  0000 L CNN
+F 2 "Resistor_SMD:R_0603_1608Metric_Pad0.98x0.95mm_HandSolder" V 3930 6000 50  0001 C CNN
+F 3 "~" H 4000 6000 50  0001 C CNN
+	1    4000 6000
+	1    0    0    -1
+$EndComp
+$Comp
+L Device:R R?
+U 1 1 60B184AC
+P 3650 5750
+AR Path="/60B184AC" Ref="R?"  Part="1"
+AR Path="/60B39FE1/60B184AC" Ref="R?"  Part="1"
+F 0 "R?" V 3750 5700 50  0000 L CNN
+F 1 "3,3k" V 3550 5650 50  0000 L CNN
+F 2 "Resistor_SMD:R_0603_1608Metric_Pad0.98x0.95mm_HandSolder" V 3580 5750 50  0001 C CNN
+F 3 "~" H 3650 5750 50  0001 C CNN
+	1    3650 5750
+	0    -1   -1   0
+$EndComp
+Wire Wire Line
+	3800 5750 4000 5750
+Wire Wire Line
+	4000 5850 4000 5750
+Connection ~ 4000 5750
+Wire Wire Line
+	4000 5750 4200 5750
+Wire Wire Line
+	4000 6150 4000 6250
+Connection ~ 4500 5550
+$Comp
+L power:GND #PWR?
+U 1 1 60B1D9CB
+P 4500 6250
+F 0 "#PWR?" H 4500 6000 50  0001 C CNN
+F 1 "GND" H 4505 6077 50  0000 C CNN
+F 2 "" H 4500 6250 50  0001 C CNN
+F 3 "" H 4500 6250 50  0001 C CNN
+	1    4500 6250
+	1    0    0    -1
+$EndComp
+Wire Wire Line
+	3500 5750 3000 5750
+Wire Wire Line
+	4000 6250 4500 6250
+Wire Wire Line
+	4500 5950 4500 6250
+Connection ~ 4500 6250
 $EndSCHEMATC

Commit message: Add files via upload
Parts:
- added R? (x2): 56k, Resistor_SMD:R_0603_1608Metric_Pad0.98x0.95mm_HandSolder, symbol Device:R
Connections:
- net +5V: now also R?.1
- net GND: now also R?.2
- net at Q?.1 (G), R?.1, R?.1: now also R?.2
- net at Q?.1 (G), R?.1, R?.1: now also R?.1
- new net: D?.1, R?.2
- new net: D?.3, R?.2
- new net: Q?.3 (C), R?.2
Other:
- moved on the sheet: D?, R?
Changed lines of the file:
@@
 L Diode:BAT54S D?
 U 1 1 60A281E0
-P 5400 4350
-F 0 "D?" V 5500 4550 50  0000 C CNN
-F 1 "BAT54S" V 5400 4484 50  0000 C CNN
-F 2 "Package_TO_SOT_SMD:SOT-23" H 5475 4475 50  0001 L CNN
-F 3 "https://www.diodes.com/assets/Datasheets/ds11005.pdf" H 5280 4350 50  0001 C CNN
-	1    5400 4350
+P 5200 4350
+F 0 "D?" V 5300 4550 50  0000 C CNN
+F 1 "BAT54S" V 5200 4484 50  0000 C CNN
+F 2 "Package_TO_SOT_SMD:SOT-23" H 5275 4475 50  0001 L CNN
+F 3 "https://www.diodes.com/assets/Datasheets/ds11005.pdf" H 5080 4350 50  0001 C CNN
+	1    5200 4350
 	0    -1   -1   0
 $EndComp
@@
 L Diode:BAT54S D?
 U 1 1 60A2A42D
-P 5400 5250
-F 0 "D?" H 5400 5475 50  0000 C CNN
-F 1 "BAT54S" H 5400 5384 50  0000 C CNN
-F 2 "Package_TO_SOT_SMD:SOT-23" H 5475 5375 50  0001 L CNN
-F 3 "https://www.diodes.com/assets/Datasheets/ds11005.pdf" H 5280 5250 50  0001 C CNN
-	1    5400 5250
+P 5200 5250
+F 0 "D?" H 5200 5475 50  0000 C CNN
+F 1 "BAT54S" H 5200 5384 50  0000 C CNN
+F 2 "Package_TO_SOT_SMD:SOT-23" H 5275 5375 50  0001 L CNN
+F 3 "https://www.diodes.com/assets/Datasheets/ds11005.pdf" H 5080 5250 50  0001 C CNN
+	1    5200 5250
 	-1   0    0    -1
 $EndComp
@@
 L Device:R R?
 U 1 1 60A272DA
-P 5950 4350
+P 5750 4350
 AR Path="/60A272DA" Ref="R?"  Part="1"
 AR Path="/609FED99/60A272DA" Ref="R?"  Part="1"
-F 0 "R?" V 5850 4300 50  0000 L CNN
-F 1 "100" V 6050 4250 50  0000 L CNN
-F 2 "Resistor_SMD:R_0603_1608Metric_Pad0.98x0.95mm_HandSolder" V 5880 4350 50  0001 C CNN
-F 3 "~" H 5950 4350 50  0001 C CNN
-	1    5950 4350
+F 0 "R?" V 5650 4300 50  0000 L CNN
+F 1 "100" V 5850 4250 50  0000 L CNN
+F 2 "Resistor_SMD:R_0603_1608Metric_Pad0.98x0.95mm_HandSolder" V 5680 4350 50  0001 C CNN
+F 3 "~" H 5750 4350 50  0001 C CNN
+	1    5750 4350
 	0    1    1    0
 $EndComp
@@
 L Device:R R?
 U 1 1 60A440E9
-P 5950 4650
+P 5750 4650
 AR Path="/60A440E9" Ref="R?"  Part="1"
 AR Path="/609FED99/60A440E9" Ref="R?"  Part="1"
-F 0 "R?" V 5850 4600 50  0000 L CNN
-F 1 "680" V 6050 4550 50  0000 L CNN
-F 2 "Resistor_SMD:R_0603_1608Metric_Pad0.98x0.95mm_HandSolder" V 5880 4650 50  0001 C CNN
-F 3 "~" H 5950 4650 50  0001 C CNN
-	1    5950 4650
+F 0 "R?" V 5650 4600 50  0000 L CNN
+F 1 "680" V 5850 4550 50  0000 L CNN
+F 2 "Resistor_SMD:R_0603_1608Metric_Pad0.98x0.95mm_HandSolder" V 5680 4650 50  0001 C CNN
+F 3 "~" H 5750 4650 50  0001 C CNN
+	1    5750 4650
 	0    1    1    0
 $EndComp
@@
 L Device:R R?
 U 1 1 60A443B1
-P 5950 5250
+P 5750 5250
 AR Path="/60A443B1" Ref="R?"  Part="1"
 AR Path="/609FED99/60A443B1" Ref="R?"  Part="1"
-F 0 "R?" V 5850 5200 50  0000 L CNN
-F 1 "1,2k" V 6050 5150 50  0000 L CNN
-F 2 "Resistor_SMD:R_0603_1608Metric_Pad0.98x0.95mm_HandSolder" V 5880 5250 50  0001 C CNN
-F 3 "~" H 5950 5250 50  0001 C CNN
-	1    5950 5250
+F 0 "R?" V 5650 5200 50  0000 L CNN
+F 1 "1,2k" V 5850 5150 50  0000 L CNN
+F 2 "Resistor_SMD:R_0603_1608Metric_Pad0.98x0.95mm_HandSolder" V 5680 5250 50  0001 C CNN
+F 3 "~" H 5750 5250 50  0001 C CNN
+	1    5750 5250
 	0    1    1    0
 $EndComp
@@
 L Device:R R?
 U 1 1 60A44627
-P 5950 5550
+P 5750 5550
 AR Path="/60A44627" Ref="R?"  Part="1"
 AR Path="/609FED99/60A44627" Ref="R?"  Part="1"
-F 0 "R?" V 5850 5500 50  0000 L CNN
-F 1 "1,2k" V 6050 5450 50  0000 L CNN
-F 2 "Resistor_SMD:R_0603_1608Metric_Pad0.98x0.95mm_HandSolder" V 5880 5550 50  0001 C CNN
-F 3 "~" H 5950 5550 50  0001 C CNN
-	1    5950 5550
+F 0 "R?" V 5650 5500 50  0000 L CNN
+F 1 "1,2k" V 5850 5450 50  0000 L CNN
+F 2 "Resistor_SMD:R_0603_1608Metric_Pad0.98x0.95mm_HandSolder" V 5680 5550 50  0001 C CNN
+F 3 "~" H 5750 5550 50  0001 C CNN
+	1    5750 5550
 	0    1    1    0
 $EndComp
@@
 	4500 3850 4500 3900
 Wire Wire Line
-	5800 5550 5400 5550
-Wire Wire Line
-	5400 5450 5400 5550
-Connection ~ 5400 5550
-Wire Wire Line
-	5400 5550 4500 5550
-Wire Wire Line
-	6100 4350 6200 4350
-Wire Wire Line
-	6200 4350 6200 4650
-Wire Wire Line
-	6200 4650 6100 4650
-Connection ~ 6200 4650
-Wire Wire Line
-	5700 5250 5800 5250
-Wire Wire Line
-	6100 5250 6200 5250
-Wire Wire Line
-	6200 5250 6200 5550
-Wire Wire Line
-	6200 5550 6100 5550
-Connection ~ 6200 5550
+	5600 5550 5200 5550
+Wire Wire Line
+	5200 5450 5200 5550
+Wire Wire Line
+	5500 5250 5600 5250
 Wire Wire Line
 	6500 4850 6500 5050
@@
 Wire Wire Line
 	4500 3900 4500 3950
-NoConn ~ 5100 5250
+NoConn ~ 4900 5250
 Text HLabel 3000 5750 0    50   Input ~ 0
 CHARGE_PUMP_CLK
@@
 Connection ~ 8900 3900
 Connection ~ 8900 4400
-Wire Wire Line
-	8900 4700 8900 5850
-Wire Wire Line
-	8900 5850 6500 5850
-Wire Wire Line
-	6500 5850 6500 5750
 Connection ~ 8900 4700
-Wire Wire Line
-	6500 5850 6500 5950
-Connection ~ 6500 5850
-$Comp
-L power:GND #PWR?
-U 1 1 60AB9561
-P 6500 5950
-F 0 "#PWR?" H 6500 5700 50  0001 C CNN
-F 1 "GND" H 6505 5777 50  0000 C CNN
-F 2 "" H 6500 5950 50  0001 C CNN
-F 3 "" H 6500 5950 50  0001 C CNN
-	1    6500 5950
-	1    0    0    -1
-$EndComp
 $Comp
 L Connector:TestPoint TP?
@@
 $EndComp
 Wire Wire Line
-	4500 4650 5400 4650
-Connection ~ 4500 4650
-Wire Wire Line
-	4500 4250 4500 4650
-Wire Wire Line
-	4500 3900 6500 3900
-Wire Wire Line
-	5400 4650 5800 4650
+	5200 4650 5600 4650
 Wire Wire Line
 	6500 5050 6500 5350
-Connection ~ 5400 4650
-Wire Wire Line
-	5600 4350 5800 4350
+Wire Wire Line
+	5400 4350 5600 4350
 NoConn ~ 5400 4050
 Wire Wire Line
@@
 Text HLabel 2900 2850 0    50   Input ~ 0
 GND_IN
-Wire Wire Line
-	4500 4650 4500 5550
 $Comp
 L Transistor_BJT:BC847 Q?
@@
 AR Path="/609C9D41/60B184A0" Ref="Q?"  Part="1"
 AR Path="/60B39FE1/60B184A0" Ref="Q?"  Part="1"
+AR Path="/609FED99/60B184A0" Ref="Q?"  Part="1"
 F 0 "Q?" H 4591 5796 50  0000 L CNN
 F 1 "BC847" H 4591 5705 50  0000 L CNN
@@
 AR Path="/60B184A6" Ref="R?"  Part="1"
 AR Path="/60B39FE1/60B184A6" Ref="R?"  Part="1"
+AR Path="/609FED99/60B184A6" Ref="R?"  Part="1"
 F 0 "R?" H 4070 6046 50  0000 L CNN
 F 1 "56k" H 4070 5955 50  0000 L CNN
@@
 AR Path="/60B184AC" Ref="R?"  Part="1"
 AR Path="/60B39FE1/60B184AC" Ref="R?"  Part="1"
+AR Path="/609FED99/60B184AC" Ref="R?"  Part="1"
 F 0 "R?" V 3750 5700 50  0000 L CNN
 F 1 "3,3k" V 3550 5650 50  0000 L CNN
@@
 Wire Wire Line
 	4000 6150 4000 6250
-Connection ~ 4500 5550
 $Comp
 L power:GND #PWR?
 U 1 1 60B1D9CB
-P 4500 6250
-F 0 "#PWR?" H 4500 6000 50  0001 C CNN
-F 1 "GND" H 4505 6077 50  0000 C CNN
-F 2 "" H 4500 6250 50  0001 C CNN
-F 3 "" H 4500 6250 50  0001 C CNN
-	1    4500 6250
+P 5400 6250
+F 0 "#PWR?" H 5400 6000 50  0001 C CNN
+F 1 "GND" H 5405 6077 50  0000 C CNN
+F 2 "" H 5400 6250 50  0001 C CNN
+F 3 "" H 5400 6250 50  0001 C CNN
+	1    5400 6250
 	1    0    0    -1
 $EndComp
@@
 	4500 5950 4500 6250
 Connection ~ 4500 6250
+$Comp
+L Device:R R?
+U 1 1 60B13DFF
+P 6100 5900
+AR Path="/60B13DFF" Ref="R?"  Part="1"
+AR Path="/60B39FE1/60B13DFF" Ref="R?"  Part="1"
+AR Path="/609FED99/60B13DFF" Ref="R?"  Part="1"
+F 0 "R?" H 6170 5946 50  0000 L CNN
+F 1 "56k" H 6170 5855 50  0000 L CNN
+F 2 "Resistor_SMD:R_0603_1608Metric_Pad0.98x0.95mm_HandSolder" V 6030 5900 50  0001 C CNN
+F 3 "~" H 6100 5900 50  0001 C CNN
+	1    6100 5900
+	1    0    0    -1
+$EndComp
+Wire Wire Line
+	4500 4250 4500 5550
+$Comp
+L Device:R R?
+U 1 1 60B1B4E2
+P 6100 4150
+AR Path="/60B1B4E2" Ref="R?"  Part="1"
+AR Path="/60B39FE1/60B1B4E2" Ref="R?"  Part="1"
+AR Path="/609FED99/60B1B4E2" Ref="R?"  Part="1"
+F 0 "R?" H 6170 4196 50  0000 L CNN
+F 1 "56k" H 6170 4105 50  0000 L CNN
+F 2 "Resistor_SMD:R_0603_1608Metric_Pad0.98x0.95mm_HandSolder" V 6030 4150 50  0001 C CNN
+F 3 "~" H 6100 4150 50  0001 C CNN
+	1    6100 4150
+	1    0    0    -1
+$EndComp
+Wire Wire Line
+	4500 3900 6100 3900
+Wire Wire Line
+	6100 4000 6100 3900
+Connection ~ 6100 3900
+Wire Wire Line
+	6100 3900 6500 3900
+Wire Wire Line
+	5900 4650 6000 4650
+Connection ~ 6100 4650
+Wire Wire Line
+	6100 4650 6200 4650
+Wire Wire Line
+	4500 6250 5400 6250
+Wire Wire Line
+	8900 4700 8900 6250
+Wire Wire Line
+	5900 5550 6000 5550
+Wire Wire Line
+	6100 5750 6100 5550
+Connection ~ 6100 5550
+Wire Wire Line
+	6100 5550 6200 5550
+Wire Wire Line
+	6100 6050 6100 6250
+Connection ~ 6100 6250
+Wire Wire Line
+	6100 6250 6500 6250
+Wire Wire Line
+	5900 5250 6000 5250
+Wire Wire Line
+	6000 5250 6000 5550
+Connection ~ 6000 5550
+Wire Wire Line
+	6000 5550 6100 5550
+Wire Wire Line
+	6100 4300 6100 4650
+Wire Wire Line
+	5900 4350 6000 4350
+Wire Wire Line
+	6000 4350 6000 4650
+Connection ~ 6000 4650
+Wire Wire Line
+	6000 4650 6100 4650
+Connection ~ 5400 6250
+Wire Wire Line
+	5400 6250 6100 6250
+Wire Wire Line
+	6500 5750 6500 6250
+Connection ~ 6500 6250
+Wire Wire Line
+	6500 6250 8900 6250
 $EndSCHEMATC

Commit message: Add files via upload
Connections:
- net at D?.1, R?.2: now also D?.3, Q?.3 (C), R?.2, R?.2
Changed lines of the file:
@@
 $EndComp
 Wire Wire Line
-	4500 4250 4500 5550
+	4500 4250 4500 4650
 $Comp
 L Device:R R?
@@
 Wire Wire Line
 	6500 6250 8900 6250
+Wire Wire Line
+	5200 4650 4500 4650
+Connection ~ 5200 4650
+Connection ~ 4500 4650
+Wire Wire Line
+	4500 4650 4500 5550
+Wire Wire Line
+	5200 5550 4500 5550
+Connection ~ 5200 5550
+Connection ~ 4500 5550
 $EndSCHEMATC
