File: furnace/furnace_controller/Power_3V3_10V.sch (KiCad schematic (older format))
At the start: 30 parts

Commit message: Add files via upload
Parts:
- gave numbers to parts that had none: 30

Commit message: Add files via upload
Parts:
- added F1: 0.2A, symbol Device:Polyfuse
Connections:
- net +5V: now also F1.1
- new net +5V_IN: F1.2
Other:
- moved on the sheet: C11, C12, C13, C14, C16, D1, TP1, TP2, TP3, U2

Commit message: Add files via upload
Changed lines of the file:
@@
 Connection ~ 6000 2500
 Wire Wire Line
-	6000 2500 6500 2500
+	6000 2500 6250 2500
 Wire Wire Line
 	6500 2400 6500 2500
@@
 	8450 3900 8900 3900
 Wire Wire Line
-	6000 3000 6500 3000
+	6000 3000 6250 3000
 Connection ~ 6000 3000
 Connection ~ 6500 3000
@@
 Connection ~ 8250 2500
 Wire Wire Line
-	8450 3900 7700 3900
+	8450 3900 8000 3900
 Connection ~ 8450 3900
 Text HLabel 3500 3000 0    50   Input ~ 0
@@
 Connection ~ 5550 3000
 Wire Wire Line
-	5550 3000 6000 3000
-Wire Wire Line
 	5550 2600 5550 2500
 Connection ~ 5550 2500
 Wire Wire Line
-	5550 2500 6000 2500
-Wire Wire Line
 	7000 2600 7000 2500
 Connection ~ 7000 2500
@@
 Wire Wire Line
 	8500 2900 8500 3000
+$Comp
+L power:PWR_FLAG #FLG0101
+U 1 1 6127C7A9
+P 8000 3900
+F 0 "#FLG0101" H 8000 3975 50  0001 C CNN
+F 1 "PWR_FLAG" H 8000 4073 50  0000 C CNN
+F 2 "" H 8000 3900 50  0001 C CNN
+F 3 "~" H 8000 3900 50  0001 C CNN
+	1    8000 3900
+	1    0    0    -1
+$EndComp
+Connection ~ 8000 3900
+Wire Wire Line
+	8000 3900 7700 3900
+$Comp
+L power:PWR_FLAG #FLG0102
+U 1 1 612826C0
+P 6250 3000
+F 0 "#FLG0102" H 6250 3075 50  0001 C CNN
+F 1 "PWR_FLAG" H 6250 2950 50  0000 C CNN
+F 2 "" H 6250 3000 50  0001 C CNN
+F 3 "~" H 6250 3000 50  0001 C CNN
+	1    6250 3000
+	1    0    0    -1
+$EndComp
+Connection ~ 6250 3000
+Wire Wire Line
+	6250 3000 6500 3000
+Wire Wire Line
+	5550 3000 6000 3000
+$Comp
+L power:PWR_FLAG #FLG0103
+U 1 1 61282069
+P 6250 2500
+F 0 "#FLG0103" H 6250 2575 50  0001 C CNN
+F 1 "PWR_FLAG" H 6300 2450 50  0000 C CNN
+F 2 "" H 6250 2500 50  0001 C CNN
+F 3 "~" H 6250 2500 50  0001 C CNN
+	1    6250 2500
+	1    0    0    -1
+$EndComp
+Wire Wire Line
+	5550 2500 6000 2500
+Connection ~ 6250 2500
+Wire Wire Line
+	6250 2500 6500 2500
 $EndSCHEMATC

Commit message: Add files via upload
Parts:
- C11: footprint (none) -> Capacitor_THT:CP_Radial_D5.0mm_P2.00mm
- C12, C13: footprint Capacitor_SMD:C_0603_1608Metric_Pad1.08x0.95mm_HandSolder -> Capacitor_SMD:C_0603_1608Metric_Pad1.05x0.95mm_HandSolder
- C14, C15, C16, C17, C18, C19: footprint Capacitor_SMD:C_1206_3216Metric_Pad1.33x1.80mm_HandSolder -> Capacitor_SMD:C_1206_3216Metric_Pad1.42x1.75mm_HandSolder
- D1: footprint (none) -> Diode_SMD:D_SMB_Handsoldering
- F1: footprint (none) -> Fuse:Fuse_1206_3216Metric_Pad1.42x1.75mm_HandSolder
- R10, R11, R12, R13, R14, R15, R16, R8, R9: footprint Resistor_SMD:R_0603_1608Metric_Pad0.98x0.95mm_HandSolder -> Resistor_SMD:R_0603_1608Metric_Pad1.05x0.95mm_HandSolder
- TP1, TP2, TP3, TP4: footprint (none) -> furnace_controller:TP
Changed lines of the file:
@@
 encoding utf-8
 Sheet 2 18
-Title ""
-Date ""
-Rev ""
-Comp ""
+Title "Furnace controller"
+Date "2021-08-26"
+Rev "1.0"
+Comp "Yuriy Volkov"
 Comment1 ""
 Comment2 ""
@@
 F 0 "C14" H 8115 2796 50  0000 L CNN
 F 1 "10u" H 8115 2705 50  0000 L CNN
-F 2 "Capacitor_SMD:C_1206_3216Metric_Pad1.33x1.80mm_HandSolder" H 8038 2600 50  0001 C CNN
+F 2 "Capacitor_SMD:C_1206_3216Metric_Pad1.42x1.75mm_HandSolder" H 8038 2600 50  0001 C CNN
 F 3 "~" H 8000 2750 50  0001 C CNN
 	1    8000 2750
@@
 F 0 "C13" H 7115 2796 50  0000 L CNN
 F 1 "0,1" H 7115 2705 50  0000 L CNN
-F 2 "Capacitor_SMD:C_0603_1608Metric_Pad1.08x0.95mm_HandSolder" H 7038 2600 50  0001 C CNN
+F 2 "Capacitor_SMD:C_0603_1608Metric_Pad1.05x0.95mm_HandSolder" H 7038 2600 50  0001 C CNN
 F 3 "~" H 7000 2750 50  0001 C CNN
 	1    7000 2750
@@
 F 0 "C16" H 8615 2796 50  0000 L CNN
 F 1 "10u" H 8615 2705 50  0000 L CNN
-F 2 "Capacitor_SMD:C_1206_3216Metric_Pad1.33x1.80mm_HandSolder" H 8538 2600 50  0001 C CNN
+F 2 "Capacitor_SMD:C_1206_3216Metric_Pad1.42x1.75mm_HandSolder" H 8538 2600 50  0001 C CNN
 F 3 "~" H 8500 2750 50  0001 C CNN
 	1    8500 2750
@@
 F 0 "C15" H 7515 4596 50  0000 L CNN
 F 1 "10u" H 7515 4505 50  0000 L CNN
-F 2 "Capacitor_SMD:C_1206_3216Metric_Pad1.33x1.80mm_HandSolder" H 7438 4400 50  0001 C CNN
+F 2 "Capacitor_SMD:C_1206_3216Metric_Pad1.42x1.75mm_HandSolder" H 7438 4400 50  0001 C CNN
 F 3 "~" H 7400 4550 50  0001 C CNN
 	1    7400 4550
@@
 F 0 "C17" H 8015 4596 50  0000 L CNN
 F 1 "10u" H 8015 4505 50  0000 L CNN
-F 2 "Capacitor_SMD:C_1206_3216Metric_Pad1.33x1.80mm_HandSolder" H 7938 4400 50  0001 C CNN
+F 2 "Capacitor_SMD:C_1206_3216Metric_Pad1.42x1.75mm_HandSolder" H 7938 4400 50  0001 C CNN
 F 3 "~" H 7900 4550 50  0001 C CNN
 	1    7900 4550
@@
 F 0 "C18" H 9015 4596 50  0000 L CNN
 F 1 "10u" H 9015 4505 50  0000 L CNN
-F 2 "Capacitor_SMD:C_1206_3216Metric_Pad1.33x1.80mm_HandSolder" H 8938 4400 50  0001 C CNN
+F 2 "Capacitor_SMD:C_1206_3216Metric_Pad1.42x1.75mm_HandSolder" H 8938 4400 50  0001 C CNN
 F 3 "~" H 8900 4550 50  0001 C CNN
 	1    8900 4550
@@
 F 0 "C19" H 9515 4596 50  0000 L CNN
 F 1 "10u" H 9515 4505 50  0000 L CNN
-F 2 "Capacitor_SMD:C_1206_3216Metric_Pad1.33x1.80mm_HandSolder" H 9438 4400 50  0001 C CNN
+F 2 "Capacitor_SMD:C_1206_3216Metric_Pad1.42x1.75mm_HandSolder" H 9438 4400 50  0001 C CNN
 F 3 "~" H 9400 4550 50  0001 C CNN
 	1    9400 4550
@@
 F 0 "R11" V 5650 4300 50  0000 L CNN
 F 1 "100" V 5850 4250 50  0000 L CNN
-F 2 "Resistor_SMD:R_0603_1608Metric_Pad0.98x0.95mm_HandSolder" V 5680 4350 50  0001 C CNN
+F 2 "Resistor_SMD:R_0603_1608Metric_Pad1.05x0.95mm_HandSolder" V 5680 4350 50  0001 C CNN
 F 3 "~" H 5750 4350 50  0001 C CNN
 	1    5750 4350
@@
 F 0 "R12" V 5650 4600 50  0000 L CNN
 F 1 "680" V 5850 4550 50  0000 L CNN
-F 2 "Resistor_SMD:R_0603_1608Metric_Pad0.98x0.95mm_HandSolder" V 5680 4650 50  0001 C CNN
+F 2 "Resistor_SMD:R_0603_1608Metric_Pad1.05x0.95mm_HandSolder" V 5680 4650 50  0001 C CNN
 F 3 "~" H 5750 4650 50  0001 C CNN
 	1    5750 4650
@@
 F 0 "R13" V 5650 5200 50  0000 L CNN
 F 1 "1,2k" V 5850 5150 50  0000 L CNN
-F 2 "Resistor_SMD:R_0603_1608Metric_Pad0.98x0.95mm_HandSolder" V 5680 5250 50  0001 C CNN
+F 2 "Resistor_SMD:R_0603_1608Metric_Pad1.05x0.95mm_HandSolder" V 5680 5250 50  0001 C CNN
 F 3 "~" H 5750 5250 50  0001 C CNN
 	1    5750 5250
@@
 F 0 "R14" V 5650 5500 50  0000 L CNN
 F 1 "1,2k" V 5850 5450 50  0000 L CNN
-F 2 "Resistor_SMD:R_0603_1608Metric_Pad0.98x0.95mm_HandSolder" V 5680 5550 50  0001 C CNN
+F 2 "Resistor_SMD:R_0603_1608Metric_Pad1.05x0.95mm_HandSolder" V 5680 5550 50  0001 C CNN
 F 3 "~" H 5750 5550 50  0001 C CNN
 	1    5750 5550
@@
 F 0 "R10" H 4570 4146 50  0000 L CNN
 F 1 "330" H 4570 4055 50  0000 L CNN
-F 2 "Resistor_SMD:R_0603_1608Metric_Pad0.98x0.95mm_HandSolder" V 4430 4100 50  0001 C CNN
+F 2 "Resistor_SMD:R_0603_1608Metric_Pad1.05x0.95mm_HandSolder" V 4430 4100 50  0001 C CNN
 F 3 "~" H 4500 4100 50  0001 C CNN
 	1    4500 4100
@@
 F 0 "TP3" H 8308 2618 50  0000 L CNN
 F 1 "TestPoint" H 8308 2527 50  0001 L CNN
-F 2 "" H 8450 2500 50  0001 C CNN
+F 2 "furnace_controller:TP" H 8450 2500 50  0001 C CNN
 F 3 "~" H 8450 2500 50  0001 C CNN
 	1    8250 2500
@@
 F 0 "TP4" H 8508 4018 50  0000 L CNN
 F 1 "TestPoint" H 8508 3927 50  0001 L CNN
-F 2 "" H 8650 3900 50  0001 C CNN
+F 2 "furnace_controller:TP" H 8650 3900 50  0001 C CNN
 F 3 "~" H 8650 3900 50  0001 C CNN
 	1    8450 3900
@@
 F 0 "TP1" H 6058 2618 50  0000 L CNN
 F 1 "TestPoint" H 6058 2527 50  0001 L CNN
-F 2 "" H 6200 2500 50  0001 C CNN
+F 2 "furnace_controller:TP" H 6200 2500 50  0001 C CNN
 F 3 "~" H 6200 2500 50  0001 C CNN
 	1    6000 2500
@@
 F 0 "C12" H 5165 2796 50  0000 L CNN
 F 1 "1u" H 5165 2705 50  0000 L CNN
-F 2 "Capacitor_SMD:C_0603_1608Metric_Pad1.08x0.95mm_HandSolder" H 5088 2600 50  0001 C CNN
+F 2 "Capacitor_SMD:C_0603_1608Metric_Pad1.05x0.95mm_HandSolder" H 5088 2600 50  0001 C CNN
 F 3 "~" H 5050 2750 50  0001 C CNN
 	1    5050 2750
@@
 F 0 "D1" V 5596 2670 50  0000 R CNN
 F 1 "SMAJ5.0CA" V 5505 2670 50  0000 R CNN
-F 2 "" H 5550 2750 50  0001 C CNN
+F 2 "Diode_SMD:D_SMB_Handsoldering" H 5550 2750 50  0001 C CNN
 F 3 "~" H 5550 2750 50  0001 C CNN
 	1    5550 2750
@@
 F 0 "C11" H 4618 2796 50  0000 L CNN
 F 1 "100u" H 4618 2705 50  0000 L CNN
-F 2 "" H 4538 2600 50  0001 C CNN
+F 2 "Capacitor_THT:CP_Radial_D5.0mm_P2.00mm" H 4538 2600 50  0001 C CNN
 F 3 "~" H 4500 2750 50  0001 C CNN
 	1    4500 2750
@@
 F 0 "TP2" H 6058 3118 50  0000 L CNN
 F 1 "TestPoint" H 6058 3027 50  0001 L CNN
-F 2 "" H 6200 3000 50  0001 C CNN
+F 2 "furnace_controller:TP" H 6200 3000 50  0001 C CNN
 F 3 "~" H 6200 3000 50  0001 C CNN
 	1    6000 3000
@@
 F 0 "R9" H 4070 6046 50  0000 L CNN
 F 1 "56k" H 4070 5955 50  0000 L CNN
-F 2 "Resistor_SMD:R_0603_1608Metric_Pad0.98x0.95mm_HandSolder" V 3930 6000 50  0001 C CNN
+F 2 "Resistor_SMD:R_0603_1608Metric_Pad1.05x0.95mm_HandSolder" V 3930 6000 50  0001 C CNN
 F 3 "~" H 4000 6000 50  0001 C CNN
 	1    4000 6000
@@
 F 0 "R8" V 3750 5700 50  0000 L CNN
 F 1 "3,3k" V 3550 5650 50  0000 L CNN
-F 2 "Resistor_SMD:R_0603_1608Metric_Pad0.98x0.95mm_HandSolder" V 3580 5750 50  0001 C CNN
+F 2 "Resistor_SMD:R_0603_1608Metric_Pad1.05x0.95mm_HandSolder" V 3580 5750 50  0001 C CNN
 F 3 "~" H 3650 5750 50  0001 C CNN
 	1    3650 5750
@@
 F 0 "R16" H 6170 5946 50  0000 L CNN
 F 1 "56k" H 6170 5855 50  0000 L CNN
-F 2 "Resistor_SMD:R_0603_1608Metric_Pad0.98x0.95mm_HandSolder" V 6030 5900 50  0001 C CNN
+F 2 "Resistor_SMD:R_0603_1608Metric_Pad1.05x0.95mm_HandSolder" V 6030 5900 50  0001 C CNN
 F 3 "~" H 6100 5900 50  0001 C CNN
 	1    6100 5900
@@
 F 0 "R15" H 6170 4196 50  0000 L CNN
 F 1 "56k" H 6170 4105 50  0000 L CNN
-F 2 "Resistor_SMD:R_0603_1608Metric_Pad0.98x0.95mm_HandSolder" V 6030 4150 50  0001 C CNN
+F 2 "Resistor_SMD:R_0603_1608Metric_Pad1.05x0.95mm_HandSolder" V 6030 4150 50  0001 C CNN
 F 3 "~" H 6100 4150 50  0001 C CNN
 	1    6100 4150
@@
 F 0 "F1" V 3950 2500 50  0000 C CNN
 F 1 "0.2A" V 4150 2500 50  0000 C CNN
-F 2 "" H 4100 2300 50  0001 L CNN
+F 2 "Fuse:Fuse_1206_3216Metric_Pad1.42x1.75mm_HandSolder" H 4100 2300 50  0001 L CNN
 F 3 "~" H 4050 2500 50  0001 C CNN
 	1    4050 2500

Commit message: Add files via upload
Parts:
- C2: renamed from C12; footprint Capacitor_SMD:C_0603_1608Metric_Pad1.05x0.95mm_HandSolder -> Capacitor_SMD:C_0603_1608Metric_Pad1.08x0.95mm_HandSolder
- C3: renamed from C13; footprint Capacitor_SMD:C_0603_1608Metric_Pad1.05x0.95mm_HandSolder -> Capacitor_SMD:C_0603_1608Metric_Pad1.08x0.95mm_HandSolder
- C4: renamed from C15; footprint Capacitor_SMD:C_1206_3216Metric_Pad1.42x1.75mm_HandSolder -> Capacitor_SMD:C_1206_3216Metric_Pad1.33x1.80mm_HandSolder
- C5: renamed from C17; footprint Capacitor_SMD:C_1206_3216Metric_Pad1.42x1.75mm_HandSolder -> Capacitor_SMD:C_1206_3216Metric_Pad1.33x1.80mm_HandSolder
- C6: renamed from C14; footprint Capacitor_SMD:C_1206_3216Metric_Pad1.42x1.75mm_HandSolder -> Capacitor_SMD:C_1206_3216Metric_Pad1.33x1.80mm_HandSolder
- C7: renamed from C16; footprint Capacitor_SMD:C_1206_3216Metric_Pad1.42x1.75mm_HandSolder -> Capacitor_SMD:C_1206_3216Metric_Pad1.33x1.80mm_HandSolder
- C8: renamed from C18; footprint Capacitor_SMD:C_1206_3216Metric_Pad1.42x1.75mm_HandSolder -> Capacitor_SMD:C_1206_3216Metric_Pad1.33x1.80mm_HandSolder
- C9: renamed from C19; footprint Capacitor_SMD:C_1206_3216Metric_Pad1.42x1.75mm_HandSolder -> Capacitor_SMD:C_1206_3216Metric_Pad1.33x1.80mm_HandSolder
- R1: renamed from R8; footprint Resistor_SMD:R_0603_1608Metric_Pad1.05x0.95mm_HandSolder -> Resistor_SMD:R_0603_1608Metric_Pad0.98x0.95mm_HandSolder
- R2: renamed from R9; footprint Resistor_SMD:R_0603_1608Metric_Pad1.05x0.95mm_HandSolder -> Resistor_SMD:R_0603_1608Metric_Pad0.98x0.95mm_HandSolder
- R3: renamed from R10; footprint Resistor_SMD:R_0603_1608Metric_Pad1.05x0.95mm_HandSolder -> Resistor_SMD:R_0603_1608Metric_Pad0.98x0.95mm_HandSolder
- R4: renamed from R11; footprint Resistor_SMD:R_0603_1608Metric_Pad1.05x0.95mm_HandSolder -> Resistor_SMD:R_0603_1608Metric_Pad0.98x0.95mm_HandSolder
- R5: renamed from R12; footprint Resistor_SMD:R_0603_1608Metric_Pad1.05x0.95mm_HandSolder -> Resistor_SMD:R_0603_1608Metric_Pad0.98x0.95mm_HandSolder
- R6: renamed from R13; footprint Resistor_SMD:R_0603_1608Metric_Pad1.05x0.95mm_HandSolder -> Resistor_SMD:R_0603_1608Metric_Pad0.98x0.95mm_HandSolder
- R7: renamed from R14; footprint Resistor_SMD:R_0603_1608Metric_Pad1.05x0.95mm_HandSolder -> Resistor_SMD:R_0603_1608Metric_Pad0.98x0.95mm_HandSolder
- R8: renamed from R15; footprint Resistor_SMD:R_0603_1608Metric_Pad1.05x0.95mm_HandSolder -> Resistor_SMD:R_0603_1608Metric_Pad0.98x0.95mm_HandSolder
- R9: renamed from R16; footprint Resistor_SMD:R_0603_1608Metric_Pad1.05x0.95mm_HandSolder -> Resistor_SMD:R_0603_1608Metric_Pad0.98x0.95mm_HandSolder
- renumbered C11 to C1, D2 to D1, D3 to D2, D1 to D3, Q2 to Q1, Q3 to Q2, Q4 to Q3, U2 to U1
