File: furnace/furnace_controller/+3V3_isolated.sch (KiCad schematic (older format))
At the start: 13 parts

Commit message: Add files via upload
Parts:
- PS?: symbol B0505S-1WR2:B0505S-1WR2 -> furnace_controller-rescue:B0505S-1WR2-B0505S-1WR2
- U?: symbol Regulator_Linear:LM317L_SO8 -> furnace_controller-rescue:LM317L_SO8-Regulator_Linear
Changed lines of the file:
@@
 $Descr A4 11693 8268
 encoding utf-8
-Sheet 7 13
+Sheet 7 14
 Title ""
 Date ""
@@
 $EndDescr
 $Comp
-L B0505S-1WR2:B0505S-1WR2 PS?
+L furnace_controller-rescue:B0505S-1WR2-B0505S-1WR2 PS?
 U 1 1 60AE766F
 P 4050 3600
@@
 	4750 3500 4550 3500
 $Comp
-L Regulator_Linear:LM317L_SO8 U?
+L furnace_controller-rescue:LM317L_SO8-Regulator_Linear U?
 U 1 1 60AE76B8
 P 6900 3500

Commit message: Add files via upload
Other:
- moved on the sheet: TP?
Changed lines of the file:
@@
 $Descr A4 11693 8268
 encoding utf-8
-Sheet 6 15
+Sheet 6 18
 Title ""
 Date ""
@@
 GND_ISO
 Wire Wire Line
-	9050 3500 8550 3500
-Connection ~ 8100 3500
-Wire Wire Line
 	9050 4500 8550 4500
 Wire Wire Line
@@
 L Connector:TestPoint TP?
 U 1 1 60B566B5
-P 8550 4100
+P 8550 4200
 AR Path="/60B566B5" Ref="TP?"  Part="1"
 AR Path="/609CA6A8/60AE5653/60B566B5" Ref="TP?"  Part="1"
-F 0 "TP?" H 8608 4218 50  0000 L CNN
-F 1 "TestPoint" H 8608 4127 50  0001 L CNN
-F 2 "" H 8750 4100 50  0001 C CNN
-F 3 "~" H 8750 4100 50  0001 C CNN
-	1    8550 4100
+F 0 "TP?" H 8608 4318 50  0000 L CNN
+F 1 "TestPoint" H 8608 4227 50  0001 L CNN
+F 2 "" H 8750 4200 50  0001 C CNN
+F 3 "~" H 8750 4200 50  0001 C CNN
+	1    8550 4200
 	1    0    0    -1
 $EndComp
@@
 L Connector:TestPoint TP?
 U 1 1 60B56DD4
-P 8550 3400
+P 8550 3500
 AR Path="/60B56DD4" Ref="TP?"  Part="1"
 AR Path="/609CA6A8/60AE5653/60B56DD4" Ref="TP?"  Part="1"
-F 0 "TP?" H 8608 3518 50  0000 L CNN
-F 1 "TestPoint" H 8608 3427 50  0001 L CNN
-F 2 "" H 8750 3400 50  0001 C CNN
-F 3 "~" H 8750 3400 50  0001 C CNN
-	1    8550 3400
-	1    0    0    -1
-$EndComp
-Wire Wire Line
-	8550 4100 8550 4200
+F 0 "TP?" H 8608 3618 50  0000 L CNN
+F 1 "TestPoint" H 8608 3527 50  0001 L CNN
+F 2 "" H 8750 3500 50  0001 C CNN
+F 3 "~" H 8750 3500 50  0001 C CNN
+	1    8550 3500
+	1    0    0    -1
+$EndComp
 Connection ~ 8550 4200
 Wire Wire Line
-	8550 3400 8550 3500
+	8100 3500 8550 3500
+Connection ~ 8100 3500
+Wire Wire Line
+	8550 3500 9050 3500
 Connection ~ 8550 3500
-Wire Wire Line
-	8550 3500 8100 3500
 $EndSCHEMATC

Commit message: Add files via upload
Parts:
- gave numbers to parts that had none: 13
Changed lines of the file:
@@
 AR Path="/60AE766F" Ref="PS?"  Part="1"
 AR Path="/609CA6A8/60AE766F" Ref="PS?"  Part="1"
-AR Path="/609CA6A8/60AE5653/60AE766F" Ref="PS?"  Part="1"
-F 0 "PS?" H 4050 3967 50  0000 C CNN
+AR Path="/609CA6A8/60AE5653/60AE766F" Ref="PS1"  Part="1"
+F 0 "PS1" H 4050 3967 50  0000 C CNN
 F 1 "B0505S-1WR2" H 4050 3876 50  0000 C CNN
 F 2 "CONV_B0505S-1WR2" H 4050 3600 50  0001 L BNN
@@
 AR Path="/609CA6A8/60A0A922/60AE7675" Ref="C?"  Part="1"
 AR Path="/609CA6A8/60AE7675" Ref="C?"  Part="1"
-AR Path="/609CA6A8/60AE5653/60AE7675" Ref="C?"  Part="1"
-F 0 "C?" H 6365 3696 50  0000 L CNN
+AR Path="/609CA6A8/60AE5653/60AE7675" Ref="C29"  Part="1"
+F 0 "C29" H 6365 3696 50  0000 L CNN
 F 1 "0,1" H 6365 3605 50  0000 L CNN
 F 2 "Capacitor_SMD:C_0603_1608Metric_Pad1.08x0.95mm_HandSolder" H 6288 3500 50  0001 C CNN
@@
 AR Path="/609CA6A8/60A0A922/60AE767B" Ref="C?"  Part="1"
 AR Path="/609CA6A8/60AE767B" Ref="C?"  Part="1"
-AR Path="/609CA6A8/60AE5653/60AE767B" Ref="C?"  Part="1"
-F 0 "C?" H 3365 3696 50  0000 L CNN
+AR Path="/609CA6A8/60AE5653/60AE767B" Ref="C27"  Part="1"
+F 0 "C27" H 3365 3696 50  0000 L CNN
 F 1 "4,7" H 3365 3605 50  0000 L CNN
 F 2 "Capacitor_SMD:C_1206_3216Metric_Pad1.33x1.80mm_HandSolder" H 3288 3500 50  0001 C CNN
@@
 AR Path="/609CA6A8/60A0A922/60AE7681" Ref="C?"  Part="1"
 AR Path="/609CA6A8/60AE7681" Ref="C?"  Part="1"
-AR Path="/609CA6A8/60AE5653/60AE7681" Ref="C?"  Part="1"
-F 0 "C?" H 4865 3696 50  0000 L CNN
+AR Path="/609CA6A8/60AE5653/60AE7681" Ref="C28"  Part="1"
+F 0 "C28" H 4865 3696 50  0000 L CNN
 F 1 "10u" H 4865 3605 50  0000 L CNN
 F 2 "Capacitor_SMD:C_1206_3216Metric_Pad1.33x1.80mm_HandSolder" H 4788 3500 50  0001 C CNN
@@
 AR Path="/60AE7692" Ref="R?"  Part="1"
 AR Path="/609CA6A8/60AE7692" Ref="R?"  Part="1"
-AR Path="/609CA6A8/60AE5653/60AE7692" Ref="R?"  Part="1"
-F 0 "R?" H 5220 3696 50  0000 L CNN
+AR Path="/609CA6A8/60AE5653/60AE7692" Ref="R45"  Part="1"
+F 0 "R45" H 5220 3696 50  0000 L CNN
 F 1 "680" H 5220 3605 50  0000 L CNN
 F 2 "Resistor_SMD:R_0603_1608Metric_Pad0.98x0.95mm_HandSolder" V 5080 3650 50  0001 C CNN
@@
 AR Path="/60AE7698" Ref="R?"  Part="1"
 AR Path="/609CA6A8/60AE7698" Ref="R?"  Part="1"
-AR Path="/609CA6A8/60AE5653/60AE7698" Ref="R?"  Part="1"
-F 0 "R?" H 5620 3696 50  0000 L CNN
+AR Path="/609CA6A8/60AE5653/60AE7698" Ref="R46"  Part="1"
+F 0 "R46" H 5620 3696 50  0000 L CNN
 F 1 "680" H 5620 3605 50  0000 L CNN
 F 2 "Resistor_SMD:R_0603_1608Metric_Pad0.98x0.95mm_HandSolder" V 5480 3650 50  0001 C CNN
@@
 AR Path="/609CA6A8/60A0A922/60AE769E" Ref="C?"  Part="1"
 AR Path="/609CA6A8/60AE769E" Ref="C?"  Part="1"
-AR Path="/609CA6A8/60AE5653/60AE769E" Ref="C?"  Part="1"
-F 0 "C?" H 8215 3696 50  0000 L CNN
+AR Path="/609CA6A8/60AE5653/60AE769E" Ref="C31"  Part="1"
+F 0 "C31" H 8215 3696 50  0000 L CNN
 F 1 "1u" H 8215 3605 50  0000 L CNN
 F 2 "Capacitor_SMD:C_0603_1608Metric_Pad1.08x0.95mm_HandSolder" H 8138 3500 50  0001 C CNN
@@
 AR Path="/609CA6A8/60A0A922/60AE76A4" Ref="C?"  Part="1"
 AR Path="/609CA6A8/60AE76A4" Ref="C?"  Part="1"
-AR Path="/609CA6A8/60AE5653/60AE76A4" Ref="C?"  Part="1"
-F 0 "C?" H 7015 4096 50  0000 L CNN
+AR Path="/609CA6A8/60AE5653/60AE76A4" Ref="C30"  Part="1"
+F 0 "C30" H 7015 4096 50  0000 L CNN
 F 1 "10u" H 7015 4005 50  0000 L CNN
 F 2 "Capacitor_SMD:C_1206_3216Metric_Pad1.33x1.80mm_HandSolder" H 6938 3900 50  0001 C CNN
@@
 AR Path="/60AE76AA" Ref="R?"  Part="1"
 AR Path="/609CA6A8/60AE76AA" Ref="R?"  Part="1"
-AR Path="/609CA6A8/60AE5653/60AE76AA" Ref="R?"  Part="1"
-F 0 "R?" H 7570 3696 50  0000 L CNN
+AR Path="/609CA6A8/60AE5653/60AE76AA" Ref="R47"  Part="1"
+F 0 "R47" H 7570 3696 50  0000 L CNN
 F 1 "240 1%" H 7570 3605 50  0000 L CNN
 F 2 "Resistor_SMD:R_0603_1608Metric_Pad0.98x0.95mm_HandSolder" V 7430 3650 50  0001 C CNN
@@
 AR Path="/60AE76B0" Ref="R?"  Part="1"
 AR Path="/609CA6A8/60AE76B0" Ref="R?"  Part="1"
-AR Path="/609CA6A8/60AE5653/60AE76B0" Ref="R?"  Part="1"
-F 0 "R?" H 7570 4096 50  0000 L CNN
+AR Path="/609CA6A8/60AE5653/60AE76B0" Ref="R48"  Part="1"
+F 0 "R48" H 7570 4096 50  0000 L CNN
 F 1 "390 1%" H 7570 4005 50  0000 L CNN
 F 2 "Resistor_SMD:R_0603_1608Metric_Pad0.98x0.95mm_HandSolder" V 7430 4050 50  0001 C CNN
@@
 P 6900 3500
 AR Path="/609CA6A8/60AE76B8" Ref="U?"  Part="1"
-AR Path="/609CA6A8/60AE5653/60AE76B8" Ref="U?"  Part="1"
-F 0 "U?" H 6900 3742 50  0000 C CNN
+AR Path="/609CA6A8/60AE5653/60AE76B8" Ref="U5"  Part="1"
+F 0 "U5" H 6900 3742 50  0000 C CNN
 F 1 "LM317L_SO8" H 6900 3651 50  0000 C CNN
 F 2 "Package_SO:SOIC-8_3.9x4.9mm_P1.27mm" H 6900 3700 50  0001 C CIN
@@
 P 8550 4200
 AR Path="/60B566B5" Ref="TP?"  Part="1"
-AR Path="/609CA6A8/60AE5653/60B566B5" Ref="TP?"  Part="1"
-F 0 "TP?" H 8608 4318 50  0000 L CNN
+AR Path="/609CA6A8/60AE5653/60B566B5" Ref="TP6"  Part="1"
+F 0 "TP6" H 8608 4318 50  0000 L CNN
 F 1 "TestPoint" H 8608 4227 50  0001 L CNN
 F 2 "" H 8750 4200 50  0001 C CNN
@@
 P 8550 3500
 AR Path="/60B56DD4" Ref="TP?"  Part="1"
-AR Path="/609CA6A8/60AE5653/60B56DD4" Ref="TP?"  Part="1"
-F 0 "TP?" H 8608 3618 50  0000 L CNN
+AR Path="/609CA6A8/60AE5653/60B56DD4" Ref="TP5"  Part="1"
+F 0 "TP5" H 8608 3618 50  0000 L CNN
 F 1 "TestPoint" H 8608 3527 50  0001 L CNN
 F 2 "" H 8750 3500 50  0001 C CNN
