File: furnace/furnace_controller/+3V3_isolated.sch (KiCad schematic (older format))
At the start: 13 parts, among them U5 LM317L_SO8

Commit message: Add files via upload
Changed lines of the file:
@@
 GND_ISO
-Wire Wire Line
-	9050 4500 8550 4500
 Wire Wire Line
 	8550 4500 8550 4200
@@
 	8550 3500 9050 3500
 Connection ~ 8550 3500
+Wire Wire Line
+	8550 4500 9050 4500
 $EndSCHEMATC

Commit message: Add files via upload
Parts:
- C27, C28, C30: footprint Capacitor_SMD:C_1206_3216Metric_Pad1.33x1.80mm_HandSolder -> Capacitor_SMD:C_1206_3216Metric_Pad1.42x1.75mm_HandSolder
- C29, C31: footprint Capacitor_SMD:C_0603_1608Metric_Pad1.08x0.95mm_HandSolder -> Capacitor_SMD:C_0603_1608Metric_Pad1.05x0.95mm_HandSolder
- PS1: footprint CONV_B0505S-1WR2 -> furnace_controller:B_S-1WR3
- R45, R46, R47, R48: footprint Resistor_SMD:R_0603_1608Metric_Pad0.98x0.95mm_HandSolder -> Resistor_SMD:R_0603_1608Metric_Pad1.05x0.95mm_HandSolder
- TP5, TP6: footprint (none) -> furnace_controller:TP
Changed lines of the file:
@@
 encoding utf-8
 Sheet 8 18
-Title ""
-Date ""
-Rev ""
-Comp ""
+Title "Furnace controller"
+Date "2021-08-26"
+Rev "1.0"
+Comp "Yuriy Volkov"
 Comment1 ""
 Comment2 ""
@@
 F 0 "PS1" H 4050 3967 50  0000 C CNN
 F 1 "B0505S-1WR2" H 4050 3876 50  0000 C CNN
-F 2 "CONV_B0505S-1WR2" H 4050 3600 50  0001 L BNN
+F 2 "furnace_controller:B_S-1WR3" H 4050 3600 50  0001 L BNN
 F 3 "" H 4050 3600 50  0001 L BNN
 F 4 "Manufacturer Recommendations" H 4050 3600 50  0001 L BNN "STANDARD"
@@
 F 0 "C29" H 6365 3696 50  0000 L CNN
 F 1 "0,1" H 6365 3605 50  0000 L CNN
-F 2 "Capacitor_SMD:C_0603_1608Metric_Pad1.08x0.95mm_HandSolder" H 6288 3500 50  0001 C CNN
+F 2 "Capacitor_SMD:C_0603_1608Metric_Pad1.05x0.95mm_HandSolder" H 6288 3500 50  0001 C CNN
 F 3 "~" H 6250 3650 50  0001 C CNN
 	1    6250 3650
@@
 F 0 "C27" H 3365 3696 50  0000 L CNN
 F 1 "4,7" H 3365 3605 50  0000 L CNN
-F 2 "Capacitor_SMD:C_1206_3216Metric_Pad1.33x1.80mm_HandSolder" H 3288 3500 50  0001 C CNN
+F 2 "Capacitor_SMD:C_1206_3216Metric_Pad1.42x1.75mm_HandSolder" H 3288 3500 50  0001 C CNN
 F 3 "~" H 3250 3650 50  0001 C CNN
 	1    3250 3650
@@
 F 0 "C28" H 4865 3696 50  0000 L CNN
 F 1 "10u" H 4865 3605 50  0000 L CNN
-F 2 "Capacitor_SMD:C_1206_3216Metric_Pad1.33x1.80mm_HandSolder" H 4788 3500 50  0001 C CNN
+F 2 "Capacitor_SMD:C_1206_3216Metric_Pad1.42x1.75mm_HandSolder" H 4788 3500 50  0001 C CNN
 F 3 "~" H 4750 3650 50  0001 C CNN
 	1    4750 3650
@@
 F 0 "R45" H 5220 3696 50  0000 L CNN
 F 1 "680" H 5220 3605 50  0000 L CNN
-F 2 "Resistor_SMD:R_0603_1608Metric_Pad0.98x0.95mm_HandSolder" V 5080 3650 50  0001 C CNN
+F 2 "Resistor_SMD:R_0603_1608Metric_Pad1.05x0.95mm_HandSolder" V 5080 3650 50  0001 C CNN
 F 3 "~" H 5150 3650 50  0001 C CNN
 	1    5150 3650
@@
 F 0 "R46" H 5620 3696 50  0000 L CNN
 F 1 "680" H 5620 3605 50  0000 L CNN
-F 2 "Resistor_SMD:R_0603_1608Metric_Pad0.98x0.95mm_HandSolder" V 5480 3650 50  0001 C CNN
+F 2 "Resistor_SMD:R_0603_1608Metric_Pad1.05x0.95mm_HandSolder" V 5480 3650 50  0001 C CNN
 F 3 "~" H 5550 3650 50  0001 C CNN
 	1    5550 3650
@@
 F 0 "C31" H 8215 3696 50  0000 L CNN
 F 1 "1u" H 8215 3605 50  0000 L CNN
-F 2 "Capacitor_SMD:C_0603_1608Metric_Pad1.08x0.95mm_HandSolder" H 8138 3500 50  0001 C CNN
+F 2 "Capacitor_SMD:C_0603_1608Metric_Pad1.05x0.95mm_HandSolder" H 8138 3500 50  0001 C CNN
 F 3 "~" H 8100 3650 50  0001 C CNN
 	1    8100 3650
@@
 F 0 "C30" H 7015 4096 50  0000 L CNN
 F 1 "10u" H 7015 4005 50  0000 L CNN
-F 2 "Capacitor_SMD:C_1206_3216Metric_Pad1.33x1.80mm_HandSolder" H 6938 3900 50  0001 C CNN
+F 2 "Capacitor_SMD:C_1206_3216Metric_Pad1.42x1.75mm_HandSolder" H 6938 3900 50  0001 C CNN
 F 3 "~" H 6900 4050 50  0001 C CNN
 	1    6900 4050
@@
 F 0 "R47" H 7570 3696 50  0000 L CNN
 F 1 "240 1%" H 7570 3605 50  0000 L CNN
-F 2 "Resistor_SMD:R_0603_1608Metric_Pad0.98x0.95mm_HandSolder" V 7430 3650 50  0001 C CNN
+F 2 "Resistor_SMD:R_0603_1608Metric_Pad1.05x0.95mm_HandSolder" V 7430 3650 50  0001 C CNN
 F 3 "~" H 7500 3650 50  0001 C CNN
 	1    7500 3650
@@
 F 0 "R48" H 7570 4096 50  0000 L CNN
 F 1 "390 1%" H 7570 4005 50  0000 L CNN
-F 2 "Resistor_SMD:R_0603_1608Metric_Pad0.98x0.95mm_HandSolder" V 7430 4050 50  0001 C CNN
+F 2 "Resistor_SMD:R_0603_1608Metric_Pad1.05x0.95mm_HandSolder" V 7430 4050 50  0001 C CNN
 F 3 "~" H 7500 4050 50  0001 C CNN
 	1    7500 4050
@@
 F 0 "TP6" H 8608 4318 50  0000 L CNN
 F 1 "TestPoint" H 8608 4227 50  0001 L CNN
-F 2 "" H 8750 4200 50  0001 C CNN
+F 2 "furnace_controller:TP" H 8750 4200 50  0001 C CNN
 F 3 "~" H 8750 4200 50  0001 C CNN
 	1    8550 4200
@@
 F 0 "TP5" H 8608 3618 50  0000 L CNN
 F 1 "TestPoint" H 8608 3527 50  0001 L CNN
-F 2 "" H 8750 3500 50  0001 C CNN
+F 2 "furnace_controller:TP" H 8750 3500 50  0001 C CNN
 F 3 "~" H 8750 3500 50  0001 C CNN
 	1    8550 3500

Commit message: Add files via upload
Parts:
- added FB1: Ferrite_Bead, Inductor_SMD:L_0805_2012Metric_Pad1.05x1.20mm_HandSolder, symbol Device:Ferrite_Bead
- C17: renamed from C27; footprint Capacitor_SMD:C_1206_3216Metric_Pad1.42x1.75mm_HandSolder -> Capacitor_SMD:C_1206_3216Metric_Pad1.33x1.80mm_HandSolder
- C18: renamed from C28; footprint Capacitor_SMD:C_1206_3216Metric_Pad1.42x1.75mm_HandSolder -> Capacitor_SMD:C_1206_3216Metric_Pad1.33x1.80mm_HandSolder
- C19: renamed from C29; footprint Capacitor_SMD:C_0603_1608Metric_Pad1.05x0.95mm_HandSolder -> Capacitor_SMD:C_0603_1608Metric_Pad1.08x0.95mm_HandSolder
- C20: renamed from C30; footprint Capacitor_SMD:C_1206_3216Metric_Pad1.42x1.75mm_HandSolder -> Capacitor_SMD:C_1206_3216Metric_Pad1.33x1.80mm_HandSolder
- C21: renamed from C31; footprint Capacitor_SMD:C_0603_1608Metric_Pad1.05x0.95mm_HandSolder -> Capacitor_SMD:C_0603_1608Metric_Pad1.08x0.95mm_HandSolder
- R38: renamed from R45; footprint Resistor_SMD:R_0603_1608Metric_Pad1.05x0.95mm_HandSolder -> Resistor_SMD:R_0603_1608Metric_Pad0.98x0.95mm_HandSolder
- R39: renamed from R46; footprint Resistor_SMD:R_0603_1608Metric_Pad1.05x0.95mm_HandSolder -> Resistor_SMD:R_0603_1608Metric_Pad0.98x0.95mm_HandSolder
- R40: renamed from R47; footprint Resistor_SMD:R_0603_1608Metric_Pad1.05x0.95mm_HandSolder -> Resistor_SMD:R_0603_1608Metric_Pad0.98x0.95mm_HandSolder
- R41: renamed from R48; footprint Resistor_SMD:R_0603_1608Metric_Pad1.05x0.95mm_HandSolder -> Resistor_SMD:R_0603_1608Metric_Pad0.98x0.95mm_HandSolder
- renumbered U5 to U4
Connections:
- net at C19.1, R38.1, R39.1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: now also FB1.1; no longer C18.1, PS1.4 (+VO)
- new net: C18.1, FB1.2, PS1.4 (+VO)
Other:
- moved on the sheet: R38, R39
Changed lines of the file:
@@
 Sheet 8 18
 Title "Furnace controller"
-Date "2021-08-26"
+Date "2021-09-24"
 Rev "1.0"
 Comp "Yuriy Volkov"
@@
 AR Path="/609CA6A8/60A0A922/60AE7675" Ref="C?"  Part="1"
 AR Path="/609CA6A8/60AE7675" Ref="C?"  Part="1"
-AR Path="/609CA6A8/60AE5653/60AE7675" Ref="C29"  Part="1"
-F 0 "C29" H 6365 3696 50  0000 L CNN
+AR Path="/609CA6A8/60AE5653/60AE7675" Ref="C19"  Part="1"
+F 0 "C19" H 6365 3696 50  0000 L CNN
 F 1 "0,1" H 6365 3605 50  0000 L CNN
-F 2 "Capacitor_SMD:C_0603_1608Metric_Pad1.05x0.95mm_HandSolder" H 6288 3500 50  0001 C CNN
+F 2 "Capacitor_SMD:C_0603_1608Metric_Pad1.08x0.95mm_HandSolder" H 6288 3500 50  0001 C CNN
 F 3 "~" H 6250 3650 50  0001 C CNN
 	1    6250 3650
@@
 AR Path="/609CA6A8/60A0A922/60AE767B" Ref="C?"  Part="1"
 AR Path="/609CA6A8/60AE767B" Ref="C?"  Part="1"
-AR Path="/609CA6A8/60AE5653/60AE767B" Ref="C27"  Part="1"
-F 0 "C27" H 3365 3696 50  0000 L CNN
+AR Path="/609CA6A8/60AE5653/60AE767B" Ref="C17"  Part="1"
+F 0 "C17" H 3365 3696 50  0000 L CNN
 F 1 "4,7" H 3365 3605 50  0000 L CNN
-F 2 "Capacitor_SMD:C_1206_3216Metric_Pad1.42x1.75mm_HandSolder" H 3288 3500 50  0001 C CNN
+F 2 "Capacitor_SMD:C_1206_3216Metric_Pad1.33x1.80mm_HandSolder" H 3288 3500 50  0001 C CNN
 F 3 "~" H 3250 3650 50  0001 C CNN
 	1    3250 3650
@@
 AR Path="/609CA6A8/60A0A922/60AE7681" Ref="C?"  Part="1"
 AR Path="/609CA6A8/60AE7681" Ref="C?"  Part="1"
-AR Path="/609CA6A8/60AE5653/60AE7681" Ref="C28"  Part="1"
-F 0 "C28" H 4865 3696 50  0000 L CNN
+AR Path="/609CA6A8/60AE5653/60AE7681" Ref="C18"  Part="1"
+F 0 "C18" H 4865 3696 50  0000 L CNN
 F 1 "10u" H 4865 3605 50  0000 L CNN
-F 2 "Capacitor_SMD:C_1206_3216Metric_Pad1.42x1.75mm_HandSolder" H 4788 3500 50  0001 C CNN
+F 2 "Capacitor_SMD:C_1206_3216Metric_Pad1.33x1.80mm_HandSolder" H 4788 3500 50  0001 C CNN
 F 3 "~" H 4750 3650 50  0001 C CNN
 	1    4750 3650
@@
 L Device:R R?
 U 1 1 60AE7692
-P 5150 3650
+P 5500 3650
 AR Path="/60AE7692" Ref="R?"  Part="1"
 AR Path="/609CA6A8/60AE7692" Ref="R?"  Part="1"
-AR Path="/609CA6A8/60AE5653/60AE7692" Ref="R45"  Part="1"
-F 0 "R45" H 5220 3696 50  0000 L CNN
-F 1 "680" H 5220 3605 50  0000 L CNN
-F 2 "Resistor_SMD:R_0603_1608Metric_Pad1.05x0.95mm_HandSolder" V 5080 3650 50  0001 C CNN
-F 3 "~" H 5150 3650 50  0001 C CNN
-	1    5150 3650
-	1    0    0    -1
-$EndComp
-$Comp
-L Device:R R?
-U 1 1 60AE7698
-P 5550 3650
-AR Path="/60AE7698" Ref="R?"  Part="1"
-AR Path="/609CA6A8/60AE7698" Ref="R?"  Part="1"
-AR Path="/609CA6A8/60AE5653/60AE7698" Ref="R46"  Part="1"
-F 0 "R46" H 5620 3696 50  0000 L CNN
-F 1 "680" H 5620 3605 50  0000 L CNN
-F 2 "Resistor_SMD:R_0603_1608Metric_Pad1.05x0.95mm_HandSolder" V 5480 3650 50  0001 C CNN
-F 3 "~" H 5550 3650 50  0001 C CNN
-	1    5550 3650
+AR Path="/609CA6A8/60AE5653/60AE7692" Ref="R38"  Part="1"
+F 0 "R38" H 5570 3696 50  0000 L CNN
+F 1 "680" H 5570 3605 50  0000 L CNN
+F 2 "Resistor_SMD:R_0603_1608Metric_Pad0.98x0.95mm_HandSolder" V 5430 3650 50  0001 C CNN
+F 3 "~" H 5500 3650 50  0001 C CNN
+	1    5500 3650
 	1    0    0    -1
 $EndComp
@@
 AR Path="/609CA6A8/60A0A922/60AE769E" Ref="C?"  Part="1"
 AR Path="/609CA6A8/60AE769E" Ref="C?"  Part="1"
-AR Path="/609CA6A8/60AE5653/60AE769E" Ref="C31"  Part="1"
-F 0 "C31" H 8215 3696 50  0000 L CNN
+AR Path="/609CA6A8/60AE5653/60AE769E" Ref="C21"  Part="1"
+F 0 "C21" H 8215 3696 50  0000 L CNN
 F 1 "1u" H 8215 3605 50  0000 L CNN
-F 2 "Capacitor_SMD:C_0603_1608Metric_Pad1.05x0.95mm_HandSolder" H 8138 3500 50  0001 C CNN
+F 2 "Capacitor_SMD:C_0603_1608Metric_Pad1.08x0.95mm_HandSolder" H 8138 3500 50  0001 C CNN
 F 3 "~" H 8100 3650 50  0001 C CNN
 	1    8100 3650
@@
 AR Path="/609CA6A8/60A0A922/60AE76A4" Ref="C?"  Part="1"
 AR Path="/609CA6A8/60AE76A4" Ref="C?"  Part="1"
-AR Path="/609CA6A8/60AE5653/60AE76A4" Ref="C30"  Part="1"
-F 0 "C30" H 7015 4096 50  0000 L CNN
+AR Path="/609CA6A8/60AE5653/60AE76A4" Ref="C20"  Part="1"
+F 0 "C20" H 7015 4096 50  0000 L CNN
 F 1 "10u" H 7015 4005 50  0000 L CNN
-F 2 "Capacitor_SMD:C_1206_3216Metric_Pad1.42x1.75mm_HandSolder" H 6938 3900 50  0001 C CNN
+F 2 "Capacitor_SMD:C_1206_3216Metric_Pad1.33x1.80mm_HandSolder" H 6938 3900 50  0001 C CNN
 F 3 "~" H 6900 4050 50  0001 C CNN
 	1    6900 4050
@@
 AR Path="/60AE76AA" Ref="R?"  Part="1"
 AR Path="/609CA6A8/60AE76AA" Ref="R?"  Part="1"
-AR Path="/609CA6A8/60AE5653/60AE76AA" Ref="R47"  Part="1"
-F 0 "R47" H 7570 3696 50  0000 L CNN
+AR Path="/609CA6A8/60AE5653/60AE76AA" Ref="R40"  Part="1"
+F 0 "R40" H 7570 3696 50  0000 L CNN
 F 1 "240 1%" H 7570 3605 50  0000 L CNN
-F 2 "Resistor_SMD:R_0603_1608Metric_Pad1.05x0.95mm_HandSolder" V 7430 3650 50  0001 C CNN
+F 2 "Resistor_SMD:R_0603_1608Metric_Pad0.98x0.95mm_HandSolder" V 7430 3650 50  0001 C CNN
 F 3 "~" H 7500 3650 50  0001 C CNN
 	1    7500 3650
@@
 AR Path="/60AE76B0" Ref="R?"  Part="1"
 AR Path="/609CA6A8/60AE76B0" Ref="R?"  Part="1"
-AR Path="/609CA6A8/60AE5653/60AE76B0" Ref="R48"  Part="1"
-F 0 "R48" H 7570 4096 50  0000 L CNN
+AR Path="/609CA6A8/60AE5653/60AE76B0" Ref="R41"  Part="1"
+F 0 "R41" H 7570 4096 50  0000 L CNN
 F 1 "390 1%" H 7570 4005 50  0000 L CNN
-F 2 "Resistor_SMD:R_0603_1608Metric_Pad1.05x0.95mm_HandSolder" V 7430 4050 50  0001 C CNN
+F 2 "Resistor_SMD:R_0603_1608Metric_Pad0.98x0.95mm_HandSolder" V 7430 4050 50  0001 C CNN
 F 3 "~" H 7500 4050 50  0001 C CNN
 	1    7500 4050
@@
 P 6900 3500
 AR Path="/609CA6A8/60AE76B8" Ref="U?"  Part="1"
-AR Path="/609CA6A8/60AE5653/60AE76B8" Ref="U5"  Part="1"
-F 0 "U5" H 6900 3742 50  0000 C CNN
+AR Path="/609CA6A8/60AE5653/60AE76B8" Ref="U4"  Part="1"
+F 0 "U4" H 6900 3742 50  0000 C CNN
 F 1 "LM317L_SO8" H 6900 3651 50  0000 C CNN
 F 2 "Package_SO:SOIC-8_3.9x4.9mm_P1.27mm" H 6900 3700 50  0001 C CIN
@@
 $EndComp
 Wire Wire Line
-	4750 3500 5150 3500
-Connection ~ 4750 3500
-Connection ~ 5150 3500
-Wire Wire Line
-	5150 3500 5550 3500
-Connection ~ 5550 3500
-Wire Wire Line
-	5550 3500 6250 3500
+	5500 3500 5850 3500
+Connection ~ 5850 3500
 Connection ~ 6250 3500
 Wire Wire Line
 	6250 3500 6600 3500
 Wire Wire Line
-	4750 3800 5150 3800
+	4750 3800 5500 3800
 Connection ~ 4750 3800
-Connection ~ 5150 3800
-Wire Wire Line
-	5150 3800 5550 3800
-Connection ~ 5550 3800
+Connection ~ 5500 3800
+Wire Wire Line
+	5500 3800 5850 3800
+Connection ~ 5850 3800
 Wire Wire Line
 	6900 3800 6900 3850
@@
 Wire Wire Line
 	7500 3500 8100 3500
-Wire Wire Line
-	5550 3800 6250 3800
 Wire Wire Line
 	6250 3800 6250 4200
@@
 Wire Wire Line
 	8550 4500 9050 4500
+Wire Wire Line
+	5850 3800 6250 3800
+Wire Wire Line
+	5850 3500 6050 3500
+$Comp
+L Device:R R?
+U 1 1 60AE7698
+P 5850 3650
+AR Path="/60AE7698" Ref="R?"  Part="1"
+AR Path="/609CA6A8/60AE7698" Ref="R?"  Part="1"
+AR Path="/609CA6A8/60AE5653/60AE7698" Ref="R39"  Part="1"
+F 0 "R39" H 5920 3696 50  0000 L CNN
+F 1 "680" H 5920 3605 50  0000 L CNN
+F 2 "Resistor_SMD:R_0603_1608Metric_Pad0.98x0.95mm_HandSolder" V 5780 3650 50  0001 C CNN
+F 3 "~" H 5850 3650 50  0001 C CNN
+	1    5850 3650
+	1    0    0    -1
+$EndComp
+$Comp
+L Device:Ferrite_Bead FB1
+U 1 1 6150A0A5
+P 5150 3500
+F 0 "FB1" V 4968 3500 50  0000 C CNN
+F 1 "Ferrite_Bead" V 4967 3500 50  0001 C CNN
+F 2 "Inductor_SMD:L_0805_2012Metric_Pad1.05x1.20mm_HandSolder" V 5080 3500 50  0001 C CNN
+F 3 "~" H 5150 3500 50  0001 C CNN
+	1    5150 3500
+	0    1    1    0
+$EndComp
+Wire Wire Line
+	5300 3500 5500 3500
+Connection ~ 5500 3500
+Wire Wire Line
+	5000 3500 4750 3500
+Connection ~ 4750 3500
+$Comp
+L power:PWR_FLAG #FLG0101
+U 1 1 61510D88
+P 6050 3500
+F 0 "#FLG0101" H 6050 3575 50  0001 C CNN
+F 1 "PWR_FLAG" H 6050 3673 50  0000 C CNN
+F 2 "" H 6050 3500 50  0001 C CNN
+F 3 "~" H 6050 3500 50  0001 C CNN
+	1    6050 3500
+	1    0    0    -1
+$EndComp
+Connection ~ 6050 3500
+Wire Wire Line
+	6050 3500 6250 3500
 $EndSCHEMATC
