File: furnace/furnace_controller/Buzzer.sch (KiCad schematic (older format))
At the start: 4 parts, among them Q7 BC847

Commit message: Add files via upload
Parts:
- BZ1: footprint (none) -> Buzzer_Beeper:Buzzer_12x9.5RM7.6
- R52, R53: footprint Resistor_SMD:R_0603_1608Metric_Pad0.98x0.95mm_HandSolder -> Resistor_SMD:R_0603_1608Metric_Pad1.05x0.95mm_HandSolder
Changed lines of the file:
@@
 $Descr A4 11693 8268
 encoding utf-8
-Sheet 17 18
-Title ""
-Date ""
-Rev ""
-Comp ""
+Sheet 16 18
+Title "Furnace controller"
+Date "2021-08-26"
+Rev "1.0"
+Comp "Yuriy Volkov"
 Comment1 ""
 Comment2 ""
@@
 F 0 "BZ1" H 6752 3929 50  0000 L CNN
 F 1 "Buzzer" H 6752 3838 50  0000 L CNN
-F 2 "" V 6575 4000 50  0001 C CNN
+F 2 "Buzzer_Beeper:Buzzer_12x9.5RM7.6" V 6575 4000 50  0001 C CNN
 F 3 "~" V 6575 4000 50  0001 C CNN
 	1    6600 3900
@@
 F 0 "R53" H 6070 4796 50  0000 L CNN
 F 1 "56k" H 6070 4705 50  0000 L CNN
-F 2 "Resistor_SMD:R_0603_1608Metric_Pad0.98x0.95mm_HandSolder" V 5930 4750 50  0001 C CNN
+F 2 "Resistor_SMD:R_0603_1608Metric_Pad1.05x0.95mm_HandSolder" V 5930 4750 50  0001 C CNN
 F 3 "~" H 6000 4750 50  0001 C CNN
 	1    6000 4750
@@
 F 0 "R52" V 5750 4450 50  0000 L CNN
 F 1 "3,3k" V 5550 4400 50  0000 L CNN
-F 2 "Resistor_SMD:R_0603_1608Metric_Pad0.98x0.95mm_HandSolder" V 5580 4500 50  0001 C CNN
+F 2 "Resistor_SMD:R_0603_1608Metric_Pad1.05x0.95mm_HandSolder" V 5580 4500 50  0001 C CNN
 F 3 "~" H 5650 4500 50  0001 C CNN
 	1    5650 4500

Commit message: Add files via upload
Parts:
- R42: renamed from R52; footprint Resistor_SMD:R_0603_1608Metric_Pad1.05x0.95mm_HandSolder -> Resistor_SMD:R_0603_1608Metric_Pad0.98x0.95mm_HandSolder
- R43: renamed from R53; footprint Resistor_SMD:R_0603_1608Metric_Pad1.05x0.95mm_HandSolder -> Resistor_SMD:R_0603_1608Metric_Pad0.98x0.95mm_HandSolder
- renumbered Q7 to Q6
Changed lines of the file:
@@
 $Descr A4 11693 8268
 encoding utf-8
-Sheet 16 18
+Sheet 15 18
 Title "Furnace controller"
-Date "2021-08-26"
+Date "2021-09-24"
 Rev "1.0"
 Comp "Yuriy Volkov"
@@
 P 6400 4500
 AR Path="/609C9D41/60B3B2F4" Ref="Q?"  Part="1"
-AR Path="/60B39FE1/60B3B2F4" Ref="Q7"  Part="1"
-F 0 "Q7" H 6591 4546 50  0000 L CNN
+AR Path="/60B39FE1/60B3B2F4" Ref="Q6"  Part="1"
+F 0 "Q6" H 6591 4546 50  0000 L CNN
 F 1 "BC847" H 6591 4455 50  0000 L CNN
 F 2 "Package_TO_SOT_SMD:SOT-23" H 6600 4425 50  0001 L CIN
@@
 P 6000 4750
 AR Path="/60B3B65C" Ref="R?"  Part="1"
-AR Path="/60B39FE1/60B3B65C" Ref="R53"  Part="1"
-F 0 "R53" H 6070 4796 50  0000 L CNN
+AR Path="/60B39FE1/60B3B65C" Ref="R43"  Part="1"
+F 0 "R43" H 6070 4796 50  0000 L CNN
 F 1 "56k" H 6070 4705 50  0000 L CNN
-F 2 "Resistor_SMD:R_0603_1608Metric_Pad1.05x0.95mm_HandSolder" V 5930 4750 50  0001 C CNN
+F 2 "Resistor_SMD:R_0603_1608Metric_Pad0.98x0.95mm_HandSolder" V 5930 4750 50  0001 C CNN
 F 3 "~" H 6000 4750 50  0001 C CNN
 	1    6000 4750
@@
 P 6500 5000
 AR Path="/60B3B924" Ref="#PWR?"  Part="1"
-AR Path="/60B39FE1/60B3B924" Ref="#PWR058"  Part="1"
-F 0 "#PWR058" H 6500 4750 50  0001 C CNN
+AR Path="/60B39FE1/60B3B924" Ref="#PWR038"  Part="1"
+F 0 "#PWR038" H 6500 4750 50  0001 C CNN
 F 1 "GND" H 6505 4827 50  0000 C CNN
 F 2 "" H 6500 5000 50  0001 C CNN
@@
 P 5650 4500
 AR Path="/60B3CA8D" Ref="R?"  Part="1"
-AR Path="/60B39FE1/60B3CA8D" Ref="R52"  Part="1"
-F 0 "R52" V 5750 4450 50  0000 L CNN
+AR Path="/60B39FE1/60B3CA8D" Ref="R42"  Part="1"
+F 0 "R42" V 5750 4450 50  0000 L CNN
 F 1 "3,3k" V 5550 4400 50  0000 L CNN
-F 2 "Resistor_SMD:R_0603_1608Metric_Pad1.05x0.95mm_HandSolder" V 5580 4500 50  0001 C CNN
+F 2 "Resistor_SMD:R_0603_1608Metric_Pad0.98x0.95mm_HandSolder" V 5580 4500 50  0001 C CNN
 F 3 "~" H 5650 4500 50  0001 C CNN
 	1    5650 4500
@@
 P 6500 3500
 AR Path="/609FED99/60B40656" Ref="#PWR?"  Part="1"
-AR Path="/60B39FE1/60B40656" Ref="#PWR057"  Part="1"
-F 0 "#PWR057" H 6500 3350 50  0001 C CNN
+AR Path="/60B39FE1/60B40656" Ref="#PWR037"  Part="1"
+F 0 "#PWR037" H 6500 3350 50  0001 C CNN
 F 1 "+5V" H 6515 3673 50  0000 C CNN
 F 2 "" H 6500 3500 50  0001 C CNN
