File: furnace/furnace_controller/Thermocouple.sch (KiCad schematic (older format))
At the start: 5 parts

Commit message: Add files via upload
Parts:
- removed D? (x2): PESD5Z3.3, symbol Device:D_Zener
Connections:
- wire segments 24 -> 16
Changed lines of the file:
@@
 $Descr A4 11693 8268
 encoding utf-8
-Sheet 8 15
+Sheet 7 18
 Title ""
 Date ""
@@
 Wire Wire Line
 	6450 4250 7350 4250
-$Comp
-L Device:D_Zener D?
-U 1 1 60B59226
-P 4850 4650
-AR Path="/60B59226" Ref="D?"  Part="1"
-AR Path="/609CA6A8/60AD75F8/60B59226" Ref="D?"  Part="1"
-AR Path="/609CA6A8/60B0F1FC/60B59226" Ref="D?"  Part="1"
-F 0 "D?" V 4804 4730 50  0000 L CNN
-F 1 "PESD5Z3.3" V 4895 4730 50  0000 L CNN
-F 2 "" H 4850 4650 50  0001 C CNN
-F 3 "~" H 4850 4650 50  0001 C CNN
-	1    4850 4650
-	0    1    1    0
-$EndComp
-$Comp
-L Device:D_Zener D?
-U 1 1 60B594A8
-P 4550 4650
-AR Path="/60B594A8" Ref="D?"  Part="1"
-AR Path="/609CA6A8/60AD75F8/60B594A8" Ref="D?"  Part="1"
-AR Path="/609CA6A8/60B0F1FC/60B594A8" Ref="D?"  Part="1"
-F 0 "D?" V 4504 4730 50  0000 L CNN
-F 1 "PESD5Z3.3" V 4595 4730 50  0001 L CNN
-F 2 "" H 4550 4650 50  0001 C CNN
-F 3 "~" H 4550 4650 50  0001 C CNN
-	1    4550 4650
-	0    1    1    0
-$EndComp
-Wire Wire Line
-	4350 5050 4550 5050
-Wire Wire Line
-	4850 4800 4850 5050
-Connection ~ 4850 5050
-Wire Wire Line
-	4850 5050 5450 5050
-Wire Wire Line
-	4550 4800 4550 5050
-Connection ~ 4550 5050
-Wire Wire Line
-	4550 5050 4850 5050
-Wire Wire Line
-	4350 4350 4850 4350
-Wire Wire Line
-	4350 4050 4550 4050
-Wire Wire Line
-	4850 4500 4850 4350
-Connection ~ 4850 4350
-Wire Wire Line
-	4850 4350 5200 4350
-Wire Wire Line
-	4550 4500 4550 4050
-Connection ~ 4550 4050
-Wire Wire Line
-	4550 4050 5200 4050
 Wire Wire Line
 	4350 3050 6050 3050
+Wire Wire Line
+	4350 5050 5450 5050
+Wire Wire Line
+	4350 4350 5200 4350
+Wire Wire Line
+	4350 4050 5200 4050
 $EndSCHEMATC

Commit message: Add files via upload
Parts:
- gave numbers to parts that had none: 3
Changed lines of the file:
@@
 AR Path="/609CA6A8/60A4AE55/609D9CFC" Ref="U?"  Part="1"
 AR Path="/609CA6A8/60A4DCFA/609D9CFC" Ref="U?"  Part="1"
-AR Path="/609CA6A8/60AD75F8/609D9CFC" Ref="U?"  Part="1"
+AR Path="/609CA6A8/60AD75F8/609D9CFC" Ref="U3"  Part="1"
 AR Path="/609CA6A8/60B05B81/609D9CFC" Ref="U?"  Part="1"
 AR Path="/609CA6A8/60B060E7/609D9CFC" Ref="U?"  Part="1"
 AR Path="/609CA6A8/60B065BD/609D9CFC" Ref="U?"  Part="1"
 AR Path="/609CA6A8/60B06ABB/609D9CFC" Ref="U?"  Part="1"
-AR Path="/609CA6A8/60B0F1FC/609D9CFC" Ref="U?"  Part="1"
-AR Path="/609CA6A8/60B0FB30/609D9CFC" Ref="U?"  Part="1"
-AR Path="/609CA6A8/60B108D6/609D9CFC" Ref="U?"  Part="1"
-AR Path="/609CA6A8/60B118F2/609D9CFC" Ref="U?"  Part="1"
-F 0 "U?" H 6200 4650 50  0000 C CNN
+AR Path="/609CA6A8/60B0F1FC/609D9CFC" Ref="U6"  Part="1"
+AR Path="/609CA6A8/60B0FB30/609D9CFC" Ref="U7"  Part="1"
+AR Path="/609CA6A8/60B108D6/609D9CFC" Ref="U8"  Part="1"
+AR Path="/609CA6A8/60B118F2/609D9CFC" Ref="U9"  Part="1"
+F 0 "U3" H 6200 4650 50  0000 C CNN
 F 1 "MAX31855EASA" H 6400 4550 50  0000 C CNN
 F 2 "Package_SO:SOIC-8_3.9x4.9mm_P1.27mm" H 7050 3800 50  0001 C CIN
@@
 AR Path="/609CA6A8/60A4AE55/609F3008" Ref="C?"  Part="1"
 AR Path="/609CA6A8/60A4DCFA/609F3008" Ref="C?"  Part="1"
-AR Path="/609CA6A8/60AD75F8/609F3008" Ref="C?"  Part="1"
+AR Path="/609CA6A8/60AD75F8/609F3008" Ref="C24"  Part="1"
 AR Path="/609CA6A8/60B05B81/609F3008" Ref="C?"  Part="1"
 AR Path="/609CA6A8/60B060E7/609F3008" Ref="C?"  Part="1"
 AR Path="/609CA6A8/60B065BD/609F3008" Ref="C?"  Part="1"
 AR Path="/609CA6A8/60B06ABB/609F3008" Ref="C?"  Part="1"
-AR Path="/609CA6A8/60B0F1FC/609F3008" Ref="C?"  Part="1"
-AR Path="/609CA6A8/60B0FB30/609F3008" Ref="C?"  Part="1"
-AR Path="/609CA6A8/60B108D6/609F3008" Ref="C?"  Part="1"
-AR Path="/609CA6A8/60B118F2/609F3008" Ref="C?"  Part="1"
-F 0 "C?" H 5565 3696 50  0000 L CNN
+AR Path="/609CA6A8/60B0F1FC/609F3008" Ref="C33"  Part="1"
+AR Path="/609CA6A8/60B0FB30/609F3008" Ref="C35"  Part="1"
+AR Path="/609CA6A8/60B108D6/609F3008" Ref="C37"  Part="1"
+AR Path="/609CA6A8/60B118F2/609F3008" Ref="C39"  Part="1"
+F 0 "C24" H 5565 3696 50  0000 L CNN
 F 1 "0,1" H 5565 3605 50  0000 L CNN
 F 2 "Capacitor_SMD:C_0603_1608Metric_Pad1.08x0.95mm_HandSolder" H 5488 3500 50  0001 C CNN
@@
 AR Path="/609CA6A8/60A4AE55/60A063BF" Ref="C?"  Part="1"
 AR Path="/609CA6A8/60A4DCFA/60A063BF" Ref="C?"  Part="1"
-AR Path="/609CA6A8/60AD75F8/60A063BF" Ref="C?"  Part="1"
+AR Path="/609CA6A8/60AD75F8/60A063BF" Ref="C23"  Part="1"
 AR Path="/609CA6A8/60B05B81/60A063BF" Ref="C?"  Part="1"
 AR Path="/609CA6A8/60B060E7/60A063BF" Ref="C?"  Part="1"
 AR Path="/609CA6A8/60B065BD/60A063BF" Ref="C?"  Part="1"
 AR Path="/609CA6A8/60B06ABB/60A063BF" Ref="C?"  Part="1"
-AR Path="/609CA6A8/60B0F1FC/60A063BF" Ref="C?"  Part="1"
-AR Path="/609CA6A8/60B0FB30/60A063BF" Ref="C?"  Part="1"
-AR Path="/609CA6A8/60B108D6/60A063BF" Ref="C?"  Part="1"
-AR Path="/609CA6A8/60B118F2/60A063BF" Ref="C?"  Part="1"
-F 0 "C?" H 5315 4246 50  0000 L CNN
+AR Path="/609CA6A8/60B0F1FC/60A063BF" Ref="C32"  Part="1"
+AR Path="/609CA6A8/60B0FB30/60A063BF" Ref="C34"  Part="1"
+AR Path="/609CA6A8/60B108D6/60A063BF" Ref="C36"  Part="1"
+AR Path="/609CA6A8/60B118F2/60A063BF" Ref="C38"  Part="1"
+F 0 "C23" H 5315 4246 50  0000 L CNN
 F 1 "0,01" H 5315 4155 50  0000 L CNN
 F 2 "Capacitor_SMD:C_0603_1608Metric_Pad1.08x0.95mm_HandSolder" H 5238 4050 50  0001 C CNN
