File: furnace/furnace_controller/Thermocouple.sch (KiCad schematic (older format))
At the start: 3 parts, among them U3 MAX31855EASA

Commit message: Add files via upload
Parts:
- C23, C24: footprint Capacitor_SMD:C_0603_1608Metric_Pad1.08x0.95mm_HandSolder -> Capacitor_SMD:C_0603_1608Metric_Pad1.05x0.95mm_HandSolder
Changed lines of the file:
@@
 encoding utf-8
 Sheet 6 18
-Title ""
-Date ""
-Rev ""
-Comp ""
+Title "Furnace controller"
+Date "2021-08-26"
+Rev "1.0"
+Comp "Yuriy Volkov"
 Comment1 ""
 Comment2 ""
@@
 F 0 "C24" H 5565 3696 50  0000 L CNN
 F 1 "0,1" H 5565 3605 50  0000 L CNN
-F 2 "Capacitor_SMD:C_0603_1608Metric_Pad1.08x0.95mm_HandSolder" H 5488 3500 50  0001 C CNN
+F 2 "Capacitor_SMD:C_0603_1608Metric_Pad1.05x0.95mm_HandSolder" H 5488 3500 50  0001 C CNN
 F 3 "~" H 5450 3650 50  0001 C CNN
 	1    5450 3650
@@
 F 0 "C23" H 5315 4246 50  0000 L CNN
 F 1 "0,01" H 5315 4155 50  0000 L CNN
-F 2 "Capacitor_SMD:C_0603_1608Metric_Pad1.08x0.95mm_HandSolder" H 5238 4050 50  0001 C CNN
+F 2 "Capacitor_SMD:C_0603_1608Metric_Pad1.05x0.95mm_HandSolder" H 5238 4050 50  0001 C CNN
 F 3 "~" H 5200 4200 50  0001 C CNN
 	1    5200 4200

Commit message: Add files via upload
Parts:
- C13: renamed from C23; footprint Capacitor_SMD:C_0603_1608Metric_Pad1.05x0.95mm_HandSolder -> Capacitor_SMD:C_0603_1608Metric_Pad1.08x0.95mm_HandSolder
- C14: renamed from C24; footprint Capacitor_SMD:C_0603_1608Metric_Pad1.05x0.95mm_HandSolder -> Capacitor_SMD:C_0603_1608Metric_Pad1.08x0.95mm_HandSolder
- renumbered U3 to U2
Changed lines of the file:
@@
 $Descr A4 11693 8268
 encoding utf-8
-Sheet 6 18
+Sheet 11 18
 Title "Furnace controller"
-Date "2021-08-26"
+Date "2021-09-24"
 Rev "1.0"
 Comp "Yuriy Volkov"
@@
 AR Path="/609CA6A8/60A4AE55/609D9CFC" Ref="U?"  Part="1"
 AR Path="/609CA6A8/60A4DCFA/609D9CFC" Ref="U?"  Part="1"
-AR Path="/609CA6A8/60AD75F8/609D9CFC" Ref="U3"  Part="1"
+AR Path="/609CA6A8/60AD75F8/609D9CFC" Ref="U2"  Part="1"
 AR Path="/609CA6A8/60B05B81/609D9CFC" Ref="U?"  Part="1"
 AR Path="/609CA6A8/60B060E7/609D9CFC" Ref="U?"  Part="1"
 AR Path="/609CA6A8/60B065BD/609D9CFC" Ref="U?"  Part="1"
 AR Path="/609CA6A8/60B06ABB/609D9CFC" Ref="U?"  Part="1"
-AR Path="/609CA6A8/60B0F1FC/609D9CFC" Ref="U6"  Part="1"
-AR Path="/609CA6A8/60B0FB30/609D9CFC" Ref="U7"  Part="1"
-AR Path="/609CA6A8/60B108D6/609D9CFC" Ref="U8"  Part="1"
-AR Path="/609CA6A8/60B118F2/609D9CFC" Ref="U9"  Part="1"
-F 0 "U3" H 6200 4650 50  0000 C CNN
+AR Path="/609CA6A8/60B0F1FC/609D9CFC" Ref="U5"  Part="1"
+AR Path="/609CA6A8/60B0FB30/609D9CFC" Ref="U6"  Part="1"
+AR Path="/609CA6A8/60B108D6/609D9CFC" Ref="U7"  Part="1"
+AR Path="/609CA6A8/60B118F2/609D9CFC" Ref="U8"  Part="1"
+F 0 "U7" H 6200 4650 50  0000 C CNN
 F 1 "MAX31855EASA" H 6400 4550 50  0000 C CNN
 F 2 "Package_SO:SOIC-8_3.9x4.9mm_P1.27mm" H 7050 3800 50  0001 C CIN
@@
 AR Path="/609CA6A8/60A4AE55/609F3008" Ref="C?"  Part="1"
 AR Path="/609CA6A8/60A4DCFA/609F3008" Ref="C?"  Part="1"
-AR Path="/609CA6A8/60AD75F8/609F3008" Ref="C24"  Part="1"
+AR Path="/609CA6A8/60AD75F8/609F3008" Ref="C14"  Part="1"
 AR Path="/609CA6A8/60B05B81/609F3008" Ref="C?"  Part="1"
 AR Path="/609CA6A8/60B060E7/609F3008" Ref="C?"  Part="1"
 AR Path="/609CA6A8/60B065BD/609F3008" Ref="C?"  Part="1"
 AR Path="/609CA6A8/60B06ABB/609F3008" Ref="C?"  Part="1"
-AR Path="/609CA6A8/60B0F1FC/609F3008" Ref="C33"  Part="1"
-AR Path="/609CA6A8/60B0FB30/609F3008" Ref="C35"  Part="1"
-AR Path="/609CA6A8/60B108D6/609F3008" Ref="C37"  Part="1"
-AR Path="/609CA6A8/60B118F2/609F3008" Ref="C39"  Part="1"
-F 0 "C24" H 5565 3696 50  0000 L CNN
+AR Path="/609CA6A8/60B0F1FC/609F3008" Ref="C23"  Part="1"
+AR Path="/609CA6A8/60B0FB30/609F3008" Ref="C25"  Part="1"
+AR Path="/609CA6A8/60B108D6/609F3008" Ref="C27"  Part="1"
+AR Path="/609CA6A8/60B118F2/609F3008" Ref="C29"  Part="1"
+F 0 "C27" H 5565 3696 50  0000 L CNN
 F 1 "0,1" H 5565 3605 50  0000 L CNN
-F 2 "Capacitor_SMD:C_0603_1608Metric_Pad1.05x0.95mm_HandSolder" H 5488 3500 50  0001 C CNN
+F 2 "Capacitor_SMD:C_0603_1608Metric_Pad1.08x0.95mm_HandSolder" H 5488 3500 50  0001 C CNN
 F 3 "~" H 5450 3650 50  0001 C CNN
 	1    5450 3650
@@
 AR Path="/609CA6A8/60A4AE55/60A063BF" Ref="C?"  Part="1"
 AR Path="/609CA6A8/60A4DCFA/60A063BF" Ref="C?"  Part="1"
-AR Path="/609CA6A8/60AD75F8/60A063BF" Ref="C23"  Part="1"
+AR Path="/609CA6A8/60AD75F8/60A063BF" Ref="C13"  Part="1"
 AR Path="/609CA6A8/60B05B81/60A063BF" Ref="C?"  Part="1"
 AR Path="/609CA6A8/60B060E7/60A063BF" Ref="C?"  Part="1"
 AR Path="/609CA6A8/60B065BD/60A063BF" Ref="C?"  Part="1"
 AR Path="/609CA6A8/60B06ABB/60A063BF" Ref="C?"  Part="1"
-AR Path="/609CA6A8/60B0F1FC/60A063BF" Ref="C32"  Part="1"
-AR Path="/609CA6A8/60B0FB30/60A063BF" Ref="C34"  Part="1"
-AR Path="/609CA6A8/60B108D6/60A063BF" Ref="C36"  Part="1"
-AR Path="/609CA6A8/60B118F2/60A063BF" Ref="C38"  Part="1"
-F 0 "C23" H 5315 4246 50  0000 L CNN
+AR Path="/609CA6A8/60B0F1FC/60A063BF" Ref="C22"  Part="1"
+AR Path="/609CA6A8/60B0FB30/60A063BF" Ref="C24"  Part="1"
+AR Path="/609CA6A8/60B108D6/60A063BF" Ref="C26"  Part="1"
+AR Path="/609CA6A8/60B118F2/60A063BF" Ref="C28"  Part="1"
+F 0 "C26" H 5315 4246 50  0000 L CNN
 F 1 "0,01" H 5315 4155 50  0000 L CNN
-F 2 "Capacitor_SMD:C_0603_1608Metric_Pad1.05x0.95mm_HandSolder" H 5238 4050 50  0001 C CNN
+F 2 "Capacitor_SMD:C_0603_1608Metric_Pad1.08x0.95mm_HandSolder" H 5238 4050 50  0001 C CNN
 F 3 "~" H 5200 4200 50  0001 C CNN
 	1    5200 4200

Commit message: Add files via upload
Changed lines of the file:
@@
 $Descr A4 11693 8268
 encoding utf-8
-Sheet 11 18
+Sheet 6 18
 Title "Furnace controller"
-Date "2021-09-24"
+Date "2021-09-30"
 Rev "1.0"
 Comp "Yuriy Volkov"
@@
 AR Path="/609CA6A8/60B108D6/609D9CFC" Ref="U7"  Part="1"
 AR Path="/609CA6A8/60B118F2/609D9CFC" Ref="U8"  Part="1"
-F 0 "U7" H 6200 4650 50  0000 C CNN
+F 0 "U2" H 6200 4650 50  0000 C CNN
 F 1 "MAX31855EASA" H 6400 4550 50  0000 C CNN
 F 2 "Package_SO:SOIC-8_3.9x4.9mm_P1.27mm" H 7050 3800 50  0001 C CIN
@@
 AR Path="/609CA6A8/60B108D6/609F3008" Ref="C27"  Part="1"
 AR Path="/609CA6A8/60B118F2/609F3008" Ref="C29"  Part="1"
-F 0 "C27" H 5565 3696 50  0000 L CNN
+F 0 "C14" H 5565 3696 50  0000 L CNN
 F 1 "0,1" H 5565 3605 50  0000 L CNN
 F 2 "Capacitor_SMD:C_0603_1608Metric_Pad1.08x0.95mm_HandSolder" H 5488 3500 50  0001 C CNN
@@
 AR Path="/609CA6A8/60B108D6/60A063BF" Ref="C26"  Part="1"
 AR Path="/609CA6A8/60B118F2/60A063BF" Ref="C28"  Part="1"
-F 0 "C26" H 5315 4246 50  0000 L CNN
+F 0 "C13" H 5315 4246 50  0000 L CNN
 F 1 "0,01" H 5315 4155 50  0000 L CNN
 F 2 "Capacitor_SMD:C_0603_1608Metric_Pad1.08x0.95mm_HandSolder" H 5238 4050 50  0001 C CNN
