File: furnace/furnace_controller/MCU.sch (KiCad schematic (older format))
At the start: 6 parts

Commit message: Add files via upload
Parts:
- added C? (x3): 0,1, Capacitor_SMD:C_0603_1608Metric_Pad1.08x0.95mm_HandSolder, symbol Device:C
- added C?: 0,01, Capacitor_SMD:C_0603_1608Metric_Pad1.08x0.95mm_HandSolder, symbol Device:C
- added C?: 1u, Capacitor_SMD:C_0603_1608Metric_Pad1.08x0.95mm_HandSolder, symbol Device:C
- added C? (x2): 10p, Capacitor_SMD:C_0603_1608Metric_Pad1.08x0.95mm_HandSolder, symbol Device:C
- added R?: 0, Resistor_SMD:R_0603_1608Metric_Pad0.98x0.95mm_HandSolder, symbol Device:R
- added Y?: 8MHz, symbol Device:Crystal
- C?: value 0603 -> 0,1
- R?: value 0603 -> 10k
Connections:
- net +3V3: now also C?.1, C?.1, R?.1, U?.24 (VDD), U?.36 (VDD), U?.48 (VDD), U?.9 (VDDA), C?.1, C?.1, C?.1, C?.1
- net GND: now also C?.2, C?.2, U?.23 (VSS), U?.35 (VSS), U?.44 (BOOT0), U?.47 (VSS), U?.8 (VSSA), C?.2, C?.2, C?.2, C?.2, C?.2, C?.2, C?.2
- net at U?.5 (PD0): now also C?.1, Y?.1
- net at U?.6 (PD1): now also R?.2
- net at U?.7 (NRST): now also R?.2, C?.1
- new net: C?.1, R?.1, Y?.2
Other:
- moved on the sheet: C?, R?, U?

Commit message: Add files via upload
Parts:
- removed J?: PLS-5, symbol Connector:Conn_01x05_Male
- added J?: PLS-6, symbol Connector:Conn_01x06_Male
Connections:
- net +3V3: now also J?.1 (Pin_1)
- net BZ_EN: now also U?.18 (PB0)
- net CHARGE_PUMP_CLK: now also U?.29 (PA8)
- net DPY_PWR_EN: now also U?.45 (PB8)
- net GND: now also J?.3 (Pin_3), J?.6 (Pin_6)
- net ~TEMP_CS0: now reaches U?.10 (PA0)
- net ~TEMP_CS1: now reaches U?.11 (PA1)
- net ~TEMP_CS2: now reaches U?.12 (PA2)
- net ~TEMP_CS3: now reaches U?.13 (PA3)
- net ~TEMP_CS4: now reaches U?.14 (PA4)
- net SPI1_SCK: now reaches U?.15 (PA5)
- net SPI1_MISO: now reaches U?.16 (PA6)
- net KYBD2: now reaches U?.17 (PA7)
- net SWO: now reaches U?.20 (PB2)
- net SWO: now also J?.4 (Pin_4)
- net KYBD5: now reaches U?.21 (PB10)
- net KYBD4: now reaches U?.22 (PB11)
- net ~SPI2__CS: now reaches U?.25 (PB12)
- net SPI2_SCK: now reaches U?.26 (PB13)
- net SPI2_MISO: now reaches U?.27 (PB14)
- net SPI2_MOSI: now reaches U?.28 (PB15)
- net UART1_TX: now reaches U?.30 (PA9)
- net UART1_TX: now also J?.1 (Pin_1)
- net UART1_RX: now reaches U?.31 (PA10)
- net UART1_RX: now also J?.2 (Pin_2)
- net KYBD1: now reaches U?.32 (PA11)
- net KYBD0: now reaches U?.33 (PA12)
- net SWDIO: now reaches U?.34 (PA13)
- net SWDIO: now also J?.3 (Pin_3)
- net SWCLK: now reaches U?.37 (PA14)
- net SWCLK: now also J?.2 (Pin_2)
- net KYBD3: now reaches U?.38 (PA15)
- net KYBD9: now reaches U?.39 (PB3)
- net KYBD8: now reaches U?.40 (PB4)
- net KYBD7: now reaches U?.41 (PB5)
- net I2C1_SCK: now reaches U?.42 (PB6)
- net I2C1_SDA: now reaches U?.43 (PB7)
- net KYBD6: now reaches U?.46 (PB9)
- net NRST: now reaches C?.1, R?.2, U?.7 (NRST)
- net NRST: now also J?.5 (Pin_5)
Other:
- note added: "Debug_UART"
- note added: "Programming"
- moved on the sheet: J?
Changed lines of the file:
@@
-$EndComp
-$Comp
-L Connector:Conn_01x05_Male J?
-U 1 1 609DE10B
-P 1750 3900
-F 0 "J?" H 1858 4281 50  0000 C CNN
-F 1 "PLS-5" H 1858 4190 50  0000 C CNN
-F 2 "" H 1750 3900 50  0001 C CNN
-F 3 "~" H 1750 3900 50  0001 C CNN
-	1    1750 3900
-	1    0    0    -1
 $EndComp
 $Comp
 L Connector:Conn_01x03_Male J?
 U 1 1 60B5D67E
-P 1750 3150
-F 0 "J?" H 1858 3431 50  0000 C CNN
-F 1 "PLS-3" H 1858 3340 50  0000 C CNN
-F 2 "" H 1750 3150 50  0001 C CNN
-F 3 "~" H 1750 3150 50  0001 C CNN
-	1    1750 3150
-	1    0    0    -1
+P 8200 5200
+F 0 "J?" H 8308 5481 50  0000 C CNN
+F 1 "PLS-3" H 8308 5390 50  0000 C CNN
+F 2 "" H 8200 5200 50  0001 C CNN
+F 3 "~" H 8200 5200 50  0001 C CNN
+	1    8200 5200
+	-1   0    0    -1
 $EndComp
 Text Notes 6300 1100 2    197  ~ 0
@@
 	4700 2800 4700 2850
 Wire Wire Line
-	4700 2850 5300 2850
-Wire Wire Line
 	5300 2850 5300 3100
 Wire Wire Line
@@
 Text HLabel 8900 4350 0    50   Input ~ 0
 DPY_I2C_SCK
-Text HLabel 9050 4850 0    50   Input ~ 0
+Text HLabel 9700 4850 0    50   Input ~ 0
 CHARGE_PUMP_CLK
 Text HLabel 8750 5150 0    50   BiDi ~ 0
@@
 TEMP_SPI_SCK
 Text HLabel 7250 4250 2    50   Input ~ 0
-TEMP_SPI_~CS
-Text HLabel 7850 5300 0    50   BiDi ~ 0
+~TEMP_SPI_CS
+Text HLabel 9550 5350 0    50   BiDi ~ 0
 TEMP_I2C_SDA
-Text HLabel 7850 5200 0    50   Input ~ 0
-TEMP_I2C_SCL
+Text HLabel 9550 5250 0    50   Input ~ 0
+TEMP_I2C_SCK
 Text HLabel 8750 5550 0    50   Input ~ 0
 BZ_EN
@@
 SD_SPI_MOSI
 Text HLabel 7650 6100 0    50   Input ~ 0
-SD_SPI_SCL
+SD_SPI_SCK
 Text HLabel 7650 6300 0    50   Output ~ 0
 SD_SPI_MISO
@@
 Text HLabel 8500 6200 2    50   Output ~ 0
 HEATER_CTRL
+Wire Wire Line
+	6700 5500 6800 5500
+Text Label 6800 5500 0    50   ~ 0
+SWDIO
+Wire Wire Line
+	6700 5600 6800 5600
+Text Label 6800 5600 0    50   ~ 0
+SWCLK
+Text Label 5050 2850 0    50   ~ 0
+NRST
+Wire Wire Line
+	4700 2850 5300 2850
+Text Notes 3150 4650 0    50   ~ 0
+Programming
+Text Label 3600 5400 0    50   ~ 0
+NRST
+Text Label 3600 5200 0    50   ~ 0
+SWDIO
+Text Label 3600 5100 0    50   ~ 0
+SWCLK
+$Comp
+L power:GND #PWR?
+U 1 1 60A6ADB8
+P 3600 5500
+AR Path="/60A6ADB8" Ref="#PWR?"  Part="1"
+AR Path="/609C9D41/60A6ADB8" Ref="#PWR?"  Part="1"
+F 0 "#PWR?" H 3600 5250 50  0001 C CNN
+F 1 "GND" H 3605 5327 50  0000 C CNN
+F 2 "" H 3600 5500 50  0001 C CNN
+F 3 "" H 3600 5500 50  0001 C CNN
+	1    3600 5500
+	1    0    0    -1
+$EndComp
+$Comp
+L power:+3V3 #PWR?
+U 1 1 60A6B5AC
+P 3600 5000
+AR Path="/609CA6A8/60A6B5AC" Ref="#PWR?"  Part="1"
+AR Path="/609C9D41/60A6B5AC" Ref="#PWR?"  Part="1"
+F 0 "#PWR?" H 3600 4850 50  0001 C CNN
+F 1 "+3V3" H 3615 5173 50  0000 C CNN
+F 2 "" H 3600 5000 50  0001 C CNN
+F 3 "" H 3600 5000 50  0001 C CNN
+	1    3600 5000
+	1    0    0    -1
+$EndComp
+Text Label 5300 4400 2    50   ~ 0
+SWO
+Wire Wire Line
+	5300 4400 5400 4400
+Text Label 3600 5300 0    50   ~ 0
+SWO
+$Comp
+L Connector:Conn_01x06_Male J?
+U 1 1 60A6D6DF
+P 3300 5200
+F 0 "J?" H 3408 5581 50  0000 C CNN
+F 1 "PLS-6" H 3408 5490 50  0000 C CNN
+F 2 "" H 3300 5200 50  0001 C CNN
+F 3 "~" H 3300 5200 50  0001 C CNN
+	1    3300 5200
+	1    0    0    -1
+$EndComp
+Wire Wire Line
+	3600 5000 3500 5000
+Wire Wire Line
+	3600 5100 3500 5100
+Wire Wire Line
+	3600 5200 3500 5200
+Wire Wire Line
+	3600 5300 3500 5300
+Wire Wire Line
+	3600 5400 3500 5400
+Wire Wire Line
+	3600 5500 3500 5500
+Text Label 6800 4700 0    50   ~ 0
+SPI1_SCK
+Text Label 6800 4800 0    50   ~ 0
+SPI1_MISO
+Text Label 6800 4200 0    50   ~ 0
+~TEMP_CS0
+Text Label 6800 4300 0    50   ~ 0
+~TEMP_CS1
+Text Label 6800 4400 0    50   ~ 0
+~TEMP_CS2
+Text Label 6800 4500 0    50   ~ 0
+~TEMP_CS3
+Text Label 6800 4600 0    50   ~ 0
+~TEMP_CS4
+Wire Wire Line
+	6800 4200 6700 4200
+Wire Wire Line
+	6800 4300 6700 4300
+Wire Wire Line
+	6800 4400 6700 4400
+Wire Wire Line
+	6800 4500 6700 4500
+Wire Wire Line
+	6800 4600 6700 4600
+Wire Wire Line
+	6800 4700 6700 4700
+Wire Wire Line
+	6800 4800 6700 4800
+Text Label 5300 4200 2    50   ~ 0
+BZ_EN
+Wire Wire Line
+	5300 4200 5400 4200
+Text Label 5300 5600 2    50   ~ 0
+SPI2_MISO
+Text Label 5300 5400 2    50   ~ 0
+~SPI2__CS
+Text Label 5300 5500 2    50   ~ 0
+SPI2_SCK
+Text Label 5300 5700 2    50   ~ 0
+SPI2_MOSI
+Wire Wire Line
+	5300 5400 5400 5400
+Wire Wire Line
+	5300 5500 5400 5500
+Wire Wire Line
+	5300 5600 5400 5600
+Wire Wire Line
+	5300 5700 5400 5700
+Text Label 5300 4800 2    50   ~ 0
+I2C1_SCK
+Text Label 5300 4900 2    50   ~ 0
+I2C1_SDA
+Wire Wire Line
+	5300 4800 5400 4800
+Wire Wire Line
+	5300 4900 5400 4900
+Text Label 6800 5100 0    50   ~ 0
+UART1_TX
+Text Label 6800 5200 0    50   ~ 0
+UART1_RX
+Text Notes 8100 4850 0    50   ~ 0
+Debug_UART
+$Comp
+L power:GND #PWR?
+U 1 1 60AA9C84
+P 7900 5300
+AR Path="/60AA9C84" Ref="#PWR?"  Part="1"
+AR Path="/609C9D41/60AA9C84" Ref="#PWR?"  Part="1"
+F 0 "#PWR?" H 7900 5050 50  0001 C CNN
+F 1 "GND" H 7905 5127 50  0000 C CNN
+F 2 "" H 7900 5300 50  0001 C CNN
+F 3 "" H 7900 5300 50  0001 C CNN
+	1    7900 5300
+	1    0    0    -1
+$EndComp
+Wire Wire Line
+	6700 5100 8000 5100
+Wire Wire Line
+	6700 5200 8000 5200
+Wire Wire Line
+	7900 5300 8000 5300
+Text Label 5300 5000 2    50   ~ 0
+DPY_PWR_EN
+Text Label 6800 5000 0    50   ~ 0
+CHARGE_PUMP_CLK
+Wire Wire Line
+	5300 5000 5400 5000
+Text Label 6800 5400 0    50   ~ 0
+KYBD0
+Text Label 6800 5300 0    50   ~ 0
+KYBD1
+Text Label 6800 4900 0    50   ~ 0
+KYBD2
+Text Label 6800 5700 0    50   ~ 0
+KYBD3
+Text Label 5200 5300 2    50   ~ 0
+KYBD4
+Text Label 5200 5200 2    50   ~ 0
+KYBD5
+Text Label 5200 5100 2    50   ~ 0
+KYBD6
+Text Label 5300 4700 2    50   ~ 0
+KYBD7
+Text Label 5300 4600 2    50   ~ 0
+KYBD8
+Text Label 5300 4500 2    50   ~ 0
+KYBD9
+Wire Wire Line
+	5300 4500 5400 4500
+Wire Wire Line
+	5300 4600 5400 4600
+Wire Wire Line
+	5300 4700 5400 4700
+Wire Wire Line
+	5200 5100 5400 5100
+Wire Wire Line
+	5200 5200 5400 5200
+Wire Wire Line
+	5200 5300 5400 5300
+Wire Wire Line
+	6700 5700 6800 5700
+Wire Wire Line
+	6700 4900 6800 4900
+Wire Wire Line
+	6700 5300 6800 5300
+Wire Wire Line
+	6700 5400 6800 5400
+Wire Wire Line
+	6700 5000 6800 5000
 $EndSCHEMATC

Commit message: Add files via upload
Connections:
- net I2C1_SCK is gone; now on net DPY_I2C_SCK: U?.42 (PB6)
- net I2C1_SDA is gone; now on net DPY_I2C_SDA: U?.43 (PB7)
- net SPI1_MISO is gone; now on net TEMP_SPI_MISO: U?.16 (PA6)
- net SPI1_SCK is gone; now on net TEMP_SPI_SCK: U?.15 (PA5)
- net SPI2_MISO is gone; now on net SD_SPI_MISO: U?.27 (PB14)
- net SPI2_MOSI is gone; now on net SD_SPI_MOSI: U?.28 (PB15)
- net SPI2_SCK is gone; now on net SD_SPI_SCK: U?.26 (PB13)
- net UART1_RX is gone; now on net EXT_UART_RX: J?.2 (Pin_2), U?.31 (PA10)
- net UART1_TX is gone; now on net HEATER_CTRL: J?.1 (Pin_1), U?.30 (PA9)
- net KYBD7: now also U?.40 (PB4); no longer U?.41 (PB5)
- net KYBD8: now also U?.39 (PB3); no longer U?.40 (PB4)
- net KYBD9: now also U?.19 (PB1); no longer U?.39 (PB3)
- net ~DPY_RST: now also U?.41 (PB5)
- net ~SPI2__CS renamed ~SD_SPI_CS

Commit message: Add files via upload
Parts:
- added C?: 0,01, Capacitor_SMD:C_0603_1608Metric_Pad1.08x0.95mm_HandSolder, symbol Device:C
- added R?: 3,3k, Resistor_SMD:R_0603_1608Metric_Pad0.98x0.95mm_HandSolder, symbol Device:R
- added R?: 1k, Resistor_SMD:R_0603_1608Metric_Pad0.98x0.95mm_HandSolder, symbol Device:R
- added R?: 100, Resistor_SMD:R_0603_1608Metric_Pad0.98x0.95mm_HandSolder, symbol Device:R
Connections:
- net EXT_UART_RX: now also R?.1, R?.1; no longer J?.2 (Pin_2), U?.31 (PA10)
- net GND: now also C?.2, R?.2
- net HEATER_CTRL: now also R?.2; no longer J?.1 (Pin_1), U?.30 (PA9)
- new net UART1_RX: C?.1, J?.2 (Pin_2), R?.2, U?.31 (PA10)
- new net UART1_TX: J?.1 (Pin_1), R?.1, U?.30 (PA9)
Other:
- note added: "5V to 3V level converter"
Changed lines of the file:
@@
 $Descr A4 11693 8268
 encoding utf-8
-Sheet 2 17
+Sheet 2 18
 Title ""
 Date ""
@@
 Text HLabel 10000 5750 2    50   Input ~ 0
 SD_SPI_MISO
-Text HLabel 1500 2000 0    50   Input ~ 0
+Text HLabel 1500 1000 0    50   Input ~ 0
 EXT_UART_RX
 Text HLabel 10000 1500 2    50   Output ~ 0
@@
 Wire Wire Line
 	6700 5000 6800 5000
-Text Label 9500 1500 2    50   ~ 0
+Text Label 9000 1500 2    50   ~ 0
 UART1_TX
-Text Label 2000 2000 0    50   ~ 0
+Text Label 3500 1250 0    50   ~ 0
 UART1_RX
 Text Label 9500 5750 2    50   ~ 0
@@
 	9850 4000 9750 4100
 Wire Wire Line
-	1500 2000 2000 2000
+	1500 1000 2000 1000
 Wire Wire Line
 	1500 3000 2000 3000
@@
 Wire Wire Line
 	9500 5750 10000 5750
+$Comp
+L Device:R R?
+U 1 1 60ACA8BC
+P 2000 1550
+AR Path="/60ACA8BC" Ref="R?"  Part="1"
+AR Path="/609C9D41/60ACA8BC" Ref="R?"  Part="1"
+AR Path="/60B42F62/60ACA8BC" Ref="R?"  Part="1"
+F 0 "R?" H 2070 1596 50  0000 L CNN
+F 1 "3,3k" H 2070 1505 50  0000 L CNN
+F 2 "Resistor_SMD:R_0603_1608Metric_Pad0.98x0.95mm_HandSolder" V 1930 1550 50  0001 C CNN
+F 3 "~" H 2000 1550 50  0001 C CNN
+	1    2000 1550
+	1    0    0    -1
+$EndComp
+$Comp
+L power:GND #PWR?
+U 1 1 60ACF85F
+P 2000 1700
+AR Path="/60ACF85F" Ref="#PWR?"  Part="1"
+AR Path="/609C9D41/60ACF85F" Ref="#PWR?"  Part="1"
+AR Path="/60B42F62/60ACF85F" Ref="#PWR?"  Part="1"
+F 0 "#PWR?" H 2000 1450 50  0001 C CNN
+F 1 "GND" H 2005 1527 50  0000 C CNN
+F 2 "" H 2000 1700 50  0001 C CNN
+F 3 "" H 2000 1700 50  0001 C CNN
+	1    2000 1700
+	1    0    0    -1
+$EndComp
+Text Notes 950  1450 0    50   ~ 0
+5V to 3V level converter
+Wire Wire Line
+	2000 1000 2000 1250
+Wire Wire Line
+	2500 1250 2000 1250
+Connection ~ 2000 1250
+Wire Wire Line
+	2000 1250 2000 1400
+$Comp
+L Device:R R?
+U 1 1 60AF6532
+P 2650 1250
+AR Path="/60AF6532" Ref="R?"  Part="1"
+AR Path="/609C9D41/60AF6532" Ref="R?"  Part="1"
+AR Path="/60B42F62/60AF6532" Ref="R?"  Part="1"
+F 0 "R?" V 2750 1200 50  0000 L CNN
+F 1 "1k" V 2550 1200 50  0000 L CNN
+F 2 "Resistor_SMD:R_0603_1608Metric_Pad0.98x0.95mm_HandSolder" V 2580 1250 50  0001 C CNN
+F 3 "~" H 2650 1250 50  0001 C CNN
+	1    2650 1250
+	0    -1   -1   0
+$EndComp
+$Comp
+L Device:C C?
+U 1 1 60AFB0FE
+P 3000 1400
+AR Path="/60AFB0FE" Ref="C?"  Part="1"
+AR Path="/609C9D41/60AFB0FE" Ref="C?"  Part="1"
+AR Path="/60B42F62/60AFB0FE" Ref="C?"  Part="1"
+F 0 "C?" H 3115 1446 50  0000 L CNN
+F 1 "0,01" H 3115 1355 50  0000 L CNN
+F 2 "Capacitor_SMD:C_0603_1608Metric_Pad1.08x0.95mm_HandSolder" H 3038 1250 50  0001 C CNN
+F 3 "~" H 3000 1400 50  0001 C CNN
+	1    3000 1400
+	1    0    0    -1
+$EndComp
+$Comp
+L power:GND #PWR?
+U 1 1 60AFB104
+P 3000 1550
+AR Path="/60AFB104" Ref="#PWR?"  Part="1"
+AR Path="/609C9D41/60AFB104" Ref="#PWR?"  Part="1"
+AR Path="/60B42F62/60AFB104" Ref="#PWR?"  Part="1"
+F 0 "#PWR?" H 3000 1300 50  0001 C CNN
+F 1 "GND" H 3005 1377 50  0000 C CNN
+F 2 "" H 3000 1550 50  0001 C CNN
+F 3 "" H 3000 1550 50  0001 C CNN
+	1    3000 1550
+	1    0    0    -1
+$EndComp
+Wire Wire Line
+	3500 1250 3000 1250
+Connection ~ 3000 1250
+Wire Wire Line
+	3000 1250 2800 1250
+$Comp
+L Device:R R?
+U 1 1 60B10008
+P 9350 1500
+AR Path="/60B10008" Ref="R?"  Part="1"
+AR Path="/609C9D41/60B10008" Ref="R?"  Part="1"
+AR Path="/60B42F62/60B10008" Ref="R?"  Part="1"
+F 0 "R?" V 9450 1450 50  0000 L CNN
+F 1 "100" V 9250 1450 50  0000 L CNN
+F 2 "Resistor_SMD:R_0603_1608Metric_Pad0.98x0.95mm_HandSolder" V 9280 1500 50  0001 C CNN
+F 3 "~" H 9350 1500 50  0001 C CNN
+	1    9350 1500
+	0    -1   -1   0
+$EndComp
+Wire Wire Line
+	9000 1500 9200 1500
 Wire Bus Line
 	1500 2500 3500 2500

Commit message: Add files via upload
Parts:
- added Q?: BC847, Package_TO_SOT_SMD:SOT-23, symbol Transistor_BJT:BC847
- added R?: 150, Resistor_SMD:R_0603_1608Metric_Pad0.98x0.95mm_HandSolder, symbol Device:R
- added R?: 56k, Resistor_SMD:R_0603_1608Metric_Pad0.98x0.95mm_HandSolder, symbol Device:R
- R?: value 100 -> 3,3k
Connections:
- net GND: now also Q?.2 (E), R?.2
- net HEATER_CTRL: now also R?.2; no longer R?.2
- new net: Q?.1 (B), R?.1, R?.2
- new net: Q?.3 (C), R?.1
Other:
- moved on the sheet: R?
Changed lines of the file:
@@
 Text HLabel 1500 1000 0    50   Input ~ 0
 EXT_UART_RX
-Text HLabel 10000 1500 2    50   Output ~ 0
-HEATER_CTRL
 Wire Wire Line
 	6700 5500 6800 5500
@@
 Wire Wire Line
 	6700 5000 6800 5000
-Text Label 9000 1500 2    50   ~ 0
+Text Label 8000 1200 2    50   ~ 0
 UART1_TX
 Text Label 3500 1250 0    50   ~ 0
@@
 	1500 3250 2000 3250
 Wire Wire Line
-	9500 1500 10000 1500
-Wire Wire Line
 	9500 2000 10000 2000
 Wire Wire Line
@@
 L Device:R R?
 U 1 1 60B10008
-P 9350 1500
+P 8350 1200
 AR Path="/60B10008" Ref="R?"  Part="1"
 AR Path="/609C9D41/60B10008" Ref="R?"  Part="1"
 AR Path="/60B42F62/60B10008" Ref="R?"  Part="1"
-F 0 "R?" V 9450 1450 50  0000 L CNN
-F 1 "100" V 9250 1450 50  0000 L CNN
-F 2 "Resistor_SMD:R_0603_1608Metric_Pad0.98x0.95mm_HandSolder" V 9280 1500 50  0001 C CNN
-F 3 "~" H 9350 1500 50  0001 C CNN
-	1    9350 1500
+F 0 "R?" V 8450 1150 50  0000 L CNN
+F 1 "3,3k" V 8250 1150 50  0000 L CNN
+F 2 "Resistor_SMD:R_0603_1608Metric_Pad0.98x0.95mm_HandSolder" V 8280 1200 50  0001 C CNN
+F 3 "~" H 8350 1200 50  0001 C CNN
+	1    8350 1200
 	0    -1   -1   0
 $EndComp
 Wire Wire Line
-	9000 1500 9200 1500
+	8000 1200 8200 1200
+$Comp
+L Transistor_BJT:BC847 Q?
+U 1 1 60AE3B9E
+P 8900 1200
+F 0 "Q?" H 9091 1246 50  0000 L CNN
+F 1 "BC847" H 9091 1155 50  0000 L CNN
+F 2 "Package_TO_SOT_SMD:SOT-23" H 9100 1125 50  0001 L CIN
+F 3 "http://www.infineon.com/dgdl/Infineon-BC847SERIES_BC848SERIES_BC849SERIES_BC850SERIES-DS-v01_01-en.pdf?fileId=db3a304314dca389011541d4630a1657" H 8900 1200 50  0001 L CNN
+	1    8900 1200
+	1    0    0    -1
+$EndComp
+Text HLabel 10000 1000 2    50   Output ~ 0
+HEATER_CTRL
+Wire Wire Line
+	9500 1000 10000 1000
+$Comp
+L Device:R R?
+U 1 1 60AE8C55
+P 9350 1000
+AR Path="/60AE8C55" Ref="R?"  Part="1"
+AR Path="/609C9D41/60AE8C55" Ref="R?"  Part="1"
+AR Path="/60B42F62/60AE8C55" Ref="R?"  Part="1"
+F 0 "R?" V 9450 950 50  0000 L CNN
+F 1 "150" V 9250 950 50  0000 L CNN
+F 2 "Resistor_SMD:R_0603_1608Metric_Pad0.98x0.95mm_HandSolder" V 9280 1000 50  0001 C CNN
+F 3 "~" H 9350 1000 50  0001 C CNN
+	1    9350 1000
+	0    -1   -1   0
+$EndComp
+$Comp
+L Device:R R?
+U 1 1 60AF1C85
+P 8600 1350
+AR Path="/60AF1C85" Ref="R?"  Part="1"
+AR Path="/609C9D41/60AF1C85" Ref="R?"  Part="1"
+AR Path="/60B42F62/60AF1C85" Ref="R?"  Part="1"
+F 0 "R?" H 8670 1396 50  0000 L CNN
+F 1 "56k" H 8670 1305 50  0000 L CNN
+F 2 "Resistor_SMD:R_0603_1608Metric_Pad0.98x0.95mm_HandSolder" V 8530 1350 50  0001 C CNN
+F 3 "~" H 8600 1350 50  0001 C CNN
+	1    8600 1350
+	1    0    0    -1
+$EndComp
+$Comp
+L power:GND #PWR?
+U 1 1 60AF59E1
+P 9000 1500
+AR Path="/60AF59E1" Ref="#PWR?"  Part="1"
+AR Path="/609C9D41/60AF59E1" Ref="#PWR?"  Part="1"
+AR Path="/60B42F62/60AF59E1" Ref="#PWR?"  Part="1"
+F 0 "#PWR?" H 9000 1250 50  0001 C CNN
+F 1 "GND" H 9005 1327 50  0000 C CNN
+F 2 "" H 9000 1500 50  0001 C CNN
+F 3 "" H 9000 1500 50  0001 C CNN
+	1    9000 1500
+	1    0    0    -1
+$EndComp
+Wire Wire Line
+	8500 1200 8600 1200
+Wire Wire Line
+	8600 1200 8700 1200
+Connection ~ 8600 1200
+Wire Wire Line
+	9000 1000 9200 1000
+Wire Wire Line
+	9000 1400 9000 1500
+Wire Wire Line
+	8600 1500 9000 1500
+Connection ~ 9000 1500
 Wire Bus Line
 	1500 2500 3500 2500

Commit message: Add files via upload
Parts:
- gave numbers to parts that had none: 22
Connections:
- no-connect marks 0 -> 4

Commit message: Add files via upload
Parts:
- removed J7: PLS-6, symbol Connector:Conn_01x06_Male
- added J7: PLS-5, symbol Connector:Conn_01x05_Male
Connections:
- net +3V3: now also J7.1 (Pin_1)
- net GND: now also J7.5 (Pin_5)
- net NRST: now also J7.4 (Pin_4)
- net SWCLK: now also J7.2 (Pin_2)
- net SWDIO: now also J7.3 (Pin_3)
- net SWO: no longer names the net of U1.20 (PB2)
- no-connect marks 4 -> 5
Changed lines of the file:
@@
 Text Notes 3150 4650 0    50   ~ 0
 Programming
-Text Label 3600 5400 0    50   ~ 0
+Text Label 3600 5300 0    50   ~ 0
 NRST
 Text Label 3600 5200 0    50   ~ 0
@@
 L power:GND #PWR?
 U 1 1 60A6ADB8
-P 3600 5500
+P 3600 5400
 AR Path="/60A6ADB8" Ref="#PWR?"  Part="1"
 AR Path="/609C9D41/60A6ADB8" Ref="#PWR05"  Part="1"
 AR Path="/60B42F62/60A6ADB8" Ref="#PWR?"  Part="1"
-F 0 "#PWR05" H 3600 5250 50  0001 C CNN
-F 1 "GND" H 3605 5327 50  0000 C CNN
-F 2 "" H 3600 5500 50  0001 C CNN
-F 3 "" H 3600 5500 50  0001 C CNN
-	1    3600 5500
+F 0 "#PWR05" H 3600 5150 50  0001 C CNN
+F 1 "GND" H 3605 5227 50  0000 C CNN
+F 2 "" H 3600 5400 50  0001 C CNN
+F 3 "" H 3600 5400 50  0001 C CNN
+	1    3600 5400
 	1    0    0    -1
 $EndComp
@@
 	1    0    0    -1
 $EndComp
-Text Label 5300 4400 2    50   ~ 0
-SWO
-Wire Wire Line
-	5300 4400 5400 4400
-Text Label 3600 5300 0    50   ~ 0
-SWO
-$Comp
-L Connector:Conn_01x06_Male J7
-U 1 1 60A6D6DF
-P 3300 5200
-AR Path="/609C9D41/60A6D6DF" Ref="J7"  Part="1"
-AR Path="/60B42F62/60A6D6DF" Ref="J?"  Part="1"
-F 0 "J7" H 3408 5581 50  0000 C CNN
-F 1 "PLS-6" H 3408 5490 50  0000 C CNN
-F 2 "" H 3300 5200 50  0001 C CNN
-F 3 "~" H 3300 5200 50  0001 C CNN
-	1    3300 5200
-	1    0    0    -1
-$EndComp
 Wire Wire Line
 	3600 5000 3500 5000
@@
 Wire Wire Line
 	3600 5400 3500 5400
-Wire Wire Line
-	3600 5500 3500 5500
 Text Label 6800 4700 0    50   ~ 0
 SPI1_SCK
@@
 Text Label 1700 2500 0    50   ~ 0
 ~TEMP_CS[0..4]
+$Comp
+L Connector:Conn_01x05_Male J7
+U 1 1 6127CB85
+P 3300 5200
+F 0 "J7" H 3408 5581 50  0000 C CNN
+F 1 "PLS-5" H 3408 5490 50  0000 C CNN
+F 2 "" H 3300 5200 50  0001 C CNN
+F 3 "~" H 3300 5200 50  0001 C CNN
+	1    3300 5200
+	1    0    0    -1
+$EndComp
+NoConn ~ 5400 4400
 Wire Bus Line
 	1500 2500 3500 2500
