File: furnace/furnace_controller/MCU.sch (KiCad schematic (older format))
At the start: 22 parts, among them J7 PLS-5, J8 PLS-3, Q1 BC847, U1 STM32F103C6Tx, Y1 8MHz

Commit message: Add files via upload
Parts:
- C1, C10, C2, C3, C4, C5, C6, C7, C8: footprint Capacitor_SMD:C_0603_1608Metric_Pad1.08x0.95mm_HandSolder -> Capacitor_SMD:C_0603_1608Metric_Pad1.05x0.95mm_HandSolder
- C9: footprint Capacitor_SMD:C_1206_3216Metric_Pad1.33x1.80mm_HandSolder -> Capacitor_SMD:C_1206_3216Metric_Pad1.42x1.75mm_HandSolder
- J7: footprint (none) -> Connector_PinHeader_2.54mm:PinHeader_1x05_P2.54mm_Vertical
- J8: footprint (none) -> Connector_PinHeader_2.54mm:PinHeader_1x03_P2.54mm_Vertical
- R1, R2, R3, R4, R5, R6, R7: footprint Resistor_SMD:R_0603_1608Metric_Pad0.98x0.95mm_HandSolder -> Resistor_SMD:R_0603_1608Metric_Pad1.05x0.95mm_HandSolder
Changed lines of the file:
@@
 encoding utf-8
 Sheet 18 18
-Title ""
-Date ""
-Rev ""
-Comp ""
+Title "Furnace controller"
+Date "2021-08-26"
+Rev "1.0"
+Comp "Yuriy Volkov"
 Comment1 ""
 Comment2 ""
@@
 F 0 "J8" H 8308 5481 50  0000 C CNN
 F 1 "PLS-3" H 8308 5390 50  0000 C CNN
-F 2 "" H 8200 5200 50  0001 C CNN
+F 2 "Connector_PinHeader_2.54mm:PinHeader_1x03_P2.54mm_Vertical" H 8200 5200 50  0001 C CNN
 F 3 "~" H 8200 5200 50  0001 C CNN
 	1    8200 5200
@@
 F 0 "R4" H 4770 2696 50  0000 L CNN
 F 1 "10k" H 4770 2605 50  0000 L CNN
-F 2 "Resistor_SMD:R_0603_1608Metric_Pad0.98x0.95mm_HandSolder" V 4630 2650 50  0001 C CNN
+F 2 "Resistor_SMD:R_0603_1608Metric_Pad1.05x0.95mm_HandSolder" V 4630 2650 50  0001 C CNN
 F 3 "~" H 4700 2650 50  0001 C CNN
 	1    4700 2650
@@
 F 0 "C5" H 6665 2196 50  0000 L CNN
 F 1 "0,1" H 6665 2105 50  0000 L CNN
-F 2 "Capacitor_SMD:C_0603_1608Metric_Pad1.08x0.95mm_HandSolder" H 6588 2000 50  0001 C CNN
+F 2 "Capacitor_SMD:C_0603_1608Metric_Pad1.05x0.95mm_HandSolder" H 6588 2000 50  0001 C CNN
 F 3 "~" H 6550 2150 50  0001 C CNN
 	1    6550 2150
@@
 F 0 "C9" H 7865 2196 50  0000 L CNN
 F 1 "4,7" H 7865 2105 50  0000 L CNN
-F 2 "Capacitor_SMD:C_1206_3216Metric_Pad1.33x1.80mm_HandSolder" H 7788 2000 50  0001 C CNN
+F 2 "Capacitor_SMD:C_1206_3216Metric_Pad1.42x1.75mm_HandSolder" H 7788 2000 50  0001 C CNN
 F 3 "~" H 7750 2150 50  0001 C CNN
 	1    7750 2150
@@
 F 0 "C6" H 7065 2196 50  0000 L CNN
 F 1 "0,1" H 7065 2105 50  0000 L CNN
-F 2 "Capacitor_SMD:C_0603_1608Metric_Pad1.08x0.95mm_HandSolder" H 6988 2000 50  0001 C CNN
+F 2 "Capacitor_SMD:C_0603_1608Metric_Pad1.05x0.95mm_HandSolder" H 6988 2000 50  0001 C CNN
 F 3 "~" H 6950 2150 50  0001 C CNN
 	1    6950 2150
@@
 F 0 "C7" H 7465 2196 50  0000 L CNN
 F 1 "0,1" H 7465 2105 50  0000 L CNN
-F 2 "Capacitor_SMD:C_0603_1608Metric_Pad1.08x0.95mm_HandSolder" H 7388 2000 50  0001 C CNN
+F 2 "Capacitor_SMD:C_0603_1608Metric_Pad1.05x0.95mm_HandSolder" H 7388 2000 50  0001 C CNN
 F 3 "~" H 7350 2150 50  0001 C CNN
 	1    7350 2150
@@
 F 0 "C8" H 7465 3096 50  0000 L CNN
 F 1 "0,01" H 7465 3005 50  0000 L CNN
-F 2 "Capacitor_SMD:C_0603_1608Metric_Pad1.08x0.95mm_HandSolder" H 7388 2900 50  0001 C CNN
+F 2 "Capacitor_SMD:C_0603_1608Metric_Pad1.05x0.95mm_HandSolder" H 7388 2900 50  0001 C CNN
 F 3 "~" H 7350 3050 50  0001 C CNN
 	1    7350 3050
@@
 F 0 "C10" H 7865 3096 50  0000 L CNN
 F 1 "1u" H 7865 3005 50  0000 L CNN
-F 2 "Capacitor_SMD:C_0603_1608Metric_Pad1.08x0.95mm_HandSolder" H 7788 2900 50  0001 C CNN
+F 2 "Capacitor_SMD:C_0603_1608Metric_Pad1.05x0.95mm_HandSolder" H 7788 2900 50  0001 C CNN
 F 3 "~" H 7750 3050 50  0001 C CNN
 	1    7750 3050
@@
 F 0 "C2" H 3115 3796 50  0000 L CNN
 F 1 "10p" H 3115 3705 50  0000 L CNN
-F 2 "Capacitor_SMD:C_0603_1608Metric_Pad1.08x0.95mm_HandSolder" H 3038 3600 50  0001 C CNN
+F 2 "Capacitor_SMD:C_0603_1608Metric_Pad1.05x0.95mm_HandSolder" H 3038 3600 50  0001 C CNN
 F 3 "~" H 3000 3750 50  0001 C CNN
 	1    3000 3750
@@
 F 0 "C3" H 3715 3796 50  0000 L CNN
 F 1 "10p" H 3715 3705 50  0000 L CNN
-F 2 "Capacitor_SMD:C_0603_1608Metric_Pad1.08x0.95mm_HandSolder" H 3638 3600 50  0001 C CNN
+F 2 "Capacitor_SMD:C_0603_1608Metric_Pad1.05x0.95mm_HandSolder" H 3638 3600 50  0001 C CNN
 F 3 "~" H 3600 3750 50  0001 C CNN
 	1    3600 3750
@@
 F 0 "R3" V 4150 3550 50  0000 L CNN
 F 1 "0" V 3950 3600 50  0000 L CNN
-F 2 "Resistor_SMD:R_0603_1608Metric_Pad0.98x0.95mm_HandSolder" V 3980 3600 50  0001 C CNN
+F 2 "Resistor_SMD:R_0603_1608Metric_Pad1.05x0.95mm_HandSolder" V 3980 3600 50  0001 C CNN
 F 3 "~" H 4050 3600 50  0001 C CNN
 	1    4050 3600
@@
 F 0 "C4" H 4815 3096 50  0000 L CNN
 F 1 "0,1" H 4815 3005 50  0000 L CNN
-F 2 "Capacitor_SMD:C_0603_1608Metric_Pad1.08x0.95mm_HandSolder" H 4738 2900 50  0001 C CNN
+F 2 "Capacitor_SMD:C_0603_1608Metric_Pad1.05x0.95mm_HandSolder" H 4738 2900 50  0001 C CNN
 F 3 "~" H 4700 3050 50  0001 C CNN
 	1    4700 3050
@@
 F 0 "R1" H 2070 1596 50  0000 L CNN
 F 1 "3,3k" H 2070 1505 50  0000 L CNN
-F 2 "Resistor_SMD:R_0603_1608Metric_Pad0.98x0.95mm_HandSolder" V 1930 1550 50  0001 C CNN
+F 2 "Resistor_SMD:R_0603_1608Metric_Pad1.05x0.95mm_HandSolder" V 1930 1550 50  0001 C CNN
 F 3 "~" H 2000 1550 50  0001 C CNN
 	1    2000 1550
@@
 F 0 "R2" V 2750 1200 50  0000 L CNN
 F 1 "1k" V 2550 1200 50  0000 L CNN
-F 2 "Resistor_SMD:R_0603_1608Metric_Pad0.98x0.95mm_HandSolder" V 2580 1250 50  0001 C CNN
+F 2 "Resistor_SMD:R_0603_1608Metric_Pad1.05x0.95mm_HandSolder" V 2580 1250 50  0001 C CNN
 F 3 "~" H 2650 1250 50  0001 C CNN
 	1    2650 1250
@@
 F 0 "C1" H 3115 1446 50  0000 L CNN
 F 1 "0,01" H 3115 1355 50  0000 L CNN
-F 2 "Capacitor_SMD:C_0603_1608Metric_Pad1.08x0.95mm_HandSolder" H 3038 1250 50  0001 C CNN
+F 2 "Capacitor_SMD:C_0603_1608Metric_Pad1.05x0.95mm_HandSolder" H 3038 1250 50  0001 C CNN
 F 3 "~" H 3000 1400 50  0001 C CNN
 	1    3000 1400
@@
 F 0 "R5" V 8450 1150 50  0000 L CNN
 F 1 "3,3k" V 8250 1150 50  0000 L CNN
-F 2 "Resistor_SMD:R_0603_1608Metric_Pad0.98x0.95mm_HandSolder" V 8280 1200 50  0001 C CNN
+F 2 "Resistor_SMD:R_0603_1608Metric_Pad1.05x0.95mm_HandSolder" V 8280 1200 50  0001 C CNN
 F 3 "~" H 8350 1200 50  0001 C CNN
 	1    8350 1200
@@
 F 0 "R7" V 9450 950 50  0000 L CNN
 F 1 "150" V 9250 950 50  0000 L CNN
-F 2 "Resistor_SMD:R_0603_1608Metric_Pad0.98x0.95mm_HandSolder" V 9280 1000 50  0001 C CNN
+F 2 "Resistor_SMD:R_0603_1608Metric_Pad1.05x0.95mm_HandSolder" V 9280 1000 50  0001 C CNN
 F 3 "~" H 9350 1000 50  0001 C CNN
 	1    9350 1000
@@
 F 0 "R6" H 8670 1396 50  0000 L CNN
 F 1 "56k" H 8670 1305 50  0000 L CNN
-F 2 "Resistor_SMD:R_0603_1608Metric_Pad0.98x0.95mm_HandSolder" V 8530 1350 50  0001 C CNN
+F 2 "Resistor_SMD:R_0603_1608Metric_Pad1.05x0.95mm_HandSolder" V 8530 1350 50  0001 C CNN
 F 3 "~" H 8600 1350 50  0001 C CNN
 	1    8600 1350
@@
 F 0 "J7" H 3408 5581 50  0000 C CNN
 F 1 "PLS-5" H 3408 5490 50  0000 C CNN
-F 2 "" H 3300 5200 50  0001 C CNN
+F 2 "Connector_PinHeader_2.54mm:PinHeader_1x05_P2.54mm_Vertical" H 3300 5200 50  0001 C CNN
 F 3 "~" H 3300 5200 50  0001 C CNN
 	1    3300 5200

Commit message: Add files via upload
Parts:
- C34: renamed from C1; footprint Capacitor_SMD:C_0603_1608Metric_Pad1.05x0.95mm_HandSolder -> Capacitor_SMD:C_0603_1608Metric_Pad1.08x0.95mm_HandSolder
- C35: renamed from C2; footprint Capacitor_SMD:C_0603_1608Metric_Pad1.05x0.95mm_HandSolder -> Capacitor_SMD:C_0603_1608Metric_Pad1.08x0.95mm_HandSolder
- C36: renamed from C3; footprint Capacitor_SMD:C_0603_1608Metric_Pad1.05x0.95mm_HandSolder -> Capacitor_SMD:C_0603_1608Metric_Pad1.08x0.95mm_HandSolder
- C37: renamed from C4; footprint Capacitor_SMD:C_0603_1608Metric_Pad1.05x0.95mm_HandSolder -> Capacitor_SMD:C_0603_1608Metric_Pad1.08x0.95mm_HandSolder
- C38: renamed from C5; footprint Capacitor_SMD:C_0603_1608Metric_Pad1.05x0.95mm_HandSolder -> Capacitor_SMD:C_0603_1608Metric_Pad1.08x0.95mm_HandSolder
- C39: renamed from C6; footprint Capacitor_SMD:C_0603_1608Metric_Pad1.05x0.95mm_HandSolder -> Capacitor_SMD:C_0603_1608Metric_Pad1.08x0.95mm_HandSolder
- C40: renamed from C7; footprint Capacitor_SMD:C_0603_1608Metric_Pad1.05x0.95mm_HandSolder -> Capacitor_SMD:C_0603_1608Metric_Pad1.08x0.95mm_HandSolder
- C41: renamed from C8; footprint Capacitor_SMD:C_0603_1608Metric_Pad1.05x0.95mm_HandSolder -> Capacitor_SMD:C_0603_1608Metric_Pad1.08x0.95mm_HandSolder
- C42: renamed from C9; footprint Capacitor_SMD:C_1206_3216Metric_Pad1.42x1.75mm_HandSolder -> Capacitor_SMD:C_1206_3216Metric_Pad1.33x1.80mm_HandSolder
- C43: renamed from C10; footprint Capacitor_SMD:C_0603_1608Metric_Pad1.05x0.95mm_HandSolder -> Capacitor_SMD:C_0603_1608Metric_Pad1.08x0.95mm_HandSolder
- R46: renamed from R1; footprint Resistor_SMD:R_0603_1608Metric_Pad1.05x0.95mm_HandSolder -> Resistor_SMD:R_0603_1608Metric_Pad0.98x0.95mm_HandSolder
- R47: renamed from R2; footprint Resistor_SMD:R_0603_1608Metric_Pad1.05x0.95mm_HandSolder -> Resistor_SMD:R_0603_1608Metric_Pad0.98x0.95mm_HandSolder
- R48: renamed from R3; footprint Resistor_SMD:R_0603_1608Metric_Pad1.05x0.95mm_HandSolder -> Resistor_SMD:R_0603_1608Metric_Pad0.98x0.95mm_HandSolder
- R49: renamed from R4; footprint Resistor_SMD:R_0603_1608Metric_Pad1.05x0.95mm_HandSolder -> Resistor_SMD:R_0603_1608Metric_Pad0.98x0.95mm_HandSolder
- R50: renamed from R5; footprint Resistor_SMD:R_0603_1608Metric_Pad1.05x0.95mm_HandSolder -> Resistor_SMD:R_0603_1608Metric_Pad0.98x0.95mm_HandSolder
- R51: renamed from R6; footprint Resistor_SMD:R_0603_1608Metric_Pad1.05x0.95mm_HandSolder -> Resistor_SMD:R_0603_1608Metric_Pad0.98x0.95mm_HandSolder
- R52: renamed from R7; footprint Resistor_SMD:R_0603_1608Metric_Pad1.05x0.95mm_HandSolder -> Resistor_SMD:R_0603_1608Metric_Pad0.98x0.95mm_HandSolder
- Y1: footprint (none) -> Crystal:Crystal_SMD_HC49-SD
- renumbered J7 to J11, J8 to J12, Q1 to Q7, U1 to U11
Connections:
- net SD_CARD_DET: now reaches U11.20 (PB2)
- no-connect marks 5 -> 4
Other:
- moved on the sheet: C37, R49

Commit message: Add files via upload
Connections:
- net BZ_EN: now also U11.38 (PA15); no longer U11.18 (PB0)
- net CHARGE_PUMP_CLK: now also U11.11 (PA1); no longer U11.29 (PA8)
- net KYBD0: now also U11.25 (PB12); no longer U11.33 (PA12)
- net KYBD1: now also U11.29 (PA8); no longer U11.32 (PA11)
- net KYBD2: now also U11.30 (PA9); no longer U11.17 (PA7)
- net KYBD3: now also U11.31 (PA10); no longer U11.38 (PA15)
- net KYBD4: now also U11.32 (PA11); no longer U11.22 (PB11)
- net KYBD5: now also U11.33 (PA12); no longer U11.21 (PB10)
- net KYBD6: now also U11.10 (PA0); no longer U11.46 (PB9)
- net KYBD7: now also U11.46 (PB9); no longer U11.40 (PB4)
- net KYBD8: now also U11.41 (PB5); no longer U11.39 (PB3)
- net KYBD9: now also U11.40 (PB4); no longer U11.19 (PB1)
- net SD_CARD_DET: now also U11.14 (PA4); no longer U11.20 (PB2)
- net SD_SPI_MISO: now also U11.16 (PA6); no longer U11.27 (PB14)
- net SD_SPI_MOSI: now also U11.17 (PA7); no longer U11.28 (PB15)
- net SD_SPI_SCK: now also U11.15 (PA5); no longer U11.26 (PB13)
- net TEMP_SPI_MISO: now also U11.27 (PB14); no longer U11.16 (PA6)
- net TEMP_SPI_SCK: now also U11.26 (PB13); no longer U11.15 (PA5)
- net ~DPY_RST: now also U11.39 (PB3); no longer U11.41 (PB5)
- net ~SD_SPI_CS: now also U11.18 (PB0); no longer U11.25 (PB12)
- net ~TEMP_CS0: now also U11.21 (PB10); no longer U11.10 (PA0)
- net ~TEMP_CS1: now also U11.22 (PB11); no longer U11.11 (PA1)
- net ~TEMP_CS2: now also U11.19 (PB1); no longer U11.12 (PA2)
- net ~TEMP_CS3: now also U11.20 (PB2); no longer U11.13 (PA3)
- net ~TEMP_CS4: now also U11.28 (PB15); no longer U11.14 (PA4)
- net UART1_RX renamed UART2_RX
- net UART2_RX: now also U11.13 (PA3); no longer U11.31 (PA10)
- net UART1_TX renamed UART2_TX
- net UART2_TX: now also U11.12 (PA2); no longer U11.30 (PA9)
Other:
- moved on the sheet: J12
