File: furnace/furnace_controller/Keyboard_connector.sch (KiCad schematic (older format))
At the start: 1 part

Commit message: Add files via upload
Parts:
- added R? (x10): 180, Resistor_SMD:R_0603_1608Metric_Pad0.98x0.95mm_HandSolder, symbol Device:R
- added R? (x10): 56k, Resistor_SMD:R_0603_1608Metric_Pad0.98x0.95mm_HandSolder, symbol Device:R
Connections:
- net at J?.1 (Pin_1): now also R?.1
- net at J?.10 (Pin_10): now also R?.1
- net at J?.2 (Pin_2): now also R?.1
- net at J?.3 (Pin_3): now also R?.1
- net at J?.4 (Pin_4): now also R?.1
- net at J?.5 (Pin_5): now also R?.1
- net at J?.6 (Pin_6): now also R?.1
- net at J?.7 (Pin_7): now also R?.1
- net at J?.8 (Pin_8): now also R?.1
- net at J?.9 (Pin_9): now also R?.1
- new net +3V3: R?.1, R?.1, R?.1, R?.1, R?.1, R?.1, R?.1, R?.1, R?.1, R?.1
- new net KYBD1: R?.2, R?.2
- new net KYBD10: R?.2, R?.2
- new net KYBD2: R?.2, R?.2
- new net KYBD3: R?.2, R?.2
- new net KYBD4: R?.2, R?.2
- new net KYBD5: R?.2, R?.2
- new net KYBD6: R?.2, R?.2
- new net KYBD7: R?.2, R?.2
- new net KYBD8: R?.2, R?.2
- new net KYBD9: R?.2, R?.2
Other:
- note added: "Connector for matrix keyboard"
- moved on the sheet: J?

Commit message: Add files via upload
Connections:
- net KYBD10 is gone; now on net KYBD9: R?.2, R?.2
- net KYBD1: now also R?.2, R?.2; no longer R?.2, R?.2
- net KYBD2: now also R?.2, R?.2; no longer R?.2, R?.2
- net KYBD3: now also R?.2, R?.2; no longer R?.2, R?.2
- net KYBD4: now also R?.2, R?.2; no longer R?.2, R?.2
- net KYBD5: now also R?.2, R?.2; no longer R?.2, R?.2
- net KYBD6: now also R?.2, R?.2; no longer R?.2, R?.2
- net KYBD7: now also R?.2, R?.2; no longer R?.2, R?.2
- net KYBD8: now also R?.2, R?.2; no longer R?.2, R?.2
- net KYBD9: no longer R?.2, R?.2
- new net KYBD0: R?.2, R?.2
Changed lines of the file:
@@
 	3000 3000 3100 3100
 Text Label 3400 2800 0    50   ~ 0
+KYBD0
+Text Label 3400 3100 0    50   ~ 0
 KYBD1
-Text Label 3400 3100 0    50   ~ 0
+Text Label 3400 3400 0    50   ~ 0
 KYBD2
-Text Label 3400 3400 0    50   ~ 0
+Text Label 3400 3700 0    50   ~ 0
 KYBD3
-Text Label 3400 3700 0    50   ~ 0
+Text Label 3400 4000 0    50   ~ 0
 KYBD4
-Text Label 3400 4000 0    50   ~ 0
+Text Label 3400 4300 0    50   ~ 0
 KYBD5
-Text Label 3400 4300 0    50   ~ 0
+Text Label 3400 4600 0    50   ~ 0
 KYBD6
-Text Label 3400 4600 0    50   ~ 0
+Text Label 3400 4900 0    50   ~ 0
 KYBD7
-Text Label 3400 4900 0    50   ~ 0
-KYBD8
 Text Label 3400 5500 0    50   ~ 0
-KYBD10
+KYBD9
 Text Label 2600 2300 0    50   ~ 0
-KYBD[1..10]
+KYBD[0..9]
 Text Notes 8000 1350 2    197  ~ 0
 Connector for matrix keyboard
 Text Label 3400 5200 0    50   ~ 0
-KYBD9
+KYBD8
 Text HLabel 2500 2300 0    50   BiDi ~ 0
 KYBD

Commit message: Add files via upload
Parts:
- gave numbers to parts that had none: 21
Changed lines of the file:
@@
 $EndDescr
 $Comp
-L Connector:Conn_01x10_Male J?
+L Connector:Conn_01x10_Male J10
 U 1 1 60A3891A
 P 9700 3200
-F 0 "J?" H 9808 3781 50  0000 C CNN
+F 0 "J10" H 9808 3781 50  0000 C CNN
 F 1 "Conn_01x10_Male" H 9808 3690 50  0000 C CNN
 F 2 "" H 9700 3200 50  0001 C CNN
@@
 P 7850 2800
 AR Path="/60A74215" Ref="R?"  Part="1"
-AR Path="/60A36559/60A74215" Ref="R?"  Part="1"
-F 0 "R?" V 7750 2750 50  0000 L CNN
+AR Path="/60A36559/60A74215" Ref="R35"  Part="1"
+F 0 "R35" V 7750 2750 50  0000 L CNN
 F 1 "180" V 7950 2700 50  0000 L CNN
 F 2 "Resistor_SMD:R_0603_1608Metric_Pad0.98x0.95mm_HandSolder" V 7780 2800 50  0001 C CNN
@@
 P 7850 3100
 AR Path="/60A74E97" Ref="R?"  Part="1"
-AR Path="/60A36559/60A74E97" Ref="R?"  Part="1"
-F 0 "R?" V 7750 3050 50  0000 L CNN
+AR Path="/60A36559/60A74E97" Ref="R36"  Part="1"
+F 0 "R36" V 7750 3050 50  0000 L CNN
 F 1 "180" V 7950 3000 50  0000 L CNN
 F 2 "Resistor_SMD:R_0603_1608Metric_Pad0.98x0.95mm_HandSolder" V 7780 3100 50  0001 C CNN
@@
 P 7850 3400
 AR Path="/60A74F36" Ref="R?"  Part="1"
-AR Path="/60A36559/60A74F36" Ref="R?"  Part="1"
-F 0 "R?" V 7750 3350 50  0000 L CNN
+AR Path="/60A36559/60A74F36" Ref="R37"  Part="1"
+F 0 "R37" V 7750 3350 50  0000 L CNN
 F 1 "180" V 7950 3300 50  0000 L CNN
 F 2 "Resistor_SMD:R_0603_1608Metric_Pad0.98x0.95mm_HandSolder" V 7780 3400 50  0001 C CNN
@@
 P 7850 3700
 AR Path="/60A7500F" Ref="R?"  Part="1"
-AR Path="/60A36559/60A7500F" Ref="R?"  Part="1"
-F 0 "R?" V 7750 3650 50  0000 L CNN
+AR Path="/60A36559/60A7500F" Ref="R38"  Part="1"
+F 0 "R38" V 7750 3650 50  0000 L CNN
 F 1 "180" V 7950 3600 50  0000 L CNN
 F 2 "Resistor_SMD:R_0603_1608Metric_Pad0.98x0.95mm_HandSolder" V 7780 3700 50  0001 C CNN
@@
 P 7850 4000
 AR Path="/60A76129" Ref="R?"  Part="1"
-AR Path="/60A36559/60A76129" Ref="R?"  Part="1"
-F 0 "R?" V 7750 3950 50  0000 L CNN
+AR Path="/60A36559/60A76129" Ref="R39"  Part="1"
+F 0 "R39" V 7750 3950 50  0000 L CNN
 F 1 "180" V 7950 3900 50  0000 L CNN
 F 2 "Resistor_SMD:R_0603_1608Metric_Pad0.98x0.95mm_HandSolder" V 7780 4000 50  0001 C CNN
@@
 P 7850 4300
 AR Path="/60A7612F" Ref="R?"  Part="1"
-AR Path="/60A36559/60A7612F" Ref="R?"  Part="1"
-F 0 "R?" V 7750 4250 50  0000 L CNN
+AR Path="/60A36559/60A7612F" Ref="R40"  Part="1"
+F 0 "R40" V 7750 4250 50  0000 L CNN
 F 1 "180" V 7950 4200 50  0000 L CNN
 F 2 "Resistor_SMD:R_0603_1608Metric_Pad0.98x0.95mm_HandSolder" V 7780 4300 50  0001 C CNN
@@
 P 7850 4600
 AR Path="/60A76135" Ref="R?"  Part="1"
-AR Path="/60A36559/60A76135" Ref="R?"  Part="1"
-F 0 "R?" V 7750 4550 50  0000 L CNN
+AR Path="/60A36559/60A76135" Ref="R41"  Part="1"
+F 0 "R41" V 7750 4550 50  0000 L CNN
 F 1 "180" V 7950 4500 50  0000 L CNN
 F 2 "Resistor_SMD:R_0603_1608Metric_Pad0.98x0.95mm_HandSolder" V 7780 4600 50  0001 C CNN
@@
 P 7850 4900
 AR Path="/60A7613B" Ref="R?"  Part="1"
-AR Path="/60A36559/60A7613B" Ref="R?"  Part="1"
-F 0 "R?" V 7750 4850 50  0000 L CNN
+AR Path="/60A36559/60A7613B" Ref="R42"  Part="1"
+F 0 "R42" V 7750 4850 50  0000 L CNN
 F 1 "180" V 7950 4800 50  0000 L CNN
 F 2 "Resistor_SMD:R_0603_1608Metric_Pad0.98x0.95mm_HandSolder" V 7780 4900 50  0001 C CNN
@@
 P 7850 5200
 AR Path="/60A767B9" Ref="R?"  Part="1"
-AR Path="/60A36559/60A767B9" Ref="R?"  Part="1"
-F 0 "R?" V 7750 5150 50  0000 L CNN
+AR Path="/60A36559/60A767B9" Ref="R43"  Part="1"
+F 0 "R43" V 7750 5150 50  0000 L CNN
 F 1 "180" V 7950 5100 50  0000 L CNN
 F 2 "Resistor_SMD:R_0603_1608Metric_Pad0.98x0.95mm_HandSolder" V 7780 5200 50  0001 C CNN
@@
 P 7850 5500
 AR Path="/60A767BF" Ref="R?"  Part="1"
-AR Path="/60A36559/60A767BF" Ref="R?"  Part="1"
-F 0 "R?" V 7750 5450 50  0000 L CNN
+AR Path="/60A36559/60A767BF" Ref="R44"  Part="1"
+F 0 "R44" V 7750 5450 50  0000 L CNN
 F 1 "180" V 7950 5400 50  0000 L CNN
 F 2 "Resistor_SMD:R_0603_1608Metric_Pad0.98x0.95mm_HandSolder" V 7780 5500 50  0001 C CNN
@@
 Text Label 3400 5500 0    50   ~ 0
 KYBD9
-Text Label 2600 2300 0    50   ~ 0
-KYBD[0..9]
 Text Notes 8000 1350 2    197  ~ 0
 Connector for matrix keyboard
@@
 KYBD8
 Text HLabel 2500 2300 0    50   BiDi ~ 0
-KYBD
+KYBD[0..9]
 $Comp
 L Device:R R?
@@
 P 6800 2500
 AR Path="/60AA213C" Ref="R?"  Part="1"
-AR Path="/60A36559/60AA213C" Ref="R?"  Part="1"
-F 0 "R?" H 6870 2546 50  0000 L CNN
+AR Path="/60A36559/60AA213C" Ref="R34"  Part="1"
+F 0 "R34" H 6870 2546 50  0000 L CNN
 F 1 "56k" H 6870 2455 50  0000 L CNN
 F 2 "Resistor_SMD:R_0603_1608Metric_Pad0.98x0.95mm_HandSolder" V 6730 2500 50  0001 C CNN
@@
 P 6500 2500
 AR Path="/60AA35DF" Ref="R?"  Part="1"
-AR Path="/60A36559/60AA35DF" Ref="R?"  Part="1"
-F 0 "R?" H 6570 2546 50  0000 L CNN
+AR Path="/60A36559/60AA35DF" Ref="R33"  Part="1"
+F 0 "R33" H 6570 2546 50  0000 L CNN
 F 1 "56k" H 6570 2455 50  0000 L CNN
 F 2 "Resistor_SMD:R_0603_1608Metric_Pad0.98x0.95mm_HandSolder" V 6430 2500 50  0001 C CNN
@@
 P 6200 2500
 AR Path="/60AA3F6A" Ref="R?"  Part="1"
-AR Path="/60A36559/60AA3F6A" Ref="R?"  Part="1"
-F 0 "R?" H 6270 2546 50  0000 L CNN
+AR Path="/60A36559/60AA3F6A" Ref="R32"  Part="1"
+F 0 "R32" H 6270 2546 50  0000 L CNN
 F 1 "56k" H 6270 2455 50  0000 L CNN
 F 2 "Resistor_SMD:R_0603_1608Metric_Pad0.98x0.95mm_HandSolder" V 6130 2500 50  0001 C CNN
@@
 P 5900 2500
 AR Path="/60AA4928" Ref="R?"  Part="1"
-AR Path="/60A36559/60AA4928" Ref="R?"  Part="1"
-F 0 "R?" H 5970 2546 50  0000 L CNN
+AR Path="/60A36559/60AA4928" Ref="R31"  Part="1"
+F 0 "R31" H 5970 2546 50  0000 L CNN
 F 1 "56k" H 5970 2455 50  0000 L CNN
 F 2 "Resistor_SMD:R_0603_1608Metric_Pad0.98x0.95mm_HandSolder" V 5830 2500 50  0001 C CNN
@@
 P 5600 2500
 AR Path="/60AA73CA" Ref="R?"  Part="1"
-AR Path="/60A36559/60AA73CA" Ref="R?"  Part="1"
-F 0 "R?" H 5670 2546 50  0000 L CNN
+AR Path="/60A36559/60AA73CA" Ref="R30"  Part="1"
+F 0 "R30" H 5670 2546 50  0000 L CNN
 F 1 "56k" H 5670 2455 50  0000 L CNN
 F 2 "Resistor_SMD:R_0603_1608Metric_Pad0.98x0.95mm_HandSolder" V 5530 2500 50  0001 C CNN
@@
 P 5300 2500
 AR Path="/60AA73D0" Ref="R?"  Part="1"
-AR Path="/60A36559/60AA73D0" Ref="R?"  Part="1"
-F 0 "R?" H 5370 2546 50  0000 L CNN
+AR Path="/60A36559/60AA73D0" Ref="R29"  Part="1"
+F 0 "R29" H 5370 2546 50  0000 L CNN
 F 1 "56k" H 5370 2455 50  0000 L CNN
 F 2 "Resistor_SMD:R_0603_1608Metric_Pad0.98x0.95mm_HandSolder" V 5230 2500 50  0001 C CNN
@@
 P 5000 2500
 AR Path="/60AA73D6" Ref="R?"  Part="1"
-AR Path="/60A36559/60AA73D6" Ref="R?"  Part="1"
-F 0 "R?" H 5070 2546 50  0000 L CNN
+AR Path="/60A36559/60AA73D6" Ref="R28"  Part="1"
+F 0 "R28" H 5070 2546 50  0000 L CNN
 F 1 "56k" H 5070 2455 50  0000 L CNN
 F 2 "Resistor_SMD:R_0603_1608Metric_Pad0.98x0.95mm_HandSolder" V 4930 2500 50  0001 C CNN
@@
 P 4700 2500
 AR Path="/60AA73DC" Ref="R?"  Part="1"
-AR Path="/60A36559/60AA73DC" Ref="R?"  Part="1"
-F 0 "R?" H 4770 2546 50  0000 L CNN
+AR Path="/60A36559/60AA73DC" Ref="R27"  Part="1"
+F 0 "R27" H 4770 2546 50  0000 L CNN
 F 1 "56k" H 4770 2455 50  0000 L CNN
 F 2 "Resistor_SMD:R_0603_1608Metric_Pad0.98x0.95mm_HandSolder" V 4630 2500 50  0001 C CNN
@@
 P 4400 2500
 AR Path="/60AA8EC2" Ref="R?"  Part="1"
-AR Path="/60A36559/60AA8EC2" Ref="R?"  Part="1"
-F 0 "R?" H 4470 2546 50  0000 L CNN
+AR Path="/60A36559/60AA8EC2" Ref="R26"  Part="1"
+F 0 "R26" H 4470 2546 50  0000 L CNN
 F 1 "56k" H 4470 2455 50  0000 L CNN
 F 2 "Resistor_SMD:R_0603_1608Metric_Pad0.98x0.95mm_HandSolder" V 4330 2500 50  0001 C CNN
@@
 P 4100 2500
 AR Path="/60AA8EC8" Ref="R?"  Part="1"
-AR Path="/60A36559/60AA8EC8" Ref="R?"  Part="1"
-F 0 "R?" H 4170 2546 50  0000 L CNN
+AR Path="/60A36559/60AA8EC8" Ref="R25"  Part="1"
+F 0 "R25" H 4170 2546 50  0000 L CNN
 F 1 "56k" H 4170 2455 50  0000 L CNN
 F 2 "Resistor_SMD:R_0603_1608Metric_Pad0.98x0.95mm_HandSolder" V 4030 2500 50  0001 C CNN
@@
 P 4100 2250
 AR Path="/609FED99/60AB0645" Ref="#PWR?"  Part="1"
-AR Path="/60A36559/60AB0645" Ref="#PWR?"  Part="1"
-F 0 "#PWR?" H 4100 2100 50  0001 C CNN
+AR Path="/60A36559/60AB0645" Ref="#PWR031"  Part="1"
+F 0 "#PWR031" H 4100 2100 50  0001 C CNN
 F 1 "+3V3" H 4115 2423 50  0000 C CNN
 F 2 "" H 4100 2250 50  0001 C CNN

Commit message: Add files via upload
Parts:
- J10: value Conn_01x10_Male -> PLS-10R; footprint (none) -> Connector_PinHeader_2.54mm:PinHeader_1x10_P2.54mm_Horizontal
- R25, R26, R27, R28, R29, R30, R31, R32, R33, R34, R35, R36, R37, R38, R39, R40, R41, R42, R43, R44: footprint Resistor_SMD:R_0603_1608Metric_Pad0.98x0.95mm_HandSolder -> Resistor_SMD:R_0603_1608Metric_Pad1.05x0.95mm_HandSolder
Changed lines of the file:
@@
 $Descr A4 11693 8268
 encoding utf-8
-Sheet 5 18
-Title ""
-Date ""
-Rev ""
-Comp ""
+Sheet 4 18
+Title "Furnace controller"
+Date "2021-08-26"
+Rev "1.0"
+Comp "Yuriy Volkov"
 Comment1 ""
 Comment2 ""
@@
 P 9700 3200
 F 0 "J10" H 9808 3781 50  0000 C CNN
-F 1 "Conn_01x10_Male" H 9808 3690 50  0000 C CNN
-F 2 "" H 9700 3200 50  0001 C CNN
+F 1 "PLS-10R" H 9808 3690 50  0000 C CNN
+F 2 "Connector_PinHeader_2.54mm:PinHeader_1x10_P2.54mm_Horizontal" H 9700 3200 50  0001 C CNN
 F 3 "~" H 9700 3200 50  0001 C CNN
 	1    9700 3200
@@
 F 0 "R35" V 7750 2750 50  0000 L CNN
 F 1 "180" V 7950 2700 50  0000 L CNN
-F 2 "Resistor_SMD:R_0603_1608Metric_Pad0.98x0.95mm_HandSolder" V 7780 2800 50  0001 C CNN
+F 2 "Resistor_SMD:R_0603_1608Metric_Pad1.05x0.95mm_HandSolder" V 7780 2800 50  0001 C CNN
 F 3 "~" H 7850 2800 50  0001 C CNN
 	1    7850 2800
@@
 F 0 "R36" V 7750 3050 50  0000 L CNN
 F 1 "180" V 7950 3000 50  0000 L CNN
-F 2 "Resistor_SMD:R_0603_1608Metric_Pad0.98x0.95mm_HandSolder" V 7780 3100 50  0001 C CNN
+F 2 "Resistor_SMD:R_0603_1608Metric_Pad1.05x0.95mm_HandSolder" V 7780 3100 50  0001 C CNN
 F 3 "~" H 7850 3100 50  0001 C CNN
 	1    7850 3100
@@
 F 0 "R37" V 7750 3350 50  0000 L CNN
 F 1 "180" V 7950 3300 50  0000 L CNN
-F 2 "Resistor_SMD:R_0603_1608Metric_Pad0.98x0.95mm_HandSolder" V 7780 3400 50  0001 C CNN
+F 2 "Resistor_SMD:R_0603_1608Metric_Pad1.05x0.95mm_HandSolder" V 7780 3400 50  0001 C CNN
 F 3 "~" H 7850 3400 50  0001 C CNN
 	1    7850 3400
@@
 F 0 "R38" V 7750 3650 50  0000 L CNN
 F 1 "180" V 7950 3600 50  0000 L CNN
-F 2 "Resistor_SMD:R_0603_1608Metric_Pad0.98x0.95mm_HandSolder" V 7780 3700 50  0001 C CNN
+F 2 "Resistor_SMD:R_0603_1608Metric_Pad1.05x0.95mm_HandSolder" V 7780 3700 50  0001 C CNN
 F 3 "~" H 7850 3700 50  0001 C CNN
 	1    7850 3700
@@
 F 0 "R39" V 7750 3950 50  0000 L CNN
 F 1 "180" V 7950 3900 50  0000 L CNN
-F 2 "Resistor_SMD:R_0603_1608Metric_Pad0.98x0.95mm_HandSolder" V 7780 4000 50  0001 C CNN
+F 2 "Resistor_SMD:R_0603_1608Metric_Pad1.05x0.95mm_HandSolder" V 7780 4000 50  0001 C CNN
 F 3 "~" H 7850 4000 50  0001 C CNN
 	1    7850 4000
@@
 F 0 "R40" V 7750 4250 50  0000 L CNN
 F 1 "180" V 7950 4200 50  0000 L CNN
-F 2 "Resistor_SMD:R_0603_1608Metric_Pad0.98x0.95mm_HandSolder" V 7780 4300 50  0001 C CNN
+F 2 "Resistor_SMD:R_0603_1608Metric_Pad1.05x0.95mm_HandSolder" V 7780 4300 50  0001 C CNN
 F 3 "~" H 7850 4300 50  0001 C CNN
 	1    7850 4300
@@
 F 0 "R41" V 7750 4550 50  0000 L CNN
 F 1 "180" V 7950 4500 50  0000 L CNN
-F 2 "Resistor_SMD:R_0603_1608Metric_Pad0.98x0.95mm_HandSolder" V 7780 4600 50  0001 C CNN
+F 2 "Resistor_SMD:R_0603_1608Metric_Pad1.05x0.95mm_HandSolder" V 7780 4600 50  0001 C CNN
 F 3 "~" H 7850 4600 50  0001 C CNN
 	1    7850 4600
@@
 F 0 "R42" V 7750 4850 50  0000 L CNN
 F 1 "180" V 7950 4800 50  0000 L CNN
-F 2 "Resistor_SMD:R_0603_1608Metric_Pad0.98x0.95mm_HandSolder" V 7780 4900 50  0001 C CNN
+F 2 "Resistor_SMD:R_0603_1608Metric_Pad1.05x0.95mm_HandSolder" V 7780 4900 50  0001 C CNN
 F 3 "~" H 7850 4900 50  0001 C CNN
 	1    7850 4900
@@
 F 0 "R43" V 7750 5150 50  0000 L CNN
 F 1 "180" V 7950 5100 50  0000 L CNN
-F 2 "Resistor_SMD:R_0603_1608Metric_Pad0.98x0.95mm_HandSolder" V 7780 5200 50  0001 C CNN
+F 2 "Resistor_SMD:R_0603_1608Metric_Pad1.05x0.95mm_HandSolder" V 7780 5200 50  0001 C CNN
 F 3 "~" H 7850 5200 50  0001 C CNN
 	1    7850 5200
@@
 F 0 "R44" V 7750 5450 50  0000 L CNN
 F 1 "180" V 7950 5400 50  0000 L CNN
-F 2 "Resistor_SMD:R_0603_1608Metric_Pad0.98x0.95mm_HandSolder" V 7780 5500 50  0001 C CNN
+F 2 "Resistor_SMD:R_0603_1608Metric_Pad1.05x0.95mm_HandSolder" V 7780 5500 50  0001 C CNN
 F 3 "~" H 7850 5500 50  0001 C CNN
 	1    7850 5500
@@
 F 0 "R34" H 6870 2546 50  0000 L CNN
 F 1 "56k" H 6870 2455 50  0000 L CNN
-F 2 "Resistor_SMD:R_0603_1608Metric_Pad0.98x0.95mm_HandSolder" V 6730 2500 50  0001 C CNN
+F 2 "Resistor_SMD:R_0603_1608Metric_Pad1.05x0.95mm_HandSolder" V 6730 2500 50  0001 C CNN
 F 3 "~" H 6800 2500 50  0001 C CNN
 	1    6800 2500
@@
 F 0 "R33" H 6570 2546 50  0000 L CNN
 F 1 "56k" H 6570 2455 50  0000 L CNN
-F 2 "Resistor_SMD:R_0603_1608Metric_Pad0.98x0.95mm_HandSolder" V 6430 2500 50  0001 C CNN
+F 2 "Resistor_SMD:R_0603_1608Metric_Pad1.05x0.95mm_HandSolder" V 6430 2500 50  0001 C CNN
 F 3 "~" H 6500 2500 50  0001 C CNN
 	1    6500 2500
@@
 F 0 "R32" H 6270 2546 50  0000 L CNN
 F 1 "56k" H 6270 2455 50  0000 L CNN
-F 2 "Resistor_SMD:R_0603_1608Metric_Pad0.98x0.95mm_HandSolder" V 6130 2500 50  0001 C CNN
+F 2 "Resistor_SMD:R_0603_1608Metric_Pad1.05x0.95mm_HandSolder" V 6130 2500 50  0001 C CNN
 F 3 "~" H 6200 2500 50  0001 C CNN
 	1    6200 2500
@@
 F 0 "R31" H 5970 2546 50  0000 L CNN
 F 1 "56k" H 5970 2455 50  0000 L CNN
-F 2 "Resistor_SMD:R_0603_1608Metric_Pad0.98x0.95mm_HandSolder" V 5830 2500 50  0001 C CNN
+F 2 "Resistor_SMD:R_0603_1608Metric_Pad1.05x0.95mm_HandSolder" V 5830 2500 50  0001 C CNN
 F 3 "~" H 5900 2500 50  0001 C CNN
 	1    5900 2500
@@
 F 0 "R30" H 5670 2546 50  0000 L CNN
 F 1 "56k" H 5670 2455 50  0000 L CNN
-F 2 "Resistor_SMD:R_0603_1608Metric_Pad0.98x0.95mm_HandSolder" V 5530 2500 50  0001 C CNN
+F 2 "Resistor_SMD:R_0603_1608Metric_Pad1.05x0.95mm_HandSolder" V 5530 2500 50  0001 C CNN
 F 3 "~" H 5600 2500 50  0001 C CNN
 	1    5600 2500
@@
 F 0 "R29" H 5370 2546 50  0000 L CNN
 F 1 "56k" H 5370 2455 50  0000 L CNN
-F 2 "Resistor_SMD:R_0603_1608Metric_Pad0.98x0.95mm_HandSolder" V 5230 2500 50  0001 C CNN
+F 2 "Resistor_SMD:R_0603_1608Metric_Pad1.05x0.95mm_HandSolder" V 5230 2500 50  0001 C CNN
 F 3 "~" H 5300 2500 50  0001 C CNN
 	1    5300 2500
@@
 F 0 "R28" H 5070 2546 50  0000 L CNN
 F 1 "56k" H 5070 2455 50  0000 L CNN
-F 2 "Resistor_SMD:R_0603_1608Metric_Pad0.98x0.95mm_HandSolder" V 4930 2500 50  0001 C CNN
+F 2 "Resistor_SMD:R_0603_1608Metric_Pad1.05x0.95mm_HandSolder" V 4930 2500 50  0001 C CNN
 F 3 "~" H 5000 2500 50  0001 C CNN
 	1    5000 2500
@@
 F 0 "R27" H 4770 2546 50  0000 L CNN
 F 1 "56k" H 4770 2455 50  0000 L CNN
-F 2 "Resistor_SMD:R_0603_1608Metric_Pad0.98x0.95mm_HandSolder" V 4630 2500 50  0001 C CNN
+F 2 "Resistor_SMD:R_0603_1608Metric_Pad1.05x0.95mm_HandSolder" V 4630 2500 50  0001 C CNN
 F 3 "~" H 4700 2500 50  0001 C CNN
 	1    4700 2500
@@
 F 0 "R26" H 4470 2546 50  0000 L CNN
 F 1 "56k" H 4470 2455 50  0000 L CNN
-F 2 "Resistor_SMD:R_0603_1608Metric_Pad0.98x0.95mm_HandSolder" V 4330 2500 50  0001 C CNN
+F 2 "Resistor_SMD:R_0603_1608Metric_Pad1.05x0.95mm_HandSolder" V 4330 2500 50  0001 C CNN
 F 3 "~" H 4400 2500 50  0001 C CNN
 	1    4400 2500
@@
 F 0 "R25" H 4170 2546 50  0000 L CNN
 F 1 "56k" H 4170 2455 50  0000 L CNN
-F 2 "Resistor_SMD:R_0603_1608Metric_Pad0.98x0.95mm_HandSolder" V 4030 2500 50  0001 C CNN
+F 2 "Resistor_SMD:R_0603_1608Metric_Pad1.05x0.95mm_HandSolder" V 4030 2500 50  0001 C CNN
 F 3 "~" H 4100 2500 50  0001 C CNN
 	1    4100 2500
