File: furnace/furnace_controller/Micro_SD_card.sch (KiCad schematic (older format))
At the start: 7 parts

Commit message: Add files via upload
Connections:
- net SCL renamed SCK
Changed lines of the file:
@@
 MOSI
 Text HLabel 4100 4700 0    50   Input ~ 0
-SCL
+SCK
 Text HLabel 4100 4900 0    50   Output ~ 0
 MISO

Commit message: Add files via upload
Parts:
- gave numbers to parts that had none: 7
Changed lines of the file:
@@
 AR Path="/60B1D1CB" Ref="J?"  Part="1"
 AR Path="/609C9D41/60B1D1CB" Ref="J?"  Part="1"
-AR Path="/60B1951B/60B1D1CB" Ref="J?"  Part="1"
-F 0 "J?" H 7150 5317 50  0000 C CNN
+AR Path="/60B1951B/60B1D1CB" Ref="J13"  Part="1"
+F 0 "J13" H 7150 5317 50  0000 C CNN
 F 1 "Micro_SD_Card" H 7150 5226 50  0000 C CNN
 F 2 "" H 8350 4900 50  0001 C CNN
@@
 AR Path="/60B1D1D1" Ref="R?"  Part="1"
 AR Path="/609C9D41/60B1D1D1" Ref="R?"  Part="1"
-AR Path="/60B1951B/60B1D1D1" Ref="R?"  Part="1"
-F 0 "R?" H 5070 3946 50  0000 L CNN
+AR Path="/60B1951B/60B1D1D1" Ref="R51"  Part="1"
+F 0 "R51" H 5070 3946 50  0000 L CNN
 F 1 "10k" H 5070 3855 50  0000 L CNN
 F 2 "Resistor_SMD:R_0603_1608Metric_Pad0.98x0.95mm_HandSolder" V 4930 3900 50  0001 C CNN
@@
 AR Path="/60B1D1D7" Ref="#PWR?"  Part="1"
 AR Path="/609C9D41/60B1D1D7" Ref="#PWR?"  Part="1"
-AR Path="/60B1951B/60B1D1D7" Ref="#PWR?"  Part="1"
-F 0 "#PWR?" H 8000 5050 50  0001 C CNN
+AR Path="/60B1951B/60B1D1D7" Ref="#PWR056"  Part="1"
+F 0 "#PWR056" H 8000 5050 50  0001 C CNN
 F 1 "GND" H 8005 5127 50  0000 C CNN
 F 2 "" H 8000 5300 50  0001 C CNN
@@
 AR Path="/60B1D1DD" Ref="C?"  Part="1"
 AR Path="/609C9D41/60B1D1DD" Ref="C?"  Part="1"
-AR Path="/60B1951B/60B1D1DD" Ref="C?"  Part="1"
-F 0 "C?" H 5915 3696 50  0000 L CNN
+AR Path="/60B1951B/60B1D1DD" Ref="C44"  Part="1"
+F 0 "C44" H 5915 3696 50  0000 L CNN
 F 1 "0,1" H 5915 3605 50  0000 L CNN
 F 2 "Capacitor_SMD:C_0603_1608Metric_Pad1.08x0.95mm_HandSolder" H 5838 3500 50  0001 C CNN
@@
 AR Path="/60B1D1E3" Ref="#PWR?"  Part="1"
 AR Path="/609C9D41/60B1D1E3" Ref="#PWR?"  Part="1"
-AR Path="/60B1951B/60B1D1E3" Ref="#PWR?"  Part="1"
-F 0 "#PWR?" H 5500 5000 50  0001 C CNN
+AR Path="/60B1951B/60B1D1E3" Ref="#PWR054"  Part="1"
+F 0 "#PWR054" H 5500 5000 50  0001 C CNN
 F 1 "GND" H 5505 5077 50  0000 C CNN
 F 2 "" H 5500 5250 50  0001 C CNN
@@
 AR Path="/609FED99/60B1D1E9" Ref="#PWR?"  Part="1"
 AR Path="/609C9D41/60B1D1E9" Ref="#PWR?"  Part="1"
-AR Path="/60B1951B/60B1D1E9" Ref="#PWR?"  Part="1"
-F 0 "#PWR?" H 5500 3100 50  0001 C CNN
+AR Path="/60B1951B/60B1D1E9" Ref="#PWR053"  Part="1"
+F 0 "#PWR053" H 5500 3100 50  0001 C CNN
 F 1 "+3V3" H 5515 3423 50  0000 C CNN
 F 2 "" H 5500 3250 50  0001 C CNN
@@
 AR Path="/60B1D1EF" Ref="#PWR?"  Part="1"
 AR Path="/609C9D41/60B1D1EF" Ref="#PWR?"  Part="1"
-AR Path="/60B1951B/60B1D1EF" Ref="#PWR?"  Part="1"
-F 0 "#PWR?" H 5800 3700 50  0001 C CNN
+AR Path="/60B1951B/60B1D1EF" Ref="#PWR055"  Part="1"
+F 0 "#PWR055" H 5800 3700 50  0001 C CNN
 F 1 "GND" H 5805 3777 50  0000 C CNN
 F 2 "" H 5800 3950 50  0001 C CNN
@@
 AR Path="/60B1D208" Ref="R?"  Part="1"
 AR Path="/609C9D41/60B1D208" Ref="R?"  Part="1"
-AR Path="/60B1951B/60B1D208" Ref="R?"  Part="1"
-F 0 "R?" H 4770 3946 50  0000 L CNN
+AR Path="/60B1951B/60B1D208" Ref="R50"  Part="1"
+F 0 "R50" H 4770 3946 50  0000 L CNN
 F 1 "10k" H 4770 3855 50  0000 L CNN
 F 2 "Resistor_SMD:R_0603_1608Metric_Pad0.98x0.95mm_HandSolder" V 4630 3900 50  0001 C CNN
@@
 AR Path="/60B1D20E" Ref="R?"  Part="1"
 AR Path="/609C9D41/60B1D20E" Ref="R?"  Part="1"
-AR Path="/60B1951B/60B1D20E" Ref="R?"  Part="1"
-F 0 "R?" H 4470 3946 50  0000 L CNN
+AR Path="/60B1951B/60B1D20E" Ref="R49"  Part="1"
+F 0 "R49" H 4470 3946 50  0000 L CNN
 F 1 "10k" H 4470 3855 50  0000 L CNN
 F 2 "Resistor_SMD:R_0603_1608Metric_Pad0.98x0.95mm_HandSolder" V 4330 3900 50  0001 C CNN
@@
 AR Path="/609FED99/60B1D21E" Ref="C?"  Part="1"
 AR Path="/609C9D41/60B1D21E" Ref="C?"  Part="1"
-AR Path="/60B1951B/60B1D21E" Ref="C?"  Part="1"
-F 0 "C?" H 6315 3696 50  0000 L CNN
+AR Path="/60B1951B/60B1D21E" Ref="C45"  Part="1"
+F 0 "C45" H 6315 3696 50  0000 L CNN
 F 1 "10u" H 6315 3605 50  0000 L CNN
 F 2 "Capacitor_SMD:C_1206_3216Metric_Pad1.33x1.80mm_HandSolder" H 6238 3500 50  0001 C CNN
@@
 MISO
 $Comp
-L Connector:Conn_01x05_Male J?
+L Connector:Conn_01x05_Male J12
 U 1 1 60B35003
 P 5200 5700
-F 0 "J?" H 5172 5724 50  0000 R CNN
+F 0 "J12" H 5172 5724 50  0000 R CNN
 F 1 "Conn_01x05_Male" H 5172 5633 50  0000 R CNN
 F 2 "" H 5200 5700 50  0001 C CNN
@@
 AR Path="/60B38C7E" Ref="#PWR?"  Part="1"
 AR Path="/609C9D41/60B38C7E" Ref="#PWR?"  Part="1"
-AR Path="/60B1951B/60B38C7E" Ref="#PWR?"  Part="1"
-F 0 "#PWR?" H 4900 5650 50  0001 C CNN
+AR Path="/60B1951B/60B38C7E" Ref="#PWR052"  Part="1"
+F 0 "#PWR052" H 4900 5650 50  0001 C CNN
 F 1 "GND" H 4905 5727 50  0000 C CNN
 F 2 "" H 4900 5900 50  0001 C CNN

Commit message: Add files via upload
Parts:
- C44: footprint Capacitor_SMD:C_0603_1608Metric_Pad1.08x0.95mm_HandSolder -> Capacitor_SMD:C_0603_1608Metric_Pad1.05x0.95mm_HandSolder
- C45: footprint Capacitor_SMD:C_1206_3216Metric_Pad1.33x1.80mm_HandSolder -> Capacitor_SMD:C_1206_3216Metric_Pad1.42x1.75mm_HandSolder
- J12: value Conn_01x05_Male -> PLS-5; footprint (none) -> Connector_PinHeader_2.54mm:PinHeader_1x05_P2.54mm_Vertical
- R49, R50, R51: footprint Resistor_SMD:R_0603_1608Metric_Pad0.98x0.95mm_HandSolder -> Resistor_SMD:R_0603_1608Metric_Pad1.05x0.95mm_HandSolder
Changed lines of the file:
@@
 $Descr A4 11693 8268
 encoding utf-8
-Sheet 16 18
-Title ""
-Date ""
-Rev ""
-Comp ""
+Sheet 15 18
+Title "Furnace controller"
+Date "2021-08-26"
+Rev "1.0"
+Comp "Yuriy Volkov"
 Comment1 ""
 Comment2 ""
@@
 F 0 "R51" H 5070 3946 50  0000 L CNN
 F 1 "10k" H 5070 3855 50  0000 L CNN
-F 2 "Resistor_SMD:R_0603_1608Metric_Pad0.98x0.95mm_HandSolder" V 4930 3900 50  0001 C CNN
+F 2 "Resistor_SMD:R_0603_1608Metric_Pad1.05x0.95mm_HandSolder" V 4930 3900 50  0001 C CNN
 F 3 "~" H 5000 3900 50  0001 C CNN
 	1    5000 3900
@@
 F 0 "C44" H 5915 3696 50  0000 L CNN
 F 1 "0,1" H 5915 3605 50  0000 L CNN
-F 2 "Capacitor_SMD:C_0603_1608Metric_Pad1.08x0.95mm_HandSolder" H 5838 3500 50  0001 C CNN
+F 2 "Capacitor_SMD:C_0603_1608Metric_Pad1.05x0.95mm_HandSolder" H 5838 3500 50  0001 C CNN
 F 3 "~" H 5800 3650 50  0001 C CNN
 	1    5800 3650
@@
 F 0 "R50" H 4770 3946 50  0000 L CNN
 F 1 "10k" H 4770 3855 50  0000 L CNN
-F 2 "Resistor_SMD:R_0603_1608Metric_Pad0.98x0.95mm_HandSolder" V 4630 3900 50  0001 C CNN
+F 2 "Resistor_SMD:R_0603_1608Metric_Pad1.05x0.95mm_HandSolder" V 4630 3900 50  0001 C CNN
 F 3 "~" H 4700 3900 50  0001 C CNN
 	1    4700 3900
@@
 F 0 "R49" H 4470 3946 50  0000 L CNN
 F 1 "10k" H 4470 3855 50  0000 L CNN
-F 2 "Resistor_SMD:R_0603_1608Metric_Pad0.98x0.95mm_HandSolder" V 4330 3900 50  0001 C CNN
+F 2 "Resistor_SMD:R_0603_1608Metric_Pad1.05x0.95mm_HandSolder" V 4330 3900 50  0001 C CNN
 F 3 "~" H 4400 3900 50  0001 C CNN
 	1    4400 3900
@@
 F 0 "C45" H 6315 3696 50  0000 L CNN
 F 1 "10u" H 6315 3605 50  0000 L CNN
-F 2 "Capacitor_SMD:C_1206_3216Metric_Pad1.33x1.80mm_HandSolder" H 6238 3500 50  0001 C CNN
+F 2 "Capacitor_SMD:C_1206_3216Metric_Pad1.42x1.75mm_HandSolder" H 6238 3500 50  0001 C CNN
 F 3 "~" H 6200 3650 50  0001 C CNN
 	1    6200 3650
@@
 P 5200 5700
 F 0 "J12" H 5172 5724 50  0000 R CNN
-F 1 "Conn_01x05_Male" H 5172 5633 50  0000 R CNN
-F 2 "" H 5200 5700 50  0001 C CNN
+F 1 "PLS-5" H 5172 5633 50  0000 R CNN
+F 2 "Connector_PinHeader_2.54mm:PinHeader_1x05_P2.54mm_Vertical" H 5200 5700 50  0001 C CNN
 F 3 "~" H 5200 5700 50  0001 C CNN
 	1    5200 5700

Commit message: Add files via upload
Parts:
- J13: value Micro_SD_Card -> CTF-11081-P
Changed lines of the file:
@@
 AR Path="/60B1951B/60B1D1CB" Ref="J13"  Part="1"
 F 0 "J13" H 7150 5317 50  0000 C CNN
-F 1 "Micro_SD_Card" H 7150 5226 50  0000 C CNN
+F 1 "CTF-11081-P" H 7150 5226 50  0000 C CNN
 F 2 "" H 8350 4900 50  0001 C CNN
 F 3 "http://katalog.we-online.de/em/datasheet/693072010801.pdf" H 7200 4600 50  0001 C CNN
