File: furnace/furnace_controller/OLED_display_connector.sch (KiCad schematic (older format))
At the start: 14 parts, among them J9 FPC-24P 0.5mm, Q5 BC847, Q6 IRLML6402

Commit message: Add files via upload
Parts:
- C10: renamed from C20; footprint Capacitor_SMD:C_0603_1608Metric_Pad1.05x0.95mm_HandSolder -> Capacitor_SMD:C_0603_1608Metric_Pad1.08x0.95mm_HandSolder
- C11: renamed from C21; footprint Capacitor_SMD:C_1206_3216Metric_Pad1.42x1.75mm_HandSolder -> Capacitor_SMD:C_1206_3216Metric_Pad1.33x1.80mm_HandSolder
- C12: renamed from C22; footprint Capacitor_SMD:C_1206_3216Metric_Pad1.42x1.75mm_HandSolder -> Capacitor_SMD:C_1206_3216Metric_Pad1.33x1.80mm_HandSolder
- J7: renamed from J9; footprint Connector_FFC-FPC:Hirose_FH12-24S-0.5SH_1x24-1MP_P0.50mm_Horizontal -> furnace_controller:Hirose_FH12-24S-0.5SH_1x24-1MP_P0.50mm_Horizontal
- R10: renamed from R17; footprint Resistor_SMD:R_0603_1608Metric_Pad1.05x0.95mm_HandSolder -> Resistor_SMD:R_0603_1608Metric_Pad0.98x0.95mm_HandSolder
- R11: renamed from R18; footprint Resistor_SMD:R_0603_1608Metric_Pad1.05x0.95mm_HandSolder -> Resistor_SMD:R_0603_1608Metric_Pad0.98x0.95mm_HandSolder
- R12: renamed from R19; footprint Resistor_SMD:R_0603_1608Metric_Pad1.05x0.95mm_HandSolder -> Resistor_SMD:R_0603_1608Metric_Pad0.98x0.95mm_HandSolder
- R13: renamed from R20; footprint Resistor_SMD:R_0603_1608Metric_Pad1.05x0.95mm_HandSolder -> Resistor_SMD:R_0603_1608Metric_Pad0.98x0.95mm_HandSolder
- R14: renamed from R21; footprint Resistor_SMD:R_0603_1608Metric_Pad1.05x0.95mm_HandSolder -> Resistor_SMD:R_0603_1608Metric_Pad0.98x0.95mm_HandSolder
- R15: renamed from R22; footprint Resistor_SMD:R_0603_1608Metric_Pad1.05x0.95mm_HandSolder -> Resistor_SMD:R_0603_1608Metric_Pad0.98x0.95mm_HandSolder
- R16: renamed from R23; footprint Resistor_SMD:R_0603_1608Metric_Pad1.05x0.95mm_HandSolder -> Resistor_SMD:R_0603_1608Metric_Pad0.98x0.95mm_HandSolder
- R17: renamed from R24; footprint Resistor_SMD:R_0603_1608Metric_Pad1.05x0.95mm_HandSolder -> Resistor_SMD:R_0603_1608Metric_Pad0.98x0.95mm_HandSolder
- renumbered Q5 to Q4, Q6 to Q5
Changed lines of the file:
@@
 Sheet 3 18
 Title "Furnace controller"
-Date "2021-08-26"
+Date "2021-09-24"
 Rev "1.0"
 Comp "Yuriy Volkov"
@@
 P 6950 3350
 AR Path="/609CA1D9/60A3B1D4" Ref="J?"  Part="1"
-AR Path="/60A364EE/60A3B1D4" Ref="J9"  Part="1"
-F 0 "J9" H 6900 4700 50  0000 L CNN
+AR Path="/60A364EE/60A3B1D4" Ref="J7"  Part="1"
+F 0 "J7" H 6900 4700 50  0000 L CNN
 F 1 "FPC-24P 0.5mm" H 6700 4600 50  0000 L CNN
-F 2 "Connector_FFC-FPC:Hirose_FH12-24S-0.5SH_1x24-1MP_P0.50mm_Horizontal" H 6950 3350 50  0001 C CNN
+F 2 "furnace_controller:Hirose_FH12-24S-0.5SH_1x24-1MP_P0.50mm_Horizontal" H 6950 3350 50  0001 C CNN
 F 3 "~" H 6950 3350 50  0001 C CNN
 	1    6950 3350
@@
 P 4000 2650
 AR Path="/609FED99/60A48DCF" Ref="#PWR?"  Part="1"
-AR Path="/60A364EE/60A48DCF" Ref="#PWR022"  Part="1"
-F 0 "#PWR022" H 4000 2500 50  0001 C CNN
+AR Path="/60A364EE/60A48DCF" Ref="#PWR07"  Part="1"
+F 0 "#PWR07" H 4000 2500 50  0001 C CNN
 F 1 "+3V3" H 4015 2823 50  0000 C CNN
 F 2 "" H 4000 2650 50  0001 C CNN
@@
 P 4300 4450
 AR Path="/609FED99/60A48DD5" Ref="#PWR?"  Part="1"
-AR Path="/60A364EE/60A48DD5" Ref="#PWR023"  Part="1"
-F 0 "#PWR023" H 4300 4300 50  0001 C CNN
+AR Path="/60A364EE/60A48DD5" Ref="#PWR08"  Part="1"
+F 0 "#PWR08" H 4300 4300 50  0001 C CNN
 F 1 "+10V" H 4315 4623 50  0000 C CNN
 F 2 "" H 4300 4450 50  0001 C CNN
@@
 P 6000 2400
 AR Path="/609FED99/60A4B340" Ref="#PWR?"  Part="1"
-AR Path="/60A364EE/60A4B340" Ref="#PWR028"  Part="1"
-F 0 "#PWR028" H 6000 2150 50  0001 C CNN
+AR Path="/60A364EE/60A4B340" Ref="#PWR013"  Part="1"
+F 0 "#PWR013" H 6000 2150 50  0001 C CNN
 F 1 "GND" H 6005 2227 50  0000 C CNN
 F 2 "" H 6000 2400 50  0001 C CNN
@@
 AR Path="/609CA6A8/60AE5653/60A4DD3E" Ref="C?"  Part="1"
 AR Path="/609FED99/60A4DD3E" Ref="C?"  Part="1"
-AR Path="/60A364EE/60A4DD3E" Ref="C20"  Part="1"
-F 0 "C20" H 5615 2846 50  0000 L CNN
+AR Path="/60A364EE/60A4DD3E" Ref="C10"  Part="1"
+F 0 "C10" H 5615 2846 50  0000 L CNN
 F 1 "1u" H 5615 2755 50  0000 L CNN
-F 2 "Capacitor_SMD:C_0603_1608Metric_Pad1.05x0.95mm_HandSolder" H 5538 2650 50  0001 C CNN
+F 2 "Capacitor_SMD:C_0603_1608Metric_Pad1.08x0.95mm_HandSolder" H 5538 2650 50  0001 C CNN
 F 3 "~" H 5500 2800 50  0001 C CNN
 	1    5500 2800
@@
 P 5500 2950
 AR Path="/609FED99/60A50DF2" Ref="#PWR?"  Part="1"
-AR Path="/60A364EE/60A50DF2" Ref="#PWR025"  Part="1"
-F 0 "#PWR025" H 5500 2700 50  0001 C CNN
+AR Path="/60A364EE/60A50DF2" Ref="#PWR010"  Part="1"
+F 0 "#PWR010" H 5500 2700 50  0001 C CNN
 F 1 "GND" H 5505 2777 50  0000 C CNN
 F 2 "" H 5500 2950 50  0001 C CNN
@@
 P 5500 5000
 AR Path="/609FED99/60A513C1" Ref="#PWR?"  Part="1"
-AR Path="/60A364EE/60A513C1" Ref="#PWR026"  Part="1"
-F 0 "#PWR026" H 5500 4750 50  0001 C CNN
+AR Path="/60A364EE/60A513C1" Ref="#PWR011"  Part="1"
+F 0 "#PWR011" H 5500 4750 50  0001 C CNN
 F 1 "GND" H 5505 4827 50  0000 C CNN
 F 2 "" H 5500 5000 50  0001 C CNN
@@
 P 6500 5000
 AR Path="/609FED99/60A53C72" Ref="#PWR?"  Part="1"
-AR Path="/60A364EE/60A53C72" Ref="#PWR030"  Part="1"
-F 0 "#PWR030" H 6500 4750 50  0001 C CNN
+AR Path="/60A364EE/60A53C72" Ref="#PWR015"  Part="1"
+F 0 "#PWR015" H 6500 4750 50  0001 C CNN
 F 1 "GND" H 6505 4827 50  0000 C CNN
 F 2 "" H 6500 5000 50  0001 C CNN
@@
 P 5750 4150
 AR Path="/609FED99/60A57558" Ref="#PWR?"  Part="1"
-AR Path="/60A364EE/60A57558" Ref="#PWR027"  Part="1"
-F 0 "#PWR027" H 5750 3900 50  0001 C CNN
+AR Path="/60A364EE/60A57558" Ref="#PWR012"  Part="1"
+F 0 "#PWR012" H 5750 3900 50  0001 C CNN
 F 1 "GND" H 5755 3977 50  0000 C CNN
 F 2 "" H 5750 4150 50  0001 C CNN
@@
 P 6000 4700
 AR Path="/60A5913A" Ref="R?"  Part="1"
-AR Path="/60A364EE/60A5913A" Ref="R24"  Part="1"
-F 0 "R24" H 6070 4746 50  0000 L CNN
+AR Path="/60A364EE/60A5913A" Ref="R17"  Part="1"
+F 0 "R17" H 6070 4746 50  0000 L CNN
 F 1 "680k" H 6070 4655 50  0000 L CNN
-F 2 "Resistor_SMD:R_0603_1608Metric_Pad1.05x0.95mm_HandSolder" V 5930 4700 50  0001 C CNN
+F 2 "Resistor_SMD:R_0603_1608Metric_Pad0.98x0.95mm_HandSolder" V 5930 4700 50  0001 C CNN
 F 3 "~" H 6000 4700 50  0001 C CNN
 	1    6000 4700
@@
 P 6000 5000
 AR Path="/609FED99/60A595A5" Ref="#PWR?"  Part="1"
-AR Path="/60A364EE/60A595A5" Ref="#PWR029"  Part="1"
-F 0 "#PWR029" H 6000 4750 50  0001 C CNN
+AR Path="/60A364EE/60A595A5" Ref="#PWR014"  Part="1"
+F 0 "#PWR014" H 6000 4750 50  0001 C CNN
 F 1 "GND" H 6005 4827 50  0000 C CNN
 F 2 "" H 6000 5000 50  0001 C CNN
@@
 	6000 4250 6750 4250
 $Comp
-L Transistor_FET:IRLML6402 Q6
+L Transistor_FET:IRLML6402 Q5
 U 1 1 60A5E9F1
 P 4950 4550
-F 0 "Q6" V 5292 4550 50  0000 C CNN
+F 0 "Q5" V 5292 4550 50  0000 C CNN
 F 1 "IRLML6402" V 5201 4550 50  0000 C CNN
 F 2 "Package_TO_SOT_SMD:SOT-23" H 5150 4475 50  0001 L CIN
@@
 P 4500 4600
 AR Path="/60A61586" Ref="R?"  Part="1"
-AR Path="/60A364EE/60A61586" Ref="R20"  Part="1"
-F 0 "R20" H 4570 4646 50  0000 L CNN
+AR Path="/60A364EE/60A61586" Ref="R13"  Part="1"
+F 0 "R13" H 4570 4646 50  0000 L CNN
 F 1 "56k" H 4570 4555 50  0000 L CNN
-F 2 "Resistor_SMD:R_0603_1608Metric_Pad1.05x0.95mm_HandSolder" V 4430 4600 50  0001 C CNN
+F 2 "Resistor_SMD:R_0603_1608Metric_Pad0.98x0.95mm_HandSolder" V 4430 4600 50  0001 C CNN
 F 3 "~" H 4500 4600 50  0001 C CNN
 	1    4500 4600
@@
 P 4950 5000
 AR Path="/60A61F55" Ref="R?"  Part="1"
-AR Path="/60A364EE/60A61F55" Ref="R22"  Part="1"
-F 0 "R22" H 5020 5046 50  0000 L CNN
+AR Path="/60A364EE/60A61F55" Ref="R15"  Part="1"
+F 0 "R15" H 5020 5046 50  0000 L CNN
 F 1 "3,3k" H 5020 4955 50  0000 L CNN
-F 2 "Resistor_SMD:R_0603_1608Metric_Pad1.05x0.95mm_HandSolder" V 4880 5000 50  0001 C CNN
+F 2 "Resistor_SMD:R_0603_1608Metric_Pad0.98x0.95mm_HandSolder" V 4880 5000 50  0001 C CNN
 F 3 "~" H 4950 5000 50  0001 C CNN
 	1    4950 5000
@@
 $EndComp
 $Comp
-L Transistor_BJT:BC847 Q5
+L Transistor_BJT:BC847 Q4
 U 1 1 60A628F7
 P 4850 5500
-F 0 "Q5" H 5041 5546 50  0000 L CNN
+F 0 "Q4" H 5041 5546 50  0000 L CNN
 F 1 "BC847" H 5041 5455 50  0000 L CNN
 F 2 "Package_TO_SOT_SMD:SOT-23" H 5050 5425 50  0001 L CIN
@@
 P 4950 5800
 AR Path="/609FED99/60A63AB4" Ref="#PWR?"  Part="1"
-AR Path="/60A364EE/60A63AB4" Ref="#PWR024"  Part="1"
-F 0 "#PWR024" H 4950 5550 50  0001 C CNN
+AR Path="/60A364EE/60A63AB4" Ref="#PWR09"  Part="1"
+F 0 "#PWR09" H 4950 5550 50  0001 C CNN
 F 1 "GND" H 4955 5627 50  0000 C CNN
 F 2 "" H 4950 5800 50  0001 C CNN
@@
 P 4500 5650
 AR Path="/60A65A06" Ref="R?"  Part="1"
-AR Path="/60A364EE/60A65A06" Ref="R21"  Part="1"
-F 0 "R21" H 4570 5696 50  0000 L CNN
+AR Path="/60A364EE/60A65A06" Ref="R14"  Part="1"
+F 0 "R14" H 4570 5696 50  0000 L CNN
 F 1 "56k" H 4570 5605 50  0000 L CNN
-F 2 "Resistor_SMD:R_0603_1608Metric_Pad1.05x0.95mm_HandSolder" V 4430 5650 50  0001 C CNN
+F 2 "Resistor_SMD:R_0603_1608Metric_Pad0.98x0.95mm_HandSolder" V 4430 5650 50  0001 C CNN
 F 3 "~" H 4500 5650 50  0001 C CNN
 	1    4500 5650
@@
 P 4200 5500
 AR Path="/60A65F80" Ref="R?"  Part="1"
-AR Path="/60A364EE/60A65F80" Ref="R18"  Part="1"
-F 0 "R18" H 4270 5546 50  0000 L CNN
+AR Path="/60A364EE/60A65F80" Ref="R11"  Part="1"
+F 0 "R11" H 4270 5546 50  0000 L CNN
 F 1 "10k" H 4270 5455 50  0000 L CNN
-F 2 "Resistor_SMD:R_0603_1608Metric_Pad1.05x0.95mm_HandSolder" V 4130 5500 50  0001 C CNN
+F 2 "Resistor_SMD:R_0603_1608Metric_Pad0.98x0.95mm_HandSolder" V 4130 5500 50  0001 C CNN
 F 3 "~" H 4200 5500 50  0001 C CNN
 	1    4200 5500
@@
 P 4000 3000
 AR Path="/60AA5C07" Ref="R?"  Part="1"
-AR Path="/60A364EE/60AA5C07" Ref="R17"  Part="1"
-F 0 "R17" H 4070 3046 50  0000 L CNN
+AR Path="/60A364EE/60AA5C07" Ref="R10"  Part="1"
+F 0 "R10" H 4070 3046 50  0000 L CNN
 F 1 "4,7k" H 4070 2955 50  0000 L CNN
-F 2 "Resistor_SMD:R_0603_1608Metric_Pad1.05x0.95mm_HandSolder" V 3930 3000 50  0001 C CNN
+F 2 "Resistor_SMD:R_0603_1608Metric_Pad0.98x0.95mm_HandSolder" V 3930 3000 50  0001 C CNN
 F 3 "~" H 4000 3000 50  0001 C CNN
 	1    4000 3000
@@
 P 4500 3000
 AR Path="/60AA6C0E" Ref="R?"  Part="1"
-AR Path="/60A364EE/60AA6C0E" Ref="R19"  Part="1"
-F 0 "R19" H 4570 3046 50  0000 L CNN
+AR Path="/60A364EE/60AA6C0E" Ref="R12"  Part="1"
+F 0 "R12" H 4570 3046 50  0000 L CNN
 F 1 "4,7k" H 4570 2955 50  0000 L CNN
-F 2 "Resistor_SMD:R_0603_1608Metric_Pad1.05x0.95mm_HandSolder" V 4430 3000 50  0001 C CNN
+F 2 "Resistor_SMD:R_0603_1608Metric_Pad0.98x0.95mm_HandSolder" V 4430 3000 50  0001 C CNN
 F 3 "~" H 4500 3000 50  0001 C CNN
 	1    4500 3000
@@
 P 5000 3000
 AR Path="/60AC582F" Ref="R?"  Part="1"
-AR Path="/60A364EE/60AC582F" Ref="R23"  Part="1"
-F 0 "R23" H 5070 3046 50  0000 L CNN
+AR Path="/60A364EE/60AC582F" Ref="R16"  Part="1"
+F 0 "R16" H 5070 3046 50  0000 L CNN
 F 1 "10k" H 5070 2955 50  0000 L CNN
-F 2 "Resistor_SMD:R_0603_1608Metric_Pad1.05x0.95mm_HandSolder" V 4930 3000 50  0001 C CNN
+F 2 "Resistor_SMD:R_0603_1608Metric_Pad0.98x0.95mm_HandSolder" V 4930 3000 50  0001 C CNN
 F 3 "~" H 5000 3000 50  0001 C CNN
 	1    5000 3000
@@
 AR Path="/609CA6A8/60AD5A10" Ref="C?"  Part="1"
 AR Path="/609CA6A8/60AE5653/60AD5A10" Ref="C?"  Part="1"
-AR Path="/60A364EE/60AD5A10" Ref="C21"  Part="1"
-F 0 "C21" H 5615 4796 50  0000 L CNN
+AR Path="/60A364EE/60AD5A10" Ref="C11"  Part="1"
+F 0 "C11" H 5615 4796 50  0000 L CNN
 F 1 "4,7" H 5615 4705 50  0000 L CNN
-F 2 "Capacitor_SMD:C_1206_3216Metric_Pad1.42x1.75mm_HandSolder" H 5538 4600 50  0001 C CNN
+F 2 "Capacitor_SMD:C_1206_3216Metric_Pad1.33x1.80mm_HandSolder" H 5538 4600 50  0001 C CNN
 F 3 "~" H 5500 4750 50  0001 C CNN
 	1    5500 4750
@@
 AR Path="/609CA6A8/60AD77C2" Ref="C?"  Part="1"
 AR Path="/609CA6A8/60AE5653/60AD77C2" Ref="C?"  Part="1"
-AR Path="/60A364EE/60AD77C2" Ref="C22"  Part="1"
-F 0 "C22" H 6615 4796 50  0000 L CNN
+AR Path="/60A364EE/60AD77C2" Ref="C12"  Part="1"
+F 0 "C12" H 6615 4796 50  0000 L CNN
 F 1 "4,7" H 6615 4705 50  0000 L CNN
-F 2 "Capacitor_SMD:C_1206_3216Metric_Pad1.42x1.75mm_HandSolder" H 6538 4600 50  0001 C CNN
+F 2 "Capacitor_SMD:C_1206_3216Metric_Pad1.33x1.80mm_HandSolder" H 6538 4600 50  0001 C CNN
 F 3 "~" H 6500 4750 50  0001 C CNN
 	1    6500 4750
