File: furnace/furnace_controller/I2C_display_connector.sch (KiCad schematic (older format))
At the start: 4 parts

Commit message: Add files via upload
Parts:
- gave numbers to parts that had none: 4
Changed lines of the file:
@@
 AR Path="/609CA1D9/60B4354B" Ref="J?"  Part="1"
 AR Path="/60B4354B" Ref="J?"  Part="1"
-AR Path="/60B3D5E3/60B4354B" Ref="J?"  Part="1"
-F 0 "J?" H 7808 4381 50  0000 C CNN
+AR Path="/60B3D5E3/60B4354B" Ref="J14"  Part="1"
+F 0 "J14" H 7808 4381 50  0000 C CNN
 F 1 "PLS-4R" H 7808 4290 50  0000 C CNN
 F 2 "" H 7700 4100 50  0001 C CNN
@@
 AR Path="/609FED99/60B43551" Ref="#PWR?"  Part="1"
 AR Path="/60B43551" Ref="#PWR?"  Part="1"
-AR Path="/60B3D5E3/60B43551" Ref="#PWR?"  Part="1"
-F 0 "#PWR?" H 7300 4050 50  0001 C CNN
+AR Path="/60B3D5E3/60B43551" Ref="#PWR061"  Part="1"
+F 0 "#PWR061" H 7300 4050 50  0001 C CNN
 F 1 "GND" H 7305 4127 50  0000 C CNN
 F 2 "" H 7300 4300 50  0001 C CNN
@@
 AR Path="/609FED99/60B43557" Ref="#PWR?"  Part="1"
 AR Path="/60B43557" Ref="#PWR?"  Part="1"
-AR Path="/60B3D5E3/60B43557" Ref="#PWR?"  Part="1"
-F 0 "#PWR?" H 5000 2850 50  0001 C CNN
+AR Path="/60B3D5E3/60B43557" Ref="#PWR059"  Part="1"
+F 0 "#PWR059" H 5000 2850 50  0001 C CNN
 F 1 "+5V" H 5015 3173 50  0000 C CNN
 F 2 "" H 5000 3000 50  0001 C CNN
@@
 P 5500 3000
 AR Path="/60B43562" Ref="JP?"  Part="1"
-AR Path="/60B3D5E3/60B43562" Ref="JP?"  Part="1"
-F 0 "JP?" H 5500 3147 50  0000 C CNN
+AR Path="/60B3D5E3/60B43562" Ref="JP1"  Part="1"
+F 0 "JP1" H 5500 3147 50  0000 C CNN
 F 1 "Jumper_NC_Dual" H 5500 3148 50  0001 C CNN
 F 2 "" H 5500 3000 50  0001 C CNN
@@
 AR Path="/609FED99/60B43568" Ref="#PWR?"  Part="1"
 AR Path="/60B43568" Ref="#PWR?"  Part="1"
-AR Path="/60B3D5E3/60B43568" Ref="#PWR?"  Part="1"
-F 0 "#PWR?" H 6000 2850 50  0001 C CNN
+AR Path="/60B3D5E3/60B43568" Ref="#PWR060"  Part="1"
+F 0 "#PWR060" H 6000 2850 50  0001 C CNN
 F 1 "+3V3" H 6015 3173 50  0000 C CNN
 F 2 "" H 6000 3000 50  0001 C CNN
@@
 AR Path="/60B4356E" Ref="R?"  Part="1"
 AR Path="/60A364EE/60B4356E" Ref="R?"  Part="1"
-AR Path="/60B3D5E3/60B4356E" Ref="R?"  Part="1"
-F 0 "R?" H 6070 3696 50  0000 L CNN
+AR Path="/60B3D5E3/60B4356E" Ref="R54"  Part="1"
+F 0 "R54" H 6070 3696 50  0000 L CNN
 F 1 "4,7k" H 6070 3605 50  0000 L CNN
 F 2 "Resistor_SMD:R_0603_1608Metric_Pad0.98x0.95mm_HandSolder" V 5930 3650 50  0001 C CNN
@@
 AR Path="/60B43574" Ref="R?"  Part="1"
 AR Path="/60A364EE/60B43574" Ref="R?"  Part="1"
-AR Path="/60B3D5E3/60B43574" Ref="R?"  Part="1"
-F 0 "R?" H 6570 3696 50  0000 L CNN
+AR Path="/60B3D5E3/60B43574" Ref="R55"  Part="1"
+F 0 "R55" H 6570 3696 50  0000 L CNN
 F 1 "4,7k" H 6570 3605 50  0000 L CNN
 F 2 "Resistor_SMD:R_0603_1608Metric_Pad0.98x0.95mm_HandSolder" V 6430 3650 50  0001 C CNN

Commit message: Add files via upload
Parts:
- J14: footprint (none) -> Connector_PinHeader_2.54mm:PinHeader_1x04_P2.54mm_Horizontal
- JP1: footprint (none) -> Connector_PinHeader_2.54mm:PinHeader_1x03_P2.54mm_Vertical
- R54, R55: footprint Resistor_SMD:R_0603_1608Metric_Pad0.98x0.95mm_HandSolder -> Resistor_SMD:R_0603_1608Metric_Pad1.05x0.95mm_HandSolder
Changed lines of the file:
@@
 encoding utf-8
 Sheet 17 18
-Title ""
-Date ""
-Rev ""
-Comp ""
+Title "Furnace controller"
+Date "2021-08-26"
+Rev "1.0"
+Comp "Yuriy Volkov"
 Comment1 ""
 Comment2 ""
@@
 F 0 "J14" H 7808 4381 50  0000 C CNN
 F 1 "PLS-4R" H 7808 4290 50  0000 C CNN
-F 2 "" H 7700 4100 50  0001 C CNN
+F 2 "Connector_PinHeader_2.54mm:PinHeader_1x04_P2.54mm_Horizontal" H 7700 4100 50  0001 C CNN
 F 3 "~" H 7700 4100 50  0001 C CNN
 	1    7700 4100
@@
 F 0 "JP1" H 5500 3147 50  0000 C CNN
 F 1 "Jumper_NC_Dual" H 5500 3148 50  0001 C CNN
-F 2 "" H 5500 3000 50  0001 C CNN
+F 2 "Connector_PinHeader_2.54mm:PinHeader_1x03_P2.54mm_Vertical" H 5500 3000 50  0001 C CNN
 F 3 "~" H 5500 3000 50  0001 C CNN
 	1    5500 3000
@@
 F 0 "R54" H 6070 3696 50  0000 L CNN
 F 1 "4,7k" H 6070 3605 50  0000 L CNN
-F 2 "Resistor_SMD:R_0603_1608Metric_Pad0.98x0.95mm_HandSolder" V 5930 3650 50  0001 C CNN
+F 2 "Resistor_SMD:R_0603_1608Metric_Pad1.05x0.95mm_HandSolder" V 5930 3650 50  0001 C CNN
 F 3 "~" H 6000 3650 50  0001 C CNN
 	1    6000 3650
@@
 F 0 "R55" H 6570 3696 50  0000 L CNN
 F 1 "4,7k" H 6570 3605 50  0000 L CNN
-F 2 "Resistor_SMD:R_0603_1608Metric_Pad0.98x0.95mm_HandSolder" V 6430 3650 50  0001 C CNN
+F 2 "Resistor_SMD:R_0603_1608Metric_Pad1.05x0.95mm_HandSolder" V 6430 3650 50  0001 C CNN
 F 3 "~" H 6500 3650 50  0001 C CNN
 	1    6500 3650

Commit message: Add files via upload
Parts:
- R44: renamed from R54; footprint Resistor_SMD:R_0603_1608Metric_Pad1.05x0.95mm_HandSolder -> Resistor_SMD:R_0603_1608Metric_Pad0.98x0.95mm_HandSolder
- R45: renamed from R55; footprint Resistor_SMD:R_0603_1608Metric_Pad1.05x0.95mm_HandSolder -> Resistor_SMD:R_0603_1608Metric_Pad0.98x0.95mm_HandSolder
- renumbered J14 to J10
Changed lines of the file:
@@
 $Descr A4 11693 8268
 encoding utf-8
-Sheet 17 18
+Sheet 16 18
 Title "Furnace controller"
-Date "2021-08-26"
+Date "2021-09-24"
 Rev "1.0"
 Comp "Yuriy Volkov"
@@
 AR Path="/609CA1D9/60B4354B" Ref="J?"  Part="1"
 AR Path="/60B4354B" Ref="J?"  Part="1"
-AR Path="/60B3D5E3/60B4354B" Ref="J14"  Part="1"
-F 0 "J14" H 7808 4381 50  0000 C CNN
+AR Path="/60B3D5E3/60B4354B" Ref="J10"  Part="1"
+F 0 "J10" H 7808 4381 50  0000 C CNN
 F 1 "PLS-4R" H 7808 4290 50  0000 C CNN
 F 2 "Connector_PinHeader_2.54mm:PinHeader_1x04_P2.54mm_Horizontal" H 7700 4100 50  0001 C CNN
@@
 AR Path="/609FED99/60B43551" Ref="#PWR?"  Part="1"
 AR Path="/60B43551" Ref="#PWR?"  Part="1"
-AR Path="/60B3D5E3/60B43551" Ref="#PWR061"  Part="1"
-F 0 "#PWR061" H 7300 4050 50  0001 C CNN
+AR Path="/60B3D5E3/60B43551" Ref="#PWR041"  Part="1"
+F 0 "#PWR041" H 7300 4050 50  0001 C CNN
 F 1 "GND" H 7305 4127 50  0000 C CNN
 F 2 "" H 7300 4300 50  0001 C CNN
@@
 AR Path="/609FED99/60B43557" Ref="#PWR?"  Part="1"
 AR Path="/60B43557" Ref="#PWR?"  Part="1"
-AR Path="/60B3D5E3/60B43557" Ref="#PWR059"  Part="1"
-F 0 "#PWR059" H 5000 2850 50  0001 C CNN
+AR Path="/60B3D5E3/60B43557" Ref="#PWR039"  Part="1"
+F 0 "#PWR039" H 5000 2850 50  0001 C CNN
 F 1 "+5V" H 5015 3173 50  0000 C CNN
 F 2 "" H 5000 3000 50  0001 C CNN
@@
 AR Path="/609FED99/60B43568" Ref="#PWR?"  Part="1"
 AR Path="/60B43568" Ref="#PWR?"  Part="1"
-AR Path="/60B3D5E3/60B43568" Ref="#PWR060"  Part="1"
-F 0 "#PWR060" H 6000 2850 50  0001 C CNN
+AR Path="/60B3D5E3/60B43568" Ref="#PWR040"  Part="1"
+F 0 "#PWR040" H 6000 2850 50  0001 C CNN
 F 1 "+3V3" H 6015 3173 50  0000 C CNN
 F 2 "" H 6000 3000 50  0001 C CNN
@@
 AR Path="/60B4356E" Ref="R?"  Part="1"
 AR Path="/60A364EE/60B4356E" Ref="R?"  Part="1"
-AR Path="/60B3D5E3/60B4356E" Ref="R54"  Part="1"
-F 0 "R54" H 6070 3696 50  0000 L CNN
+AR Path="/60B3D5E3/60B4356E" Ref="R44"  Part="1"
+F 0 "R44" H 6070 3696 50  0000 L CNN
 F 1 "4,7k" H 6070 3605 50  0000 L CNN
-F 2 "Resistor_SMD:R_0603_1608Metric_Pad1.05x0.95mm_HandSolder" V 5930 3650 50  0001 C CNN
+F 2 "Resistor_SMD:R_0603_1608Metric_Pad0.98x0.95mm_HandSolder" V 5930 3650 50  0001 C CNN
 F 3 "~" H 6000 3650 50  0001 C CNN
 	1    6000 3650
@@
 AR Path="/60B43574" Ref="R?"  Part="1"
 AR Path="/60A364EE/60B43574" Ref="R?"  Part="1"
-AR Path="/60B3D5E3/60B43574" Ref="R55"  Part="1"
-F 0 "R55" H 6570 3696 50  0000 L CNN
+AR Path="/60B3D5E3/60B43574" Ref="R45"  Part="1"
+F 0 "R45" H 6570 3696 50  0000 L CNN
 F 1 "4,7k" H 6570 3605 50  0000 L CNN
-F 2 "Resistor_SMD:R_0603_1608Metric_Pad1.05x0.95mm_HandSolder" V 6430 3650 50  0001 C CNN
+F 2 "Resistor_SMD:R_0603_1608Metric_Pad0.98x0.95mm_HandSolder" V 6430 3650 50  0001 C CNN
 F 3 "~" H 6500 3650 50  0001 C CNN
 	1    6500 3650
