File: furnace/furnace_controller/Isolated_temp_sensor.sch (KiCad schematic (older format))
At the start: 1 part

Commit message: Add files via upload
Changed lines of the file:
@@
 TC-
 Text Label 3450 2050 2    50   ~ 0
-TC+1
+TC+0
 Text Label 3450 2150 2    50   ~ 0
-TC-1
+TC-0
 Text Label 7650 3250 0    50   ~ 0
 MISO
 Text Label 7650 3150 0    50   ~ 0
-~CS1
+~CS0
 Text HLabel 1050 2750 0    50   Input ~ 0
 TC+
@@
 	2350 2750 2450 2850
 Text Label 1250 2950 0    50   ~ 0
+TC+0
+Text Label 1550 2950 0    50   ~ 0
 TC+1
-Text Label 1550 2950 0    50   ~ 0
+Text Label 1850 2950 0    50   ~ 0
 TC+2
-Text Label 1850 2950 0    50   ~ 0
+Text Label 2150 2950 0    50   ~ 0
 TC+3
-Text Label 2150 2950 0    50   ~ 0
+Text Label 2450 2950 0    50   ~ 0
 TC+4
-Text Label 2450 2950 0    50   ~ 0
-TC+5
 Wire Wire Line
 	1250 2850 1250 2950
@@
 	2450 3350 2450 3450
 Text Label 1250 3450 0    50   ~ 0
+TC-0
+Text Label 1550 3450 0    50   ~ 0
 TC-1
-Text Label 1550 3450 0    50   ~ 0
+Text Label 1850 3450 0    50   ~ 0
 TC-2
-Text Label 1850 3450 0    50   ~ 0
+Text Label 2150 3450 0    50   ~ 0
 TC-3
-Text Label 2150 3450 0    50   ~ 0
+Text Label 2450 3450 0    50   ~ 0
 TC-4
-Text Label 2450 3450 0    50   ~ 0
-TC-5
 $Sheet
 S 3550 1750 1000 700
 U 60AD75F8
-F0 "THERMOCOUPLE1" 50
+F0 "THERMOCOUPLE0" 50
 F1 "Thermocouple.sch" 50
 F2 "TC+" I L 3550 2050 50
@@
 S 6550 2750 1000 800
 U 60AD7668
-F0 "ISOLATOR1" 50
+F0 "ISOLATOR0" 50
 F1 "Isolator.sch" 50
 F2 "OUTC" O R 7550 3250 50
@@
 +3V3_ISO
 Text Label 3450 3050 2    50   ~ 0
-TC+2
+TC+1
 Text Label 3450 3150 2    50   ~ 0
-TC-2
+TC-1
 Wire Wire Line
 	3550 2850 3450 2850
@@
 S 3550 2750 1000 700
 U 60B0F1FC
-F0 "THERMOCOUPLE2" 50
+F0 "THERMOCOUPLE1" 50
 F1 "Thermocouple.sch" 50
 F2 "TC+" I L 3550 3050 50
@@
 +3V3_ISO
 Text Label 3450 4050 2    50   ~ 0
-TC+3
+TC+2
 Text Label 3450 4150 2    50   ~ 0
-TC-3
+TC-2
 Wire Wire Line
 	3550 3850 3450 3850
@@
 S 3550 3750 1000 700
 U 60B0FB30
-F0 "THERMOCOUPLE3" 50
+F0 "THERMOCOUPLE2" 50
 F1 "Thermocouple.sch" 50
 F2 "TC+" I L 3550 4050 50
@@
 +3V3_ISO
 Text Label 3450 5050 2    50   ~ 0
-TC+4
+TC+3
 Text Label 3450 5150 2    50   ~ 0
-TC-4
+TC-3
 Wire Wire Line
 	3550 4850 3450 4850
@@
 S 3550 4750 1000 700
 U 60B108D6
-F0 "THERMOCOUPLE4" 50
+F0 "THERMOCOUPLE3" 50
 F1 "Thermocouple.sch" 50
 F2 "TC+" I L 3550 5050 50
@@
 +3V3_ISO
 Text Label 3450 6050 2    50   ~ 0
-TC+5
+TC+4
 Text Label 3450 6150 2    50   ~ 0
-TC-5
+TC-4
 Wire Wire Line
 	3550 5850 3450 5850
@@
 S 3550 5750 1000 700
 U 60B118F2
-F0 "THERMOCOUPLE5" 50
+F0 "THERMOCOUPLE4" 50
 F1 "Thermocouple.sch" 50
 F2 "TC+" I L 3550 6050 50
@@
 $EndComp
 Text Label 7650 4300 0    50   ~ 0
-~CS2
+~CS1
 Wire Wire Line
 	7550 4300 7650 4300
@@
 S 6550 4000 1000 800
 U 60B14815
-F0 "ISOLATOR2" 50
+F0 "ISOLATOR1" 50
 F1 "Isolator.sch" 50
 F2 "OUTC" O R 7550 4500 50
@@
 $EndComp
 Text Label 7650 5550 0    50   ~ 0
-~CS4
+~CS3
 Wire Wire Line
 	7550 5550 7650 5550
@@
 S 6550 5250 1000 800
 U 60B180E1
-F0 "ISOLATOR3" 50
+F0 "ISOLATOR2" 50
 F1 "Isolator.sch" 50
 F2 "OUTC" O R 7550 5750 50
@@
 	6550 5350 6450 5350
 Text Label 7650 4400 0    50   ~ 0
-~CS3
+~CS2
 Text Label 7650 5650 0    50   ~ 0
-~CS5
+~CS4
 NoConn ~ 7650 4500
 NoConn ~ 7650 5750
@@
 $EndComp
 Text Label 10350 2950 0    50   ~ 0
-~CS5
+~CS4
 Text Label 10050 2950 0    50   ~ 0
-~CS4
+~CS3
 Text Label 9750 2950 0    50   ~ 0
-~CS3
+~CS2
 Text Label 9450 2950 0    50   ~ 0
-~CS2
+~CS1
 Wire Wire Line
 	10550 3750 10050 3750
@@
 	9150 2850 9150 2950
 Text Label 9150 2950 0    50   ~ 0
-~CS1
+~CS0
 Entry Wire Line
 	10250 2750 10350 2850

Commit message: Add files via upload
Parts:
- gave numbers to parts that had none: 1
Changed lines of the file:
@@
 $Descr A4 11693 8268
 encoding utf-8
-Sheet 6 18
+Sheet 5 18
 Title ""
 Date ""
@@
 AR Path="/609CA6A8/60A0A500/60A0B581" Ref="#PWR?"  Part="1"
 AR Path="/609CA6A8/60A0A922/60A0B581" Ref="#PWR?"  Part="1"
-AR Path="/609CA6A8/60A0B581" Ref="#PWR?"  Part="1"
-F 0 "#PWR?" H 7650 3200 50  0001 C CNN
+AR Path="/609CA6A8/60A0B581" Ref="#PWR046"  Part="1"
+F 0 "#PWR046" H 7650 3200 50  0001 C CNN
 F 1 "GND" H 7655 3277 50  0000 C CNN
 F 2 "" H 7650 3450 50  0001 C CNN
@@
 AR Path="/609CA6A8/60A0A500/60A0EB0A" Ref="#PWR?"  Part="1"
 AR Path="/609CA6A8/60A0A922/60A0EB0A" Ref="#PWR?"  Part="1"
-AR Path="/609CA6A8/60A0EB0A" Ref="#PWR?"  Part="1"
-F 0 "#PWR?" H 3450 2100 50  0001 C CNN
+AR Path="/609CA6A8/60A0EB0A" Ref="#PWR032"  Part="1"
+F 0 "#PWR032" H 3450 2100 50  0001 C CNN
 F 1 "GND1" H 3455 2177 50  0000 C CNN
 F 2 "" H 3450 2350 50  0001 C CNN
@@
 +3V3_ISO
 Text HLabel 1050 3250 0    50   Input ~ 0
-TC-
+TC-[0..4]
 Text Label 3450 2050 2    50   ~ 0
 TC+0
@@
 ~CS0
 Text HLabel 1050 2750 0    50   Input ~ 0
-TC+
+TC+[0..4]
 Text Label 7650 3050 0    50   ~ 0
 SCK
@@
 	7550 2850 7650 2850
 $Comp
-L power:+3V3 #PWR?
+L power:+3V3 #PWR045
 U 1 1 60A0F4F9
 P 7650 2850
-F 0 "#PWR?" H 7650 2700 50  0001 C CNN
+F 0 "#PWR045" H 7650 2700 50  0001 C CNN
 F 1 "+3V3" H 7665 3023 50  0000 C CNN
 F 2 "" H 7650 2850 50  0001 C CNN
@@
 AR Path="/609CA6A8/60A0A500/60B09F47" Ref="#PWR?"  Part="1"
 AR Path="/609CA6A8/60A0A922/60B09F47" Ref="#PWR?"  Part="1"
-AR Path="/609CA6A8/60B09F47" Ref="#PWR?"  Part="1"
-F 0 "#PWR?" H 6450 1900 50  0001 C CNN
+AR Path="/609CA6A8/60B09F47" Ref="#PWR037"  Part="1"
+F 0 "#PWR037" H 6450 1900 50  0001 C CNN
 F 1 "GND1" H 6455 1977 50  0000 C CNN
 F 2 "" H 6450 2150 50  0001 C CNN
@@
 AR Path="/609CA6A8/60A0A500/60B0A5B6" Ref="#PWR?"  Part="1"
 AR Path="/609CA6A8/60A0A922/60B0A5B6" Ref="#PWR?"  Part="1"
-AR Path="/609CA6A8/60B0A5B6" Ref="#PWR?"  Part="1"
-F 0 "#PWR?" H 6450 3200 50  0001 C CNN
+AR Path="/609CA6A8/60B0A5B6" Ref="#PWR038"  Part="1"
+F 0 "#PWR038" H 6450 3200 50  0001 C CNN
 F 1 "GND1" H 6455 3277 50  0000 C CNN
 F 2 "" H 6450 3450 50  0001 C CNN
@@
 	6450 3450 6550 3450
 $Comp
-L power:+5V #PWR?
+L power:+5V #PWR043
 U 1 1 60B0AA53
 P 7650 1850
-F 0 "#PWR?" H 7650 1700 50  0001 C CNN
+F 0 "#PWR043" H 7650 1700 50  0001 C CNN
 F 1 "+5V" H 7665 2023 50  0000 C CNN
 F 2 "" H 7650 1850 50  0001 C CNN
@@
 AR Path="/609CA6A8/60A0A500/60B0B742" Ref="#PWR?"  Part="1"
 AR Path="/609CA6A8/60A0A922/60B0B742" Ref="#PWR?"  Part="1"
-AR Path="/609CA6A8/60B0B742" Ref="#PWR?"  Part="1"
-F 0 "#PWR?" H 7650 1900 50  0001 C CNN
+AR Path="/609CA6A8/60B0B742" Ref="#PWR044"  Part="1"
+F 0 "#PWR044" H 7650 1900 50  0001 C CNN
 F 1 "GND" H 7655 1977 50  0000 C CNN
 F 2 "" H 7650 2150 50  0001 C CNN
@@
 AR Path="/609CA6A8/60A0A500/60B0F1ED" Ref="#PWR?"  Part="1"
 AR Path="/609CA6A8/60A0A922/60B0F1ED" Ref="#PWR?"  Part="1"
-AR Path="/609CA6A8/60B0F1ED" Ref="#PWR?"  Part="1"
-F 0 "#PWR?" H 3450 3100 50  0001 C CNN
+AR Path="/609CA6A8/60B0F1ED" Ref="#PWR033"  Part="1"
+F 0 "#PWR033" H 3450 3100 50  0001 C CNN
 F 1 "GND1" H 3455 3177 50  0000 C CNN
 F 2 "" H 3450 3350 50  0001 C CNN
@@
 AR Path="/609CA6A8/60A0A500/60B0FB21" Ref="#PWR?"  Part="1"
 AR Path="/609CA6A8/60A0A922/60B0FB21" Ref="#PWR?"  Part="1"
-AR Path="/609CA6A8/60B0FB21" Ref="#PWR?"  Part="1"
-F 0 "#PWR?" H 3450 4100 50  0001 C CNN
+AR Path="/609CA6A8/60B0FB21" Ref="#PWR034"  Part="1"
+F 0 "#PWR034" H 3450 4100 50  0001 C CNN
 F 1 "GND1" H 3455 4177 50  0000 C CNN
 F 2 "" H 3450 4350 50  0001 C CNN
@@
 AR Path="/609CA6A8/60A0A500/60B108C7" Ref="#PWR?"  Part="1"
 AR Path="/609CA6A8/60A0A922/60B108C7" Ref="#PWR?"  Part="1"
-AR Path="/609CA6A8/60B108C7" Ref="#PWR?"  Part="1"
-F 0 "#PWR?" H 3450 5100 50  0001 C CNN
+AR Path="/609CA6A8/60B108C7" Ref="#PWR035"  Part="1"
+F 0 "#PWR035" H 3450 5100 50  0001 C CNN
 F 1 "GND1" H 3455 5177 50  0000 C CNN
 F 2 "" H 3450 5350 50  0001 C CNN
@@
 AR Path="/609CA6A8/60A0A500/60B118E3" Ref="#PWR?"  Part="1"
 AR Path="/609CA6A8/60A0A922/60B118E3" Ref="#PWR?"  Part="1"
-AR Path="/609CA6A8/60B118E3" Ref="#PWR?"  Part="1"
-F 0 "#PWR?" H 3450 6100 50  0001 C CNN
+AR Path="/609CA6A8/60B118E3" Ref="#PWR036"  Part="1"
+F 0 "#PWR036" H 3450 6100 50  0001 C CNN
 F 1 "GND1" H 3455 6177 50  0000 C CNN
 F 2 "" H 3450 6350 50  0001 C CNN
@@
 AR Path="/609CA6A8/60A0A500/60B14803" Ref="#PWR?"  Part="1"
 AR Path="/609CA6A8/60A0A922/60B14803" Ref="#PWR?"  Part="1"
-AR Path="/609CA6A8/60B14803" Ref="#PWR?"  Part="1"
-F 0 "#PWR?" H 7650 4450 50  0001 C CNN
+AR Path="/609CA6A8/60B14803" Ref="#PWR048"  Part="1"
+F 0 "#PWR048" H 7650 4450 50  0001 C CNN
 F 1 "GND" H 7655 4527 50  0000 C CNN
 F 2 "" H 7650 4700 50  0001 C CNN
@@
 	7550 4100 7650 4100
 $Comp
-L power:+3V3 #PWR?
+L power:+3V3 #PWR047
 U 1 1 60B1481C
 P 7650 4100
-F 0 "#PWR?" H 7650 3950 50  0001 C CNN
+F 0 "#PWR047" H 7650 3950 50  0001 C CNN
 F 1 "+3V3" H 7665 4273 50  0000 C CNN
 F 2 "" H 7650 4100 50  0001 C CNN
@@
 AR Path="/609CA6A8/60A0A500/60B14823" Ref="#PWR?"  Part="1"
 AR Path="/609CA6A8/60A0A922/60B14823" Ref="#PWR?"  Part="1"
-AR Path="/609CA6A8/60B14823" Ref="#PWR?"  Part="1"
-F 0 "#PWR?" H 6450 4450 50  0001 C CNN
+AR Path="/609CA6A8/60B14823" Ref="#PWR040"  Part="1"
+F 0 "#PWR040" H 6450 4450 50  0001 C CNN
 F 1 "GND1" H 6455 4527 50  0000 C CNN
 F 2 "" H 6450 4700 50  0001 C CNN
@@
 AR Path="/609CA6A8/60A0A500/60B180CF" Ref="#PWR?"  Part="1"
 AR Path="/609CA6A8/60A0A922/60B180CF" Ref="#PWR?"  Part="1"
-AR Path="/609CA6A8/60B180CF" Ref="#PWR?"  Part="1"
-F 0 "#PWR?" H 7650 5700 50  0001 C CNN
+AR Path="/609CA6A8/60B180CF" Ref="#PWR050"  Part="1"
+F 0 "#PWR050" H 7650 5700 50  0001 C CNN
 F 1 "GND" H 7655 5777 50  0000 C CNN
 F 2 "" H 7650 5950 50  0001 C CNN
@@
 	7550 5350 7650 5350
 $Comp
-L power:+3V3 #PWR?
+L power:+3V3 #PWR049
 U 1 1 60B180E8
 P 7650 5350
-F 0 "#PWR?" H 7650 5200 50  0001 C CNN
+F 0 "#PWR049" H 7650 5200 50  0001 C CNN
 F 1 "+3V3" H 7665 5523 50  0000 C CNN
 F 2 "" H 7650 5350 50  0001 C CNN
@@
 AR Path="/609CA6A8/60A0A500/60B180EF" Ref="#PWR?"  Part="1"
 AR Path="/609CA6A8/60A0A922/60B180EF" Ref="#PWR?"  Part="1"
-AR Path="/609CA6A8/60B180EF" Ref="#PWR?"  Part="1"
-F 0 "#PWR?" H 6450 5700 50  0001 C CNN
+AR Path="/609CA6A8/60B180EF" Ref="#PWR042"  Part="1"
+F 0 "#PWR042" H 6450 5700 50  0001 C CNN
 F 1 "GND1" H 6455 5777 50  0000 C CNN
 F 2 "" H 6450 5950 50  0001 C CNN
@@
 AR Path="/609CA6A8/60A0A500/60B43E6A" Ref="#PWR?"  Part="1"
 AR Path="/609CA6A8/60A0A922/60B43E6A" Ref="#PWR?"  Part="1"
-AR Path="/609CA6A8/60B43E6A" Ref="#PWR?"  Part="1"
-F 0 "#PWR?" H 6450 4250 50  0001 C CNN
+AR Path="/609CA6A8/60B43E6A" Ref="#PWR039"  Part="1"
+F 0 "#PWR039" H 6450 4250 50  0001 C CNN
 F 1 "GND1" H 6455 4327 50  0000 C CNN
 F 2 "" H 6450 4500 50  0001 C CNN
@@
 AR Path="/609CA6A8/60A0A500/60B472DC" Ref="#PWR?"  Part="1"
 AR Path="/609CA6A8/60A0A922/60B472DC" Ref="#PWR?"  Part="1"
-AR Path="/609CA6A8/60B472DC" Ref="#PWR?"  Part="1"
-F 0 "#PWR?" H 6450 5500 50  0001 C CNN
+AR Path="/609CA6A8/60B472DC" Ref="#PWR041"  Part="1"
+F 0 "#PWR041" H 6450 5500 50  0001 C CNN
 F 1 "GND1" H 6455 5577 50  0000 C CNN
 F 2 "" H 6450 5750 50  0001 C CNN
@@
 AR Path="/609FED99/60A4EC17" Ref="#PWR?"  Part="1"
 AR Path="/60A364EE/60A4EC17" Ref="#PWR?"  Part="1"
-AR Path="/609CA6A8/60A4EC17" Ref="#PWR?"  Part="1"
-F 0 "#PWR?" H 9600 4250 50  0001 C CNN
+AR Path="/609CA6A8/60A4EC17" Ref="#PWR051"  Part="1"
+F 0 "#PWR051" H 9600 4250 50  0001 C CNN
 F 1 "GND" H 9605 4327 50  0000 C CNN
 F 2 "" H 9600 4500 50  0001 C CNN
@@
 P 9900 4400
 AR Path="/60A364EE/60A4EC11" Ref="J?"  Part="1"
-AR Path="/609CA6A8/60A4EC11" Ref="J?"  Part="1"
-F 0 "J?" H 10008 4681 50  0000 C CNN
+AR Path="/609CA6A8/60A4EC11" Ref="J11"  Part="1"
+F 0 "J11" H 10008 4681 50  0000 C CNN
 F 1 "Conn_01x03_Male" H 10008 4590 50  0000 C CNN
 F 2 "" H 9900 4400 50  0001 C CNN
@@
 SCK
 Text HLabel 10550 2750 2    50   Input ~ 0
-~CS
+~CS[0..4]
 Wire Bus Line
 	1050 2750 2550 2750

Commit message: Add files via upload
Parts:
- J11: value Conn_01x03_Male -> PLS-3; footprint (none) -> Connector_PinHeader_2.54mm:PinHeader_1x03_P2.54mm_Vertical
Changed lines of the file:
@@
 encoding utf-8
 Sheet 5 18
-Title ""
-Date ""
-Rev ""
-Comp ""
+Title "Furnace controller"
+Date "2021-08-26"
+Rev "1.0"
+Comp "Yuriy Volkov"
 Comment1 ""
 Comment2 ""
@@
 AR Path="/609CA6A8/60A4EC11" Ref="J11"  Part="1"
 F 0 "J11" H 10008 4681 50  0000 C CNN
-F 1 "Conn_01x03_Male" H 10008 4590 50  0000 C CNN
-F 2 "" H 9900 4400 50  0001 C CNN
+F 1 "PLS-3" H 10008 4590 50  0000 C CNN
+F 2 "Connector_PinHeader_2.54mm:PinHeader_1x03_P2.54mm_Vertical" H 9900 4400 50  0001 C CNN
 F 3 "~" H 9900 4400 50  0001 C CNN
 	1    9900 4400

Commit message: Add files via upload
Parts:
- renumbered J11 to J9
Changed lines of the file:
@@
 Sheet 5 18
 Title "Furnace controller"
-Date "2021-08-26"
+Date "2021-09-24"
 Rev "1.0"
 Comp "Yuriy Volkov"
@@
 AR Path="/609CA6A8/60A0A500/60A0B581" Ref="#PWR?"  Part="1"
 AR Path="/609CA6A8/60A0A922/60A0B581" Ref="#PWR?"  Part="1"
-AR Path="/609CA6A8/60A0B581" Ref="#PWR046"  Part="1"
-F 0 "#PWR046" H 7650 3200 50  0001 C CNN
+AR Path="/609CA6A8/60A0B581" Ref="#PWR031"  Part="1"
+F 0 "#PWR031" H 7650 3200 50  0001 C CNN
 F 1 "GND" H 7655 3277 50  0000 C CNN
 F 2 "" H 7650 3450 50  0001 C CNN
@@
 AR Path="/609CA6A8/60A0A500/60A0EB0A" Ref="#PWR?"  Part="1"
 AR Path="/609CA6A8/60A0A922/60A0EB0A" Ref="#PWR?"  Part="1"
-AR Path="/609CA6A8/60A0EB0A" Ref="#PWR032"  Part="1"
-F 0 "#PWR032" H 3450 2100 50  0001 C CNN
+AR Path="/609CA6A8/60A0EB0A" Ref="#PWR017"  Part="1"
+F 0 "#PWR017" H 3450 2100 50  0001 C CNN
 F 1 "GND1" H 3455 2177 50  0000 C CNN
 F 2 "" H 3450 2350 50  0001 C CNN
@@
 	7550 2850 7650 2850
 $Comp
-L power:+3V3 #PWR045
+L power:+3V3 #PWR030
 U 1 1 60A0F4F9
 P 7650 2850
-F 0 "#PWR045" H 7650 2700 50  0001 C CNN
+F 0 "#PWR030" H 7650 2700 50  0001 C CNN
 F 1 "+3V3" H 7665 3023 50  0000 C CNN
 F 2 "" H 7650 2850 50  0001 C CNN
@@
 AR Path="/609CA6A8/60A0A500/60B09F47" Ref="#PWR?"  Part="1"
 AR Path="/609CA6A8/60A0A922/60B09F47" Ref="#PWR?"  Part="1"
-AR Path="/609CA6A8/60B09F47" Ref="#PWR037"  Part="1"
-F 0 "#PWR037" H 6450 1900 50  0001 C CNN
+AR Path="/609CA6A8/60B09F47" Ref="#PWR022"  Part="1"
+F 0 "#PWR022" H 6450 1900 50  0001 C CNN
 F 1 "GND1" H 6455 1977 50  0000 C CNN
 F 2 "" H 6450 2150 50  0001 C CNN
@@
 AR Path="/609CA6A8/60A0A500/60B0A5B6" Ref="#PWR?"  Part="1"
 AR Path="/609CA6A8/60A0A922/60B0A5B6" Ref="#PWR?"  Part="1"
-AR Path="/609CA6A8/60B0A5B6" Ref="#PWR038"  Part="1"
-F 0 "#PWR038" H 6450 3200 50  0001 C CNN
+AR Path="/609CA6A8/60B0A5B6" Ref="#PWR023"  Part="1"
+F 0 "#PWR023" H 6450 3200 50  0001 C CNN
 F 1 "GND1" H 6455 3277 50  0000 C CNN
 F 2 "" H 6450 3450 50  0001 C CNN
@@
 	6450 3450 6550 3450
 $Comp
-L power:+5V #PWR043
+L power:+5V #PWR028
 U 1 1 60B0AA53
 P 7650 1850
-F 0 "#PWR043" H 7650 1700 50  0001 C CNN
+F 0 "#PWR028" H 7650 1700 50  0001 C CNN
 F 1 "+5V" H 7665 2023 50  0000 C CNN
 F 2 "" H 7650 1850 50  0001 C CNN
@@
 AR Path="/609CA6A8/60A0A500/60B0B742" Ref="#PWR?"  Part="1"
 AR Path="/609CA6A8/60A0A922/60B0B742" Ref="#PWR?"  Part="1"
-AR Path="/609CA6A8/60B0B742" Ref="#PWR044"  Part="1"
-F 0 "#PWR044" H 7650 1900 50  0001 C CNN
+AR Path="/609CA6A8/60B0B742" Ref="#PWR029"  Part="1"
+F 0 "#PWR029" H 7650 1900 50  0001 C CNN
 F 1 "GND" H 7655 1977 50  0000 C CNN
 F 2 "" H 7650 2150 50  0001 C CNN
@@
 AR Path="/609CA6A8/60A0A500/60B0F1ED" Ref="#PWR?"  Part="1"
 AR Path="/609CA6A8/60A0A922/60B0F1ED" Ref="#PWR?"  Part="1"
-AR Path="/609CA6A8/60B0F1ED" Ref="#PWR033"  Part="1"
-F 0 "#PWR033" H 3450 3100 50  0001 C CNN
+AR Path="/609CA6A8/60B0F1ED" Ref="#PWR018"  Part="1"
+F 0 "#PWR018" H 3450 3100 50  0001 C CNN
 F 1 "GND1" H 3455 3177 50  0000 C CNN
 F 2 "" H 3450 3350 50  0001 C CNN
@@
 AR Path="/609CA6A8/60A0A500/60B0FB21" Ref="#PWR?"  Part="1"
 AR Path="/609CA6A8/60A0A922/60B0FB21" Ref="#PWR?"  Part="1"
-AR Path="/609CA6A8/60B0FB21" Ref="#PWR034"  Part="1"
-F 0 "#PWR034" H 3450 4100 50  0001 C CNN
+AR Path="/609CA6A8/60B0FB21" Ref="#PWR019"  Part="1"
+F 0 "#PWR019" H 3450 4100 50  0001 C CNN
 F 1 "GND1" H 3455 4177 50  0000 C CNN
 F 2 "" H 3450 4350 50  0001 C CNN
@@
 AR Path="/609CA6A8/60A0A500/60B108C7" Ref="#PWR?"  Part="1"
 AR Path="/609CA6A8/60A0A922/60B108C7" Ref="#PWR?"  Part="1"
-AR Path="/609CA6A8/60B108C7" Ref="#PWR035"  Part="1"
-F 0 "#PWR035" H 3450 5100 50  0001 C CNN
+AR Path="/609CA6A8/60B108C7" Ref="#PWR020"  Part="1"
+F 0 "#PWR020" H 3450 5100 50  0001 C CNN
 F 1 "GND1" H 3455 5177 50  0000 C CNN
 F 2 "" H 3450 5350 50  0001 C CNN
@@
 AR Path="/609CA6A8/60A0A500/60B118E3" Ref="#PWR?"  Part="1"
 AR Path="/609CA6A8/60A0A922/60B118E3" Ref="#PWR?"  Part="1"
-AR Path="/609CA6A8/60B118E3" Ref="#PWR036"  Part="1"
-F 0 "#PWR036" H 3450 6100 50  0001 C CNN
+AR Path="/609CA6A8/60B118E3" Ref="#PWR021"  Part="1"
+F 0 "#PWR021" H 3450 6100 50  0001 C CNN
 F 1 "GND1" H 3455 6177 50  0000 C CNN
 F 2 "" H 3450 6350 50  0001 C CNN
@@
 AR Path="/609CA6A8/60A0A500/60B14803" Ref="#PWR?"  Part="1"
 AR Path="/609CA6A8/60A0A922/60B14803" Ref="#PWR?"  Part="1"
-AR Path="/609CA6A8/60B14803" Ref="#PWR048"  Part="1"
-F 0 "#PWR048" H 7650 4450 50  0001 C CNN
+AR Path="/609CA6A8/60B14803" Ref="#PWR033"  Part="1"
+F 0 "#PWR033" H 7650 4450 50  0001 C CNN
 F 1 "GND" H 7655 4527 50  0000 C CNN
 F 2 "" H 7650 4700 50  0001 C CNN
@@
 	7550 4100 7650 4100
 $Comp
-L power:+3V3 #PWR047
+L power:+3V3 #PWR032
 U 1 1 60B1481C
 P 7650 4100
-F 0 "#PWR047" H 7650 3950 50  0001 C CNN
+F 0 "#PWR032" H 7650 3950 50  0001 C CNN
 F 1 "+3V3" H 7665 4273 50  0000 C CNN
 F 2 "" H 7650 4100 50  0001 C CNN
@@
 AR Path="/609CA6A8/60A0A500/60B14823" Ref="#PWR?"  Part="1"
 AR Path="/609CA6A8/60A0A922/60B14823" Ref="#PWR?"  Part="1"
-AR Path="/609CA6A8/60B14823" Ref="#PWR040"  Part="1"
-F 0 "#PWR040" H 6450 4450 50  0001 C CNN
+AR Path="/609CA6A8/60B14823" Ref="#PWR025"  Part="1"
+F 0 "#PWR025" H 6450 4450 50  0001 C CNN
 F 1 "GND1" H 6455 4527 50  0000 C CNN
 F 2 "" H 6450 4700 50  0001 C CNN
@@
 AR Path="/609CA6A8/60A0A500/60B180CF" Ref="#PWR?"  Part="1"
 AR Path="/609CA6A8/60A0A922/60B180CF" Ref="#PWR?"  Part="1"
-AR Path="/609CA6A8/60B180CF" Ref="#PWR050"  Part="1"
-F 0 "#PWR050" H 7650 5700 50  0001 C CNN
+AR Path="/609CA6A8/60B180CF" Ref="#PWR035"  Part="1"
+F 0 "#PWR035" H 7650 5700 50  0001 C CNN
 F 1 "GND" H 7655 5777 50  0000 C CNN
 F 2 "" H 7650 5950 50  0001 C CNN
@@
 	7550 5350 7650 5350
 $Comp
-L power:+3V3 #PWR049
+L power:+3V3 #PWR034
 U 1 1 60B180E8
 P 7650 5350
-F 0 "#PWR049" H 7650 5200 50  0001 C CNN
+F 0 "#PWR034" H 7650 5200 50  0001 C CNN
 F 1 "+3V3" H 7665 5523 50  0000 C CNN
 F 2 "" H 7650 5350 50  0001 C CNN
@@
 AR Path="/609CA6A8/60A0A500/60B180EF" Ref="#PWR?"  Part="1"
 AR Path="/609CA6A8/60A0A922/60B180EF" Ref="#PWR?"  Part="1"
-AR Path="/609CA6A8/60B180EF" Ref="#PWR042"  Part="1"
-F 0 "#PWR042" H 6450 5700 50  0001 C CNN
+AR Path="/609CA6A8/60B180EF" Ref="#PWR027"  Part="1"
+F 0 "#PWR027" H 6450 5700 50  0001 C CNN
 F 1 "GND1" H 6455 5777 50  0000 C CNN
 F 2 "" H 6450 5950 50  0001 C CNN
@@
 AR Path="/609CA6A8/60A0A500/60B43E6A" Ref="#PWR?"  Part="1"
 AR Path="/609CA6A8/60A0A922/60B43E6A" Ref="#PWR?"  Part="1"
-AR Path="/609CA6A8/60B43E6A" Ref="#PWR039"  Part="1"
-F 0 "#PWR039" H 6450 4250 50  0001 C CNN
+AR Path="/609CA6A8/60B43E6A" Ref="#PWR024"  Part="1"
+F 0 "#PWR024" H 6450 4250 50  0001 C CNN
 F 1 "GND1" H 6455 4327 50  0000 C CNN
 F 2 "" H 6450 4500 50  0001 C CNN
@@
 AR Path="/609CA6A8/60A0A500/60B472DC" Ref="#PWR?"  Part="1"
 AR Path="/609CA6A8/60A0A922/60B472DC" Ref="#PWR?"  Part="1"
-AR Path="/609CA6A8/60B472DC" Ref="#PWR041"  Part="1"
-F 0 "#PWR041" H 6450 5500 50  0001 C CNN
+AR Path="/609CA6A8/60B472DC" Ref="#PWR026"  Part="1"
+F 0 "#PWR026" H 6450 5500 50  0001 C CNN
 F 1 "GND1" H 6455 5577 50  0000 C CNN
 F 2 "" H 6450 5750 50  0001 C CNN
@@
 AR Path="/609FED99/60A4EC17" Ref="#PWR?"  Part="1"
 AR Path="/60A364EE/60A4EC17" Ref="#PWR?"  Part="1"
-AR Path="/609CA6A8/60A4EC17" Ref="#PWR051"  Part="1"
-F 0 "#PWR051" H 9600 4250 50  0001 C CNN
+AR Path="/609CA6A8/60A4EC17" Ref="#PWR036"  Part="1"
+F 0 "#PWR036" H 9600 4250 50  0001 C CNN
 F 1 "GND" H 9605 4327 50  0000 C CNN
 F 2 "" H 9600 4500 50  0001 C CNN
@@
 P 9900 4400
 AR Path="/60A364EE/60A4EC11" Ref="J?"  Part="1"
-AR Path="/609CA6A8/60A4EC11" Ref="J11"  Part="1"
-F 0 "J11" H 10008 4681 50  0000 C CNN
+AR Path="/609CA6A8/60A4EC11" Ref="J9"  Part="1"
+F 0 "J9" H 10008 4681 50  0000 C CNN
 F 1 "PLS-3" H 10008 4590 50  0000 C CNN
 F 2 "Connector_PinHeader_2.54mm:PinHeader_1x03_P2.54mm_Vertical" H 9900 4400 50  0001 C CNN
