File: furnace/furnace_controller/furnace_controller.kicad_pcb (KiCad board)
At the start: 2 copper layers, 90 x 100 mm, 153 parts, among them J1 DG141R-2.54-02P, J10 PLS-4R, J11 PLS-5, J12 PLS-3, J13 PLS-5, J14 CTF-11081-P, J2 DG141R-2.54-02P, J3 DG141R-2.54-02P, J4 DG141R-2.54-02P, J5 DG141R-2.54-02P, J6 IDC-6, J7 FPC-24P 0.5mm, J8 PLS-10R, J9 PLS-3, Q1 BC847, Q2 IRLML6402, Q3 IRLML2402, Q4 BC847, Q5 IRLML6402, Q6 BC847, Q7 BC847, U1 AMS1117-3.3, U10 ADuM1301, U11 STM32F103C6Tx, U2 MAX31855EASA, U3 ADuM1301, U4 LM317L_SO8, U5 MAX31855EASA, U6 MAX31855EASA, U7 MAX31855EASA, U8 MAX31855EASA, U9 ADuM1301, Y1 8MHz

Commit message: Add files via upload
Parts:
- added H4: MountingHole, furnace_controller:hole_D3.5mm, F.Cu at (10.0, 5.00)
- added H5: MountingHole, furnace_controller:hole_D3.5mm, F.Cu at (80.0, 5.00)
- J8: footprint Connector_PinHeader_2.54mm:PinHeader_1x10_P2.54mm_Horizontal -> Connector_PinHeader_2.54mm:PinHeader_1x10_P2.54mm_Vertical
- moved BZ1 89.1 mm to (70.0, 13.5), turned to 0 degrees
- moved Q6 81.1 mm to (75.0, 23.5), turned to 0 degrees
- moved G1 76.9 mm to (12.0, 54.5)
- moved R43 75.4 mm to (71.0, 23.4), turned to 270 degrees
- moved R42 72.8 mm to (68.1, 22.5), turned to 0 degrees
- moved R53 69.3 mm to (30.0, 62.9)
- moved R54 66.1 mm to (32.0, 62.9)
- moved R56 63.0 mm to (34.0, 62.9)
- moved R55 53.8 mm to (36.0, 62.9), turned to 90 degrees
- moved J14 52.5 mm to (38.0, 52.0), turned to 90 degrees
- moved J12 46.8 mm to (14.4, 63.0)
- moved C44 46.4 mm to (42.0, 50.1), turned to 90 degrees
- moved TP2 45.6 mm to (29.0, 95.5)
- moved C45 44.9 mm to (42.0, 56.1), turned to 270 degrees
- moved R52 40.9 mm to (12.9, 87.5), turned to 0 degrees
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Connections:
- C34 pad 1: /MCU/UART1_RX -> /MCU/UART2_RX
- J1 pad 1: /TC-0 -> /TC+0
- J1 pad 2: /TC+0 -> /TC-0
- J12 pad 1: /MCU/UART1_TX -> /MCU/UART2_TX
- J12 pad 2: /MCU/UART1_RX -> /MCU/UART2_RX
- J2 pad 1: /TC-1 -> /TC+1
- J2 pad 2: /TC+1 -> /TC-1
- J3 pad 1: /TC-2 -> /TC+2
- J3 pad 2: /TC+2 -> /TC-2
- J4 pad 1: /TC-3 -> /TC+3
- J4 pad 2: /TC+3 -> /TC-3
- J5 pad 1: /TC-4 -> /TC+4
- J5 pad 2: /TC+4 -> /TC-4
- R47 pad 2: /MCU/UART1_RX -> /MCU/UART2_RX
- R50 pad 1: /MCU/UART1_TX -> /MCU/UART2_TX
- U10 pad 12: GND1 -> /ISOLATED_TEMP_SENSOR/ISOLATOR2/INC
- U10 pad 3: /ISOLATED_TEMP_SENSOR/~CS3 -> /ISOLATED_TEMP_SENSOR/~CS4
- U10 pad 4: /ISOLATED_TEMP_SENSOR/~CS4 -> /ISOLATED_TEMP_SENSOR/SCK
- U10 pad 5: /ISOLATED_TEMP_SENSOR/ISOLATOR2/OUTC -> /ISOLATED_TEMP_SENSOR/MISO
- U11 pad 10: /ISOLATED_TEMP_SENSOR/~CS0 -> /KEYBOARD_CONNECTOR/KYBD6
- U11 pad 11: /ISOLATED_TEMP_SENSOR/~CS1 -> /MCU/CHARGE_PUMP_CLK
- U11 pad 12: /ISOLATED_TEMP_SENSOR/~CS2 -> /MCU/UART2_TX
- U11 pad 13: /ISOLATED_TEMP_SENSOR/~CS3 -> /MCU/UART2_RX
- U11 pad 14: /ISOLATED_TEMP_SENSOR/~CS4 -> /MICRO_SD_CARD/CARD_DET
- U11 pad 15: /ISOLATED_TEMP_SENSOR/SCK -> /MICRO_SD_CARD/SCK
- U11 pad 16: /ISOLATED_TEMP_SENSOR/MISO -> /MICRO_SD_CARD/MISO
- U11 pad 17: /KEYBOARD_CONNECTOR/KYBD2 -> /MICRO_SD_CARD/MOSI
- U11 pad 18: /MCU/BZ_EN -> /MICRO_SD_CARD/~CS~
- U11 pad 19: /KEYBOARD_CONNECTOR/KYBD9 -> /ISOLATED_TEMP_SENSOR/~CS2
- U11 pad 20: /MICRO_SD_CARD/CARD_DET -> /ISOLATED_TEMP_SENSOR/~CS3
- U11 pad 21: /KEYBOARD_CONNECTOR/KYBD5 -> /ISOLATED_TEMP_SENSOR/~CS0
- U11 pad 22: /KEYBOARD_CONNECTOR/KYBD4 -> /ISOLATED_TEMP_SENSOR/~CS1
- U11 pad 25: /MICRO_SD_CARD/~CS~ -> /KEYBOARD_CONNECTOR/KYBD0
- U11 pad 26: /MICRO_SD_CARD/SCK -> /ISOLATED_TEMP_SENSOR/SCK
- U11 pad 27: /MICRO_SD_CARD/MISO -> /ISOLATED_TEMP_SENSOR/MISO
- U11 pad 28: /MICRO_SD_CARD/MOSI -> /ISOLATED_TEMP_SENSOR/~CS4
- U11 pad 29: /MCU/CHARGE_PUMP_CLK -> /KEYBOARD_CONNECTOR/KYBD1
- U11 pad 30: /MCU/UART1_TX -> /KEYBOARD_CONNECTOR/KYBD2
- U11 pad 31: /MCU/UART1_RX -> /KEYBOARD_CONNECTOR/KYBD3
- U11 pad 32: /KEYBOARD_CONNECTOR/KYBD1 -> /KEYBOARD_CONNECTOR/KYBD4
- U11 pad 33: /KEYBOARD_CONNECTOR/KYBD0 -> /KEYBOARD_CONNECTOR/KYBD5
- U11 pad 38: /KEYBOARD_CONNECTOR/KYBD3 -> /MCU/BZ_EN
- U11 pad 39: /KEYBOARD_CONNECTOR/KYBD8 -> /MCU/~DPY_RST
- U11 pad 40: /KEYBOARD_CONNECTOR/KYBD7 -> /KEYBOARD_CONNECTOR/KYBD9
- U11 pad 41: /MCU/~DPY_RST -> /KEYBOARD_CONNECTOR/KYBD8
- U11 pad 46: /KEYBOARD_CONNECTOR/KYBD6 -> /KEYBOARD_CONNECTOR/KYBD7
- U2 pad 5: /ISOLATED_TEMP_SENSOR/ISOLATOR0/OUTA -> /ISOLATED_TEMP_SENSOR/ISOLATOR2/OUTB
- U2 pad 7: /ISOLATED_TEMP_SENSOR/ISOLATOR0/INC -> /ISOLATED_TEMP_SENSOR/ISOLATOR2/INC
- U3 pad 12: /ISOLATED_TEMP_SENSOR/ISOLATOR0/INC -> GND1
- U3 pad 3: /ISOLATED_TEMP_SENSOR/SCK -> /ISOLATED_TEMP_SENSOR/~CS0
- U3 pad 4: /ISOLATED_TEMP_SENSOR/~CS0 -> /ISOLATED_TEMP_SENSOR/~CS1
- U3 pad 5: /ISOLATED_TEMP_SENSOR/MISO -> /ISOLATED_TEMP_SENSOR/ISOLATOR0/OUTC
- U5 pad 5: /ISOLATED_TEMP_SENSOR/ISOLATOR0/OUTA -> /ISOLATED_TEMP_SENSOR/ISOLATOR2/OUTB
- U5 pad 6: /ISOLATED_TEMP_SENSOR/ISOLATOR1/OUTA -> /ISOLATED_TEMP_SENSOR/ISOLATOR0/OUTA
- U5 pad 7: /ISOLATED_TEMP_SENSOR/ISOLATOR0/INC -> /ISOLATED_TEMP_SENSOR/ISOLATOR2/INC
- U6 pad 5: /ISOLATED_TEMP_SENSOR/ISOLATOR0/OUTA -> /ISOLATED_TEMP_SENSOR/ISOLATOR2/OUTB
- U6 pad 7: /ISOLATED_TEMP_SENSOR/ISOLATOR0/INC -> /ISOLATED_TEMP_SENSOR/ISOLATOR2/INC
- U7 pad 5: /ISOLATED_TEMP_SENSOR/ISOLATOR0/OUTA -> /ISOLATED_TEMP_SENSOR/ISOLATOR2/OUTB
- U7 pad 6: /ISOLATED_TEMP_SENSOR/ISOLATOR2/OUTA -> /ISOLATED_TEMP_SENSOR/ISOLATOR1/OUTA
- U7 pad 7: /ISOLATED_TEMP_SENSOR/ISOLATOR0/INC -> /ISOLATED_TEMP_SENSOR/ISOLATOR2/INC
- U8 pad 5: /ISOLATED_TEMP_SENSOR/ISOLATOR0/OUTA -> /ISOLATED_TEMP_SENSOR/ISOLATOR2/OUTB
- U8 pad 6: /ISOLATED_TEMP_SENSOR/ISOLATOR2/OUTB -> /ISOLATED_TEMP_SENSOR/ISOLATOR2/OUTA
- U8 pad 7: /ISOLATED_TEMP_SENSOR/ISOLATOR0/INC -> /ISOLATED_TEMP_SENSOR/ISOLATOR2/INC
- U9 pad 3: /ISOLATED_TEMP_SENSOR/~CS1 -> /ISOLATED_TEMP_SENSOR/~CS2
- U9 pad 4: /ISOLATED_TEMP_SENSOR/~CS2 -> /ISOLATED_TEMP_SENSOR/~CS3
Routing:
- net +3V3: track 0.00 -> 320.0 mm, vias 0 -> 28
- net +5V: track 0.00 -> 219.3 mm, vias 0 -> 7
- net /ISOLATED_TEMP_SENSOR/+3V3_ISO: track 0.00 -> 163.2 mm, vias 0 -> 12
- net /MCU/UART2_TX: track 0.00 -> 73.2 mm
- net /ISOLATED_TEMP_SENSOR/ISOLATOR2/INC: track 0.00 -> 59.6 mm, vias 0 -> 6
- net /MCU/UART2_RX: track 0.00 -> 56.0 mm
- net /ISOLATED_TEMP_SENSOR/ISOLATOR2/OUTB: track 0.00 -> 51.8 mm
- net /ISOLATED_TEMP_SENSOR/~CS1: track 0.00 -> 48.8 mm
- net /ISOLATED_TEMP_SENSOR/~CS0: track 0.00 -> 47.1 mm
- net /MICRO_SD_CARD/CARD_DET: track 0.00 -> 42.6 mm
- net /KEYBOARD_CONNECTOR/KYBD5: track 0.00 -> 41.8 mm, vias 0 -> 2
- net /MICRO_SD_CARD/MISO: track 0.00 -> 41.6 mm
- net /KEYBOARD_CONNECTOR/KYBD4: track 0.00 -> 40.5 mm, vias 0 -> 2
- net /KEYBOARD_CONNECTOR/KYBD3: track 0.00 -> 39.8 mm, vias 0 -> 2
- net /KEYBOARD_CONNECTOR/KYBD2: track 0.00 -> 39.1 mm, vias 0 -> 2
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- added copper zone on B.Cu, net GND
- added copper zone on F.Cu, net GND
- added copper zone on B.Cu, net GND1
- added copper zone on F.Cu, net GND1
Other:
- board size 90 x 100 mm -> 88 x 100 mm
- board text added: "-0+"
- board text added: "-1+"
- board text added: "-2+"
- board text added: "-3+"
- board text added: "-4+"
- board text added: "0"
- board text added: "9"
- board text added: "SCK SDA VCC GND"
- board text added: "furnace controller 1.0"
- board text added: "keyboard"
- board text added: "thermocouple type k"
