File: furnace/furnace_230V/Current_sensor.sch (KiCad schematic (older format))
At the start: 0 parts

Commit message: Add files via upload
Parts:
- added C?: 0,1, Capacitor_SMD:C_0603_1608Metric_Pad1.08x0.95mm_HandSolder, symbol Device:C
- added D?: BAT54S, Package_TO_SOT_SMD:SOT-23, symbol Diode:BAT54S
- added L?: L, symbol Device:L
- added R?: 680, Resistor_SMD:R_0603_1608Metric_Pad0.98x0.95mm_HandSolder, symbol Device:R
- added R? (x2): 100, Resistor_SMD:R_0603_1608Metric_Pad1.05x0.95mm_HandSolder, symbol Device:R
- added TP? (x2): TestPoint, symbol Connector:TestPoint
Changed lines of the file:
@@
 $Descr A4 11693 8268
 encoding utf-8
-Sheet 1 9
+Sheet 7 9
 Title ""
 Date ""
@@
 Comment4 ""
 $EndDescr
+$Comp
+L Device:L L?
+U 1 1 60AC7E83
+P 5650 4300
+F 0 "L?" V 5840 4300 50  0000 C CNN
+F 1 "L" V 5749 4300 50  0000 C CNN
+F 2 "" H 5650 4300 50  0001 C CNN
+F 3 "~" H 5650 4300 50  0001 C CNN
+	1    5650 4300
+	0    -1   -1   0
+$EndComp
+$Comp
+L Device:R R?
+U 1 1 60AC8E28
+P 6050 4500
+AR Path="/60AC8E28" Ref="R?"  Part="1"
+AR Path="/609CA6A8/60AC8E28" Ref="R?"  Part="1"
+AR Path="/609CA6A8/60AE5653/60AC8E28" Ref="R?"  Part="1"
+AR Path="/60AAC605/60AC8E28" Ref="R?"  Part="1"
+AR Path="/60AAE212/60AC8E28" Ref="R?"  Part="1"
+F 0 "R?" H 6120 4546 50  0000 L CNN
+F 1 "680" H 6120 4455 50  0000 L CNN
+F 2 "Resistor_SMD:R_0603_1608Metric_Pad0.98x0.95mm_HandSolder" V 5980 4500 50  0001 C CNN
+F 3 "~" H 6050 4500 50  0001 C CNN
+	1    6050 4500
+	1    0    0    -1
+$EndComp
+$Comp
+L Device:R R?
+U 1 1 60AC9714
+P 7600 4250
+AR Path="/60AAE0B8/60AC9714" Ref="R?"  Part="1"
+AR Path="/60AAEC6C/60AC9714" Ref="R?"  Part="1"
+AR Path="/60AAE4BD/60AC9714" Ref="R?"  Part="1"
+AR Path="/60AAE212/60AC9714" Ref="R?"  Part="1"
+F 0 "R?" V 7393 4250 50  0000 C CNN
+F 1 "100" V 7484 4250 50  0000 C CNN
+F 2 "Resistor_SMD:R_0603_1608Metric_Pad1.05x0.95mm_HandSolder" V 7530 4250 50  0001 C CNN
+F 3 "~" H 7600 4250 50  0001 C CNN
+	1    7600 4250
+	0    1    1    0
+$EndComp
+$Comp
+L Device:C C?
+U 1 1 60AC971A
+P 8200 4500
+AR Path="/60AC971A" Ref="C?"  Part="1"
+AR Path="/609CA6A8/609D24C0/60AC971A" Ref="C?"  Part="1"
+AR Path="/609CA6A8/60A08E0B/60AC971A" Ref="C?"  Part="1"
+AR Path="/609CA6A8/60A0A46E/60AC971A" Ref="C?"  Part="1"
+AR Path="/609CA6A8/60A0A500/60AC971A" Ref="C?"  Part="1"
+AR Path="/609CA6A8/60A0A922/60AC971A" Ref="C?"  Part="1"
+AR Path="/609CA6A8/60AC971A" Ref="C?"  Part="1"
+AR Path="/609CA6A8/60AE5653/60AC971A" Ref="C?"  Part="1"
+AR Path="/60AAC605/60AC971A" Ref="C?"  Part="1"
+AR Path="/60AAE4BD/60AC971A" Ref="C?"  Part="1"
+AR Path="/60AAE212/60AC971A" Ref="C?"  Part="1"
+F 0 "C?" H 8315 4546 50  0000 L CNN
+F 1 "0,1" H 8315 4455 50  0000 L CNN
+F 2 "Capacitor_SMD:C_0603_1608Metric_Pad1.08x0.95mm_HandSolder" H 8238 4350 50  0001 C CNN
+F 3 "~" H 8200 4500 50  0001 C CNN
+	1    8200 4500
+	1    0    0    -1
+$EndComp
+$Comp
+L Device:R R?
+U 1 1 60ACAD1A
+P 6250 4250
+AR Path="/60AAE0B8/60ACAD1A" Ref="R?"  Part="1"
+AR Path="/60AAEC6C/60ACAD1A" Ref="R?"  Part="1"
+AR Path="/60AAE4BD/60ACAD1A" Ref="R?"  Part="1"
+AR Path="/60AAE212/60ACAD1A" Ref="R?"  Part="1"
+F 0 "R?" V 6043 4250 50  0000 C CNN
+F 1 "100" V 6134 4250 50  0000 C CNN
+F 2 "Resistor_SMD:R_0603_1608Metric_Pad1.05x0.95mm_HandSolder" V 6180 4250 50  0001 C CNN
+F 3 "~" H 6250 4250 50  0001 C CNN
+	1    6250 4250
+	0    1    1    0
+$EndComp
+$Comp
+L Diode:BAT54S D?
+U 1 1 60ACAD20
+P 6900 4250
+F 0 "D?" V 6946 4338 50  0000 L CNN
+F 1 "BAT54S" V 6855 4338 50  0000 L CNN
+F 2 "Package_TO_SOT_SMD:SOT-23" H 6975 4375 50  0001 L CNN
+F 3 "https://www.diodes.com/assets/Datasheets/ds11005.pdf" H 6780 4250 50  0001 C CNN
+	1    6900 4250
+	0    -1   -1   0
+$EndComp
+$Comp
+L Connector:TestPoint TP?
+U 1 1 60ACFCB9
+P 5950 4250
+AR Path="/60ACFCB9" Ref="TP?"  Part="1"
+AR Path="/609CA6A8/60AE5653/60ACFCB9" Ref="TP?"  Part="1"
+AR Path="/60AAC605/60ACFCB9" Ref="TP?"  Part="1"
+AR Path="/60AAE212/60ACFCB9" Ref="TP?"  Part="1"
+F 0 "TP?" H 6008 4368 50  0000 L CNN
+F 1 "TestPoint" H 6008 4277 50  0001 L CNN
+F 2 "" H 6150 4250 50  0001 C CNN
+F 3 "~" H 6150 4250 50  0001 C CNN
+	1    5950 4250
+	1    0    0    -1
+$EndComp
+$Comp
+L Connector:TestPoint TP?
+U 1 1 60ACFF73
+P 8000 4250
+AR Path="/60ACFF73" Ref="TP?"  Part="1"
+AR Path="/609CA6A8/60AE5653/60ACFF73" Ref="TP?"  Part="1"
+AR Path="/60AAC605/60ACFF73" Ref="TP?"  Part="1"
+AR Path="/60AAE212/60ACFF73" Ref="TP?"  Part="1"
+F 0 "TP?" H 8058 4368 50  0000 L CNN
+F 1 "TestPoint" H 8058 4277 50  0001 L CNN
+F 2 "" H 8200 4250 50  0001 C CNN
+F 3 "~" H 8200 4250 50  0001 C CNN
+	1    8000 4250
+	1    0    0    -1
+$EndComp
 $EndSCHEMATC
