File: furnace/furnace_230V/Voltage_divider.sch (KiCad schematic (older format))
At the start: 0 parts

Commit message: Add files via upload
Parts:
- added C? (x2): 100, Capacitor_SMD:C_0603_1608Metric_Pad1.08x0.95mm_HandSolder, symbol Device:C
- added C?: 10u, Capacitor_SMD:C_0603_1608Metric_Pad1.08x0.95mm_HandSolder, symbol Device:C
- added D?: BAT54S, Package_TO_SOT_SMD:SOT-23, symbol Diode:BAT54S
- added D?: D_TVS, symbol Device:D_TVS
- added D?: ES1J, symbol Device:D
- added R? (x2): 180k 0,25W 1%, symbol Device:R
- added R?: 100, Resistor_SMD:R_0603_1608Metric_Pad1.05x0.95mm_HandSolder, symbol Device:R
- added R?: 1k, Resistor_SMD:R_0603_1608Metric_Pad1.05x0.95mm_HandSolder, symbol Device:R
- added R?: 3,3k 1%, Resistor_SMD:R_0603_1608Metric_Pad0.98x0.95mm_HandSolder, symbol Device:R
- added TP? (x3): TestPoint, symbol Connector:TestPoint
Connections:
- net labels added: +3V3, AC1, AC2, GND, VOLT
- wire segments 0 -> 33
Other:
- note added: "Input 230V voltage mesurement circuit"
