File: furnace/furnace_230V/+3V3_isolated.sch (KiCad schematic (older format))
At the start: 13 parts

Commit message: Add files via upload
Parts:
- C10, C11, C12, C8, C9: renamed from C?; symbol Device:C -> furnace_230V-rescue:C-Device
- PS2: renamed from PS?; footprint CONV_B0505S-1WR2 -> (none)
- R2, R3, R4, R5: renamed from R?; symbol Device:R -> furnace_230V-rescue:R-Device
- TP4, TP5: renamed from TP?; symbol Connector:TestPoint -> furnace_230V-rescue:TestPoint-Connector
- gave numbers to parts that had none: 1
Changed lines of the file:
@@
 AR Path="/609CA6A8/60AE766F" Ref="PS?"  Part="1"
 AR Path="/609CA6A8/60AE5653/60AE766F" Ref="PS?"  Part="1"
-AR Path="/60AAC605/60AE766F" Ref="PS?"  Part="1"
-F 0 "PS?" H 4050 3967 50  0000 C CNN
+AR Path="/60AAC605/60AE766F" Ref="PS2"  Part="1"
+F 0 "PS2" H 4050 3967 50  0000 C CNN
 F 1 "B0505S-1WR2" H 4050 3876 50  0000 C CNN
-F 2 "CONV_B0505S-1WR2" H 4050 3600 50  0001 L BNN
+F 2 "" H 4050 3600 50  0001 L BNN
 F 3 "" H 4050 3600 50  0001 L BNN
 F 4 "Manufacturer Recommendations" H 4050 3600 50  0001 L BNN "STANDARD"
@@
 $EndComp
 $Comp
-L Device:C C?
+L furnace_230V-rescue:C-Device C?
 U 1 1 60AE7675
 P 6250 3650
@@
 AR Path="/609CA6A8/60AE7675" Ref="C?"  Part="1"
 AR Path="/609CA6A8/60AE5653/60AE7675" Ref="C?"  Part="1"
-AR Path="/60AAC605/60AE7675" Ref="C?"  Part="1"
-F 0 "C?" H 6365 3696 50  0000 L CNN
+AR Path="/60AAC605/60AE7675" Ref="C10"  Part="1"
+F 0 "C10" H 6365 3696 50  0000 L CNN
 F 1 "0,1" H 6365 3605 50  0000 L CNN
 F 2 "Capacitor_SMD:C_0603_1608Metric_Pad1.08x0.95mm_HandSolder" H 6288 3500 50  0001 C CNN
@@
 $EndComp
 $Comp
-L Device:C C?
+L furnace_230V-rescue:C-Device C?
 U 1 1 60AE767B
 P 3250 3650
@@
 AR Path="/609CA6A8/60AE767B" Ref="C?"  Part="1"
 AR Path="/609CA6A8/60AE5653/60AE767B" Ref="C?"  Part="1"
-AR Path="/60AAC605/60AE767B" Ref="C?"  Part="1"
-F 0 "C?" H 3365 3696 50  0000 L CNN
+AR Path="/60AAC605/60AE767B" Ref="C8"  Part="1"
+F 0 "C8" H 3365 3696 50  0000 L CNN
 F 1 "4,7" H 3365 3605 50  0000 L CNN
 F 2 "Capacitor_SMD:C_1206_3216Metric_Pad1.33x1.80mm_HandSolder" H 3288 3500 50  0001 C CNN
@@
 $EndComp
 $Comp
-L Device:C C?
+L furnace_230V-rescue:C-Device C?
 U 1 1 60AE7681
 P 4750 3650
@@
 AR Path="/609CA6A8/60AE7681" Ref="C?"  Part="1"
 AR Path="/609CA6A8/60AE5653/60AE7681" Ref="C?"  Part="1"
-AR Path="/60AAC605/60AE7681" Ref="C?"  Part="1"
-F 0 "C?" H 4865 3696 50  0000 L CNN
+AR Path="/60AAC605/60AE7681" Ref="C9"  Part="1"
+F 0 "C9" H 4865 3696 50  0000 L CNN
 F 1 "10u" H 4865 3605 50  0000 L CNN
 F 2 "Capacitor_SMD:C_1206_3216Metric_Pad1.33x1.80mm_HandSolder" H 4788 3500 50  0001 C CNN
@@
 	3550 3800 3550 3700
 $Comp
-L Device:R R?
+L furnace_230V-rescue:R-Device R?
 U 1 1 60AE7692
 P 5150 3650
@@
 AR Path="/609CA6A8/60AE7692" Ref="R?"  Part="1"
 AR Path="/609CA6A8/60AE5653/60AE7692" Ref="R?"  Part="1"
-AR Path="/60AAC605/60AE7692" Ref="R?"  Part="1"
-F 0 "R?" H 5220 3696 50  0000 L CNN
+AR Path="/60AAC605/60AE7692" Ref="R2"  Part="1"
+F 0 "R2" H 5220 3696 50  0000 L CNN
 F 1 "680" H 5220 3605 50  0000 L CNN
 F 2 "Resistor_SMD:R_0603_1608Metric_Pad0.98x0.95mm_HandSolder" V 5080 3650 50  0001 C CNN
@@
 $EndComp
 $Comp
-L Device:R R?
+L furnace_230V-rescue:R-Device R?
 U 1 1 60AE7698
 P 5550 3650
@@
 AR Path="/609CA6A8/60AE7698" Ref="R?"  Part="1"
 AR Path="/609CA6A8/60AE5653/60AE7698" Ref="R?"  Part="1"
-AR Path="/60AAC605/60AE7698" Ref="R?"  Part="1"
-F 0 "R?" H 5620 3696 50  0000 L CNN
+AR Path="/60AAC605/60AE7698" Ref="R3"  Part="1"
+F 0 "R3" H 5620 3696 50  0000 L CNN
 F 1 "680" H 5620 3605 50  0000 L CNN
 F 2 "Resistor_SMD:R_0603_1608Metric_Pad0.98x0.95mm_HandSolder" V 5480 3650 50  0001 C CNN
@@
 $EndComp
 $Comp
-L Device:C C?
+L furnace_230V-rescue:C-Device C?
 U 1 1 60AE769E
 P 8100 3650
@@
 AR Path="/609CA6A8/60AE769E" Ref="C?"  Part="1"
 AR Path="/609CA6A8/60AE5653/60AE769E" Ref="C?"  Part="1"
-AR Path="/60AAC605/60AE769E" Ref="C?"  Part="1"
-F 0 "C?" H 8215 3696 50  0000 L CNN
+AR Path="/60AAC605/60AE769E" Ref="C12"  Part="1"
+F 0 "C12" H 8215 3696 50  0000 L CNN
 F 1 "1u" H 8215 3605 50  0000 L CNN
 F 2 "Capacitor_SMD:C_0603_1608Metric_Pad1.08x0.95mm_HandSolder" H 8138 3500 50  0001 C CNN
@@
 $EndComp
 $Comp
-L Device:C C?
+L furnace_230V-rescue:C-Device C?
 U 1 1 60AE76A4
 P 6900 4050
@@
 AR Path="/609CA6A8/60AE76A4" Ref="C?"  Part="1"
 AR Path="/609CA6A8/60AE5653/60AE76A4" Ref="C?"  Part="1"
-AR Path="/60AAC605/60AE76A4" Ref="C?"  Part="1"
-F 0 "C?" H 7015 4096 50  0000 L CNN
+AR Path="/60AAC605/60AE76A4" Ref="C11"  Part="1"
+F 0 "C11" H 7015 4096 50  0000 L CNN
 F 1 "10u" H 7015 4005 50  0000 L CNN
 F 2 "Capacitor_SMD:C_1206_3216Metric_Pad1.33x1.80mm_HandSolder" H 6938 3900 50  0001 C CNN
@@
 $EndComp
 $Comp
-L Device:R R?
+L furnace_230V-rescue:R-Device R?
 U 1 1 60AE76AA
 P 7500 3650
@@
 AR Path="/609CA6A8/60AE76AA" Ref="R?"  Part="1"
 AR Path="/609CA6A8/60AE5653/60AE76AA" Ref="R?"  Part="1"
-AR Path="/60AAC605/60AE76AA" Ref="R?"  Part="1"
-F 0 "R?" H 7570 3696 50  0000 L CNN
+AR Path="/60AAC605/60AE76AA" Ref="R4"  Part="1"
+F 0 "R4" H 7570 3696 50  0000 L CNN
 F 1 "240 1%" H 7570 3605 50  0000 L CNN
 F 2 "Resistor_SMD:R_0603_1608Metric_Pad0.98x0.95mm_HandSolder" V 7430 3650 50  0001 C CNN
@@
 $EndComp
 $Comp
-L Device:R R?
+L furnace_230V-rescue:R-Device R?
 U 1 1 60AE76B0
 P 7500 4050
@@
 AR Path="/609CA6A8/60AE76B0" Ref="R?"  Part="1"
 AR Path="/609CA6A8/60AE5653/60AE76B0" Ref="R?"  Part="1"
-AR Path="/60AAC605/60AE76B0" Ref="R?"  Part="1"
-F 0 "R?" H 7570 4096 50  0000 L CNN
+AR Path="/60AAC605/60AE76B0" Ref="R5"  Part="1"
+F 0 "R5" H 7570 4096 50  0000 L CNN
 F 1 "390 1%" H 7570 4005 50  0000 L CNN
 F 2 "Resistor_SMD:R_0603_1608Metric_Pad0.98x0.95mm_HandSolder" V 7430 4050 50  0001 C CNN
@@
 AR Path="/609CA6A8/60AE76B8" Ref="U?"  Part="1"
 AR Path="/609CA6A8/60AE5653/60AE76B8" Ref="U?"  Part="1"
-AR Path="/60AAC605/60AE76B8" Ref="U?"  Part="1"
-F 0 "U?" H 6900 3742 50  0000 C CNN
+AR Path="/60AAC605/60AE76B8" Ref="U2"  Part="1"
+F 0 "U2" H 6900 3742 50  0000 C CNN
 F 1 "LM317L_SO8" H 6900 3651 50  0000 C CNN
 F 2 "Package_SO:SOIC-8_3.9x4.9mm_P1.27mm" H 6900 3700 50  0001 C CIN
@@
 Connection ~ 3250 3800
 $Comp
-L Connector:TestPoint TP?
+L furnace_230V-rescue:TestPoint-Connector TP?
 U 1 1 60B566B5
 P 8550 4200
 AR Path="/60B566B5" Ref="TP?"  Part="1"
 AR Path="/609CA6A8/60AE5653/60B566B5" Ref="TP?"  Part="1"
-AR Path="/60AAC605/60B566B5" Ref="TP?"  Part="1"
-F 0 "TP?" H 8608 4318 50  0000 L CNN
+AR Path="/60AAC605/60B566B5" Ref="TP5"  Part="1"
+F 0 "TP5" H 8608 4318 50  0000 L CNN
 F 1 "TestPoint" H 8608 4227 50  0001 L CNN
 F 2 "" H 8750 4200 50  0001 C CNN
@@
 $EndComp
 $Comp
-L Connector:TestPoint TP?
+L furnace_230V-rescue:TestPoint-Connector TP?
 U 1 1 60B56DD4
 P 8550 3500
 AR Path="/60B56DD4" Ref="TP?"  Part="1"
 AR Path="/609CA6A8/60AE5653/60B56DD4" Ref="TP?"  Part="1"
-AR Path="/60AAC605/60B56DD4" Ref="TP?"  Part="1"
-F 0 "TP?" H 8608 3618 50  0000 L CNN
+AR Path="/60AAC605/60B56DD4" Ref="TP4"  Part="1"
+F 0 "TP4" H 8608 3618 50  0000 L CNN
 F 1 "TestPoint" H 8608 3527 50  0001 L CNN
 F 2 "" H 8750 3500 50  0001 C CNN

Commit message: Add files via upload
Parts:
- TP4, TP5: footprint (none) -> MountingHole:MountingHole_2.2mm_M2_DIN965_Pad_TopBottom
Changed lines of the file:
@@
 F 0 "TP5" H 8608 4318 50  0000 L CNN
 F 1 "TestPoint" H 8608 4227 50  0001 L CNN
-F 2 "" H 8750 4200 50  0001 C CNN
+F 2 "MountingHole:MountingHole_2.2mm_M2_DIN965_Pad_TopBottom" H 8750 4200 50  0001 C CNN
 F 3 "~" H 8750 4200 50  0001 C CNN
 	1    8550 4200
@@
 F 0 "TP4" H 8608 3618 50  0000 L CNN
 F 1 "TestPoint" H 8608 3527 50  0001 L CNN
-F 2 "" H 8750 3500 50  0001 C CNN
+F 2 "MountingHole:MountingHole_2.2mm_M2_DIN965_Pad_TopBottom" H 8750 3500 50  0001 C CNN
 F 3 "~" H 8750 3500 50  0001 C CNN
 	1    8550 3500

Commit message: Add files via upload
Parts:
- C10, C12: footprint Capacitor_SMD:C_0603_1608Metric_Pad1.08x0.95mm_HandSolder -> Capacitor_SMD:C_0603_1608Metric_Pad1.05x0.95mm_HandSolder
- C11, C8, C9: footprint Capacitor_SMD:C_1206_3216Metric_Pad1.33x1.80mm_HandSolder -> Capacitor_SMD:C_1206_3216Metric_Pad1.42x1.75mm_HandSolder
- PS2: footprint (none) -> furnace_230V:B_S-1WR3
- R2, R3, R4, R5: footprint Resistor_SMD:R_0603_1608Metric_Pad0.98x0.95mm_HandSolder -> Resistor_SMD:R_0603_1608Metric_Pad1.05x0.95mm_HandSolder
- TP4, TP5: footprint MountingHole:MountingHole_2.2mm_M2_DIN965_Pad_TopBottom -> furnace_230V:TP
Changed lines of the file:
@@
 F 0 "PS2" H 4050 3967 50  0000 C CNN
 F 1 "B0505S-1WR2" H 4050 3876 50  0000 C CNN
-F 2 "" H 4050 3600 50  0001 L BNN
+F 2 "furnace_230V:B_S-1WR3" H 4050 3600 50  0001 L BNN
 F 3 "" H 4050 3600 50  0001 L BNN
 F 4 "Manufacturer Recommendations" H 4050 3600 50  0001 L BNN "STANDARD"
@@
 F 0 "C10" H 6365 3696 50  0000 L CNN
 F 1 "0,1" H 6365 3605 50  0000 L CNN
-F 2 "Capacitor_SMD:C_0603_1608Metric_Pad1.08x0.95mm_HandSolder" H 6288 3500 50  0001 C CNN
+F 2 "Capacitor_SMD:C_0603_1608Metric_Pad1.05x0.95mm_HandSolder" H 6288 3500 50  0001 C CNN
 F 3 "~" H 6250 3650 50  0001 C CNN
 	1    6250 3650
@@
 F 0 "C8" H 3365 3696 50  0000 L CNN
 F 1 "4,7" H 3365 3605 50  0000 L CNN
-F 2 "Capacitor_SMD:C_1206_3216Metric_Pad1.33x1.80mm_HandSolder" H 3288 3500 50  0001 C CNN
+F 2 "Capacitor_SMD:C_1206_3216Metric_Pad1.42x1.75mm_HandSolder" H 3288 3500 50  0001 C CNN
 F 3 "~" H 3250 3650 50  0001 C CNN
 	1    3250 3650
@@
 F 0 "C9" H 4865 3696 50  0000 L CNN
 F 1 "10u" H 4865 3605 50  0000 L CNN
-F 2 "Capacitor_SMD:C_1206_3216Metric_Pad1.33x1.80mm_HandSolder" H 4788 3500 50  0001 C CNN
+F 2 "Capacitor_SMD:C_1206_3216Metric_Pad1.42x1.75mm_HandSolder" H 4788 3500 50  0001 C CNN
 F 3 "~" H 4750 3650 50  0001 C CNN
 	1    4750 3650
@@
 F 0 "R2" H 5220 3696 50  0000 L CNN
 F 1 "680" H 5220 3605 50  0000 L CNN
-F 2 "Resistor_SMD:R_0603_1608Metric_Pad0.98x0.95mm_HandSolder" V 5080 3650 50  0001 C CNN
+F 2 "Resistor_SMD:R_0603_1608Metric_Pad1.05x0.95mm_HandSolder" V 5080 3650 50  0001 C CNN
 F 3 "~" H 5150 3650 50  0001 C CNN
 	1    5150 3650
@@
 F 0 "R3" H 5620 3696 50  0000 L CNN
 F 1 "680" H 5620 3605 50  0000 L CNN
-F 2 "Resistor_SMD:R_0603_1608Metric_Pad0.98x0.95mm_HandSolder" V 5480 3650 50  0001 C CNN
+F 2 "Resistor_SMD:R_0603_1608Metric_Pad1.05x0.95mm_HandSolder" V 5480 3650 50  0001 C CNN
 F 3 "~" H 5550 3650 50  0001 C CNN
 	1    5550 3650
@@
 F 0 "C12" H 8215 3696 50  0000 L CNN
 F 1 "1u" H 8215 3605 50  0000 L CNN
-F 2 "Capacitor_SMD:C_0603_1608Metric_Pad1.08x0.95mm_HandSolder" H 8138 3500 50  0001 C CNN
+F 2 "Capacitor_SMD:C_0603_1608Metric_Pad1.05x0.95mm_HandSolder" H 8138 3500 50  0001 C CNN
 F 3 "~" H 8100 3650 50  0001 C CNN
 	1    8100 3650
@@
 F 0 "C11" H 7015 4096 50  0000 L CNN
 F 1 "10u" H 7015 4005 50  0000 L CNN
-F 2 "Capacitor_SMD:C_1206_3216Metric_Pad1.33x1.80mm_HandSolder" H 6938 3900 50  0001 C CNN
+F 2 "Capacitor_SMD:C_1206_3216Metric_Pad1.42x1.75mm_HandSolder" H 6938 3900 50  0001 C CNN
 F 3 "~" H 6900 4050 50  0001 C CNN
 	1    6900 4050
@@
 F 0 "R4" H 7570 3696 50  0000 L CNN
 F 1 "240 1%" H 7570 3605 50  0000 L CNN
-F 2 "Resistor_SMD:R_0603_1608Metric_Pad0.98x0.95mm_HandSolder" V 7430 3650 50  0001 C CNN
+F 2 "Resistor_SMD:R_0603_1608Metric_Pad1.05x0.95mm_HandSolder" V 7430 3650 50  0001 C CNN
 F 3 "~" H 7500 3650 50  0001 C CNN
 	1    7500 3650
@@
 F 0 "R5" H 7570 4096 50  0000 L CNN
 F 1 "390 1%" H 7570 4005 50  0000 L CNN
-F 2 "Resistor_SMD:R_0603_1608Metric_Pad0.98x0.95mm_HandSolder" V 7430 4050 50  0001 C CNN
+F 2 "Resistor_SMD:R_0603_1608Metric_Pad1.05x0.95mm_HandSolder" V 7430 4050 50  0001 C CNN
 F 3 "~" H 7500 4050 50  0001 C CNN
 	1    7500 4050
@@
 F 0 "TP5" H 8608 4318 50  0000 L CNN
 F 1 "TestPoint" H 8608 4227 50  0001 L CNN
-F 2 "MountingHole:MountingHole_2.2mm_M2_DIN965_Pad_TopBottom" H 8750 4200 50  0001 C CNN
+F 2 "furnace_230V:TP" H 8750 4200 50  0001 C CNN
 F 3 "~" H 8750 4200 50  0001 C CNN
 	1    8550 4200
@@
 F 0 "TP4" H 8608 3618 50  0000 L CNN
 F 1 "TestPoint" H 8608 3527 50  0001 L CNN
-F 2 "MountingHole:MountingHole_2.2mm_M2_DIN965_Pad_TopBottom" H 8750 3500 50  0001 C CNN
+F 2 "furnace_230V:TP" H 8750 3500 50  0001 C CNN
 F 3 "~" H 8750 3500 50  0001 C CNN
 	1    8550 3500
