File: furnace/furnace_230V/AC-DC 5V.sch (KiCad schematic (older format))
At the start: 13 parts

Commit message: Add files via upload
Changed lines of the file:
@@
 	4250 4000 4750 4000
 Wire Wire Line
-	4750 4000 5500 4000
+	4750 4000 5250 4000
 Connection ~ 4750 4000
 Wire Wire Line
@@
 Connection ~ 4750 4500
 Wire Wire Line
-	4750 4500 5500 4500
+	4750 4500 5250 4500
 Wire Wire Line
 	3000 4300 3000 4500
@@
 Connection ~ 9000 4000
 Wire Wire Line
-	9000 4000 10000 4000
+	9000 4000 9500 4000
 Wire Wire Line
 	6750 4300 6750 4500
@@
 	8500 4300 8500 4500
 Connection ~ 8500 4500
+$Comp
+L power:PWR_FLAG #FLG0101
+U 1 1 6127E67A
+P 5250 4000
+F 0 "#FLG0101" H 5250 4075 50  0001 C CNN
+F 1 "PWR_FLAG" H 5250 4173 50  0000 C CNN
+F 2 "" H 5250 4000 50  0001 C CNN
+F 3 "~" H 5250 4000 50  0001 C CNN
+	1    5250 4000
+	1    0    0    -1
+$EndComp
+Connection ~ 5250 4000
+Wire Wire Line
+	5250 4000 5500 4000
+$Comp
+L power:PWR_FLAG #FLG0102
+U 1 1 6127F32F
+P 5250 4500
+F 0 "#FLG0102" H 5250 4575 50  0001 C CNN
+F 1 "PWR_FLAG" H 5250 4673 50  0000 C CNN
+F 2 "" H 5250 4500 50  0001 C CNN
+F 3 "~" H 5250 4500 50  0001 C CNN
+	1    5250 4500
+	1    0    0    -1
+$EndComp
+Connection ~ 5250 4500
+Wire Wire Line
+	5250 4500 5500 4500
+$Comp
+L power:PWR_FLAG #FLG0103
+U 1 1 61281158
+P 9500 4000
+F 0 "#FLG0103" H 9500 4075 50  0001 C CNN
+F 1 "PWR_FLAG" H 9500 4173 50  0000 C CNN
+F 2 "" H 9500 4000 50  0001 C CNN
+F 3 "~" H 9500 4000 50  0001 C CNN
+	1    9500 4000
+	1    0    0    -1
+$EndComp
+Connection ~ 9500 4000
+Wire Wire Line
+	9500 4000 10000 4000
 $EndSCHEMATC
