File: furnace/furnace_230V/Isolated_TRIAC.sch (KiCad schematic (older format))
At the start: 6 parts, among them Q1 BTA16-600B, U3 MOC3052M

Commit message: Add files via upload
Parts:
- removed HS1: HS 304-50, furnace_230V:HS_304-50, symbol Mechanical:Heatsink
- added C13: 0,01 630V, Capacitor_THT:C_Disc_D10.5mm_W5.0mm_P10.00mm, symbol furnace_230V-rescue:C-Device
- added F2: 10A, Fuse:Fuseholder_Cylinder-5x20mm_Stelvio-Kontek_PTF78_Horizontal_Open, symbol furnace_230V-rescue:Fuse-Device
- added R8: 33 1W, Resistor_THT:R_Axial_DIN0414_L11.9mm_D4.5mm_P20.32mm_Horizontal, symbol furnace_230V-rescue:R-Device
- added RV1: 471KD20, Varistor:RV_Disc_D21.5mm_W6.1mm_P7.5mm, symbol Device:Varistor
- D3: footprint LED_SMD:LED_1206_3216Metric_ReverseMount_Hole1.8x2.4mm -> LED_SMD:LED_1206_3216Metric_Pad1.42x1.75mm_HandSolder
- Q1: footprint furnace_230V:TRIAC -> (none)
Connections:
- net AC: now also R8.1, RV1.1
- net LOAD: now also F2.1; no longer Q1.1 (A1)
- new net: C13.2, F2.2, Q1.1 (A1), RV1.2
- new net: C13.1, R8.2
Other:
- moved on the sheet: R7
Changed lines of the file:
@@
 F 0 "Q1" H 6129 4196 50  0000 L CNN
 F 1 "BTA16-600B" H 6129 4105 50  0000 L CNN
-F 2 "furnace_230V:TRIAC" H 6200 4075 50  0001 L CIN
+F 2 "" H 6200 4075 50  0001 L CIN
 F 3 "https://www.st.com/resource/en/datasheet/bta16.pdf" H 6000 4150 50  0001 L CNN
 	1    6000 4150
@@
 L furnace_230V-rescue:R-Device R7
 U 1 1 60AB3416
-P 5250 3750
-F 0 "R7" H 5320 3796 50  0000 L CNN
-F 1 "470 0,5W" H 5320 3705 50  0000 L CNN
-F 2 "Resistor_THT:R_Axial_DIN0309_L9.0mm_D3.2mm_P15.24mm_Horizontal" V 5180 3750 50  0001 C CNN
-F 3 "~" H 5250 3750 50  0001 C CNN
-	1    5250 3750
+P 5000 3650
+F 0 "R7" H 5070 3696 50  0000 L CNN
+F 1 "470 0,5W" H 5070 3605 50  0000 L CNN
+F 2 "Resistor_THT:R_Axial_DIN0309_L9.0mm_D3.2mm_P15.24mm_Horizontal" V 4930 3650 50  0001 C CNN
+F 3 "~" H 5000 3650 50  0001 C CNN
+	1    5000 3650
 	1    0    0    -1
 $EndComp
@@
 $EndComp
 $Comp
+L furnace_230V-rescue:R-Device R8
+U 1 1 60ABF950
+P 7000 3800
+F 0 "R8" H 7070 3846 50  0000 L CNN
+F 1 "33 1W" H 7070 3755 50  0000 L CNN
+F 2 "Resistor_THT:R_Axial_DIN0414_L11.9mm_D4.5mm_P20.32mm_Horizontal" V 6930 3800 50  0001 C CNN
+F 3 "~" H 7000 3800 50  0001 C CNN
+	1    7000 3800
+	1    0    0    -1
+$EndComp
+$Comp
+L furnace_230V-rescue:C-Device C13
+U 1 1 60ABFAB6
+P 7000 4200
+F 0 "C13" H 7115 4246 50  0000 L CNN
+F 1 "0,01 630V" H 7115 4155 50  0000 L CNN
+F 2 "Capacitor_THT:C_Disc_D10.5mm_W5.0mm_P10.00mm" H 7038 4050 50  0001 C CNN
+F 3 "~" H 7000 4200 50  0001 C CNN
+	1    7000 4200
+	1    0    0    -1
+$EndComp
+$Comp
 L furnace_230V-rescue:LED-Device D3
 U 1 1 60AD0B5E
@@
 F 0 "D3" H 3843 3745 50  0000 C CNN
 F 1 "LED" H 3843 3836 50  0000 C CNN
-F 2 "LED_SMD:LED_1206_3216Metric_ReverseMount_Hole1.8x2.4mm" H 3850 4000 50  0001 C CNN
+F 2 "LED_SMD:LED_1206_3216Metric_Pad1.42x1.75mm_HandSolder" H 3850 4000 50  0001 C CNN
 F 3 "~" H 3850 4000 50  0001 C CNN
 	1    3850 4000
@@
 Text Notes 7800 2450 2    197  ~ 0
 Isolated TRIAC control circuit
-Text HLabel 7500 3500 2    50   Input ~ 0
+$Comp
+L furnace_230V-rescue:Fuse-Device F2
+U 1 1 60B1BB7E
+P 8250 4500
+F 0 "F2" V 8150 4500 50  0000 C CNN
+F 1 "10A" V 8350 4500 50  0000 C CNN
+F 2 "Fuse:Fuseholder_Cylinder-5x20mm_Stelvio-Kontek_PTF78_Horizontal_Open" V 8180 4500 50  0001 C CNN
+F 3 "~" H 8250 4500 50  0001 C CNN
+	1    8250 4500
+	0    1    1    0
+$EndComp
+Text HLabel 9000 3500 2    50   Input ~ 0
 AC
-Text HLabel 7500 4500 2    50   Output ~ 0
+Text HLabel 9000 4500 2    50   Output ~ 0
 LOAD
 Text HLabel 2500 4000 0    50   Input ~ 0
@@
 	4400 4500 2500 4500
 Wire Wire Line
+	5000 4000 5000 3800
+Wire Wire Line
 	5000 4200 5000 4250
 Wire Wire Line
 	5000 4250 5850 4250
 Wire Wire Line
+	5000 3500 6000 3500
+Wire Wire Line
 	6000 4000 6000 3500
+Connection ~ 6000 3500
 Wire Wire Line
 	6000 4300 6000 4500
+Wire Wire Line
+	8400 4500 9000 4500
+Wire Wire Line
+	6000 4500 7000 4500
+Wire Wire Line
+	6000 3500 7000 3500
+Wire Wire Line
+	7000 3650 7000 3500
+Connection ~ 7000 3500
+Wire Wire Line
+	7000 3500 7750 3500
+Wire Wire Line
+	7000 3950 7000 4050
+Wire Wire Line
+	7000 4350 7000 4500
+Connection ~ 7000 4500
 $Comp
-L Mechanical:Heatsink HS1
-U 1 1 610DEB43
-P 6200 3950
-F 0 "HS1" H 6341 4071 50  0000 L CNN
-F 1 "HS 304-50" H 6341 3980 50  0000 L CNN
-F 2 "furnace_230V:HS_304-50" H 6212 3950 50  0001 C CNN
-F 3 "~" H 6212 3950 50  0001 C CNN
-	1    6200 3950
+L Device:Varistor RV1
+U 1 1 6105DA3F
+P 7750 4000
+F 0 "RV1" H 7853 4046 50  0000 L CNN
+F 1 "471KD20" H 7853 3955 50  0000 L CNN
+F 2 "Varistor:RV_Disc_D21.5mm_W6.1mm_P7.5mm" V 7680 4000 50  0001 C CNN
+F 3 "~" H 7750 4000 50  0001 C CNN
+	1    7750 4000
 	1    0    0    -1
 $EndComp
 Wire Wire Line
-	5250 3600 5250 3500
+	7750 4150 7750 4500
 Wire Wire Line
-	5250 3500 6000 3500
+	7000 4500 7750 4500
+Connection ~ 7750 4500
 Wire Wire Line
-	5250 3900 5250 4000
+	7750 4500 8100 4500
 Wire Wire Line
-	5250 4000 5000 4000
+	7750 3850 7750 3500
+Connection ~ 7750 3500
 Wire Wire Line
-	6000 4500 7500 4500
-Wire Wire Line
-	7500 3500 6000 3500
-Connection ~ 6000 3500
+	7750 3500 9000 3500
 $EndSCHEMATC
