File: furnace/furnace_230V/Isolated_TRIAC.sch (KiCad schematic (older format))
At the start: 4 parts

Commit message: Add files via upload
Parts:
- added C?: 0,01, symbol Device:C
- added D?: LED, symbol Device:LED
- added F?: 10A, symbol Device:Fuse
- added R?: 33 0,5W, symbol Device:R
- R?: value 100 -> 150
Connections:
- net labels added: +5V, AC, LOAD, ~EN
- wire segments 0 -> 19
Other:
- note added: "Isolated TRIAC control circuit"
- moved on the sheet: Q?
Changed lines of the file:
@@
 L furnace_230V-rescue:BTA16-600B-Triac_Thyristor Q?
 U 1 1 60AB340A
-P 6300 3850
-F 0 "Q?" H 6429 3896 50  0000 L CNN
-F 1 "BTA16-600B" H 6429 3805 50  0000 L CNN
-F 2 "Package_TO_SOT_THT:TO-220-3_Vertical" H 6500 3775 50  0001 L CIN
-F 3 "https://www.st.com/resource/en/datasheet/bta16.pdf" H 6300 3850 50  0001 L CNN
-	1    6300 3850
+P 6500 4150
+F 0 "Q?" H 6629 4196 50  0000 L CNN
+F 1 "BTA16-600B" H 6629 4105 50  0000 L CNN
+F 2 "Package_TO_SOT_THT:TO-220-3_Vertical" H 6700 4075 50  0001 L CIN
+F 3 "https://www.st.com/resource/en/datasheet/bta16.pdf" H 6500 4150 50  0001 L CNN
+	1    6500 4150
 	1    0    0    -1
 $EndComp
@@
 L Relay_SolidState:MOC3052M U?
 U 1 1 60AB3410
-P 5100 4100
-F 0 "U?" H 5100 4425 50  0000 C CNN
-F 1 "MOC3052M" H 5100 4334 50  0000 C CNN
-F 2 "" H 4900 3900 50  0001 L CIN
-F 3 "https://www.onsemi.com/pub/Collateral/MOC3052M-D.PDF" H 5100 4100 50  0001 L CNN
-	1    5100 4100
+P 5200 4100
+F 0 "U?" H 5200 4425 50  0000 C CNN
+F 1 "MOC3052M" H 5200 4334 50  0000 C CNN
+F 2 "" H 5000 3900 50  0001 L CIN
+F 3 "https://www.onsemi.com/pub/Collateral/MOC3052M-D.PDF" H 5200 4100 50  0001 L CNN
+	1    5200 4100
 	1    0    0    -1
 $EndComp
@@
 L Device:R R?
 U 1 1 60AB3416
-P 5450 3450
-F 0 "R?" H 5520 3496 50  0000 L CNN
-F 1 "470 0,5W" H 5520 3405 50  0000 L CNN
-F 2 "" V 5380 3450 50  0001 C CNN
-F 3 "~" H 5450 3450 50  0001 C CNN
-	1    5450 3450
+P 5500 3650
+F 0 "R?" H 5570 3696 50  0000 L CNN
+F 1 "470 0,5W" H 5570 3605 50  0000 L CNN
+F 2 "" V 5430 3650 50  0001 C CNN
+F 3 "~" H 5500 3650 50  0001 C CNN
+	1    5500 3650
 	1    0    0    -1
 $EndComp
@@
 L Device:R R?
 U 1 1 60B5C7C1
-P 4100 4000
-F 0 "R?" V 3893 4000 50  0000 C CNN
-F 1 "100" V 3984 4000 50  0000 C CNN
-F 2 "Resistor_SMD:R_0603_1608Metric_Pad1.05x0.95mm_HandSolder" V 4030 4000 50  0001 C CNN
-F 3 "~" H 4100 4000 50  0001 C CNN
-	1    4100 4000
+P 3850 4000
+F 0 "R?" V 3643 4000 50  0000 C CNN
+F 1 "150" V 3734 4000 50  0000 C CNN
+F 2 "Resistor_SMD:R_0603_1608Metric_Pad1.05x0.95mm_HandSolder" V 3780 4000 50  0001 C CNN
+F 3 "~" H 3850 4000 50  0001 C CNN
+	1    3850 4000
 	0    1    1    0
 $EndComp
+$Comp
+L Device:R R?
+U 1 1 60ABF950
+P 7500 3800
+F 0 "R?" H 7570 3846 50  0000 L CNN
+F 1 "33 0,5W" H 7570 3755 50  0000 L CNN
+F 2 "" V 7430 3800 50  0001 C CNN
+F 3 "~" H 7500 3800 50  0001 C CNN
+	1    7500 3800
+	1    0    0    -1
+$EndComp
+$Comp
+L Device:C C?
+U 1 1 60ABFAB6
+P 7500 4200
+F 0 "C?" H 7615 4246 50  0000 L CNN
+F 1 "0,01" H 7615 4155 50  0000 L CNN
+F 2 "" H 7538 4050 50  0001 C CNN
+F 3 "~" H 7500 4200 50  0001 C CNN
+	1    7500 4200
+	1    0    0    -1
+$EndComp
+$Comp
+L Device:LED D?
+U 1 1 60AD0B5E
+P 4350 4000
+F 0 "D?" H 4343 3745 50  0000 C CNN
+F 1 "LED" H 4343 3836 50  0000 C CNN
+F 2 "" H 4350 4000 50  0001 C CNN
+F 3 "~" H 4350 4000 50  0001 C CNN
+	1    4350 4000
+	-1   0    0    1
+$EndComp
+Text Notes 7800 2450 2    197  ~ 0
+Isolated TRIAC control circuit
+$Comp
+L Device:Fuse F?
+U 1 1 60B1BB7E
+P 8350 4500
+F 0 "F?" V 8250 4500 50  0000 C CNN
+F 1 "10A" V 8450 4500 50  0000 C CNN
+F 2 "" V 8280 4500 50  0001 C CNN
+F 3 "~" H 8350 4500 50  0001 C CNN
+	1    8350 4500
+	0    1    1    0
+$EndComp
+Text HLabel 9000 3500 2    50   Input ~ 0
+AC
+Text HLabel 9000 4500 2    50   Output ~ 0
+LOAD
+Text HLabel 3000 4000 0    50   Input ~ 0
++5V
+Text HLabel 3000 4500 0    50   Input ~ 0
+~EN
+Wire Wire Line
+	3000 4000 3700 4000
+Wire Wire Line
+	4000 4000 4200 4000
+Wire Wire Line
+	4500 4000 4900 4000
+Wire Wire Line
+	4900 4200 4900 4500
+Wire Wire Line
+	4900 4500 3000 4500
+Wire Wire Line
+	5500 4000 5500 3800
+Wire Wire Line
+	5500 4200 5500 4250
+Wire Wire Line
+	5500 4250 6350 4250
+Wire Wire Line
+	5500 3500 6500 3500
+Wire Wire Line
+	6500 4000 6500 3500
+Connection ~ 6500 3500
+Wire Wire Line
+	6500 4300 6500 4500
+Wire Wire Line
+	8500 4500 9000 4500
+Wire Wire Line
+	6500 4500 7500 4500
+Wire Wire Line
+	6500 3500 7500 3500
+Wire Wire Line
+	7500 3650 7500 3500
+Connection ~ 7500 3500
+Wire Wire Line
+	7500 3500 9000 3500
+Wire Wire Line
+	7500 3950 7500 4050
+Wire Wire Line
+	7500 4350 7500 4500
+Connection ~ 7500 4500
+Wire Wire Line
+	7500 4500 8200 4500
 $EndSCHEMATC

Commit message: Add files via upload
Parts:
- added RV1: 471KD20, symbol Device:Varistor
- C13: renamed from C?; value 0,01 -> 0,01 630V; footprint (none) -> Capacitor_THT:C_Disc_D10.5mm_W5.0mm_P10.00mm; symbol Device:C -> furnace_230V-rescue:C-Device
- D3: renamed from D?; footprint (none) -> LED_SMD:LED_1206_3216Metric_Pad1.42x1.75mm_HandSolder; symbol Device:LED -> furnace_230V-rescue:LED-Device
- F2: renamed from F?; footprint (none) -> Fuse:Fuseholder_Cylinder-5x20mm_Stelvio-Kontek_PTF78_Horizontal_Open; symbol Device:Fuse -> furnace_230V-rescue:Fuse-Device
- R6, R7: renamed from R?; symbol Device:R -> furnace_230V-rescue:R-Device
- R8: renamed from R?; value 33 0,5W -> 33 1W; symbol Device:R -> furnace_230V-rescue:R-Device
- U3: renamed from U?; symbol Relay_SolidState:MOC3052M -> furnace_230V-rescue:MOC3052M-Relay_SolidState
- gave numbers to parts that had none: 1
Connections:
- wire segments 19 -> 23
Other:
- moved on the sheet: Q1
Changed lines of the file:
@@
 $EndDescr
 $Comp
-L furnace_230V-rescue:BTA16-600B-Triac_Thyristor Q?
+L furnace_230V-rescue:BTA16-600B-Triac_Thyristor Q1
 U 1 1 60AB340A
-P 6500 4150
-F 0 "Q?" H 6629 4196 50  0000 L CNN
-F 1 "BTA16-600B" H 6629 4105 50  0000 L CNN
-F 2 "Package_TO_SOT_THT:TO-220-3_Vertical" H 6700 4075 50  0001 L CIN
-F 3 "https://www.st.com/resource/en/datasheet/bta16.pdf" H 6500 4150 50  0001 L CNN
-	1    6500 4150
+P 6000 4150
+F 0 "Q1" H 6129 4196 50  0000 L CNN
+F 1 "BTA16-600B" H 6129 4105 50  0000 L CNN
+F 2 "Package_TO_SOT_THT:TO-220-3_Vertical" H 6200 4075 50  0001 L CIN
+F 3 "https://www.st.com/resource/en/datasheet/bta16.pdf" H 6000 4150 50  0001 L CNN
+	1    6000 4150
 	1    0    0    -1
 $EndComp
 $Comp
-L Relay_SolidState:MOC3052M U?
+L furnace_230V-rescue:MOC3052M-Relay_SolidState U3
 U 1 1 60AB3410
-P 5200 4100
-F 0 "U?" H 5200 4425 50  0000 C CNN
-F 1 "MOC3052M" H 5200 4334 50  0000 C CNN
-F 2 "" H 5000 3900 50  0001 L CIN
-F 3 "https://www.onsemi.com/pub/Collateral/MOC3052M-D.PDF" H 5200 4100 50  0001 L CNN
-	1    5200 4100
+P 4700 4100
+F 0 "U3" H 4700 4425 50  0000 C CNN
+F 1 "MOC3052M" H 4700 4334 50  0000 C CNN
+F 2 "" H 4500 3900 50  0001 L CIN
+F 3 "https://www.onsemi.com/pub/Collateral/MOC3052M-D.PDF" H 4700 4100 50  0001 L CNN
+	1    4700 4100
 	1    0    0    -1
 $EndComp
 $Comp
-L Device:R R?
+L furnace_230V-rescue:R-Device R7
 U 1 1 60AB3416
-P 5500 3650
-F 0 "R?" H 5570 3696 50  0000 L CNN
-F 1 "470 0,5W" H 5570 3605 50  0000 L CNN
-F 2 "" V 5430 3650 50  0001 C CNN
-F 3 "~" H 5500 3650 50  0001 C CNN
-	1    5500 3650
+P 5000 3650
+F 0 "R7" H 5070 3696 50  0000 L CNN
+F 1 "470 0,5W" H 5070 3605 50  0000 L CNN
+F 2 "" V 4930 3650 50  0001 C CNN
+F 3 "~" H 5000 3650 50  0001 C CNN
+	1    5000 3650
 	1    0    0    -1
 $EndComp
 $Comp
-L Device:R R?
+L furnace_230V-rescue:R-Device R6
 U 1 1 60B5C7C1
-P 3850 4000
-F 0 "R?" V 3643 4000 50  0000 C CNN
-F 1 "150" V 3734 4000 50  0000 C CNN
-F 2 "Resistor_SMD:R_0603_1608Metric_Pad1.05x0.95mm_HandSolder" V 3780 4000 50  0001 C CNN
-F 3 "~" H 3850 4000 50  0001 C CNN
-	1    3850 4000
+P 3350 4000
+F 0 "R6" V 3143 4000 50  0000 C CNN
+F 1 "150" V 3234 4000 50  0000 C CNN
+F 2 "Resistor_SMD:R_0603_1608Metric_Pad1.05x0.95mm_HandSolder" V 3280 4000 50  0001 C CNN
+F 3 "~" H 3350 4000 50  0001 C CNN
+	1    3350 4000
 	0    1    1    0
 $EndComp
 $Comp
-L Device:R R?
+L furnace_230V-rescue:R-Device R8
 U 1 1 60ABF950
-P 7500 3800
-F 0 "R?" H 7570 3846 50  0000 L CNN
-F 1 "33 0,5W" H 7570 3755 50  0000 L CNN
-F 2 "" V 7430 3800 50  0001 C CNN
-F 3 "~" H 7500 3800 50  0001 C CNN
-	1    7500 3800
+P 7000 3800
+F 0 "R8" H 7070 3846 50  0000 L CNN
+F 1 "33 1W" H 7070 3755 50  0000 L CNN
+F 2 "" V 6930 3800 50  0001 C CNN
+F 3 "~" H 7000 3800 50  0001 C CNN
+	1    7000 3800
 	1    0    0    -1
 $EndComp
 $Comp
-L Device:C C?
+L furnace_230V-rescue:C-Device C13
 U 1 1 60ABFAB6
-P 7500 4200
-F 0 "C?" H 7615 4246 50  0000 L CNN
-F 1 "0,01" H 7615 4155 50  0000 L CNN
-F 2 "" H 7538 4050 50  0001 C CNN
-F 3 "~" H 7500 4200 50  0001 C CNN
-	1    7500 4200
+P 7000 4200
+F 0 "C13" H 7115 4246 50  0000 L CNN
+F 1 "0,01 630V" H 7115 4155 50  0000 L CNN
+F 2 "Capacitor_THT:C_Disc_D10.5mm_W5.0mm_P10.00mm" H 7038 4050 50  0001 C CNN
+F 3 "~" H 7000 4200 50  0001 C CNN
+	1    7000 4200
 	1    0    0    -1
 $EndComp
 $Comp
-L Device:LED D?
+L furnace_230V-rescue:LED-Device D3
 U 1 1 60AD0B5E
-P 4350 4000
-F 0 "D?" H 4343 3745 50  0000 C CNN
-F 1 "LED" H 4343 3836 50  0000 C CNN
-F 2 "" H 4350 4000 50  0001 C CNN
-F 3 "~" H 4350 4000 50  0001 C CNN
-	1    4350 4000
+P 3850 4000
+F 0 "D3" H 3843 3745 50  0000 C CNN
+F 1 "LED" H 3843 3836 50  0000 C CNN
+F 2 "LED_SMD:LED_1206_3216Metric_Pad1.42x1.75mm_HandSolder" H 3850 4000 50  0001 C CNN
+F 3 "~" H 3850 4000 50  0001 C CNN
+	1    3850 4000
 	-1   0    0    1
 $EndComp
@@
 Isolated TRIAC control circuit
 $Comp
-L Device:Fuse F?
+L furnace_230V-rescue:Fuse-Device F2
 U 1 1 60B1BB7E
-P 8350 4500
-F 0 "F?" V 8250 4500 50  0000 C CNN
-F 1 "10A" V 8450 4500 50  0000 C CNN
-F 2 "" V 8280 4500 50  0001 C CNN
-F 3 "~" H 8350 4500 50  0001 C CNN
-	1    8350 4500
+P 8250 4500
+F 0 "F2" V 8150 4500 50  0000 C CNN
+F 1 "10A" V 8350 4500 50  0000 C CNN
+F 2 "Fuse:Fuseholder_Cylinder-5x20mm_Stelvio-Kontek_PTF78_Horizontal_Open" V 8180 4500 50  0001 C CNN
+F 3 "~" H 8250 4500 50  0001 C CNN
+	1    8250 4500
 	0    1    1    0
 $EndComp
@@
 Text HLabel 9000 4500 2    50   Output ~ 0
 LOAD
-Text HLabel 3000 4000 0    50   Input ~ 0
+Text HLabel 2500 4000 0    50   Input ~ 0
 +5V
-Text HLabel 3000 4500 0    50   Input ~ 0
+Text HLabel 2500 4500 0    50   Input ~ 0
 ~EN
 Wire Wire Line
-	3000 4000 3700 4000
+	2500 4000 3200 4000
 Wire Wire Line
-	4000 4000 4200 4000
+	3500 4000 3700 4000
 Wire Wire Line
-	4500 4000 4900 4000
+	4000 4000 4400 4000
 Wire Wire Line
-	4900 4200 4900 4500
+	4400 4200 4400 4500
 Wire Wire Line
-	4900 4500 3000 4500
+	4400 4500 2500 4500
 Wire Wire Line
-	5500 4000 5500 3800
+	5000 4000 5000 3800
 Wire Wire Line
-	5500 4200 5500 4250
+	5000 4200 5000 4250
 Wire Wire Line
-	5500 4250 6350 4250
+	5000 4250 5850 4250
 Wire Wire Line
-	5500 3500 6500 3500
+	5000 3500 6000 3500
 Wire Wire Line
-	6500 4000 6500 3500
-Connection ~ 6500 3500
+	6000 4000 6000 3500
+Connection ~ 6000 3500
 Wire Wire Line
-	6500 4300 6500 4500
+	6000 4300 6000 4500
 Wire Wire Line
-	8500 4500 9000 4500
+	8400 4500 9000 4500
 Wire Wire Line
-	6500 4500 7500 4500
+	6000 4500 7000 4500
 Wire Wire Line
-	6500 3500 7500 3500
+	6000 3500 7000 3500
 Wire Wire Line
-	7500 3650 7500 3500
-Connection ~ 7500 3500
+	7000 3650 7000 3500
+Connection ~ 7000 3500
 Wire Wire Line
-	7500 3500 9000 3500
+	7000 3500 7750 3500
 Wire Wire Line
-	7500 3950 7500 4050
+	7000 3950 7000 4050
 Wire Wire Line
-	7500 4350 7500 4500
-Connection ~ 7500 4500
+	7000 4350 7000 4500
+Connection ~ 7000 4500
+$Comp
+L Device:Varistor RV1
+U 1 1 6105DA3F
+P 7750 4000
+F 0 "RV1" H 7853 4046 50  0000 L CNN
+F 1 "471KD20" H 7853 3955 50  0000 L CNN
+F 2 "" V 7680 4000 50  0001 C CNN
+F 3 "~" H 7750 4000 50  0001 C CNN
+	1    7750 4000
+	1    0    0    -1
+$EndComp
 Wire Wire Line
-	7500 4500 8200 4500
+	7750 4150 7750 4500
+Wire Wire Line
+	7000 4500 7750 4500
+Connection ~ 7750 4500
+Wire Wire Line
+	7750 4500 8100 4500
+Wire Wire Line
+	7750 3850 7750 3500
+Connection ~ 7750 3500
+Wire Wire Line
+	7750 3500 9000 3500
 $EndSCHEMATC

Commit message: Add files via upload
Parts:
- Q1: footprint Package_TO_SOT_THT:TO-220-3_Vertical -> (none)
- R7: footprint (none) -> Resistor_THT:R_Axial_DIN0309_L9.0mm_D3.2mm_P15.24mm_Horizontal
- R8: footprint (none) -> Resistor_THT:R_Axial_DIN0414_L11.9mm_D4.5mm_P20.32mm_Horizontal
- RV1: footprint (none) -> Varistor:RV_Disc_D21.5mm_W6.1mm_P7.5mm
- U3: footprint (none) -> Package_DIP:DIP-6_W7.62mm_LongPads
Changed lines of the file:
@@
 F 0 "Q1" H 6129 4196 50  0000 L CNN
 F 1 "BTA16-600B" H 6129 4105 50  0000 L CNN
-F 2 "Package_TO_SOT_THT:TO-220-3_Vertical" H 6200 4075 50  0001 L CIN
+F 2 "" H 6200 4075 50  0001 L CIN
 F 3 "https://www.st.com/resource/en/datasheet/bta16.pdf" H 6000 4150 50  0001 L CNN
 	1    6000 4150
@@
 F 0 "U3" H 4700 4425 50  0000 C CNN
 F 1 "MOC3052M" H 4700 4334 50  0000 C CNN
-F 2 "" H 4500 3900 50  0001 L CIN
+F 2 "Package_DIP:DIP-6_W7.62mm_LongPads" H 4500 3900 50  0001 L CIN
 F 3 "https://www.onsemi.com/pub/Collateral/MOC3052M-D.PDF" H 4700 4100 50  0001 L CNN
 	1    4700 4100
@@
 F 0 "R7" H 5070 3696 50  0000 L CNN
 F 1 "470 0,5W" H 5070 3605 50  0000 L CNN
-F 2 "" V 4930 3650 50  0001 C CNN
+F 2 "Resistor_THT:R_Axial_DIN0309_L9.0mm_D3.2mm_P15.24mm_Horizontal" V 4930 3650 50  0001 C CNN
 F 3 "~" H 5000 3650 50  0001 C CNN
 	1    5000 3650
@@
 F 0 "R8" H 7070 3846 50  0000 L CNN
 F 1 "33 1W" H 7070 3755 50  0000 L CNN
-F 2 "" V 6930 3800 50  0001 C CNN
+F 2 "Resistor_THT:R_Axial_DIN0414_L11.9mm_D4.5mm_P20.32mm_Horizontal" V 6930 3800 50  0001 C CNN
 F 3 "~" H 7000 3800 50  0001 C CNN
 	1    7000 3800
@@
 F 0 "RV1" H 7853 4046 50  0000 L CNN
 F 1 "471KD20" H 7853 3955 50  0000 L CNN
-F 2 "" V 7680 4000 50  0001 C CNN
+F 2 "Varistor:RV_Disc_D21.5mm_W6.1mm_P7.5mm" V 7680 4000 50  0001 C CNN
 F 3 "~" H 7750 4000 50  0001 C CNN
 	1    7750 4000

Commit message: Add files via upload
Parts:
- removed C13: 0,01 630V, Capacitor_THT:C_Disc_D10.5mm_W5.0mm_P10.00mm, symbol furnace_230V-rescue:C-Device
- removed F2: 10A, Fuse:Fuseholder_Cylinder-5x20mm_Stelvio-Kontek_PTF78_Horizontal_Open, symbol furnace_230V-rescue:Fuse-Device
- removed R8: 33 1W, Resistor_THT:R_Axial_DIN0414_L11.9mm_D4.5mm_P20.32mm_Horizontal, symbol furnace_230V-rescue:R-Device
- removed RV1: 471KD20, Varistor:RV_Disc_D21.5mm_W6.1mm_P7.5mm, symbol Device:Varistor
- added HS1: HS 304-50, furnace_230V:HS_304-50, symbol Mechanical:Heatsink
- D3: footprint LED_SMD:LED_1206_3216Metric_Pad1.42x1.75mm_HandSolder -> LED_SMD:LED_1206_3216Metric_ReverseMount_Hole1.8x2.4mm
- Q1: footprint (none) -> furnace_230V:TRIAC
Connections:
- net LOAD: now also Q1.1 (A1)
Other:
- moved on the sheet: R7
Changed lines of the file:
@@
 F 0 "Q1" H 6129 4196 50  0000 L CNN
 F 1 "BTA16-600B" H 6129 4105 50  0000 L CNN
-F 2 "" H 6200 4075 50  0001 L CIN
+F 2 "furnace_230V:TRIAC" H 6200 4075 50  0001 L CIN
 F 3 "https://www.st.com/resource/en/datasheet/bta16.pdf" H 6000 4150 50  0001 L CNN
 	1    6000 4150
@@
 L furnace_230V-rescue:R-Device R7
 U 1 1 60AB3416
-P 5000 3650
-F 0 "R7" H 5070 3696 50  0000 L CNN
-F 1 "470 0,5W" H 5070 3605 50  0000 L CNN
-F 2 "Resistor_THT:R_Axial_DIN0309_L9.0mm_D3.2mm_P15.24mm_Horizontal" V 4930 3650 50  0001 C CNN
-F 3 "~" H 5000 3650 50  0001 C CNN
-	1    5000 3650
+P 5250 3750
+F 0 "R7" H 5320 3796 50  0000 L CNN
+F 1 "470 0,5W" H 5320 3705 50  0000 L CNN
+F 2 "Resistor_THT:R_Axial_DIN0309_L9.0mm_D3.2mm_P15.24mm_Horizontal" V 5180 3750 50  0001 C CNN
+F 3 "~" H 5250 3750 50  0001 C CNN
+	1    5250 3750
 	1    0    0    -1
 $EndComp
@@
 $EndComp
 $Comp
-L furnace_230V-rescue:R-Device R8
-U 1 1 60ABF950
-P 7000 3800
-F 0 "R8" H 7070 3846 50  0000 L CNN
-F 1 "33 1W" H 7070 3755 50  0000 L CNN
-F 2 "Resistor_THT:R_Axial_DIN0414_L11.9mm_D4.5mm_P20.32mm_Horizontal" V 6930 3800 50  0001 C CNN
-F 3 "~" H 7000 3800 50  0001 C CNN
-	1    7000 3800
-	1    0    0    -1
-$EndComp
-$Comp
-L furnace_230V-rescue:C-Device C13
-U 1 1 60ABFAB6
-P 7000 4200
-F 0 "C13" H 7115 4246 50  0000 L CNN
-F 1 "0,01 630V" H 7115 4155 50  0000 L CNN
-F 2 "Capacitor_THT:C_Disc_D10.5mm_W5.0mm_P10.00mm" H 7038 4050 50  0001 C CNN
-F 3 "~" H 7000 4200 50  0001 C CNN
-	1    7000 4200
-	1    0    0    -1
-$EndComp
-$Comp
 L furnace_230V-rescue:LED-Device D3
 U 1 1 60AD0B5E
@@
 F 0 "D3" H 3843 3745 50  0000 C CNN
 F 1 "LED" H 3843 3836 50  0000 C CNN
-F 2 "LED_SMD:LED_1206_3216Metric_Pad1.42x1.75mm_HandSolder" H 3850 4000 50  0001 C CNN
+F 2 "LED_SMD:LED_1206_3216Metric_ReverseMount_Hole1.8x2.4mm" H 3850 4000 50  0001 C CNN
 F 3 "~" H 3850 4000 50  0001 C CNN
 	1    3850 4000
@@
 Text Notes 7800 2450 2    197  ~ 0
 Isolated TRIAC control circuit
-$Comp
-L furnace_230V-rescue:Fuse-Device F2
-U 1 1 60B1BB7E
-P 8250 4500
-F 0 "F2" V 8150 4500 50  0000 C CNN
-F 1 "10A" V 8350 4500 50  0000 C CNN
-F 2 "Fuse:Fuseholder_Cylinder-5x20mm_Stelvio-Kontek_PTF78_Horizontal_Open" V 8180 4500 50  0001 C CNN
-F 3 "~" H 8250 4500 50  0001 C CNN
-	1    8250 4500
-	0    1    1    0
-$EndComp
-Text HLabel 9000 3500 2    50   Input ~ 0
+Text HLabel 7500 3500 2    50   Input ~ 0
 AC
-Text HLabel 9000 4500 2    50   Output ~ 0
+Text HLabel 7500 4500 2    50   Output ~ 0
 LOAD
 Text HLabel 2500 4000 0    50   Input ~ 0
@@
 	4400 4500 2500 4500
 Wire Wire Line
-	5000 4000 5000 3800
-Wire Wire Line
 	5000 4200 5000 4250
 Wire Wire Line
 	5000 4250 5850 4250
 Wire Wire Line
-	5000 3500 6000 3500
-Wire Wire Line
 	6000 4000 6000 3500
-Connection ~ 6000 3500
 Wire Wire Line
 	6000 4300 6000 4500
-Wire Wire Line
-	8400 4500 9000 4500
-Wire Wire Line
-	6000 4500 7000 4500
-Wire Wire Line
-	6000 3500 7000 3500
-Wire Wire Line
-	7000 3650 7000 3500
-Connection ~ 7000 3500
-Wire Wire Line
-	7000 3500 7750 3500
-Wire Wire Line
-	7000 3950 7000 4050
-Wire Wire Line
-	7000 4350 7000 4500
-Connection ~ 7000 4500
 $Comp
-L Device:Varistor RV1
-U 1 1 6105DA3F
-P 7750 4000
-F 0 "RV1" H 7853 4046 50  0000 L CNN
-F 1 "471KD20" H 7853 3955 50  0000 L CNN
-F 2 "Varistor:RV_Disc_D21.5mm_W6.1mm_P7.5mm" V 7680 4000 50  0001 C CNN
-F 3 "~" H 7750 4000 50  0001 C CNN
-	1    7750 4000
+L Mechanical:Heatsink HS1
+U 1 1 610DEB43
+P 6200 3950
+F 0 "HS1" H 6341 4071 50  0000 L CNN
+F 1 "HS 304-50" H 6341 3980 50  0000 L CNN
+F 2 "furnace_230V:HS_304-50" H 6212 3950 50  0001 C CNN
+F 3 "~" H 6212 3950 50  0001 C CNN
+	1    6200 3950
 	1    0    0    -1
 $EndComp
 Wire Wire Line
-	7750 4150 7750 4500
+	5250 3600 5250 3500
 Wire Wire Line
-	7000 4500 7750 4500
-Connection ~ 7750 4500
+	5250 3500 6000 3500
 Wire Wire Line
-	7750 4500 8100 4500
+	5250 3900 5250 4000
 Wire Wire Line
-	7750 3850 7750 3500
-Connection ~ 7750 3500
+	5250 4000 5000 4000
 Wire Wire Line
-	7750 3500 9000 3500
+	6000 4500 7500 4500
+Wire Wire Line
+	7500 3500 6000 3500
+Connection ~ 6000 3500
 $EndSCHEMATC

Commit message: Add files via upload
Parts:
- R7: footprint Resistor_THT:R_Axial_DIN0309_L9.0mm_D3.2mm_P15.24mm_Horizontal -> Resistor_THT:R_Axial_DIN0309_L9.0mm_D3.2mm_P12.70mm_Horizontal
Changed lines of the file:
@@
 F 0 "R7" H 5320 3796 50  0000 L CNN
 F 1 "470 0,5W" H 5320 3705 50  0000 L CNN
-F 2 "Resistor_THT:R_Axial_DIN0309_L9.0mm_D3.2mm_P15.24mm_Horizontal" V 5180 3750 50  0001 C CNN
+F 2 "Resistor_THT:R_Axial_DIN0309_L9.0mm_D3.2mm_P12.70mm_Horizontal" V 5180 3750 50  0001 C CNN
 F 3 "~" H 5250 3750 50  0001 C CNN
 	1    5250 3750
