File: furnace/furnace_230V/MCU.sch (KiCad schematic (older format))
At the start: 1 part

Commit message: Add files via upload
Parts:
- added C?: 1u, Capacitor_SMD:C_0603_1608Metric_Pad1.08x0.95mm_HandSolder, symbol Device:C
- added C?: 0,1, Capacitor_SMD:C_0603_1608Metric_Pad1.08x0.95mm_HandSolder, symbol Device:C
- added TP?: TestPoint, symbol Connector:TestPoint
Connections:
- net labels added: +3V3, 1-WIRE, AIN2, AIN6, CURR, GND, SWIM, TEMP_SDA, UART_TX, VOLT
- wire segments 0 -> 22
Other:
- note added: "MCU"
- note added: "Programming"
Changed lines of the file:
@@
 L MCU_ST_STM8:STM8S001J3M U?
 U 1 1 60AACB00
-P 5550 3800
-F 0 "U?" H 5550 4381 50  0000 C CNN
-F 1 "STM8S001J3M" H 5550 4290 50  0000 C CNN
-F 2 "Package_SO:SO-8_3.9x4.9mm_P1.27mm" H 5600 4350 50  0001 L CNN
-F 3 "https://www.st.com/resource/en/datasheet/stm8s001j3.pdf" H 5450 3900 50  0001 C CNN
-	1    5550 3800
+P 6300 4300
+F 0 "U?" H 6850 4800 50  0000 C CNN
+F 1 "STM8S001J3M" H 7000 4700 50  0000 C CNN
+F 2 "Package_SO:SO-8_3.9x4.9mm_P1.27mm" H 6350 4850 50  0001 L CNN
+F 3 "https://www.st.com/resource/en/datasheet/stm8s001j3.pdf" H 6200 4400 50  0001 C CNN
+	1    6300 4300
 	1    0    0    -1
 $EndComp
+$Comp
+L Device:C C?
+U 1 1 60ACBC6E
+P 5500 4650
+AR Path="/60ACBC6E" Ref="C?"  Part="1"
+AR Path="/609CA6A8/609D24C0/60ACBC6E" Ref="C?"  Part="1"
+AR Path="/609CA6A8/60A08E0B/60ACBC6E" Ref="C?"  Part="1"
+AR Path="/609CA6A8/60A0A46E/60ACBC6E" Ref="C?"  Part="1"
+AR Path="/609CA6A8/60A0A500/60ACBC6E" Ref="C?"  Part="1"
+AR Path="/609CA6A8/60A0A922/60ACBC6E" Ref="C?"  Part="1"
+AR Path="/609CA6A8/60ACBC6E" Ref="C?"  Part="1"
+AR Path="/609CA6A8/60AE5653/60ACBC6E" Ref="C?"  Part="1"
+AR Path="/60AAC605/60ACBC6E" Ref="C?"  Part="1"
+AR Path="/60AABDBE/60ACBC6E" Ref="C?"  Part="1"
+F 0 "C?" H 5615 4696 50  0000 L CNN
+F 1 "1u" H 5615 4605 50  0000 L CNN
+F 2 "Capacitor_SMD:C_0603_1608Metric_Pad1.08x0.95mm_HandSolder" H 5538 4500 50  0001 C CNN
+F 3 "~" H 5500 4650 50  0001 C CNN
+	1    5500 4650
+	1    0    0    -1
+$EndComp
+$Comp
+L Device:C C?
+U 1 1 60ACBEC0
+P 5500 3650
+AR Path="/60ACBEC0" Ref="C?"  Part="1"
+AR Path="/609CA6A8/609D24C0/60ACBEC0" Ref="C?"  Part="1"
+AR Path="/609CA6A8/60A08E0B/60ACBEC0" Ref="C?"  Part="1"
+AR Path="/609CA6A8/60A0A46E/60ACBEC0" Ref="C?"  Part="1"
+AR Path="/609CA6A8/60A0A500/60ACBEC0" Ref="C?"  Part="1"
+AR Path="/609CA6A8/60A0A922/60ACBEC0" Ref="C?"  Part="1"
+AR Path="/609CA6A8/60ACBEC0" Ref="C?"  Part="1"
+AR Path="/609CA6A8/60AE5653/60ACBEC0" Ref="C?"  Part="1"
+AR Path="/60AAC605/60ACBEC0" Ref="C?"  Part="1"
+AR Path="/60AABDBE/60ACBEC0" Ref="C?"  Part="1"
+F 0 "C?" H 5615 3696 50  0000 L CNN
+F 1 "0,1" H 5615 3605 50  0000 L CNN
+F 2 "Capacitor_SMD:C_0603_1608Metric_Pad1.08x0.95mm_HandSolder" H 5538 3500 50  0001 C CNN
+F 3 "~" H 5500 3650 50  0001 C CNN
+	1    5500 3650
+	1    0    0    -1
+$EndComp
+Text Notes 6600 2250 2    197  ~ 0
+MCU
+Text Label 5800 4200 2    50   ~ 0
+1-WIRE
+Text Label 6800 4400 0    50   ~ 0
+AIN2
+Text Label 6800 4200 0    50   ~ 0
+AIN6
+Text Label 5800 4300 2    50   ~ 0
+UART_TX
+Text Label 6800 4300 0    50   ~ 0
+SWIM
+$Comp
+L Connector:TestPoint TP?
+U 1 1 60B590E5
+P 4500 4000
+AR Path="/60B590E5" Ref="TP?"  Part="1"
+AR Path="/609CA6A8/60AE5653/60B590E5" Ref="TP?"  Part="1"
+AR Path="/60AAC605/60B590E5" Ref="TP?"  Part="1"
+AR Path="/60AAE4BD/60B590E5" Ref="TP?"  Part="1"
+F 0 "TP?" V 4558 4118 50  0000 L CNN
+F 1 "TestPoint" H 4558 4027 50  0001 L CNN
+F 2 "" H 4700 4000 50  0001 C CNN
+F 3 "~" H 4700 4000 50  0001 C CNN
+	1    4500 4000
+	0    -1   -1   0
+$EndComp
+Text Notes 4500 3800 2    50   ~ 0
+Programming
+Text Label 4600 4000 0    50   ~ 0
+SWIM
+Text HLabel 8500 4000 2    50   Output ~ 0
+UART_TX
+Text HLabel 3000 3000 0    50   Input ~ 0
++3V3
+Text HLabel 3000 5000 0    50   Input ~ 0
+GND
+Text HLabel 3000 4000 0    50   Input ~ 0
+VOLT
+Text HLabel 3000 3500 0    50   BiDi ~ 0
+TEMP_SDA
+Text HLabel 3000 4500 0    50   Input ~ 0
+CURR
+Text Label 3500 4000 0    50   ~ 0
+AIN2
+Text Label 3500 4500 0    50   ~ 0
+AIN6
+Text Label 3500 3500 0    50   ~ 0
+1-WIRE
+Wire Wire Line
+	4500 4000 4600 4000
+Wire Wire Line
+	5800 4200 5900 4200
+Wire Wire Line
+	5800 4300 5900 4300
+Wire Wire Line
+	6700 4200 6800 4200
+Wire Wire Line
+	6700 4300 6800 4300
+Wire Wire Line
+	6700 4400 6800 4400
+Wire Wire Line
+	5500 4500 5900 4500
+Wire Wire Line
+	3000 3500 3500 3500
+Wire Wire Line
+	3000 4000 3500 4000
+Wire Wire Line
+	3000 4500 3500 4500
+Wire Wire Line
+	3000 5000 5250 5000
+Wire Wire Line
+	6300 5000 6300 4700
+Wire Wire Line
+	5500 4800 5500 5000
+Connection ~ 5500 5000
+Wire Wire Line
+	5500 5000 6300 5000
+Wire Wire Line
+	5500 3800 5250 3800
+Wire Wire Line
+	5250 3800 5250 5000
+Connection ~ 5250 5000
+Wire Wire Line
+	5250 5000 5500 5000
+Wire Wire Line
+	3000 3000 5500 3000
+Wire Wire Line
+	6300 3000 6300 3900
+Wire Wire Line
+	5500 3500 5500 3000
+Connection ~ 5500 3000
+Wire Wire Line
+	5500 3000 6300 3000
+Text Label 8000 4000 2    50   ~ 0
+UART_TX
+Wire Wire Line
+	8000 4000 8500 4000
 $EndSCHEMATC

Commit message: Add files via upload
Parts:
- C6, C7: renamed from C?; symbol Device:C -> furnace_230V-rescue:C-Device
- TP3: renamed from TP?; symbol Connector:TestPoint -> furnace_230V-rescue:TestPoint-Connector
- U1: renamed from U?; symbol MCU_ST_STM8:STM8S001J3M -> furnace_230V-rescue:STM8S001J3M-MCU_ST_STM8
Changed lines of the file:
@@
 $EndDescr
 $Comp
-L MCU_ST_STM8:STM8S001J3M U?
+L furnace_230V-rescue:STM8S001J3M-MCU_ST_STM8 U1
 U 1 1 60AACB00
 P 6300 4300
-F 0 "U?" H 6850 4800 50  0000 C CNN
+F 0 "U1" H 6850 4800 50  0000 C CNN
 F 1 "STM8S001J3M" H 7000 4700 50  0000 C CNN
 F 2 "Package_SO:SO-8_3.9x4.9mm_P1.27mm" H 6350 4850 50  0001 L CNN
@@
 $EndComp
 $Comp
-L Device:C C?
+L furnace_230V-rescue:C-Device C?
 U 1 1 60ACBC6E
 P 5500 4650
@@
 AR Path="/609CA6A8/60AE5653/60ACBC6E" Ref="C?"  Part="1"
 AR Path="/60AAC605/60ACBC6E" Ref="C?"  Part="1"
-AR Path="/60AABDBE/60ACBC6E" Ref="C?"  Part="1"
-F 0 "C?" H 5615 4696 50  0000 L CNN
+AR Path="/60AABDBE/60ACBC6E" Ref="C7"  Part="1"
+F 0 "C7" H 5615 4696 50  0000 L CNN
 F 1 "1u" H 5615 4605 50  0000 L CNN
 F 2 "Capacitor_SMD:C_0603_1608Metric_Pad1.08x0.95mm_HandSolder" H 5538 4500 50  0001 C CNN
@@
 $EndComp
 $Comp
-L Device:C C?
+L furnace_230V-rescue:C-Device C?
 U 1 1 60ACBEC0
 P 5500 3650
@@
 AR Path="/609CA6A8/60AE5653/60ACBEC0" Ref="C?"  Part="1"
 AR Path="/60AAC605/60ACBEC0" Ref="C?"  Part="1"
-AR Path="/60AABDBE/60ACBEC0" Ref="C?"  Part="1"
-F 0 "C?" H 5615 3696 50  0000 L CNN
+AR Path="/60AABDBE/60ACBEC0" Ref="C6"  Part="1"
+F 0 "C6" H 5615 3696 50  0000 L CNN
 F 1 "0,1" H 5615 3605 50  0000 L CNN
 F 2 "Capacitor_SMD:C_0603_1608Metric_Pad1.08x0.95mm_HandSolder" H 5538 3500 50  0001 C CNN
@@
 SWIM
 $Comp
-L Connector:TestPoint TP?
+L furnace_230V-rescue:TestPoint-Connector TP?
 U 1 1 60B590E5
 P 4500 4000
@@
 AR Path="/60AAC605/60B590E5" Ref="TP?"  Part="1"
 AR Path="/60AAE4BD/60B590E5" Ref="TP?"  Part="1"
-AR Path="/60AABDBE/60B590E5" Ref="TP?"  Part="1"
-F 0 "TP?" V 4558 4118 50  0000 L CNN
+AR Path="/60AABDBE/60B590E5" Ref="TP3"  Part="1"
+F 0 "TP3" V 4558 4118 50  0000 L CNN
 F 1 "TestPoint" H 4558 4027 50  0001 L CNN
 F 2 "" H 4700 4000 50  0001 C CNN

Commit message: Add files via upload
Parts:
- TP3: footprint (none) -> MountingHole:MountingHole_2.2mm_M2_DIN965_Pad_TopBottom
Changed lines of the file:
@@
 F 0 "TP3" V 4558 4118 50  0000 L CNN
 F 1 "TestPoint" H 4558 4027 50  0001 L CNN
-F 2 "" H 4700 4000 50  0001 C CNN
+F 2 "MountingHole:MountingHole_2.2mm_M2_DIN965_Pad_TopBottom" H 4700 4000 50  0001 C CNN
 F 3 "~" H 4700 4000 50  0001 C CNN
 	1    4500 4000

Commit message: Add files via upload
Parts:
- C6, C7: footprint Capacitor_SMD:C_0603_1608Metric_Pad1.08x0.95mm_HandSolder -> Capacitor_SMD:C_0603_1608Metric_Pad1.05x0.95mm_HandSolder
- TP3: footprint MountingHole:MountingHole_2.2mm_M2_DIN965_Pad_TopBottom -> furnace_230V:TP
- U1: footprint Package_SO:SO-8_3.9x4.9mm_P1.27mm -> Package_SO:SOIC-8_3.9x4.9mm_P1.27mm
Changed lines of the file:
@@
 F 0 "U1" H 6850 4800 50  0000 C CNN
 F 1 "STM8S001J3M" H 7000 4700 50  0000 C CNN
-F 2 "Package_SO:SO-8_3.9x4.9mm_P1.27mm" H 6350 4850 50  0001 L CNN
+F 2 "Package_SO:SOIC-8_3.9x4.9mm_P1.27mm" H 6350 4850 50  0001 L CNN
 F 3 "https://www.st.com/resource/en/datasheet/stm8s001j3.pdf" H 6200 4400 50  0001 C CNN
 	1    6300 4300
@@
 F 0 "C7" H 5615 4696 50  0000 L CNN
 F 1 "1u" H 5615 4605 50  0000 L CNN
-F 2 "Capacitor_SMD:C_0603_1608Metric_Pad1.08x0.95mm_HandSolder" H 5538 4500 50  0001 C CNN
+F 2 "Capacitor_SMD:C_0603_1608Metric_Pad1.05x0.95mm_HandSolder" H 5538 4500 50  0001 C CNN
 F 3 "~" H 5500 4650 50  0001 C CNN
 	1    5500 4650
@@
 F 0 "C6" H 5615 3696 50  0000 L CNN
 F 1 "0,1" H 5615 3605 50  0000 L CNN
-F 2 "Capacitor_SMD:C_0603_1608Metric_Pad1.08x0.95mm_HandSolder" H 5538 3500 50  0001 C CNN
+F 2 "Capacitor_SMD:C_0603_1608Metric_Pad1.05x0.95mm_HandSolder" H 5538 3500 50  0001 C CNN
 F 3 "~" H 5500 3650 50  0001 C CNN
 	1    5500 3650
@@
 F 0 "TP3" V 4558 4118 50  0000 L CNN
 F 1 "TestPoint" H 4558 4027 50  0001 L CNN
-F 2 "MountingHole:MountingHole_2.2mm_M2_DIN965_Pad_TopBottom" H 4700 4000 50  0001 C CNN
+F 2 "furnace_230V:TP" H 4700 4000 50  0001 C CNN
 F 3 "~" H 4700 4000 50  0001 C CNN
 	1    4500 4000

Commit message: Add files via upload
Parts:
- C6, C7: footprint Capacitor_SMD:C_0603_1608Metric_Pad1.05x0.95mm_HandSolder -> Capacitor_SMD:C_0603_1608Metric_Pad1.08x0.95mm_HandSolder
- TP3: footprint furnace_230V:TP -> MountingHole:MountingHole_2.2mm_M2_DIN965_Pad_TopBottom
- U1: footprint Package_SO:SOIC-8_3.9x4.9mm_P1.27mm -> Package_SO:SO-8_3.9x4.9mm_P1.27mm
Changed lines of the file:
@@
 F 0 "U1" H 6850 4800 50  0000 C CNN
 F 1 "STM8S001J3M" H 7000 4700 50  0000 C CNN
-F 2 "Package_SO:SOIC-8_3.9x4.9mm_P1.27mm" H 6350 4850 50  0001 L CNN
+F 2 "Package_SO:SO-8_3.9x4.9mm_P1.27mm" H 6350 4850 50  0001 L CNN
 F 3 "https://www.st.com/resource/en/datasheet/stm8s001j3.pdf" H 6200 4400 50  0001 C CNN
 	1    6300 4300
@@
 F 0 "C7" H 5615 4696 50  0000 L CNN
 F 1 "1u" H 5615 4605 50  0000 L CNN
-F 2 "Capacitor_SMD:C_0603_1608Metric_Pad1.05x0.95mm_HandSolder" H 5538 4500 50  0001 C CNN
+F 2 "Capacitor_SMD:C_0603_1608Metric_Pad1.08x0.95mm_HandSolder" H 5538 4500 50  0001 C CNN
 F 3 "~" H 5500 4650 50  0001 C CNN
 	1    5500 4650
@@
 F 0 "C6" H 5615 3696 50  0000 L CNN
 F 1 "0,1" H 5615 3605 50  0000 L CNN
-F 2 "Capacitor_SMD:C_0603_1608Metric_Pad1.05x0.95mm_HandSolder" H 5538 3500 50  0001 C CNN
+F 2 "Capacitor_SMD:C_0603_1608Metric_Pad1.08x0.95mm_HandSolder" H 5538 3500 50  0001 C CNN
 F 3 "~" H 5500 3650 50  0001 C CNN
 	1    5500 3650
@@
 F 0 "TP3" V 4558 4118 50  0000 L CNN
 F 1 "TestPoint" H 4558 4027 50  0001 L CNN
-F 2 "furnace_230V:TP" H 4700 4000 50  0001 C CNN
+F 2 "MountingHole:MountingHole_2.2mm_M2_DIN965_Pad_TopBottom" H 4700 4000 50  0001 C CNN
 F 3 "~" H 4700 4000 50  0001 C CNN
 	1    4500 4000
