File: furnace/furnace_230V/Optoisolator.sch (KiCad schematic (older format))
At the start: 4 parts, among them U5 H11L1

Commit message: Add files via upload
Parts:
- TP10: footprint furnace_230V:TP -> MountingHole:MountingHole_2.2mm_M2_DIN965_Pad_TopBottom
- U5: footprint Package_DIP:DIP-6_W7.62mm_LongPads -> Package_DIP:DIP-6_W7.62mm_SMDSocket_SmallPads
- renumbered R14 to R15, R15 to R16
Changed lines of the file:
@@
 F 0 "U5" H 6644 4146 50  0000 L CNN
 F 1 "H11L1" H 6644 4055 50  0000 L CNN
-F 2 "Package_DIP:DIP-6_W7.62mm_LongPads" H 6210 4100 50  0001 C CNN
+F 2 "Package_DIP:DIP-6_W7.62mm_SMDSocket_SmallPads" H 6210 4100 50  0001 C CNN
 F 3 "https://www.onsemi.com/pub/Collateral/H11L3M-D.PDF" H 6210 4100 50  0001 C CNN
 	1    6300 4100
@@
 P 5350 4000
 AR Path="/60AAE0B8/60AC1EDD" Ref="R?"  Part="1"
-AR Path="/60AAEC6C/60AC1EDD" Ref="R14"  Part="1"
-F 0 "R14" V 5250 4000 50  0000 C CNN
+AR Path="/60AAEC6C/60AC1EDD" Ref="R15"  Part="1"
+F 0 "R15" V 5250 4000 50  0000 C CNN
 F 1 "680" V 5450 4000 50  0000 C CNN
 F 2 "Resistor_SMD:R_0603_1608Metric_Pad1.05x0.95mm_HandSolder" V 5280 4000 50  0001 C CNN
@@
 P 7000 3850
 AR Path="/60AAE0B8/60AC2929" Ref="R?"  Part="1"
-AR Path="/60AAEC6C/60AC2929" Ref="R15"  Part="1"
-F 0 "R15" H 7100 3950 50  0000 C CNN
+AR Path="/60AAEC6C/60AC2929" Ref="R16"  Part="1"
+F 0 "R16" H 7100 3950 50  0000 C CNN
 F 1 "3,3k" H 7150 3850 50  0000 C CNN
 F 2 "Resistor_SMD:R_0603_1608Metric_Pad1.05x0.95mm_HandSolder" V 6930 3850 50  0001 C CNN
@@
 F 0 "TP10" H 5058 4118 50  0000 L CNN
 F 1 "TestPoint" H 5058 4027 50  0001 L CNN
-F 2 "furnace_230V:TP" H 5200 4000 50  0001 C CNN
+F 2 "MountingHole:MountingHole_2.2mm_M2_DIN965_Pad_TopBottom" H 5200 4000 50  0001 C CNN
 F 3 "~" H 5200 4000 50  0001 C CNN
 	1    5000 4000
