File: furnace/furnace_230V/Optoisolator.sch (KiCad schematic (older format))
At the start: 1 part

Commit message: Add files via upload
Parts:
- added R?: 680, Resistor_SMD:R_0603_1608Metric_Pad1.05x0.95mm_HandSolder, symbol Device:R
- added R?: 3,3k, Resistor_SMD:R_0603_1608Metric_Pad1.05x0.95mm_HandSolder, symbol Device:R
- added TP?: TestPoint, symbol Connector:TestPoint
Connections:
- net labels added: +5V, GND1, GND2, IN, OUT
- wire segments 0 -> 14
Other:
- note added: "UART isolator"
Changed lines of the file:
@@
 L Isolator:H11L1 U?
 U 1 1 60AB014C
-P 5300 3950
-F 0 "U?" H 5644 3996 50  0000 L CNN
-F 1 "H11L1" H 5644 3905 50  0000 L CNN
-F 2 "" H 5210 3950 50  0001 C CNN
-F 3 "https://www.onsemi.com/pub/Collateral/H11L3M-D.PDF" H 5210 3950 50  0001 C CNN
-	1    5300 3950
+P 6300 4100
+F 0 "U?" H 6644 4146 50  0000 L CNN
+F 1 "H11L1" H 6644 4055 50  0000 L CNN
+F 2 "" H 6210 4100 50  0001 C CNN
+F 3 "https://www.onsemi.com/pub/Collateral/H11L3M-D.PDF" H 6210 4100 50  0001 C CNN
+	1    6300 4100
 	1    0    0    -1
 $EndComp
+$Comp
+L Device:R R?
+U 1 1 60AC1EDD
+P 5350 4000
+AR Path="/60AAE0B8/60AC1EDD" Ref="R?"  Part="1"
+AR Path="/60AAEC6C/60AC1EDD" Ref="R?"  Part="1"
+F 0 "R?" V 5250 4000 50  0000 C CNN
+F 1 "680" V 5450 4000 50  0000 C CNN
+F 2 "Resistor_SMD:R_0603_1608Metric_Pad1.05x0.95mm_HandSolder" V 5280 4000 50  0001 C CNN
+F 3 "~" H 5350 4000 50  0001 C CNN
+	1    5350 4000
+	0    1    1    0
+$EndComp
+$Comp
+L Device:R R?
+U 1 1 60AC2929
+P 7000 3850
+AR Path="/60AAE0B8/60AC2929" Ref="R?"  Part="1"
+AR Path="/60AAEC6C/60AC2929" Ref="R?"  Part="1"
+F 0 "R?" H 7100 3950 50  0000 C CNN
+F 1 "3,3k" H 7150 3850 50  0000 C CNN
+F 2 "Resistor_SMD:R_0603_1608Metric_Pad1.05x0.95mm_HandSolder" V 6930 3850 50  0001 C CNN
+F 3 "~" H 7000 3850 50  0001 C CNN
+	1    7000 3850
+	1    0    0    -1
+$EndComp
+$Comp
+L Connector:TestPoint TP?
+U 1 1 60ACF622
+P 5000 4000
+AR Path="/60ACF622" Ref="TP?"  Part="1"
+AR Path="/609CA6A8/60AE5653/60ACF622" Ref="TP?"  Part="1"
+AR Path="/60AAC605/60ACF622" Ref="TP?"  Part="1"
+AR Path="/60AAEC6C/60ACF622" Ref="TP?"  Part="1"
+F 0 "TP?" H 5058 4118 50  0000 L CNN
+F 1 "TestPoint" H 5058 4027 50  0001 L CNN
+F 2 "" H 5200 4000 50  0001 C CNN
+F 3 "~" H 5200 4000 50  0001 C CNN
+	1    5000 4000
+	1    0    0    -1
+$EndComp
+Text Notes 7100 2300 2    197  ~ 0
+UART isolator
+Text HLabel 4500 4000 0    50   Input ~ 0
+IN
+Text HLabel 4500 4500 0    50   Input ~ 0
+GND1
+Text HLabel 7500 3500 2    50   Input ~ 0
++5V
+Text HLabel 7500 4500 2    50   Input ~ 0
+GND2
+Text HLabel 7500 4000 2    50   Output ~ 0
+OUT
+Wire Wire Line
+	4500 4000 5000 4000
+Wire Wire Line
+	5000 4000 5200 4000
+Connection ~ 5000 4000
+Wire Wire Line
+	5500 4000 6000 4000
+Wire Wire Line
+	6000 4200 6000 4500
+Wire Wire Line
+	6000 4500 4500 4500
+Wire Wire Line
+	6300 3800 6300 3500
+Wire Wire Line
+	6300 3500 7000 3500
+Wire Wire Line
+	7000 3700 7000 3500
+Connection ~ 7000 3500
+Wire Wire Line
+	7000 3500 7500 3500
+Wire Wire Line
+	6600 4100 7000 4100
+Wire Wire Line
+	7000 4100 7000 4000
+Wire Wire Line
+	7000 4000 7500 4000
+Connection ~ 7000 4000
+Wire Wire Line
+	6300 4400 6300 4500
+Wire Wire Line
+	6300 4500 7500 4500
 $EndSCHEMATC

Commit message: Add files via upload
Parts:
- R15, R16: renamed from R?; symbol Device:R -> furnace_230V-rescue:R-Device
- TP10: renamed from TP?; symbol Connector:TestPoint -> furnace_230V-rescue:TestPoint-Connector
- U5: renamed from U?; symbol Isolator:H11L1 -> furnace_230V-rescue:H11L1-Isolator
Changed lines of the file:
@@
 $Descr A4 11693 8268
 encoding utf-8
-Sheet 9 9
+Sheet 8 9
 Title ""
 Date ""
@@
 $EndDescr
 $Comp
-L Isolator:H11L1 U?
+L furnace_230V-rescue:H11L1-Isolator U5
 U 1 1 60AB014C
 P 6300 4100
-F 0 "U?" H 6644 4146 50  0000 L CNN
+F 0 "U5" H 6644 4146 50  0000 L CNN
 F 1 "H11L1" H 6644 4055 50  0000 L CNN
 F 2 "" H 6210 4100 50  0001 C CNN
@@
 $EndComp
 $Comp
-L Device:R R?
+L furnace_230V-rescue:R-Device R?
 U 1 1 60AC1EDD
 P 5350 4000
 AR Path="/60AAE0B8/60AC1EDD" Ref="R?"  Part="1"
-AR Path="/60AAEC6C/60AC1EDD" Ref="R?"  Part="1"
-F 0 "R?" V 5250 4000 50  0000 C CNN
+AR Path="/60AAEC6C/60AC1EDD" Ref="R15"  Part="1"
+F 0 "R15" V 5250 4000 50  0000 C CNN
 F 1 "680" V 5450 4000 50  0000 C CNN
 F 2 "Resistor_SMD:R_0603_1608Metric_Pad1.05x0.95mm_HandSolder" V 5280 4000 50  0001 C CNN
@@
 $EndComp
 $Comp
-L Device:R R?
+L furnace_230V-rescue:R-Device R?
 U 1 1 60AC2929
 P 7000 3850
 AR Path="/60AAE0B8/60AC2929" Ref="R?"  Part="1"
-AR Path="/60AAEC6C/60AC2929" Ref="R?"  Part="1"
-F 0 "R?" H 7100 3950 50  0000 C CNN
+AR Path="/60AAEC6C/60AC2929" Ref="R16"  Part="1"
+F 0 "R16" H 7100 3950 50  0000 C CNN
 F 1 "3,3k" H 7150 3850 50  0000 C CNN
 F 2 "Resistor_SMD:R_0603_1608Metric_Pad1.05x0.95mm_HandSolder" V 6930 3850 50  0001 C CNN
@@
 $EndComp
 $Comp
-L Connector:TestPoint TP?
+L furnace_230V-rescue:TestPoint-Connector TP?
 U 1 1 60ACF622
 P 5000 4000
@@
 AR Path="/609CA6A8/60AE5653/60ACF622" Ref="TP?"  Part="1"
 AR Path="/60AAC605/60ACF622" Ref="TP?"  Part="1"
-AR Path="/60AAEC6C/60ACF622" Ref="TP?"  Part="1"
-F 0 "TP?" H 5058 4118 50  0000 L CNN
+AR Path="/60AAEC6C/60ACF622" Ref="TP10"  Part="1"
+F 0 "TP10" H 5058 4118 50  0000 L CNN
 F 1 "TestPoint" H 5058 4027 50  0001 L CNN
 F 2 "" H 5200 4000 50  0001 C CNN

Commit message: Add files via upload
Parts:
- TP10: footprint (none) -> MountingHole:MountingHole_2.2mm_M2_DIN965_Pad_TopBottom
- U5: footprint (none) -> Package_DIP:DIP-6_W7.62mm_SMDSocket_SmallPads
Changed lines of the file:
@@
 F 0 "U5" H 6644 4146 50  0000 L CNN
 F 1 "H11L1" H 6644 4055 50  0000 L CNN
-F 2 "" H 6210 4100 50  0001 C CNN
+F 2 "Package_DIP:DIP-6_W7.62mm_SMDSocket_SmallPads" H 6210 4100 50  0001 C CNN
 F 3 "https://www.onsemi.com/pub/Collateral/H11L3M-D.PDF" H 6210 4100 50  0001 C CNN
 	1    6300 4100
@@
 F 0 "TP10" H 5058 4118 50  0000 L CNN
 F 1 "TestPoint" H 5058 4027 50  0001 L CNN
-F 2 "" H 5200 4000 50  0001 C CNN
+F 2 "MountingHole:MountingHole_2.2mm_M2_DIN965_Pad_TopBottom" H 5200 4000 50  0001 C CNN
 F 3 "~" H 5200 4000 50  0001 C CNN
 	1    5000 4000

Commit message: Add files via upload
Parts:
- TP10: footprint MountingHole:MountingHole_2.2mm_M2_DIN965_Pad_TopBottom -> furnace_230V:TP
- U5: footprint Package_DIP:DIP-6_W7.62mm_SMDSocket_SmallPads -> Package_DIP:DIP-6_W7.62mm_LongPads
- renumbered R15 to R14, R16 to R15
Changed lines of the file:
@@
 F 0 "U5" H 6644 4146 50  0000 L CNN
 F 1 "H11L1" H 6644 4055 50  0000 L CNN
-F 2 "Package_DIP:DIP-6_W7.62mm_SMDSocket_SmallPads" H 6210 4100 50  0001 C CNN
+F 2 "Package_DIP:DIP-6_W7.62mm_LongPads" H 6210 4100 50  0001 C CNN
 F 3 "https://www.onsemi.com/pub/Collateral/H11L3M-D.PDF" H 6210 4100 50  0001 C CNN
 	1    6300 4100
@@
 P 5350 4000
 AR Path="/60AAE0B8/60AC1EDD" Ref="R?"  Part="1"
-AR Path="/60AAEC6C/60AC1EDD" Ref="R15"  Part="1"
-F 0 "R15" V 5250 4000 50  0000 C CNN
+AR Path="/60AAEC6C/60AC1EDD" Ref="R14"  Part="1"
+F 0 "R14" V 5250 4000 50  0000 C CNN
 F 1 "680" V 5450 4000 50  0000 C CNN
 F 2 "Resistor_SMD:R_0603_1608Metric_Pad1.05x0.95mm_HandSolder" V 5280 4000 50  0001 C CNN
@@
 P 7000 3850
 AR Path="/60AAE0B8/60AC2929" Ref="R?"  Part="1"
-AR Path="/60AAEC6C/60AC2929" Ref="R16"  Part="1"
-F 0 "R16" H 7100 3950 50  0000 C CNN
+AR Path="/60AAEC6C/60AC2929" Ref="R15"  Part="1"
+F 0 "R15" H 7100 3950 50  0000 C CNN
 F 1 "3,3k" H 7150 3850 50  0000 C CNN
 F 2 "Resistor_SMD:R_0603_1608Metric_Pad1.05x0.95mm_HandSolder" V 6930 3850 50  0001 C CNN
@@
 F 0 "TP10" H 5058 4118 50  0000 L CNN
 F 1 "TestPoint" H 5058 4027 50  0001 L CNN
-F 2 "MountingHole:MountingHole_2.2mm_M2_DIN965_Pad_TopBottom" H 5200 4000 50  0001 C CNN
+F 2 "furnace_230V:TP" H 5200 4000 50  0001 C CNN
 F 3 "~" H 5200 4000 50  0001 C CNN
 	1    5000 4000
