File: furnace/furnace_230V/furnace_230V.sch (KiCad schematic (older format))
At the start: 9 parts

Commit message: Add files via upload
Parts:
- removed Q?: BTA16-600B, Package_TO_SOT_THT:TO-220-3_Vertical, symbol Triac_Thyristor:BTA16-600B
- removed R?: 470 0,5W, symbol Device:R
- removed U?: MOC3052M, symbol Relay_SolidState:MOC3052M
- removed U?: LM321, Package_TO_SOT_SMD:SOT-23-5, symbol Amplifier_Operational:LM321
- removed U?: DS18B20, Package_TO_SOT_THT:TO-92_Inline, symbol Sensor_Temperature:DS18B20
- removed U?: STM8S001J3M, Package_SO:SO-8_3.9x4.9mm_P1.27mm, symbol MCU_ST_STM8:STM8S001J3M
- removed U?: H11L1, symbol Isolator:H11L1
- removed U?: TLV70233_SOT23-5, Package_TO_SOT_SMD:SOT-23-5, symbol Regulator_Linear:TLV70233_SOT23-5
- added J?: CWF-4R, symbol Connector_Generic:Conn_01x04
- added J? (x2): TC0, symbol Connector:Screw_Terminal_01x02
Changed lines of the file:
@@
 $Descr A4 11693 8268
 encoding utf-8
-Sheet 1 1
+Sheet 1 9
 Title ""
 Date ""
@@
 Comment4 ""
 $EndDescr
-$Comp
-L Triac_Thyristor:BTA16-600B Q?
-U 1 1 609B5246
-P 5000 3850
-F 0 "Q?" H 5129 3896 50  0000 L CNN
-F 1 "BTA16-600B" H 5129 3805 50  0000 L CNN
-F 2 "Package_TO_SOT_THT:TO-220-3_Vertical" H 5200 3775 50  0001 L CIN
-F 3 "https://www.st.com/resource/en/datasheet/bta16.pdf" H 5000 3850 50  0001 L CNN
-	1    5000 3850
-	1    0    0    -1
-$EndComp
-$Comp
-L Relay_SolidState:MOC3052M U?
-U 1 1 609B6C4B
-P 3800 4100
-F 0 "U?" H 3800 4425 50  0000 C CNN
-F 1 "MOC3052M" H 3800 4334 50  0000 C CNN
-F 2 "" H 3600 3900 50  0001 L CIN
-F 3 "https://www.onsemi.com/pub/Collateral/MOC3052M-D.PDF" H 3800 4100 50  0001 L CNN
-	1    3800 4100
-	1    0    0    -1
-$EndComp
-$Comp
-L Device:R R?
-U 1 1 609B85C9
-P 4150 3450
-F 0 "R?" H 4220 3496 50  0000 L CNN
-F 1 "470 0,5W" H 4220 3405 50  0000 L CNN
-F 2 "" V 4080 3450 50  0001 C CNN
-F 3 "~" H 4150 3450 50  0001 C CNN
-	1    4150 3450
-	1    0    0    -1
-$EndComp
 $Comp
 L Amplifier_Operational:LM321 U?
@@
 $EndComp
 $Comp
-L Amplifier_Operational:LM321 U?
-U 1 1 609BC368
-P 4600 4750
-F 0 "U?" H 4944 4796 50  0000 L CNN
-F 1 "LM321" H 4944 4705 50  0000 L CNN
-F 2 "Package_TO_SOT_SMD:SOT-23-5" H 4600 4750 50  0001 C CNN
-F 3 "http://www.ti.com/lit/ds/symlink/lm321.pdf" H 4600 4750 50  0001 C CNN
-	1    4600 4750
+L Connector_Generic:Conn_01x04 J?
+U 1 1 60AAE60F
+P 2650 2400
+AR Path="/60AAC03E/60AAE60F" Ref="J?"  Part="1"
+AR Path="/60AAE60F" Ref="J?"  Part="1"
+F 0 "J?" H 2730 2392 50  0000 L CNN
+F 1 "CWF-4R" H 2730 2301 50  0000 L CNN
+F 2 "" H 2650 2400 50  0001 C CNN
+F 3 "~" H 2650 2400 50  0001 C CNN
+	1    2650 2400
 	1    0    0    -1
 $EndComp
 $Comp
-L Sensor_Temperature:DS18B20 U?
-U 1 1 609BCB04
-P 2750 3950
-F 0 "U?" H 2520 3996 50  0000 R CNN
-F 1 "DS18B20" H 2520 3905 50  0000 R CNN
-F 2 "Package_TO_SOT_THT:TO-92_Inline" H 1750 3700 50  0001 C CNN
-F 3 "http://datasheets.maximintegrated.com/en/ds/DS18B20.pdf" H 2600 4200 50  0001 C CNN
-	1    2750 3950
-	1    0    0    -1
+L Connector:Screw_Terminal_01x02 J?
+U 1 1 60AAEFEC
+P 1600 2850
+F 0 "J?" H 1680 2842 50  0000 L CNN
+F 1 "TC0" H 1680 2751 50  0000 L CNN
+F 2 "" H 1600 2850 50  0001 C CNN
+F 3 "~" H 1600 2850 50  0001 C CNN
+	1    1600 2850
+	-1   0    0    -1
 $EndComp
+$Sheet
+S 5000 5000 1000 500
+U 60AABABA
+F0 "AC-DC 5V" 50
+F1 "AC-DC 5V.sch" 50
+$EndSheet
+$Sheet
+S 5000 6000 1000 500
+U 60AABDBE
+F0 "MCU" 50
+F1 "MCU.sch" 50
+$EndSheet
+$Sheet
+S 6500 5000 1000 500
+U 60AAC605
+F0 "+3V3_ISOLATED" 50
+F1 "+3V3_isolated.sch" 50
+$EndSheet
+$Sheet
+S 6500 6000 1000 500
+U 60AAE0B8
+F0 "ISOLATED_TRIAC" 50
+F1 "Isolated_TRIAC.sch" 50
+$EndSheet
+$Sheet
+S 8000 5000 1000 500
+U 60AAE178
+F0 "TEMP_SENSOR" 50
+F1 "Temp_sensor.sch" 50
+$EndSheet
+$Sheet
+S 8000 6000 1000 500
+U 60AAE212
+F0 "CURRENT_SENSOR" 50
+F1 "Current_sensor.sch" 50
+$EndSheet
+$Sheet
+S 6000 4000 1000 500
+U 60AAE4BD
+F0 "VOLTAGE_DIVIDER" 50
+F1 "Voltage_divider.sch" 50
+$EndSheet
+$Sheet
+S 3000 6000 1000 500
+U 60AAEC6C
+F0 "OPTOISOLATOR" 50
+F1 "Optoisolator.sch" 50
+$EndSheet
 $Comp
-L MCU_ST_STM8:STM8S001J3M U?
-U 1 1 609BDB3F
-P 3500 5600
-F 0 "U?" H 3500 6181 50  0000 C CNN
-F 1 "STM8S001J3M" H 3500 6090 50  0000 C CNN
-F 2 "Package_SO:SO-8_3.9x4.9mm_P1.27mm" H 3550 6150 50  0001 L CNN
-F 3 "https://www.st.com/resource/en/datasheet/stm8s001j3.pdf" H 3400 5700 50  0001 C CNN
-	1    3500 5600
-	1    0    0    -1
-$EndComp
-$Comp
-L Isolator:H11L1 U?
-U 1 1 609BF0FD
-P 2100 5550
-F 0 "U?" H 2444 5596 50  0000 L CNN
-F 1 "H11L1" H 2444 5505 50  0000 L CNN
-F 2 "" H 2010 5550 50  0001 C CNN
-F 3 "https://www.onsemi.com/pub/Collateral/H11L3M-D.PDF" H 2010 5550 50  0001 C CNN
-	1    2100 5550
-	1    0    0    -1
-$EndComp
-$Comp
-L Regulator_Linear:TLV70233_SOT23-5 U?
-U 1 1 609C005A
-P 6200 4750
-F 0 "U?" H 6200 5092 50  0000 C CNN
-F 1 "TLV70233_SOT23-5" H 6200 5001 50  0000 C CNN
-F 2 "Package_TO_SOT_SMD:SOT-23-5" H 6200 5075 50  0001 C CIN
-F 3 "http://www.ti.com/lit/ds/symlink/tlv702.pdf" H 6200 4800 50  0001 C CNN
-	1    6200 4750
-	1    0    0    -1
+L Connector:Screw_Terminal_01x02 J?
+U 1 1 60AB629C
+P 1600 3400
+F 0 "J?" H 1680 3392 50  0000 L CNN
+F 1 "TC0" H 1680 3301 50  0000 L CNN
+F 2 "" H 1600 3400 50  0001 C CNN
+F 3 "~" H 1600 3400 50  0001 C CNN
+	1    1600 3400
+	-1   0    0    -1
 $EndComp
 $EndSCHEMATC

Commit message: Add files via upload
Changed lines of the file:
@@
 $EndComp
 $Sheet
-S 5000 5000 1000 500
+S 8500 2000 1000 500
 U 60AABABA
 F0 "AC-DC 5V" 50
 F1 "AC-DC 5V.sch" 50
+F2 "+5V" O R 9500 2100 50
+F3 "GND" O R 9500 2400 50
+F4 "AC1" I L 8500 2100 50
+F5 "AC2" I L 8500 2400 50
 $EndSheet
 $Sheet
-S 5000 6000 1000 500
+S 5000 4000 1000 800
 U 60AABDBE
 F0 "MCU" 50
 F1 "MCU.sch" 50
+F2 "UART_TX" O R 6000 4100 50
+F3 "+3V3" I L 5000 4100 50
+F4 "GND" I L 5000 4700 50
+F5 "VOLT" I L 5000 4400 50
+F6 "TEMP_SDA" B L 5000 4300 50
+F7 "CURR" I L 5000 4500 50
 $EndSheet
 $Sheet
-S 6500 5000 1000 500
+S 4000 2000 1000 500
 U 60AAC605
 F0 "+3V3_ISOLATED" 50
 F1 "+3V3_isolated.sch" 50
+F2 "+3V3_ISO" O R 5000 2100 50
+F3 "GND_ISO" O R 5000 2400 50
+F4 "+5V" I L 4000 2100 50
+F5 "GND" I L 4000 2400 50
 $EndSheet
 $Sheet
-S 6500 6000 1000 500
+S 7000 2000 1000 500
 U 60AAE0B8
 F0 "ISOLATED_TRIAC" 50
 F1 "Isolated_TRIAC.sch" 50
+F2 "AC" I R 8000 2100 50
+F3 "LOAD" O R 8000 2400 50
+F4 "+5V" I L 7000 2100 50
+F5 "~EN" I L 7000 2400 50
 $EndSheet
 $Sheet
-S 8000 5000 1000 500
+S 5000 3000 1000 500
 U 60AAE178
 F0 "TEMP_SENSOR" 50
 F1 "Temp_sensor.sch" 50
+F2 "SDA" B R 6000 3100 50
+F3 "+3V3" I L 5000 3100 50
+F4 "GND" I L 5000 3400 50
 $EndSheet
 $Sheet
-S 8000 6000 1000 500
+S 6000 5500 1000 500
 U 60AAE212
 F0 "CURRENT_SENSOR" 50
@@
 $EndSheet
 $Sheet
-S 6000 4000 1000 500
+S 6500 3000 1000 500
 U 60AAE4BD
 F0 "VOLTAGE_DIVIDER" 50
 F1 "Voltage_divider.sch" 50
+F2 "AC1" I L 6500 3100 50
+F3 "AC2" I L 6500 3400 50
+F4 "VOLT" O R 7500 3250 50
+F5 "+3V3" I R 7500 3100 50
+F6 "GND" I R 7500 3400 50
 $EndSheet
 $Sheet
-S 3000 6000 1000 500
+S 5500 2000 1000 500
 U 60AAEC6C
 F0 "OPTOISOLATOR" 50
 F1 "Optoisolator.sch" 50
+F2 "IN" I L 5500 2250 50
+F3 "GND1" I L 5500 2400 50
+F4 "+5V" I R 6500 2100 50
+F5 "GND2" I R 6500 2400 50
+F6 "OUT" O R 6500 2250 50
 $EndSheet
 $Comp

Commit message: Add files via upload
Parts:
- removed U?: LM321, Package_TO_SOT_SMD:SOT-23-5, symbol Amplifier_Operational:LM321
Changed lines of the file:
@@
 $EndDescr
-$Comp
-L Amplifier_Operational:LM321 U?
-U 1 1 609BBA47
-P 2800 4700
-F 0 "U?" H 3144 4746 50  0000 L CNN
-F 1 "LM321" H 3144 4655 50  0000 L CNN
-F 2 "Package_TO_SOT_SMD:SOT-23-5" H 2800 4700 50  0001 C CNN
-F 3 "http://www.ti.com/lit/ds/symlink/lm321.pdf" H 2800 4700 50  0001 C CNN
-	1    2800 4700
-	1    0    0    -1
-$EndComp
 $Comp
 L Connector_Generic:Conn_01x04 J?
@@
 $EndSheet
 $Sheet
-S 6000 5500 1000 500
-U 60AAE212
-F0 "CURRENT_SENSOR" 50
-F1 "Current_sensor.sch" 50
-$EndSheet
-$Sheet
 S 6500 3000 1000 500
 U 60AAE4BD
@@
 	-1   0    0    -1
 $EndComp
+$Sheet
+S 6500 4000 1000 500
+U 60AAE212
+F0 "CURRENT_SENSOR" 50
+F1 "Current_sensor.sch" 50
+F2 "CURR" O R 7500 4250 50
+F3 "+3V3" I R 7500 4100 50
+F4 "GND" I R 7500 4400 50
+$EndSheet
 $EndSCHEMATC

Commit message: Add files via upload
Connections:
- wire segments 0 -> 81
Other:
- note added: "+5V"
- note added: "230V"
- note added: "AC 230V input"
- note added: "GND"
- note added: "Heater"
- note added: "Isolation"
- note added: "Load"
- note added: "Load wire \nshould pass throught\nthe current \ntransformer hole"
- note added: "Temp sensor placed \non the same heatsink\nas the TRIAC"
- note added: "UART_TX"

Commit message: Add files via upload
Parts:
- removed J?: CWF-4R, symbol Connector_Generic:Conn_01x04
- added J3: IDC-6, Connector_IDC:IDC-Header_2x03_P2.54mm_Vertical, symbol Connector_Generic:Conn_01x06
- J1, J2: renamed from J?; symbol Connector:Screw_Terminal_01x02 -> furnace_230V-rescue:Screw_Terminal_01x02-Connector
Connections:
- wire segments 81 -> 87
Changed lines of the file:
@@
 $EndDescr
 $Comp
-L Connector_Generic:Conn_01x04 J?
-U 1 1 60AAE60F
-P 10200 3200
-AR Path="/60AAC03E/60AAE60F" Ref="J?"  Part="1"
-AR Path="/60AAE60F" Ref="J?"  Part="1"
-F 0 "J?" H 10150 2800 50  0000 L CNN
-F 1 "CWF-4R" H 10050 2900 50  0000 L CNN
-F 2 "" H 10200 3200 50  0001 C CNN
-F 3 "~" H 10200 3200 50  0001 C CNN
-	1    10200 3200
-	1    0    0    1
-$EndComp
-$Comp
-L Connector:Screw_Terminal_01x02 J?
+L furnace_230V-rescue:Screw_Terminal_01x02-Connector J1
 U 1 1 60AAEFEC
 P 1800 1500
-F 0 "J?" H 1880 1492 50  0000 L CNN
+F 0 "J1" H 1880 1492 50  0000 L CNN
 F 1 "TC0" H 1880 1401 50  0000 L CNN
 F 2 "" H 1800 1500 50  0001 C CNN
@@
 $EndSheet
 $Comp
-L Connector:Screw_Terminal_01x02 J?
+L furnace_230V-rescue:Screw_Terminal_01x02-Connector J2
 U 1 1 60AB629C
 P 1800 2500
-F 0 "J?" H 1880 2492 50  0000 L CNN
+F 0 "J2" H 1880 2492 50  0000 L CNN
 F 1 "TC0" H 1880 2401 50  0000 L CNN
 F 2 "" H 1800 2500 50  0001 C CNN
@@
 Text Notes 6150 1050 2    197  ~ 0
 230V
-Text Notes 10500 3050 0    50   ~ 0
+Text Notes 10300 3000 0    50   ~ 0
 +5V
-Text Notes 10500 3350 0    50   ~ 0
+Text Notes 10300 3400 0    50   ~ 0
 GND
-Text Notes 10500 3150 0    50   ~ 0
+Text Notes 10300 3150 0    50   ~ 0
 UART_TX
-Text Notes 10500 3250 0    50   ~ 0
+Text Notes 10300 3250 0    50   ~ 0
 Heater
 Wire Wire Line
@@
 	9250 2400 8500 2400
 Wire Wire Line
-	10000 3000 9000 3000
+	10000 3000 9900 3000
 Connection ~ 9000 3000
 Wire Wire Line
 	9000 3000 9000 2100
 Wire Wire Line
-	10000 3300 9250 3300
+	10000 3300 9900 3300
 Connection ~ 9250 3300
 Wire Wire Line
@@
 Wire Wire Line
 	7300 5250 7500 5250
+$Comp
+L Connector_Generic:Conn_01x06 J3
+U 1 1 610690C6
+P 10200 3100
+F 0 "J3" H 10150 3550 50  0000 L CNN
+F 1 "IDC-6" H 10100 3450 50  0000 L CNN
+F 2 "Connector_IDC:IDC-Header_2x03_P2.54mm_Vertical" H 10200 3100 50  0001 C CNN
+F 3 "~" H 10200 3100 50  0001 C CNN
+	1    10200 3100
+	1    0    0    -1
+$EndComp
+Wire Wire Line
+	10000 2900 9900 2900
+Wire Wire Line
+	9900 2900 9900 3000
+Connection ~ 9900 3000
+Wire Wire Line
+	9900 3000 9000 3000
+Wire Wire Line
+	10000 3400 9900 3400
+Wire Wire Line
+	9900 3400 9900 3300
+Connection ~ 9900 3300
+Wire Wire Line
+	9900 3300 9250 3300
 $EndSCHEMATC

Commit message: Add files via upload
Parts:
- J1, J2: value TC0 -> (none)
Changed lines of the file:
@@
 P 1800 1500
 F 0 "J1" H 1880 1492 50  0000 L CNN
-F 1 "TC0" H 1880 1401 50  0000 L CNN
+F 1 " " H 1880 1401 50  0000 L CNN
 F 2 "" H 1800 1500 50  0001 C CNN
 F 3 "~" H 1800 1500 50  0001 C CNN
@@
 P 1800 2500
 F 0 "J2" H 1880 2492 50  0000 L CNN
-F 1 "TC0" H 1880 2401 50  0000 L CNN
+F 1 " " H 1880 2401 50  0000 L CNN
 F 2 "" H 1800 2500 50  0001 C CNN
 F 3 "~" H 1800 2500 50  0001 C CNN

Commit message: Add files via upload
Parts:
- added F1: 10A, Fuse:Fuseholder_Cylinder-5x20mm_Stelvio-Kontek_PTF78_Horizontal_Open, symbol furnace_230V-rescue:Fuse-Device
- added F2: 0,1A, Fuse:Fuseholder_Cylinder-5x20mm_Stelvio-Kontek_PTF78_Horizontal_Open, symbol furnace_230V-rescue:Fuse-Device
- added G1: LOGO, furnace_230V:stamp, symbol stamp:LOGO
- added H1, H2, H3, H4: MountingHole, furnace_230V:hole_D3.5mm, symbol Mechanical:MountingHole
- J1, J2: footprint (none) -> furnace_230V:KF7.62-2P
Connections:
- net AC-DC 5V/AC1: now also F2.1; no longer J1.1 (Pin_1)
- new net: F1.2, F2.2, J1.1 (Pin_1)
- new net ISOLATED_TRIAC/AC: F1.1
Other:
- moved on the sheet: J1, J2
Changed lines of the file:
@@
 L furnace_230V-rescue:Screw_Terminal_01x02-Connector J1
 U 1 1 60AAEFEC
-P 1800 1500
-F 0 "J1" H 1880 1492 50  0000 L CNN
-F 1 " " H 1880 1401 50  0000 L CNN
-F 2 "" H 1800 1500 50  0001 C CNN
-F 3 "~" H 1800 1500 50  0001 C CNN
-	1    1800 1500
+P 1300 1500
+F 0 "J1" H 1380 1492 50  0000 L CNN
+F 1 " " H 1380 1401 50  0000 L CNN
+F 2 "furnace_230V:KF7.62-2P" H 1300 1500 50  0001 C CNN
+F 3 "~" H 1300 1500 50  0001 C CNN
+	1    1300 1500
 	-1   0    0    -1
 $EndComp
@@
 L furnace_230V-rescue:Screw_Terminal_01x02-Connector J2
 U 1 1 60AB629C
-P 1800 2500
-F 0 "J2" H 1880 2492 50  0000 L CNN
-F 1 " " H 1880 2401 50  0000 L CNN
-F 2 "" H 1800 2500 50  0001 C CNN
-F 3 "~" H 1800 2500 50  0001 C CNN
-	1    1800 2500
+P 1300 2500
+F 0 "J2" H 1380 2492 50  0000 L CNN
+F 1 " " H 1380 2401 50  0000 L CNN
+F 2 "furnace_230V:KF7.62-2P" H 1300 2500 50  0001 C CNN
+F 3 "~" H 1300 2500 50  0001 C CNN
+	1    1300 2500
 	-1   0    0    -1
 $EndComp
@@
 F4 "GND" I L 3000 5400 50
 $EndSheet
-Text Notes 1550 1300 0    50   ~ 0
+Text Notes 1100 1300 0    50   ~ 0
 AC 230V input
 Wire Notes Line rgb(255, 0, 0)
 	8000 1500 8000 6000
 Wire Notes Line
-	1750 2600 1500 2600
+	1300 2650 1300 5250
 Wire Notes Line
-	1500 2600 1500 5250
-Wire Notes Line
-	1500 5250 3000 5250
+	1300 5250 3000 5250
 Wire Notes Line
 	7500 3250 4000 3250
 Text Notes 7850 1350 0    50   ~ 0
 Isolation
-Text Notes 650  3050 0    50   ~ 0
+Text Notes 850  3100 0    50   ~ 0
 Load wire \nshould pass throught\nthe current \ntransformer hole
 Text Notes 4200 3200 0    50   ~ 0
 Temp sensor placed \non the same heatsink\nas the TRIAC
-Text Notes 1700 2300 0    50   ~ 0
+Text Notes 1200 2300 0    50   ~ 0
 Load
 Wire Wire Line
-	6500 1500 6500 2100
-Wire Wire Line
-	6500 2100 7500 2100
-Wire Wire Line
 	7500 3100 6500 3100
 Wire Wire Line
-	6500 3100 6500 2100
-Connection ~ 6500 2100
-Wire Wire Line
 	7500 3400 6000 3400
 Wire Wire Line
 	7500 2400 6250 2400
 Wire Wire Line
-	6250 2400 6250 1600
-Wire Wire Line
-	2000 1500 2250 1500
-Wire Wire Line
-	2000 1600 2150 1600
+	6250 2400 6250 2000
 Wire Wire Line
 	6000 3400 6000 2500
-Wire Wire Line
-	6000 2500 2000 2500
-Wire Wire Line
-	2000 2600 2500 2600
-Wire Wire Line
-	2500 2600 2500 1600
-Connection ~ 2500 1600
-Wire Wire Line
-	2500 1600 6250 1600
 Text Notes 6150 1050 2    197  ~ 0
 230V
@@
 	2500 5400 2500 4500
 Wire Wire Line
-	3000 4100 2250 4100
-Wire Wire Line
-	2250 4100 2250 1500
-Connection ~ 2250 1500
-Wire Wire Line
-	2250 1500 6500 1500
-Wire Wire Line
-	3000 4200 2150 4200
-Wire Wire Line
-	2150 4200 2150 1600
-Connection ~ 2150 1600
-Wire Wire Line
-	2150 1600 2500 1600
+	3000 4100 2400 4100
+Wire Wire Line
+	2400 4100 2400 2000
+Wire Wire Line
+	3000 4200 2300 4200
+Wire Wire Line
+	2300 4200 2300 1800
 Wire Wire Line
 	5000 5700 4750 5700
@@
 Wire Wire Line
 	9900 3300 9250 3300
+$Comp
+L stamp:LOGO G1
+U 1 1 610EDF1B
+P 10300 6050
+F 0 "G1" H 10300 5928 60  0001 C CNN
+F 1 "LOGO" H 10300 6172 60  0001 C CNN
+F 2 "furnace_230V:stamp" H 10300 6050 50  0001 C CNN
+F 3 "" H 10300 6050 50  0001 C CNN
+	1    10300 6050
+	1    0    0    -1
+$EndComp
+$Comp
+L Mechanical:MountingHole H1
+U 1 1 6110929D
+P 8500 6000
+F 0 "H1" H 8550 6150 50  0000 L CNN
+F 1 "MountingHole" H 8350 5850 50  0000 L CNN
+F 2 "furnace_230V:hole_D3.5mm" H 8500 6000 50  0001 C CNN
+F 3 "~" H 8500 6000 50  0001 C CNN
+	1    8500 6000
+	1    0    0    -1
+$EndComp
+$Comp
+L Mechanical:MountingHole H2
+U 1 1 6110B2E7
+P 8750 6000
+F 0 "H2" H 8800 6150 50  0000 L CNN
+F 1 "MountingHole" H 8600 5850 50  0001 L CNN
+F 2 "furnace_230V:hole_D3.5mm" H 8750 6000 50  0001 C CNN
+F 3 "~" H 8750 6000 50  0001 C CNN
+	1    8750 6000
+	1    0    0    -1
+$EndComp
+$Comp
+L Mechanical:MountingHole H3
+U 1 1 6110B4DC
+P 9000 6000
+F 0 "H3" H 9050 6150 50  0000 L CNN
+F 1 "MountingHole" H 8850 5850 50  0001 L CNN
+F 2 "furnace_230V:hole_D3.5mm" H 9000 6000 50  0001 C CNN
+F 3 "~" H 9000 6000 50  0001 C CNN
+	1    9000 6000
+	1    0    0    -1
+$EndComp
+$Comp
+L Mechanical:MountingHole H4
+U 1 1 6110B613
+P 9250 6000
+F 0 "H4" H 9300 6150 50  0000 L CNN
+F 1 "MountingHole" H 9100 5850 50  0001 L CNN
+F 2 "furnace_230V:hole_D3.5mm" H 9250 6000 50  0001 C CNN
+F 3 "~" H 9250 6000 50  0001 C CNN
+	1    9250 6000
+	1    0    0    -1
+$EndComp
+$Comp
+L furnace_230V-rescue:Fuse-Device F?
+U 1 1 61103E7E
+P 2150 1800
+AR Path="/60AABABA/61103E7E" Ref="F?"  Part="1"
+AR Path="/61103E7E" Ref="F2"  Part="1"
+F 0 "F2" V 2050 1800 50  0000 C CNN
+F 1 "0,1A" V 2250 1800 50  0000 C CNN
+F 2 "Fuse:Fuseholder_Cylinder-5x20mm_Stelvio-Kontek_PTF78_Horizontal_Open" V 2080 1800 50  0001 C CNN
+F 3 "~" H 2150 1800 50  0001 C CNN
+	1    2150 1800
+	0    1    1    0
+$EndComp
+$Comp
+L furnace_230V-rescue:Fuse-Device F?
+U 1 1 61107140
+P 2150 1500
+AR Path="/60AAE0B8/61107140" Ref="F?"  Part="1"
+AR Path="/61107140" Ref="F1"  Part="1"
+F 0 "F1" V 2050 1500 50  0000 C CNN
+F 1 "10A" V 2250 1500 50  0000 C CNN
+F 2 "Fuse:Fuseholder_Cylinder-5x20mm_Stelvio-Kontek_PTF78_Horizontal_Open" V 2080 1500 50  0001 C CNN
+F 3 "~" H 2150 1500 50  0001 C CNN
+	1    2150 1500
+	0    1    1    0
+$EndComp
+Wire Wire Line
+	6500 1500 6500 3100
+Wire Wire Line
+	1600 2600 1600 2000
+Wire Wire Line
+	1600 1600 1500 1600
+Wire Wire Line
+	6250 2000 2400 2000
+Connection ~ 1600 2000
+Wire Wire Line
+	1600 2000 1600 1600
+Connection ~ 2400 2000
+Wire Wire Line
+	2400 2000 1600 2000
+Wire Wire Line
+	1500 1500 1900 1500
+Wire Wire Line
+	2000 1800 1900 1800
+Wire Wire Line
+	1900 1800 1900 1500
+Connection ~ 1900 1500
+Wire Wire Line
+	1900 1500 2000 1500
+Wire Wire Line
+	2300 1500 6500 1500
+Wire Wire Line
+	2300 1800 7000 1800
+Wire Wire Line
+	7000 1800 7000 2100
+Wire Wire Line
+	7000 2100 7500 2100
+Connection ~ 2300 1800
+Wire Wire Line
+	1600 2600 1500 2600
+Wire Wire Line
+	1500 2500 6000 2500
 $EndSCHEMATC
