File: furnace/furnace_230V/furnace_230V.sch (KiCad schematic (older format))
At the start: 10 parts, among them J1 , J2 , J3 IDC-6

Commit message: Add files via upload
Connections:
- net +3V3_ISOLATED/+5V: now also J3.5 (Pin_5), J3.6 (Pin_6); no longer J3.1 (Pin_1), J3.2 (Pin_2)
- net +3V3_ISOLATED/GND: now also J3.1 (Pin_1), J3.2 (Pin_2); no longer J3.5 (Pin_5), J3.6 (Pin_6)
Changed lines of the file:
@@
 Text Notes 6150 1050 2    197  ~ 0
 230V
+Text Notes 10300 3400 0    50   ~ 0
++5V
 Text Notes 10300 3000 0    50   ~ 0
-+5V
-Text Notes 10300 3400 0    50   ~ 0
 GND
 Text Notes 10300 3150 0    50   ~ 0
@@
 	9250 2400 8500 2400
 Wire Wire Line
-	10000 3000 9900 3000
-Connection ~ 9000 3000
-Wire Wire Line
-	9000 3000 9000 2100
-Wire Wire Line
-	10000 3300 9900 3300
-Connection ~ 9250 3300
-Wire Wire Line
-	9250 3300 9250 2400
-Wire Wire Line
 	8500 3100 9000 3100
 Connection ~ 9000 3100
 Wire Wire Line
-	9000 3100 9000 3000
-Wire Wire Line
 	8500 4100 9000 4100
 Connection ~ 9000 4100
 Wire Wire Line
-	9000 4100 9000 3100
+	9000 4100 9000 3300
 Wire Wire Line
 	8500 4400 9250 4400
 Connection ~ 9250 4400
-Wire Wire Line
-	9250 4400 9250 3300
 Wire Wire Line
 	7500 4100 5500 4100
@@
 	1    0    0    -1
 $EndComp
-Wire Wire Line
-	10000 2900 9900 2900
-Wire Wire Line
-	9900 2900 9900 3000
-Connection ~ 9900 3000
-Wire Wire Line
-	9900 3000 9000 3000
-Wire Wire Line
-	10000 3400 9900 3400
-Wire Wire Line
-	9900 3400 9900 3300
-Connection ~ 9900 3300
-Wire Wire Line
-	9900 3300 9250 3300
 $Comp
 L stamp:LOGO G1
@@
 Wire Wire Line
 	1500 2500 6000 2500
+Wire Wire Line
+	9000 2100 9000 3100
+Wire Wire Line
+	9250 2400 9250 3000
+Wire Wire Line
+	10000 3300 9900 3300
+Wire Wire Line
+	9900 3300 9900 3400
+Wire Wire Line
+	9900 3400 10000 3400
+Wire Wire Line
+	10000 2900 9900 2900
+Wire Wire Line
+	9900 2900 9900 3000
+Wire Wire Line
+	9900 3000 10000 3000
+Wire Wire Line
+	9900 3300 9000 3300
+Connection ~ 9900 3300
+Connection ~ 9000 3300
+Wire Wire Line
+	9000 3300 9000 3100
+Wire Wire Line
+	9900 3000 9250 3000
+Connection ~ 9900 3000
+Connection ~ 9250 3000
+Wire Wire Line
+	9250 3000 9250 4400
 $EndSCHEMATC
