File: furnace/furnace_230V/furnace_230V.kicad_pcb (KiCad board)
At the start: 2 copper layers, 85 x 90 mm, 82 parts, among them J1 , J2 , J3 IDC-6, Q1 BTA16-600B, T1 ZMCT103C, U1 STM8S001J3M, U2 LM317L_SO8, U3 MOC3052M, U4 DS18B20, U5 H11L1

Commit message: Add files via upload
Parts:
- R7: footprint Resistor_THT:R_Axial_DIN0309_L9.0mm_D3.2mm_P15.24mm_Horizontal -> Resistor_THT:R_Axial_DIN0309_L9.0mm_D3.2mm_P5.08mm_Vertical
- moved R7 7.06 mm to (40.1, 63.5)
- moved R1 6.21 mm to (77.5, 49.7)
- moved F1 3.00 mm to (48.0, 71.0)
- moved J1 2.30 mm to (11.0, 81.3)
- moved J2 2.26 mm to (11.0, 66.0)
- moved J3 2.00 mm to (82.3, 42.0)
- moved L1 1.92 mm to (62.6, 73.0)
- moved D4 1.69 mm to (67.7, 79.6)
- moved C1 1.57 mm to (55.0, 71.9)
- moved T1 1.41 mm to (3.00, 61.0)
- moved D2 1.14 mm to (81.0, 50.5), turned to 180 degrees
- moved F2 1.01 mm to (48.0, 83.0)
- moved R11 0.71 mm to (54.0, 58.3)
- moved PS2 0.67 mm to (81.7, 22.1)
- moved R9 0.55 mm to (58.0, 68.5)

Commit message: Add files via upload
Parts:
- R7: footprint Resistor_THT:R_Axial_DIN0309_L9.0mm_D3.2mm_P5.08mm_Vertical -> Resistor_THT:R_Axial_DIN0309_L9.0mm_D3.2mm_P12.70mm_Horizontal
- moved TP8 59.1 mm to (52.7, 58.4)
- moved TP12 52.6 mm to (31.8, 2.54)
- moved TP11 46.7 mm to (28.6, 2.54)
- moved TP7 30.4 mm to (60.3, 58.4)
- moved TP6 26.3 mm to (55.2, 2.54)
- moved D3 21.3 mm to (83.2, 49.9), turned to 270 degrees
- moved R6 17.8 mm to (82.5, 45.5)
- moved TP13 15.9 mm to (41.9, 2.54)
- moved C18 14.3 mm to (43.2, 30.9), turned to 90 degrees
- moved C17 13.1 mm to (33.7, 33.5)
- moved R16 13.1 mm to (33.7, 35.5)
- moved TP3 11.7 mm to (52.7, 2.54)
- moved R17 10.6 mm to (39.6, 35.7), turned to 180 degrees
- moved D7 8.47 mm to (40.3, 30.8), turned to 180 degrees
- moved TP5 7.45 mm to (70.5, 11.4)
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Connections:
- J3 pad 1: /+3V3_ISOLATED/+5V -> /+3V3_ISOLATED/GND
- J3 pad 2: /+3V3_ISOLATED/+5V -> /+3V3_ISOLATED/GND
- J3 pad 5: /+3V3_ISOLATED/GND -> /+3V3_ISOLATED/+5V
- J3 pad 6: /+3V3_ISOLATED/GND -> /+3V3_ISOLATED/+5V
Routing:
- net /+3V3_ISOLATED/+5V: track 0.00 -> 95.9 mm, vias 0 -> 4
- net Net-(C17-Pad2): track 0.00 -> 91.9 mm, vias 0 -> 2
- net /CURRENT_SENSOR/+3V3: track 0.00 -> 86.7 mm, vias 0 -> 4
- net /VOLTAGE_DIVIDER/AC1: track 0.00 -> 84.1 mm
- net Net-(C17-Pad1): track 0.00 -> 77.6 mm
- net /+3V3_ISOLATED/GND: track 0.00 -> 66.9 mm, vias 0 -> 12
- net /TEMP_SENSOR/SDA: track 0.00 -> 63.7 mm
- net /CURRENT_SENSOR/GND: track 0.00 -> 59.7 mm, vias 0 -> 67
- net Net-(D3-Pad1): track 0.00 -> 56.8 mm, vias 0 -> 2
- net Net-(C2-Pad2): track 0.00 -> 50.6 mm
- net /ISOLATED_TRIAC/~EN: track 0.00 -> 42.2 mm
- net /OPTOISOLATOR/OUT: track 0.00 -> 36.5 mm
- net Net-(F1-Pad2): track 0.00 -> 33.8 mm
- net Net-(Q1-Pad3): track 0.00 -> 33.4 mm
- net /CURRENT_SENSOR/CURR: track 0.00 -> 30.8 mm
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- added copper zone on B.Cu, net /+3V3_ISOLATED/GND
- added copper zone on F.Cu, net /+3V3_ISOLATED/GND
- added copper zone on B.Cu, net /CURRENT_SENSOR/GND
- added copper zone on F.Cu, net /CURRENT_SENSOR/GND
- added copper zone on B.Cu, net /ISOLATED_TRIAC/AC
- added copper zone on B.Cu, net /ISOLATED_TRIAC/LOAD
- added copper zone on B.Cu, net Net-(F1-Pad2)
Other:
- net class Default: clearance 0.2 -> 0.3
- rule trace_clearance: 0.2 -> 0.3

Commit message: Add files via upload
Other:
- rule trace_min: 0.2 -> 0.16

Commit message: Add files via upload
Other:
- board text added: "furnace 230V 1.0"

Commit message: Add files via upload
Other:
- board text added: "0,1A 10A"
- board text added: "AC IN"
- board text added: "LOAD"
