File: furnace_230V_HW/furnace_230V.kicad_pcb (KiCad board)
At the start: 2 copper layers, 85 x 90 mm, 82 parts, among them J1 , J2 , J3 IDC-6, Q1 BTA16-600B, T1 ZMCT103C, U1 STM8S001J3M, U2 LM317L_SO8, U3 MOC3052M, U4 DS18B20, U5 H11L1

Commit message: Resave in KiCad 8
Connections:
- net /ISOLATED_TRIAC/~EN renamed /ISOLATED_TRIAC/~{EN}
Other:
- net class Default removed
