File: furnace_controller_HW/furnace_controller.kicad_pcb (KiCad board)
At the start: 2 copper layers, 88 x 100 mm, 155 parts, among them J1 DG141R-2.54-02P, J10 PLS-4R, J11 PLS-5, J12 PLS-3, J13 PLS-5, J14 CTF-11081-P, J2 DG141R-2.54-02P, J3 DG141R-2.54-02P, J4 DG141R-2.54-02P, J5 DG141R-2.54-02P, J6 IDC-6, J7 FPC-24P 0.5mm, J8 PLS-10R, J9 PLS-3, Q1 BC847, Q2 IRLML6402, Q3 IRLML2402, Q4 BC847, Q5 IRLML6402, Q6 BC847, Q7 BC847, U1 AMS1117-3.3, U10 ADuM1301, U11 STM32F103C6Tx, U2 MAX31855EASA, U3 ADuM1301, U4 LM317L_SO8, U5 MAX31855EASA, U6 MAX31855EASA, U7 MAX31855EASA, U8 MAX31855EASA, U9 ADuM1301, Y1 8MHz

Commit message: Resave in Kicad 9
Connections:
- net /ISOLATED_TEMP_SENSOR/~CS0 renamed /ISOLATED_TEMP_SENSOR/~{CS0}
- net /ISOLATED_TEMP_SENSOR/~CS1 renamed /ISOLATED_TEMP_SENSOR/~{CS1}
- net /ISOLATED_TEMP_SENSOR/~CS2 renamed /ISOLATED_TEMP_SENSOR/~{CS2}
- net /ISOLATED_TEMP_SENSOR/~CS3 renamed /ISOLATED_TEMP_SENSOR/~{CS3}
- net /ISOLATED_TEMP_SENSOR/~CS4 renamed /ISOLATED_TEMP_SENSOR/~{CS4}
- net /MCU/~DPY_RST renamed /MCU/~{DPY_RST}
- net /MICRO_SD_CARD/~CS~ renamed /MICRO_SD_CARD/~{CS}
Other:
- net class Default removed
